File: KiCad/DiKo_PreAmp.kicad_sch (KiCad schematic)
At the start: 454 parts, among them J1 R_Phono_In, J10 VCC_IN, J11 VCC_OUT, J2 L_Phono_In, J3 R_Line_In, J4 L_Line_In, J5 Mic_In, J6 Effekt_In, J7 AUX_RET_1, J8 AUX_RET_2, J9 AUX_RET_3, SW1 SW_SPDT, SW2 SW_SPDT, SW3 SW_SPDT, SW4 SW_SPDT, SW5 SW_SPDT, SW6 SW_SPDT, SW7 SW_DPST, SW8 SW_SPDT, U1 TL074, U10 TL074, U11 TL074, U12 TL074, U13 TL074, U14 INA128U, U15 TL074, U16 TL074, U17 TL074, U18 TL074, U19 TL074, U2 TL074, U20 TL074, U21 REC10K-2409, U22 REC10K-2415, U23 TL074, U3 TL074, U4 TL074, U5 TL074, U6 TL074, U7 TL074, U8 TL074, U9 TL074

Commit message: Schaltplan Update
Parts:
- removed RV27: 47k lin, symbol Device:R_Potentiometer_US
- added R122, R123: 22k, symbol Device:R_US
- renumbered C4 to C2, C25 to C24, C26 to C25, C27 to C26, C28 to C27, C24 to C28, C32 to C29, C5 to C3, C33 to C30, C34 to C31, C29 to C32, C35 to C33, C36 to C34, C37 to C35, C30 to C36, C31 to C37, C6 to C4, C46 to C45, C47 to C46, C48 to C47, C45 to C48, C7 to C5, C95 to C50, C96 to C51, C50 to C52, C51 to C53, C52 to C54, C53 to C55, C54 to C56, C55 to C57, C56 to C58, C57 to C59, C2 to C6, C73 to C60, C58 to C61, C59 to C62, C60 to C63, C61 to C64, C62 to C65, C63 to C66, C64 to C67, C65 to C68, C66 to C69, C3 to C7, C67 to C70, C68 to C71, C69 to C72, C70 to C73, C71 to C74, C72 to C75, C97 to C76, C74 to C77, C75 to C78, C76 to C79, C92 to C80, C93 to C81, C94 to C82, C77 to C83, C78 to C84, C79 to C85, C80 to C86, C81 to C87, C82 to C88, C83 to C89, C84 to C90, C85 to C91, C86 to C92, C87 to C93, C88 to C94, C89 to C95, C90 to C96, C91 to C97, R6 to R1, R13 to R10, R93 to R100, R95 to R101, R117 to R104, R118 to R105, R113 to R106, R119 to R107, R114 to R108, R120 to R109, R14 to R11, R121 to R110, R115 to R111, R116 to R112, R104 to R113, R105 to R114, R106 to R115, R107 to R116, R108 to R117, R109 to R118, R110 to R119, R5 to R12, R111 to R120, R112 to R121, R16 to R13, R17 to R14, R18 to R15, R10 to R16, R12 to R17, R19 to R18, R20 to R19, R7 to R2, R21 to R20, R22 to R21, R23 to R22, R24 to R23, R15 to R24, R27 to R25, R28 to R26, R32 to R27, R33 to R28, R25 to R29, R1 to R3, R26 to R30, R35 to R31, R36 to R32, R37 to R33, R39 to R34, R40 to R35, R41 to R36, R42 to R37, R43 to R38, R44 to R39, R2 to R4, R29 to R40, R30 to R41, R31 to R42, R45 to R43, R34 to R44, R38 to R45, R8 to R5, R55 to R54, R56 to R55, R58 to R56, R59 to R57, R60 to R58, R62 to R59, R9 to R6, R63 to R60, R64 to R61, R54 to R62, R65 to R63, R66 to R64, R67 to R65, R57 to R66, R70 to R67, R61 to R68, R71 to R69, R3 to R7, R72 to R70, R73 to R71, R74 to R72, R75 to R73, R76 to R74, R77 to R75, R78 to R76, R68 to R77, R69 to R78, R11 to R8, R85 to R84, R86 to R85, R87 to R86, R88 to R87, R89 to R88, R90 to R89, R4 to R9, R94 to R90, R84 to R91, R96 to R92, R97 to R93, R98 to R94, R99 to R95, R100 to R96, R101 to R97, R91 to R98, R92 to R99, RV14 to RV12, RV15 to RV13, RV12 to RV14, RV13 to RV15, RV17 to RV16, RV16 to RV17, RV23 to RV21, RV21 to RV22, RV22 to RV23, RV6 to RV5, RV5 to RV6, SW3 to SW2, SW2 to SW3, SW8 to SW6, SW6 to SW7, SW7 to SW8, U3 to U1, U18 to U17, U4 to U2, U23 to U21, U21 to U22, U22 to U23, U1 to U3, U2 to U4, Z8 to Z10, Z117 to Z108, Z118 to Z109, Z9 to Z11, Z119 to Z110, Z120 to Z111, Z121 to Z112, Z122 to Z113, Z123 to Z114, Z108 to Z115, Z109 to Z116, Z110 to Z117, Z111 to Z118, Z112 to Z119, Z10 to Z12, Z113 to Z120, Z114 to Z121, Z115 to Z122, Z116 to Z123, Z156 to Z125, Z157 to Z126, Z158 to Z127, Z159 to Z128, Z160 to Z129, Z20 to Z13, Z161 to Z130, Z128 to Z131, Z129 to Z132, Z130 to Z133, Z131 to Z134, Z132 to Z135, Z133 to Z136, Z125 to Z137, Z126 to Z138, Z127 to Z139, Z11 to Z14, Z134 to Z140, Z135 to Z141, Z136 to Z142, Z137 to Z143, Z138 to Z144, Z139 to Z145, Z140 to Z146, Z141 to Z147, Z142 to Z148, Z143 to Z149, Z12 to Z15, Z144 to Z150, Z145 to Z151, Z146 to Z152, Z147 to Z153, Z148 to Z154, Z149 to Z155, Z150 to Z156, Z151 to Z157, Z152 to Z158, Z153 to Z159, Z13 to Z16, Z154 to Z160, Z155 to Z161, Z24 to Z17, Z25 to Z18, Z14 to Z19, Z26 to Z20, Z17 to Z21, Z18 to Z22, Z19 to Z23, Z21 to Z24, Z22 to Z25, Z27 to Z26, Z28 to Z27, Z29 to Z28, Z30 to Z29, Z23 to Z30, Z33 to Z31, Z34 to Z32, Z31 to Z33, Z32 to Z34, Z48 to Z38, Z49 to Z39, Z15 to Z4, Z50 to Z40, Z51 to Z41, Z38 to Z42, Z52 to Z43, Z53 to Z44, Z54 to Z45, Z55 to Z46, Z39 to Z47, Z40 to Z48, Z41 to Z49, Z16 to Z5, Z42 to Z50, Z43 to Z51, Z56 to Z52, Z44 to Z53, Z45 to Z54, Z46 to Z55, Z47 to Z56, Z64 to Z57, Z65 to Z58, Z66 to Z59, Z4 to Z6, Z67 to Z60, Z68 to Z61, Z69 to Z62, Z70 to Z63, Z57 to Z64, Z58 to Z65, Z59 to Z66, Z60 to Z67, Z61 to Z68, Z62 to Z69, Z5 to Z7, Z63 to Z70, Z76 to Z71, Z77 to Z72, Z78 to Z73, Z79 to Z74, Z83 to Z75, Z84 to Z76, Z87 to Z77, Z88 to Z78, Z71 to Z79, Z6 to Z8, Z91 to Z80, Z72 to Z81, Z73 to Z82, Z74 to Z83, Z75 to Z84, Z80 to Z85, Z81 to Z86, Z82 to Z87, Z85 to Z88, Z86 to Z89, Z7 to Z9, Z92 to Z90, Z93 to Z91, Z94 to Z92, Z95 to Z93, Z96 to Z94, Z89 to Z95, Z90 to Z96
Connections:
- net GND: no longer C50.1, R106.1, R108.2, RV25.2, RV25.3, RV26.1, RV26.2, U20.12 (+), U20.13 (-)
- net at R106.2, U20.14, Z127.2: now also R122.2
- net at R108.1, Z126.1: now also R123.1
- net at U20.10 (+): now also R122.1, R123.2
- net at U7.7: now also R105.2, Z125.2
- new net: C50.1, RV25.2, RV25.3, RV26.1, RV26.2, U20.12 (+)
- new net: R106.1, R108.2, U20.13 (-)
Other:
- moved on the sheet: U21C, U21D
