File: KiCad/DiKo_PreAmp.kicad_sch (KiCad schematic)
At the start: 607 parts, among them J1 Bass_Out, J10 Effekt_In, J11 AUX_Send_1, J12 Line_Out_L, J13 AUX_RET_1, J14 AUX_Send_2, J15 Line_Out_R, J16 VU Meter, J17 AUX_RET_2, J18 AUX_Send_3, J19 AUX_RET_3, J2 R_Phono_In, J20 VCC_IN, J21 VCC_OUT, J22 Phono/Line_Out, J23 Phono/Line_In, J24 Effect_Mic_Out, J25 Effect_Mic_In, J26 Effect_Mic_Out, J27 Pegel_In, J28 Effect_Mic_Out, J29 Effect_Mic_In, J3 L_Phono_In, J30 Aux_Ret_Out, J31 Aux_Ret_In, J32 Masse_Sternpunkt, J33 Masse_Sternpunkt, J34 Pegel_In, J35 Aux_Ret_Out, J36 Pegel_In, J37 Aux_Ret_Out, J4 Kick_Out, J5 R_Line_In, J6 L_Line_In, J7 Mid_Out, J8 Mic_In, J9 High_Out, SW1 SW_SPDT, SW10 Pegel_Selector, SW11 SW_SPDT, SW12 SW_DPST, SW2 SW_SPDT, SW3 SW_SPDT, SW4 SW_SPDT, SW5 SW_SPDT, SW6 SW_SPDT, SW7 SW_SPDT, SW8 SW_SPDT, SW9 SW_SPDT, U1 TL074, U10 TL074, U11 TL074, U12 TL074, U13 TL074, U14 TL074, U15 TL074, U16 TL074, U17 INA128U, U18 TL074, U19 TL074, U2 TL074, U20 TL074, U21 TL074, U22 TL074, U23 TL074, U24 TL074, U25 TL074, U26 TL074, U27 REC10K-2409, U28 REC10K-2415, U3 TL074, U4 TL074, U5 TL074, U6 TL074, U7 TL074, U8 TL074, U9 TL074

Commit message: Schaltplan Update
Parts:
- removed J22: Phono/Line_Out, symbol Connector:Conn_01x01_Socket
- removed J23: Phono/Line_In, symbol Connector:Conn_01x01_Pin
- removed J24, J26, J28: Effect_Mic_Out, symbol Connector:Conn_01x01_Socket
- removed J25, J29: Effect_Mic_In, symbol Connector:Conn_01x01_Pin
- removed J27, J34, J36: Pegel_In, symbol Connector:Conn_01x01_Pin
- removed J30, J35, J37: Aux_Ret_Out, symbol Connector:Conn_01x01_Socket
- removed J31: Aux_Ret_In, symbol Connector:Conn_01x01_Pin
- removed J32: Masse_Sternpunkt, symbol Connector:Conn_01x01_Socket
- removed J33: Masse_Sternpunkt, symbol Connector:Conn_01x01_Pin
- added C112, C113, C114, C115: 100n, Capacitor_SMD:C_0805_2012Metric_Pad1.18x1.45mm_HandSolder, symbol Device:C_Small
- added J22: Phono/Line_In, Connector_PinHeader_2.54mm:PinHeader_1x02_P2.54mm_Vertical, symbol Connector:Conn_01x02_Pin
- added J23, J25, J26, J30, J35: Mic_Effekt_Out, Connector_PinSocket_2.54mm:PinSocket_1x02_P2.54mm_Vertical, symbol Connector:Conn_01x02_Socket
- added J24, J28, J31: Mic_Effekt_In, Connector_PinHeader_2.54mm:PinHeader_1x02_P2.54mm_Vertical, symbol Connector:Conn_01x02_Pin
- added J27, J29, J34, J36: Pegel_In, Connector_PinHeader_2.54mm:PinHeader_1x02_P2.54mm_Vertical, symbol Connector:Conn_01x02_Pin
- added J32, J33, J41: EMK_In, Connector_PinHeader_2.54mm:PinHeader_1x05_P2.54mm_Vertical, symbol Connector:Conn_01x05_Pin
- added J37, J42: Pegel_Out, Connector_PinSocket_2.54mm:PinSocket_1x02_P2.54mm_Vertical, symbol Connector:Conn_01x02_Socket
- added J38, J39, J40: EMK_Out, Connector_PinSocket_2.54mm:PinSocket_1x05_P2.54mm_Vertical, symbol Connector:Conn_01x05_Socket
- added J44: LED_In, Connector_PinHeader_2.54mm:PinHeader_1x02_P2.54mm_Vertical, symbol Connector:Conn_01x02_Pin
- added J45: LED_Out, Connector_PinSocket_2.54mm:PinSocket_1x02_P2.54mm_Vertical, symbol Connector:Conn_01x02_Socket
- added J46: Phono/Line_Out, Connector_PinSocket_2.54mm:PinSocket_1x02_P2.54mm_Vertical, symbol Connector:Conn_01x02_Socket
- added unit 5 of U25
- added U3: TL074, Package_DIP:DIP-14_W7.62mm_Socket_LongPads, symbol Amplifier_Operational:TL074
- added Z126, Z146, Z178, Z186, Z211, Z243, Z244, Z245, Z247, Z248, Z249, Z250, Z253, Z254, Z255, Z256, Z39: ~, Resistor_SMD:R_0805_2012Metric_Pad1.20x1.40mm_HandSolder, symbol Device:R
- C1, C10, C100, C101, C102, C103, C104, C105, C106, C107, C108, C109, C11, C110, C111, C12, C13, C14, C15, C16, C17, C18, C19, C2, C20, C21, C22, C23, C24, C25, C26, C27, C28, C29, C3, C30, C31, C32, C33, C34, C35, C36, C37, C38, C39, C4, C40, C41, C42, C43, C44, C45, C46, C47, C48, C49, C5, C50, C51, C52, C53, C54, C55, C56, C57, C58, C59, C6, C60, C61, C62, C63, C64, C65, C66, C67, C68, C69, C7, C70, C71, C72, C73, C74, C75, C76, C77, C78, C79, C8, C80, C81, C82, C83, C84, C85, C86, C87, C88, C89, C9, C90, C91, C92, C93, C94, C95, C96, C97, C98, C99: footprint (none) -> Capacitor_SMD:C_0805_2012Metric_Pad1.18x1.45mm_HandSolder
- D1, D2, D4: footprint (none) -> Diode_SMD:D_0805_2012Metric_Pad1.15x1.40mm_HandSolder
- D3: footprint (none) -> LED_THT:LED_D3.0mm
- J1, J11, J12, J14, J15, J18, J4, J7, J9, L3, L5: footprint (none) -> Connector_PinSocket_2.54mm:PinSocket_1x02_P2.54mm_Vertical
- J10, J13, J17, J19, J2, J20, J21, J3, J5, J6: footprint (none) -> Connector_PinHeader_2.54mm:PinHeader_1x02_P2.54mm_Vertical
- J16: value VU Meter -> VU_Meter_Out; footprint (none) -> Connector_PinSocket_2.54mm:PinSocket_1x04_P2.54mm_Vertical
- J8: footprint (none) -> Connector_PinHeader_2.54mm:PinHeader_1x03_P2.54mm_Vertical
- L1: value L_Ferrite -> Dämpfungsperle, 220 Ohm @ 100MHz, 0.5A; footprint (none) -> Connector_PinSocket_2.54mm:PinSocket_1x02_P2.54mm_Vertical
- L2: value ~ -> Dämpfungsperle, 220 Ohm @ 100MHz, 0.5A; footprint (none) -> Connector_PinSocket_2.54mm:PinSocket_1x02_P2.54mm_Vertical
- R1, R10, R100, R101, R102, R103, R104, R105, R106, R107, R108, R109, R11, R110, R111, R112, R113, R114, R115, R116, R117, R118, R119, R12, R120, R121, R122, R123, R124, R125, R126, R127, R128, R129, R13, R130, R131, R132, R133, R134, R135, R136, R137, R138, R139, R14, R140, R141, R142, R143, R144, R145, R146, R147, R148, R149, R15, R16, R17, R18, R19, R2, R20, R21, R22, R23, R24, R25, R26, R27, R28, R29, R3, R30, R31, R32, R33, R34, R35, R36, R37, R38, R39, R4, R40, R41, R42, R43, R44, R45, R46, R47, R48, R49, R5, R50, R51, R52, R53, R54, R55, R56, R57, R58, R59, R6, R60, R61, R62, R63, R64, R65, R66, R67, R68, R69, R7, R70, R71, R72, R73, R74, R75, R76, R77, R78, R79, R8, R80, R81, R82, R83, R84, R85, R86, R87, R88, R89, R9, R90, R91, R92, R93, R94, R95, R96, R97, R98, R99, Z1, Z100, Z102, Z103, Z105, Z106, Z11, Z112, Z113, Z114, Z115, Z116, Z117, Z118, Z119, Z12, Z120, Z121, Z122, Z123, Z125, Z128, Z129, Z130, Z131, Z132, Z133, Z134, Z135, Z136, Z137, Z143, Z148, Z149, Z150, Z151, Z152, Z153, Z154, Z155, Z156, Z157, Z158, Z159, Z160, Z162, Z165, Z166, Z167, Z168, Z169, Z170, Z171, Z172, Z173, Z174, Z18, Z182, Z183, Z184, Z187, Z188, Z189, Z190, Z198, Z2, Z202, Z203, Z216, Z217, Z218, Z219, Z220, Z221, Z222, Z223, Z224, Z225, Z226, Z227, Z228, Z229, Z230, Z231, Z232, Z233, Z234, Z235, Z236, Z237, Z238, Z239, Z24, Z240, Z241, Z242, Z25, Z26, Z27, Z28, Z29, Z3, Z30, Z31, Z33, Z4, Z41, Z42, Z43, Z44, Z46, Z47, Z48, Z49, Z5, Z50, Z54, Z6, Z62, Z63, Z64, Z65, Z66, Z67, Z68, Z69, Z7, Z70, Z77, Z78, Z79, Z80, Z81, Z82, Z83, Z84, Z85, Z86, Z87, Z88, Z89, Z95, Z96, Z97, Z98, Z99: footprint (none) -> Resistor_SMD:R_0805_2012Metric_Pad1.20x1.40mm_HandSolder
- RV1, RV10, RV11, RV13, RV14, RV16, RV18, RV20, RV21, RV22, RV3, RV4, RV5, RV7, RV8, SW1, SW11, SW2, SW3, SW4, SW5, SW6, SW7, SW8, SW9: footprint (none) -> Connector_PinSocket_2.54mm:PinSocket_1x03_P2.54mm_Vertical
- RV12, RV15, RV17, RV19, RV2, RV6, RV9: footprint (none) -> Connector_PinSocket_2.54mm:PinSocket_1x06_P2.54mm_Vertical
- SW10: footprint (none) -> Connector_PinSocket_2.54mm:PinSocket_1x05_P2.54mm_Vertical
- SW12: footprint (none) -> Connector_PinSocket_2.54mm:PinSocket_1x04_P2.54mm_Vertical
- U1: renamed from U4; footprint (none) -> Package_DIP:DIP-14_W7.62mm_Socket_LongPads
- U1, U10, U11, U12, U13, U14, U15, U16, U18, U19, U2, U20, U21, U22, U23, U24, U25, U26, U3, U4, U5, U6, U7, U8, U9: footprint (none) -> Package_DIP:DIP-14_W7.62mm_Socket_LongPads
- U2: renamed from U9; footprint (none) -> Package_DIP:DIP-14_W7.62mm_Socket_LongPads
- U2, U5: renamed from U24; footprint (none) -> Package_DIP:DIP-14_W7.62mm_Socket_LongPads
- U3: renamed from U2; footprint (none) -> Package_DIP:DIP-14_W7.62mm_Socket_LongPads
- U3, U4: renamed from U10; footprint (none) -> Package_DIP:DIP-14_W7.62mm_Socket_LongPads
- U3, U4: renamed from U1; footprint (none) -> Package_DIP:DIP-14_W7.62mm_Socket_LongPads
- U4: renamed from U14; footprint (none) -> Package_DIP:DIP-14_W7.62mm_Socket_LongPads
- U5: renamed from U22; footprint (none) -> Package_DIP:DIP-14_W7.62mm_Socket_LongPads
- Z1: renamed from Z15; footprint (none) -> Resistor_SMD:R_0805_2012Metric_Pad1.20x1.40mm_HandSolder
- Z10: renamed from Z34; footprint (none) -> Resistor_SMD:R_0805_2012Metric_Pad1.20x1.40mm_HandSolder
- Z101: renamed from Z94; footprint (none) -> Resistor_SMD:R_0805_2012Metric_Pad1.20x1.40mm_HandSolder
- Z104: renamed from Z101; footprint (none) -> Resistor_SMD:R_0805_2012Metric_Pad1.20x1.40mm_HandSolder
- Z107: renamed from Z104; footprint (none) -> Resistor_SMD:R_0805_2012Metric_Pad1.20x1.40mm_HandSolder
- Z108: renamed from Z107; footprint (none) -> Resistor_SMD:R_0805_2012Metric_Pad1.20x1.40mm_HandSolder
- Z109: renamed from Z108; footprint (none) -> Resistor_SMD:R_0805_2012Metric_Pad1.20x1.40mm_HandSolder
- Z11: renamed from Z38; footprint (none) -> Resistor_SMD:R_0805_2012Metric_Pad1.20x1.40mm_HandSolder
- Z110: renamed from Z109; footprint (none) -> Resistor_SMD:R_0805_2012Metric_Pad1.20x1.40mm_HandSolder
- Z111: renamed from Z110; footprint (none) -> Resistor_SMD:R_0805_2012Metric_Pad1.20x1.40mm_HandSolder
- Z12: renamed from Z35; footprint (none) -> Resistor_SMD:R_0805_2012Metric_Pad1.20x1.40mm_HandSolder
- Z124: renamed from Z111; footprint (none) -> Resistor_SMD:R_0805_2012Metric_Pad1.20x1.40mm_HandSolder
- Z127: renamed from Z138; footprint (none) -> Resistor_SMD:R_0805_2012Metric_Pad1.20x1.40mm_HandSolder
- Z13: renamed from Z21; footprint (none) -> Resistor_SMD:R_0805_2012Metric_Pad1.20x1.40mm_HandSolder
- Z138: renamed from Z139; footprint (none) -> Resistor_SMD:R_0805_2012Metric_Pad1.20x1.40mm_HandSolder
- Z139: renamed from Z140; footprint (none) -> Resistor_SMD:R_0805_2012Metric_Pad1.20x1.40mm_HandSolder
- Z14: renamed from Z13; footprint (none) -> Resistor_SMD:R_0805_2012Metric_Pad1.20x1.40mm_HandSolder
- Z140: renamed from Z142; footprint (none) -> Resistor_SMD:R_0805_2012Metric_Pad1.20x1.40mm_HandSolder
- Z141: renamed from Z207; footprint (none) -> Resistor_SMD:R_0805_2012Metric_Pad1.20x1.40mm_HandSolder
- Z142: renamed from Z141; footprint (none) -> Resistor_SMD:R_0805_2012Metric_Pad1.20x1.40mm_HandSolder
- Z144: renamed from Z208; footprint (none) -> Resistor_SMD:R_0805_2012Metric_Pad1.20x1.40mm_HandSolder
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Connections:
- net +15V: now also C112.2, C114.2, J32.3 (Pin_3), J33.3 (Pin_3), J38.3 (Pin_3), J39.3 (Pin_3), J40.3 (Pin_3), J41.3 (Pin_3), U25.4 (V+), U3.4 (V+)
- net +9V: now also J32.1 (Pin_1), J33.1 (Pin_1), J38.1 (Pin_1), J39.1 (Pin_1), J40.1 (Pin_1), J41.1 (Pin_1)
- net -15V: now also C113.2, C115.2, J32.4 (Pin_4), J33.4 (Pin_4), J38.4 (Pin_4), J39.4 (Pin_4), J40.4 (Pin_4), J41.4 (Pin_4), U25.11 (V-), U3.11 (V-)
- net 9V_GND: now also J32.2 (Pin_2), J33.2 (Pin_2), J38.2 (Pin_2), J39.2 (Pin_2), J40.2 (Pin_2), J41.2 (Pin_2)
- net GND: now also C112.1, C113.1, C114.1, C115.1, J32.5 (Pin_5), J33.5 (Pin_5), J38.5 (Pin_5), J39.5 (Pin_5), J40.5 (Pin_5), J41.5 (Pin_5), Z126.2, Z146.2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; no longer D3.1 (K)
- net Pegel_Post: no longer U24.10 (+), U24.12 (+), Z160.2, Z231.1, Z232.1
- net at Z225.1, Z226.1: now also J29.1 (Pin_1)
- net at Z37.2, Z38.1: now also J46.1 (Pin_1)
- net at Z180.2, Z192.1: now also U4.12 (+); no longer U4.5 (+)
- net at Z237.2, Z238.1: now also J42.1 (Pin_1)
- net at Z228.1, Z229.1: now also J34.1 (Pin_1)
- net at Z113.1, Z171.1: now also J24.1 (Pin_1)
- net at Z240.1, Z241.1: now also J31.1 (Pin_1)
- net at Z234.1, Z235.1: now also J28.1 (Pin_1)
- net at R141.1: now also J45.1 (Pin_1); no longer D3.2 (A)
- net at Z163.2, Z177.1: now also J25.1 (Pin_1)
- net at Z179.2, Z185.1: now also J26.1 (Pin_1)
- net at Z205.2, Z210.1: now also J30.1 (Pin_1), J35.1 (Pin_1)
- net at Z222.1, Z223.1: now also J27.1 (Pin_1)
- net at Z141.2, Z145.1: now also J23.1 (Pin_1)
- net at Z2.1, Z42.1: now also J22.1 (Pin_1)
- new net: J23.2 (Pin_2), Z146.1
- new net: J34.2 (Pin_2), Z249.1
- new net: J36.1 (Pin_1), Z231.1, Z232.1
- new net: J22.2 (Pin_2), Z126.1
- new net: J37.1 (Pin_1), U24.10 (+), U24.12 (+), Z160.2
- new net: J42.2 (Pin_2), Z254.1
- new net: J28.2 (Pin_2), Z245.1
- new net: U4.13 (-), U4.14, Z175.2
- new net: J24.2 (Pin_2), Z243.1
- new net: J36.2 (Pin_2), Z250.1
- new net: J27.2 (Pin_2), Z247.1
- new net: J37.2 (Pin_2), Z255.1
- new net: J25.2 (Pin_2), Z178.1
- new net: J26.2 (Pin_2), Z186.1
- new net: J46.2 (Pin_2), Z39.1
- new net: J35.2 (Pin_2), Z244.1
- new net: J30.2 (Pin_2), Z211.1
- new net: D3.2 (A), J44.1 (Pin_1)
- new net: D3.1 (K), J44.2 (Pin_2)
- new net: J31.2 (Pin_2), Z253.1
- new net: J45.2 (Pin_2), Z256.1
- new net: J29.2 (Pin_2), Z248.1
Other:
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
Commit message: Schaltplan Update
Parts:
- renumbered Z244 to Z100, Z92 to Z40, Z91 to Z41, Z93 to Z42, Z109 to Z43, Z107 to Z44, Z110 to Z45, Z94 to Z46, Z104 to Z47, Z101 to Z48, Z108 to Z49, Z111 to Z50, Z124 to Z51, Z127 to Z52, Z142 to Z53, Z138 to Z54, Z191 to Z55, Z180 to Z56, Z192 to Z57, Z175 to Z58, Z164 to Z59, Z147 to Z60, Z161 to Z61, Z139 to Z62, Z143 to Z63, Z140 to Z64, Z144 to Z65, Z141 to Z66, Z145 to Z67, Z146 to Z68, Z176 to Z69, Z163 to Z70, Z177 to Z71, Z178 to Z72, Z181 to Z73, Z179 to Z74, Z185 to Z75, Z186 to Z76, Z196 to Z77, Z193 to Z78, Z197 to Z79, Z194 to Z80, Z199 to Z81, Z195 to Z82, Z206 to Z83, Z200 to Z84, Z207 to Z85, Z201 to Z86, Z208 to Z87, Z204 to Z88, Z246 to Z89, Z213 to Z90, Z251 to Z91, Z214 to Z92, Z252 to Z93, Z215 to Z94, Z212 to Z95, Z209 to Z96, Z205 to Z97, Z210 to Z98, Z211 to Z99
Other:
- note added: "LEGENDE"
- note added: "Leiterbahn"
- note added: "Leiterkabel"
- note added: "Platinen Bereich"
- moved on the sheet: Z239

Commit message: Footprint Update
Parts:
- J1, J11, J12, J14, J15, J18, J23, J25, J26, J30, J35, J37, J4, J42, J45, J46, J7, J9, L1, L2, L3, L5: footprint Connector_PinSocket_2.54mm:PinSocket_1x02_P2.54mm_Vertical -> Connector_PinSocket_2.54mm_LongPads:PinSocket_1x02_P2.54mm_Vertical_LongPads
- J10, J13, J17, J19, J2, J20, J21, J22, J24, J27, J28, J29, J3, J31, J34, J36, J44, J5, J6: footprint Connector_PinHeader_2.54mm:PinHeader_1x02_P2.54mm_Vertical -> Connector_PinHeader_2.54mm_LongPads:PinHeader_1x02_P2.54mm_Vertical_LongPads
- J16, SW12: footprint Connector_PinSocket_2.54mm:PinSocket_1x04_P2.54mm_Vertical -> Connector_PinSocket_2.54mm_LongPads:PinSocket_1x04_P2.54mm_Vertical_LongPdas
- J32, J33, J41: footprint Connector_PinHeader_2.54mm:PinHeader_1x05_P2.54mm_Vertical -> Connector_PinHeader_2.54mm_LongPads:PinHeader_1x05_P2.54mm_Vertical_LongPads
- J38, J39, J40, SW10: footprint Connector_PinSocket_2.54mm:PinSocket_1x05_P2.54mm_Vertical -> Connector_PinSocket_2.54mm_LongPads:PinSocket_1x05_P2.54mm_Vertical_LongPads
- J8: footprint Connector_PinHeader_2.54mm:PinHeader_1x03_P2.54mm_Vertical -> Connector_PinHeader_2.54mm_LongPads:PinHeader_1x03_P2.54mm_Vertical_LongPads
- RV1, RV10, RV11, RV13, RV14, RV16, RV18, RV20, RV21, RV22, RV3, RV4, RV5, RV7, RV8, SW1, SW11, SW2, SW3, SW4, SW5, SW6, SW7, SW8, SW9: footprint Connector_PinSocket_2.54mm:PinSocket_1x03_P2.54mm_Vertical -> Connector_PinSocket_2.54mm_LongPads:PinSocket_1x03_P2.54mm_Vertical_LongPads
- RV12, RV15, RV17, RV19, RV2, RV6, RV9: footprint Connector_PinSocket_2.54mm:PinSocket_1x06_P2.54mm_Vertical -> Connector_PinSocket_2.54mm_LongPads:PinSocket_1x06_P2.54mm_Vertical_LongPads

Commit message: Schaltplan Update
Parts:
- removed C110, C112, C113, C67, C85, C92: 100n, Capacitor_SMD:C_0805_2012Metric_Pad1.18x1.45mm_HandSolder, symbol Device:C_Small
- removed unit 5 of U12
- removed unit 5 of U22
- removed U3: TL074, Package_DIP:DIP-14_W7.62mm_Socket_LongPads, symbol Amplifier_Operational:TL074
- added C28, C29: 100n, Capacitor_SMD:C_0805_2012Metric_Pad1.18x1.45mm_HandSolder, symbol Device:C_Small
- added unit 2 of U22
- added unit 3 of U22
- added unit 4 of U22
- added unit 5 of U5
- renumbered C49 to C1, C57 to C10, C81 to C100, C106 to C101, C74 to C102, C99 to C103, C82 to C104, C107 to C105, C75 to C106, C100 to C107, C78 to C108, C103 to C109, C58 to C11, C76 to C110, C101 to C111, C89 to C12, C65 to C13, C90 to C14, C7 to C15, C66 to C16, C91 to C17, C55 to C18, C61 to C19, C62 to C2, C64 to C20, C1 to C21, C37 to C22, C54 to C23, C56 to C24, C60 to C25, C88 to C26, C2 to C27, C48 to C3, C36 to C30, C68 to C31, C93 to C32, C114 to C33, C115 to C34, C50 to C35, C52 to C36, C51 to C37, C13 to C38, C23 to C39, C59 to C4, C34 to C40, C47 to C41, C10 to C42, C20 to C43, C31 to C44, C44 to C45, C83 to C46, C108 to C47, C3 to C48, C14 to C49, C63 to C5, C24 to C50, C38 to C51, C8 to C52, C18 to C53, C29 to C54, C42 to C55, C84 to C56, C109 to C57, C4 to C58, C15 to C59, C87 to C6, C25 to C60, C39 to C61, C11 to C62, C21 to C63, C32 to C64, C45 to C65, C69 to C66, C94 to C67, C86 to C68, C111 to C69, C28 to C7, C5 to C70, C16 to C71, C26 to C72, C40 to C73, C9 to C74, C19 to C75, C30 to C76, C43 to C77, C70 to C78, C95 to C79, C35 to C8, C77 to C80, C102 to C81, C6 to C82, C17 to C83, C27 to C84, C41 to C85, C12 to C86, C22 to C87, C33 to C88, C46 to C89, C53 to C9, C71 to C90, C96 to C91, C79 to C92, C104 to C93, C72 to C94, C97 to C95, C80 to C96, C105 to C97, C73 to C98, C98 to C99, D2 to D1, D1 to D2, D4 to D3, D3 to D4, J2 to J1, J20 to J10, J21 to J11, J33 to J12, J38 to J13, J40 to J14, J26 to J15, J25 to J16, J30 to J17, J35 to J18, J46 to J19, J3 to J2, J23 to J20, J39 to J21, J41 to J22, J32 to J23, J28 to J24, J31 to J25, J22 to J26, J24 to J27, J42 to J28, J37 to J29, J5 to J3, J27 to J30, J29 to J31, J34 to J32, J36 to J33, J45 to J34, J44 to J35, J16 to J36, J18 to J37, J11 to J38, J14 to J39, J6 to J4, J1 to J40, J4 to J41, J7 to J42, J9 to J43, J12 to J44, J15 to J45, J8 to J5, J10 to J6, J13 to J7, J17 to J8, J19 to J9, L4 to L1, L1 to L2, L2 to L3, L3 to L4, R102 to R1, R127 to R10, R116 to R100, R5 to R101, R30 to R102, R53 to R103, R79 to R104, R16 to R105, R40 to R106, R65 to R107, R89 to R108, R3 to R109, R145 to R11, R26 to R110, R50 to R111, R76 to R112, R17 to R113, R41 to R114, R66 to R115, R90 to R116, R9 to R117, R31 to R118, R55 to R119, R88 to R12, R81 to R120, R109 to R121, R117 to R122, R128 to R124, R118 to R125, R132 to R126, R18 to R127, R42 to R128, R67 to R129, R8 to R13, R91 to R130, R110 to R131, R124 to R132, R4 to R133, R27 to R134, R51 to R135, R77 to R136, R19 to R137, R43 to R138, R68 to R139, R33 to R14, R92 to R140, R10 to R141, R32 to R142, R56 to R143, R82 to R144, R104 to R145, R20 to R146, R44 to R147, R69 to R148, R93 to R149, R137 to R15, R97 to R16, R99 to R17, R15 to R18, R98 to R19, R64 to R2, R6 to R20, R74 to R21, R7 to R22, R63 to R23, R75 to R24, R146 to R25, R148 to R26, R149 to R27, R36 to R29, R96 to R3, R61 to R30, R39 to R31, R29 to R32, R105 to R33, R121 to R34, R47 to R35, R54 to R36, R72 to R37, R80 to R38, R1 to R39, R103 to R4, R13 to R40, R24 to R41, R35 to R42, R100 to R43, R108 to R44, R119 to R45, R122 to R46, R57 to R47, R83 to R48, R14 to R49, R11 to R5, R38 to R50, R114 to R51, R125 to R52, R48 to R53, R73 to R54, R2 to R55, R25 to R56, R101 to R57, R120 to R58, R134 to R59, R23 to R6, R135 to R60, R52 to R61, R58 to R62, R62 to R63, R78 to R64, R84 to R65, R87 to R66, R129 to R67, R136 to R68, R106 to R69, R37 to R7, R115 to R70, R130 to R71, R142 to R72, R59 to R73, R85 to R74, R143 to R75, R107 to R76, R138 to R77, R144 to R78, R111 to R79, R49 to R8, R147 to R80, R131 to R81, R140 to R82, R139 to R83, R141 to R84, R112 to R85, R133 to R86, R21 to R87, R45 to R88, R70 to R89, R126 to R9, R94 to R90, R12 to R91, R22 to R92, R34 to R93, R46 to R94, R60 to R95, R71 to R96, R86 to R97, R95 to R98, R113 to R99, RV18 to RV1, RV4 to RV10, RV22 to RV11, RV3 to RV12, RV7 to RV13, RV11 to RV14, RV16 to RV15, RV19 to RV16, RV2 to RV17, RV6 to RV18, RV9 to RV19, RV10 to RV2, RV15 to RV20, RV20 to RV21, RV21 to RV22, RV17 to RV3, RV13 to RV4, RV12 to RV5, RV5 to RV6, RV8 to RV7, RV14 to RV8, RV1 to RV9, SW12 to SW1, SW11 to SW10, SW7 to SW11, SW9 to SW12, SW4 to SW3, SW5 to SW4, SW1 to SW5, SW3 to SW6, SW6 to SW7, SW10 to SW9, U15 to U10, U16 to U10, U5 to U10, U6 to U10, U14 to U10, U7 to U11, U20 to U11, U18 to U11, U15 to U11, U14 to U11, U8 to U12, U7 to U12, U22 to U12, U6 to U13, U23 to U13, U9 to U13, U25 to U14, U12 to U14, U10 to U14, U7 to U15, U11 to U15, U2 to U15, U10 to U16, U23 to U16, U3 to U16, U13 to U17, U19 to U17, U20 to U18, U15 to U18, U23 to U18, U3 to U19, U16 to U19, U11 to U19, U13 to U20, U21 to U20, U18 to U20, U19 to U21, U15 to U21, U24 to U21, U14 to U22, U24 to U22, U26 to U23, U8 to U23, U20 to U23, U19 to U23, U21 to U24, U16 to U24, U5 to U24, U17 to U25, U4 to U3, U25 to U4, U27 to U6, U28 to U7, U5 to U8, U3 to U8, U6 to U8, U1 to U8, U12 to U9, U8 to U9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
Connections:
- net +15V: now also C28.2, U5.4 (V+)
- net -15V: now also C29.2, U5.11 (V-)
- net GND: now also C28.1, C29.1, U22.10 (+), U22.12 (+), U22.5 (+)
- net Pegel_Aux_Return: now also U23.8, U23.9 (-); no longer U23.13 (-), U23.14
- net Pegel_Post: now also U23.13 (-), U23.14; no longer U23.6 (-), U23.7
- net Pegel_Pre: now also U23.1, U23.2 (-); no longer U23.8, U23.9 (-)
- net at R35.1, RV7.1, SW3.1 (A): now also U10.1; no longer U10.14
- net at R36.1, RV7.2, RV7.3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: now also U10.2 (-); no longer U10.13 (-)
- net at C70.1, R109.2: now also U15.1, U15.2 (-); no longer U15.8, U15.9 (-)
- net at R57.1, Z142.1: now also U12.14; no longer U12.7
- net at R43.1, R57.2: now also U12.13 (-); no longer U12.6 (-)
- net at C37.1, R85.1: now also U13.5 (+); no longer U13.10 (+)
- net at R145.1, Z225.1: now also U21.8; no longer U21.1
- net at R145.2, R146.2, R147.2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: now also U21.9 (-); no longer U21.2 (-)
- net at Z211.1: now also U21.10 (+); no longer U21.3 (+)
- net at Z133.2, Z137.1: now also U23.12 (+); no longer U23.5 (+)
- net at R29.2, R31.2: now also U3.3 (+); no longer U3.9 (-)
- net at C59.2, R118.2: now also U16.3 (+); no longer U16.10 (+)
- net at R83.1, Z175.1, Z176.1: now also U14.7; no longer U14.14
- net at C61.2, R120.2: now also U18.3 (+); no longer U18.10 (+)
- net at R37.2, R54.1: now also U11.9 (-); no longer U11.2 (-)
- net at R54.2, Z139.1: now also U11.8; no longer U11.1
- net at R37.1, RV8.1, SW4.1 (A): now also U11.7; no longer U11.14
- net at R38.1, RV8.2, RV8.3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: now also U11.6 (-); no longer U11.13 (-)
- net at R55.2, Z140.1: now also U8.7; no longer U8.1
- net at R39.2, R55.1: now also U8.6 (-); no longer U8.2 (-)
- net at R40.2, R49.2: now also U8.5 (+); no longer U8.3 (+)
- net at J29.1 (Pin_1), Z226.2: now also U21.12 (+), U22.3 (+); no longer U21.10 (+), U22.12 (+)
- net at C72.1, R111.2: now also U17.1, U17.2 (-); no longer U17.8, U17.9 (-)
- net at RV14.2: now also U10.12 (+); no longer U10.5 (+)
- net at R58.1, Z143.1: now also U13.14; no longer U13.7
- net at R69.1, R70.1, R76.2: now also U13.2 (-); no longer U13.12 (+)
- net at Z158.1: now also U13.3 (+); no longer U13.13 (-)
- net at R76.1, Z163.1: now also U13.1; no longer U13.14
- net at R102.2, RV13.3, Z182.1: now also U9.14; no longer U9.1
- net at R102.1, R93.2: now also U9.13 (-); no longer U9.2 (-)
- net at C43.1, RV18.1, RV18.2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: now also U9.12 (+); no longer U9.3 (+)
- net at C82.2, R141.2: now also U15.5 (+); no longer U15.12 (+)
- net at R61.2, R62.2, R63.2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: now also U10.9 (-); no longer U10.13 (-)
- net at R73.2, Z159.1: now also U10.8; no longer U10.14
- net at C60.2, R119.2: now also U17.3 (+); no longer U17.10 (+)
- net at Z236.1, Z246.1: now also U22.1, U22.2 (-); no longer U22.13 (-), U22.14
- net at Z132.2, Z136.1: now also U23.10 (+); no longer U23.12 (+)
- net at R32.2, Z84.1, Z89.1: now also U3.1; no longer U3.8
- net at R34.1, R45.2, SW8.1 (A): now also U13.8; no longer U13.1
- net at R34.2, R46.2, SW8.2 (B): now also U13.9 (-); no longer U13.2 (-)
- net at Z112.2, Z116.1: now also U13.10 (+); no longer U13.3 (+)
- net at C58.2, R117.2: now also U15.3 (+); no longer U15.10 (+)
- net at RV1.2: now also U3.12 (+); no longer U3.5 (+)
- net at R30.2, RV4.3, Z78.1: now also U3.8; no longer U3.1
- net at R23.2, R30.1: now also U3.9 (-); no longer U3.2 (-)
- net at C30.1, RV5.1, RV5.2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: now also U3.10 (+); no longer U3.3 (+)
- net at R41.2, R56.1: now also U9.6 (-); no longer U9.2 (-)
- net at R56.2, Z141.1: now also U9.7; no longer U9.1
- net at R71.2, U24.10 (+), U24.7: now also U24.12 (+); no longer U24.10 (+)
- net at R42.1, RV10.2, RV10.3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: now also U9.2 (-); no longer U9.13 (-)
- net at R41.1, RV10.1, SW6.1 (A): now also U9.1; no longer U9.14
- net at R122.1, R125.1: now also U21.5 (+); no longer U21.12 (+)
- net at R42.2, R50.2: now also U9.5 (+); no longer U9.3 (+)
- net at R99.1, RV16.3, Z178.1: now also U13.7; no longer U13.8
- net at C84.2, R143.2: now also U17.5 (+); no longer U17.12 (+)
- net at C42.1, RV17.1, RV17.2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: now also U8.12 (+); no longer U8.3 (+)
- net at R131.1, Z205.1, Z207.1: now also U21.7; no longer U21.14
- net at R121.1, R131.2: now also U21.6 (-); no longer U21.13 (-)
- net at R33.1, R43.2, SW7.1 (A): now also U12.8; no longer U12.1
- net at R33.2, R44.2, SW7.2 (B): now also U12.9 (-); no longer U12.2 (-)
- net at RV12.2: now also U8.10 (+); no longer U8.5 (+)
- net at R101.2, RV12.3, Z181.1: now also U8.14; no longer U8.1
- net at R100.1, R99.2: now also U13.6 (-); no longer U13.9 (-)
- net at Z235.1, Z245.1: now also U21.13 (-), U21.14; no longer U21.8, U21.9 (-)
- net at R38.2, R48.2: now also U11.10 (+); no longer U11.3 (+)
- net at R101.1, R91.2: now also U8.13 (-); no longer U8.2 (-)
- net at R136.2, Z188.1: now also U18.6 (-), U18.7; no longer U18.13 (-), U18.14
- net at U14.10 (+), Z180.2: now also U14.3 (+), U21.3 (+); no longer U14.10 (+), U21.10 (+)
- net at R35.2, R53.1: now also U10.6 (-); no longer U10.2 (-)
- net at R53.2, Z138.1: now also U10.7; no longer U10.1
- net at R46.1, R52.1: now also U13.12 (+); no longer U13.5 (+)
- net at Z156.1: now also U10.10 (+); no longer U10.12 (+)
- net at R45.1, R58.2: now also U13.13 (-); no longer U13.6 (-)
- net at R133.2, Z185.2: now also U15.6 (-), U15.7; no longer U15.13 (-), U15.14
- net at R122.2, RV21.2, RV21.3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: now also U21.2 (-); no longer U21.9 (-)
- net at R78.1, R80.1: now also U14.5 (+); no longer U14.12 (+)
- new net: C40.2, U10.13 (-), U10.14
- new net: U10.3 (+), U11.5 (+), U12.10 (+), U8.3 (+), U9.3 (+), Z110.2, Z114.1, Z119.1, Z121.1
- new net: C39.2, U9.8, U9.9 (-)
- new net: C1.2, U3.13 (-), U3.14
- new net: U22.6 (-), U22.7
- new net: U22.8, U22.9 (-)
- new net: U24.13 (-), U24.14, Z167.1
- new net: C38.2, U8.8, U8.9 (-)
- new net: U22.13 (-), U22.14
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Other:
- note removed: "LEGENDE"
- note removed: "Leiterbahn"
- note removed: "Leiterkabel"
- note removed: "Platinen Bereich"
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
Commit message: final PCB Update
Parts:
- removed C7, C8: 0.1uF, Capacitor_SMD:C_0805_2012Metric_Pad1.18x1.45mm_HandSolder, symbol Device:C_Small
- removed J12, J22, J23: EMK_In, Connector_PinHeader_2.54mm_LongPads:PinHeader_1x05_P2.54mm_Vertical_LongPads, symbol Connector:Conn_01x05_Pin
- removed J13, J14, J21: EMK_Out, Connector_PinSocket_2.54mm_LongPads:PinSocket_1x05_P2.54mm_Vertical_LongPads, symbol Connector:Conn_01x05_Socket
- removed L1: 470uF, 1.6A, WE-SL575:WE-SL575, symbol Device:L_Coupled
- removed R2: 100R, Resistor_SMD:R_0805_2012Metric_Pad1.20x1.40mm_HandSolder, symbol Device:R
- removed R25, R26, R27: 22R, Resistor_SMD:R_0805_2012Metric_Pad1.20x1.40mm_HandSolder, symbol Device:R
- removed SW10, SW11, SW12, SW3, SW4, SW5, SW6, SW7, SW8: SW_SPDT, Connector_PinSocket_2.54mm_LongPads:PinSocket_1x03_P2.54mm_Vertical_LongPads, symbol Switch:SW_SPDT
- removed SW9: Pegel_Selector, Connector_PinSocket_2.54mm_LongPads:PinSocket_1x05_P2.54mm_Vertical_LongPads, symbol Switch:SW_Rotary_1x4_MP
- removed unit 5 of U10
- removed unit 5 of U12
- removed unit 5 of U13
- removed unit 4 of U2
- removed U25: INA128U, INA128U:INA128U_L, symbol INA128U:INA128U
- removed unit 1 of U4
- removed Z185, Z193, Z198: ~, Resistor_SMD:R_0805_2012Metric_Pad1.20x1.40mm_HandSolder, symbol Device:R_Small
- added C100, C89: 10n, Capacitor_SMD:C_0805_2012Metric_Pad1.18x1.45mm_HandSolder, symbol Device:C_Small
- added C114, C118, C91: 10u, Capacitor_THT:CP_Radial_D5.0mm_P2.50mm, symbol Device:C_Polarized_Small
- added C3, C4, C85: 10n, Capacitor_SMD:C_1210_3225Metric_Pad1.33x2.70mm_HandSolder, symbol Device:C_Small
- added C52, C53, C59, C60: 100n, Capacitor_SMD:C_0805_2012Metric_Pad1.18x1.45mm_HandSolder, symbol Device:C_Small
- added H1, H10, H11, H13, H14, H15, H16, H2, H5, H6, H7, H8, H9: MountingHole, MountingHole:MountingHole_3.2mm_M3_Pad, symbol Mechanical:MountingHole
- added H12, H3, H4: MountingHole_Pad, MountingHole:MountingHole_3.2mm_M3_Pad, symbol Mechanical:MountingHole_Pad
- added J30, J31, J40, J41: Conn_02x07_Odd_Even, Connector_PinHeader_2.54mm:PinHeader_2x07_P2.54mm_Vertical, symbol Connector_Generic:Conn_02x07_Odd_Even
- added L4: ~, WE-SL575:WE-SL575, symbol Common_Mode_Choke:Common_Mode_Choke
- added R52, R53, R57, R67, R75, R80: 10k, Resistor_SMD:R_0805_2012Metric_Pad1.20x1.40mm_HandSolder, symbol Device:R
- added SW1, SW10, SW3, SW4, SW5, SW6, SW7, SW8, SW9: SW_SPDT, Connector_PinHeader_2.54mm_LongPads:PinHeader_1x02_P2.54mm_Vertical_LongPads, symbol sw_spdt_2:SW_SPDT
- added SW11: SW_Rotary_1x4, Connector_PinHeader_2.54mm_LongPads:PinHeader_1x05_P2.54mm_Vertical_LongPads, symbol SW_Rotary_1x4:SW_Rotary_1x4_MP
- added unit 1 of U11
- added unit 3 of U11
- added unit 4 of U11
- added unit 2 of U11
- added unit 3 of U17
- added unit 5 of U18
- added unit 4 of U19
- added unit 5 of U2
- added unit 5 of U5
- added unit 5 of U7
- added unit 4 of U8
- added unit 2 of U8
- added unit 5 of U8
- added unit 3 of U8
- added unit 4 of U9
- added Z231, Z234, Z235, Z241, Z255, Z258, Z28, Z29, Z36: ~, Resistor_SMD:R_0805_2012Metric_Pad1.20x1.40mm_HandSolder, symbol Device:R
- C115: renamed from C2; footprint Capacitor_SMD:C_0805_2012Metric_Pad1.18x1.45mm_HandSolder -> Capacitor_SMD:C_1210_3225Metric_Pad1.33x2.70mm_HandSolder
- C116: renamed from C5; footprint Capacitor_SMD:C_0805_2012Metric_Pad1.18x1.45mm_HandSolder -> Capacitor_SMD:C_1210_3225Metric_Pad1.33x2.70mm_HandSolder
- renumbered C21 to C1, C52 to C10, C36 to C101, C24 to C102, C10 to C103, C67 to C104, C79 to C105, C97 to C106, C101 to C107, C105 to C108, C74 to C11, C11 to C110, C25 to C111, C4 to C112, C19 to C113, C20 to C117, C6 to C119, C43 to C12, C26 to C120, C12 to C121, C62 to C13, C86 to C14, C39 to C15, C49 to C16, C59 to C17, C71 to C18, C83 to C19, C27 to C2, C53 to C20, C75 to C21, C42 to C22, C63 to C23, C87 to C24, C38 to C25, C50 to C26, C60 to C27, C72 to C28, C84 to C29, C54 to C30, C76 to C31, C44 to C32, C3 to C33, C64 to C34, C88 to C35, C40 to C36, C1 to C37, C51 to C38, C61 to C39, C73 to C40, C85 to C41, C55 to C42, C77 to C43, C45 to C44, C65 to C45, C89 to C46, C41 to C47, C30 to C48, C22 to C49, C48 to C5, C35 to C50, C37 to C51, C13 to C54, C16 to C55, C31 to C56, C33 to C57, C28 to C58, C58 to C6, C14 to C61, C17 to C62, C32 to C63, C34 to C64, C29 to C65, C110 to C66, C68 to C67, C80 to C68, C92 to C69, C70 to C7, C111 to C70, C69 to C71, C81 to C72, C93 to C73, C90 to C74, C94 to C75, C98 to C76, C102 to C77, C106 to C78, C91 to C79, C82 to C8, C95 to C80, C99 to C81, C103 to C82, C107 to C83, C9 to C84, C23 to C86, C46 to C87, C56 to C88, C15 to C9, C18 to C90, C47 to C92, C57 to C93, C66 to C94, C78 to C95, C100 to C97, C104 to C98, C108 to C99, D2 to D1, D1 to D2, D4 to D3, D3 to D4, J40 to J1, J42 to J10, J43 to J11, J20 to J12, J27 to J13, J16 to J14, J24 to J15, J15 to J16, J7 to J17, J38 to J18, J44 to J19, J1 to J2, J6 to J20, J45 to J21, J8 to J22, J17 to J23, J25 to J24, J37 to J25, J39 to J26, J18 to J27, J9 to J28, J28 to J29, J2 to J3, J29 to J32, J30 to J33, J36 to J34, J31 to J35, J32 to J36, J34 to J37, J35 to J38, J10 to J39, J19 to J4, J33 to J42, J11 to J43, J26 to J5, J41 to J6, J3 to J7, J4 to J8, J5 to J9, R39 to R1, R117 to R10, R98 to R100, R23 to R101, R16 to R102, R19 to R103, R17 to R104, R21 to R105, R24 to R106, R43 to R107, R57 to R108, R145 to R109, R141 to R11, R33 to R110, R69 to R111, R76 to R112, R44 to R113, R121 to R114, R131 to R115, R79 to R116, R85 to R117, R99 to R118, R51 to R119, R93 to R12, R70 to R120, R100 to R121, R125 to R123, R45 to R124, R58 to R125, R9 to R126, R34 to R127, R46 to R128, R77 to R129, R40 to R13, R83 to R130, R123 to R131, R52 to R133, R10 to R134, R15 to R135, R78 to R136, R124 to R137, R80 to R138, R126 to R139, R49 to R14, R11 to R140, R67 to R141, R71 to R142, R81 to R143, R86 to R144, R59 to R145, R60 to R146, R68 to R147, R82 to R148, R84 to R149, R18 to R15, R72 to R150, R75 to R151, R6 to R16, R105 to R17, R113 to R18, R127 to R19, R55 to R2, R137 to R20, R146 to R21, R88 to R22, R94 to R23, R28 to R24, R32 to R25, R41 to R26, R56 to R27, R110 to R28, R134 to R29, R20 to R3, R14 to R30, R101 to R31, R29 to R32, R7 to R33, R118 to R34, R142 to R35, R31 to R36, R91 to R37, R42 to R38, R50 to R39, R22 to R4, R106 to R40, R114 to R41, R128 to R42, R138 to R43, R147 to R44, R8 to R45, R87 to R46, R92 to R47, R35 to R48, R53 to R49, R109 to R5, R111 to R50, R135 to R51, R61 to R54, R103 to R55, R36 to R56, R12 to R58, R119 to R59, R133 to R6, R143 to R60, R47 to R61, R73 to R63, R95 to R64, R3 to R65, R63 to R66, R107 to R68, R115 to R69, R13 to R7, R129 to R70, R139 to R71, R148 to R72, R89 to R73, R96 to R74, R1 to R76, R4 to R77, R37 to R78, R54 to R79, R102 to R8, R112 to R81, R136 to R82, R64 to R83, R104 to R84, R38 to R85, R120 to R86, R144 to R87, R48 to R88, R65 to R89, R5 to R9, R74 to R90, R97 to R91, R66 to R92, R30 to R93, R108 to R94, R116 to R95, R130 to R96, R140 to R97, R149 to R98, R90 to R99, RV9 to RV1, RV14 to RV12, RV1 to RV13, RV8 to RV14, RV15 to RV16, RV4 to RV18, RV21 to RV20, RV11 to RV21, RV13 to RV3, RV6 to RV4, RV10 to RV5, RV12 to RV7, RV7 to RV8, RV2 to RV9, SW1 to SW12, U8 to U1, U9 to U1, U11 to U10, U9 to U10, U17 to U12, U18 to U12, U16 to U12, U20 to U13, U18 to U13, U10 to U14, U12 to U14, U11 to U14, U3 to U15, U17 to U16, U18 to U16, U4 to U17, U5 to U17, U13 to U18, U12 to U18, U5 to U19, U16 to U2, U15 to U2, U21 to U20, U22 to U20, U13 to U21, U22 to U21, U14 to U21, U14 to U22, U21 to U22, U20 to U22, U24 to U23, U23 to U24, U6 to U25, U7 to U26, U19 to U3, U1 to U4, U9 to U5, U8 to U5, U15 to U6, U16 to U6, U10 to U7, U22 to U7, U11 to U7, U4 to U8, U2 to U9, Z238 to Z1, Z68 to Z10, Z58 to Z100, Z214 to Z101, Z223 to Z102, Z187 to Z103, Z203 to Z104, Z232 to Z105, Z252 to Z106, Z156 to Z107, Z218 to Z108, Z19 to Z109, Z5 to Z11, Z195 to Z110, Z242 to Z111, Z9 to Z112, Z29 to Z113, Z243 to Z114, Z139 to Z115, Z151 to Z116, Z184 to Z117, Z201 to Z118, Z233 to Z119, Z25 to Z12, Z253 to Z120, Z145 to Z121, Z192 to Z122, Z160 to Z123, Z165 to Z124, Z162 to Z125, Z215 to Z126, Z224 to Z127, Z188 to Z128, Z204 to Z129, Z190 to Z13, Z234 to Z130, Z254 to Z131, Z157 to Z132, Z219 to Z133, Z78 to Z134, Z79 to Z135, Z71 to Z136, Z76 to Z137, Z196 to Z138, Z244 to Z139, Z41 to Z14, Z85 to Z140, Z111 to Z141, Z73 to Z142, Z77 to Z143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
Connections:
- net Pegel_Aux_Return: now also U24.1, U24.2 (-), SW11.2; no longer U24.8, U24.9 (-)
- net Pegel_Mic_Effekt: now also SW11.3
- net Pegel_Post: now also U24.6 (-), U24.7, SW11.1; no longer U24.13 (-), U24.14
- net Pegel_Pre: now also SW11.4
- net at R7.2, Z9.1: now also U4.14; no longer U4.8
- net at R48.1, RV8.1, U10.1: now also SW4.1 (A)
- net at R56.1, RV8.2, RV8.3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: now also SW4.2 (B)
- net at R12.1, RV3.1: now also Z18.2; no longer Z61.2
- net at U13.5 (+), Z102.2: now also U13.10 (+); no longer U13.3 (+)
- net at C51.1, R117.1: now also U21.10 (+); no longer U21.5 (+)
- net at C1.1, C9.2, R3.2: now also U4.9 (-); no longer U4.13 (-)
- net at RV9.1: now also R67.2, U11.2 (-)
- net at RV9.2, RV9.3: now also R57.1, U11.6 (-)
- net at R135.1, Z204.1, Z211.1: now also U19.8; no longer U19.7
- net at R126.1, R134.1, R135.2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: now also U19.9 (-); no longer U19.6 (-)
- net at Z1.1, Z7.1: now also U3.8, U3.9 (-); no longer U3.1, U3.2 (-)
- net at Z259.2, Z262.1: now also U24.5 (+); no longer U24.12 (+)
- net at R32.1, RV4.2, RV4.3: now also U8.6 (-)
- net at R32.2, R36.2: now also U8.10 (+); no longer U15.3 (+)
- net at R83.2, R89.2, R90.1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: now also U7.6 (-); no longer U7.13 (-)
- net at C17.2, R34.2: now also U2.5 (+); no longer U2.3 (+)
- net at Z189.2, Z193.1: now also U17.3 (+); no longer U17.12 (+)
- net at R130.1, Z208.1, Z219.1: now also U21.14; no longer U21.7
- net at C117.2, C120.1, C121.2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: now also Z258.1
- net at C39.2, R86.2: now also U12.5 (+); no longer U12.3 (+)
- net at C110.2, C111.2, C113.1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: now also Z255.1
- net at R78.1, RV14.1, U10.7: now also SW5.1 (A)
- net at R85.1, RV14.2, RV14.3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: now also SW5.2 (B)
- net at R13.2, R14.2: now also U1.12 (+); no longer U1.5 (+)
- net at R1.2, R2.1: now also U1.13 (-); no longer U1.6 (-)
- net at R2.2, Z17.1: now also U1.14; no longer U1.7
- net at R131.2, RV22.1, U22.8: now also SW10.1 (A)
- net at R137.2, RV22.2, RV22.3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: now also SW10.2 (B)
- net at Z201.2, Z207.1: now also U19.3 (+); no longer U19.12 (+)
- net at R102.2, R103.1, R104.2: now also U17.13 (-); no longer U17.9 (-)
- net at R103.2, Z136.1: now also U17.14; no longer U17.8
- net at C35.2, R71.2: now also U16.5 (+); no longer U16.12 (+)
- net at RV12.2: now also U14.3 (+); no longer U14.12 (+)
- net at D2.1 (K), R145.2, R146.1: now also U23.13 (-); no longer U23.2 (-)
- net at R125.1, Z195.1: now also U18.8; no longer U18.14
- net at C115.1, SW12.4: now also L4.1
- net at C110.1, C112.2, C116.1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: now also C89.2, L4.2
- net at C115.2, SW12.2: now also L4.4
- net at C103.1, C116.2, C119.1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: now also C100.1, L4.3
- net at R112.1, Z164.1: now also U21.7; no longer U21.1
- net at R111.1, R112.2, R120.1: now also U21.6 (-); no longer U21.2 (-)
- net at Z182.1: now also U21.5 (+); no longer U21.3 (+)
- net at C44.1, RV15.1, RV15.2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: now also U14.10 (+); no longer U14.3 (+)
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Other:
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
Commit message: final pcb update
Parts:
- added R152, R153, R154, R155, R156, R157: 10k, Resistor_SMD:R_0805_2012Metric_Pad1.20x1.40mm_HandSolder, symbol Device:R
- added Z263, Z264, Z265, Z266, Z267, Z268, Z269, Z270, Z271, Z272, Z273, Z274: ~, Resistor_SMD:R_0805_2012Metric_Pad1.20x1.40mm_HandSolder, symbol Device:R
- C1, C100, C101, C102, C103, C110, C111, C112, C113, C114, C115, C116, C117, C118, C119, C120, C121, C2, C3, C33, C37, C48, C49, C52, C53, C54, C55, C56, C57, C58, C59, C60, C61, C62, C63, C64, C65, C84, C85, C86, C87, C88, C89, C9, C90, C91, C92, C93, D1, D2, D3, D4, H1, H10, H11, H12, H13, H14, H15, H16, H3, H6, H7, H9, J12, J14, J16, J17, J2, J20, J22, J23, J27, J28, J3, J30, J33, J34, J35, J36, J37, J38, J39, J4, J40, J41, J42, J43, J7, J8, J9, L1, L2, L3, L4, L5, R101, R102, R103, R104, R105, R106, R126, R134, R135, R140, R141, R142, R143, R144, R145, R146, R147, R148, R149, R15, R150, R151, R16, R24, R25, R3, R30, R32, R33, R36, R4, R45, R52, R53, R57, R58, R65, R67, R7, R75, R76, R77, R80, R9, R93, RV11, RV13, RV17, RV18, RV4, RV9, SW11, SW12, SW2, U11, U15, U17, U19, U23, U24, U25, U26, U4, U8, U9, Z10, Z100, Z109, Z11, Z112, Z113, Z12, Z134, Z135, Z136, Z137, Z14, Z140, Z142, Z143, Z144, Z145, Z146, Z15, Z150, Z151, Z152, Z154, Z155, Z156, Z157, Z158, Z16, Z175, Z176, Z177, Z178, Z179, Z180, Z181, Z189, Z19, Z190, Z191, Z192, Z193, Z194, Z2, Z201, Z202, Z203, Z204, Z206, Z207, Z21, Z210, Z211, Z212, Z213, Z22, Z224, Z225, Z226, Z227, Z228, Z229, Z23, Z230, Z232, Z237, Z238, Z239, Z240, Z241, Z242, Z243, Z244, Z245, Z246, Z247, Z248, Z249, Z250, Z251, Z252, Z253, Z254, Z255, Z256, Z257, Z258, Z259, Z26, Z260, Z261, Z262, Z27, Z32, Z33, Z35, Z38, Z40, Z41, Z42, Z49, Z5, Z50, Z51, Z54, Z55, Z57, Z58, Z59, Z6, Z62, Z63, Z67, Z72, Z73, Z75, Z76, Z79, Z80, Z86, Z87, Z9, Z94, Z95, Z97, Z98, Z99: now left out of the parts list
Connections:
- net GND_O: now also Z265.2, Z266.2, Z269.2, Z270.2, Z271.2, Z274.2; no longer U20.5 (+), U7.10 (+), U7.12 (+)
- net at R37.1, RV7.1: now also Z268.2; no longer Z61.2
- net at U20.8, Z166.1: now also R109.2; no longer R109.1
- net at R21.2, R44.2, R72.2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: now also R109.1; no longer R109.2
- net at U20.12 (+), U20.3 (+), Z231.2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: now also Z273.2; no longer Z174.2
- net at U20.7: now also R156.1, Z272.1; no longer U20.6 (-)
- net at U7.13 (-): now also R152.1, R153.2; no longer U7.14
- net at R12.1, RV3.1: now also Z264.2; no longer Z18.2
- net at U7.9 (-): now also R154.1, R155.2; no longer U7.8
- new net: R155.1, Z61.2
- new net: U20.5 (+), Z271.1
- new net: R157.1, Z174.2
- new net: Z272.2, Z273.1, Z274.1
- new net: Z267.2, Z268.1, Z269.1
- new net: U7.12 (+), Z266.1
- new net: R152.2, U7.14, Z263.1
- new net: R156.2, R157.2, U20.6 (-)
- new net: U7.10 (+), Z270.1
- new net: R154.2, U7.8, Z267.1
- new net: R153.1, Z18.2
- new net: Z263.2, Z264.1, Z265.1
Other:
- moved on the sheet: C1, C10, C100, C101, C102, C103, C104, C105, C106, C107, C108, C109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

Commit message: Bezeichner und BOM Update
Other:
- title: DiKo Vorverstärker -> Vorverstärker 1
- moved on the sheet: C101, C104, C105, C106, C107, C108, C109, C87, C88, C94, C95, C96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
