File: KiCad/DiKo_PreAmp.kicad_sch (KiCad schematic)
At the start: 683 parts, among them J1 Bass_Out, J10 Mid_Out, J11 High_Out, J12 Mic_Effekt_Out, J13 Mic_Effekt_In, J14 Mic_Effekt_Out, J15 Mic_Effekt_In, J16 Mic_Effekt_Out, J17 Effekt_In, J18 AUX_Send_1, J19 Line_Out_L, J2 R_Phono_In, J20 AUX_RET_1, J21 Line_Out_R, J22 AUX_RET_2, J23 Mic_Effekt_Out, J24 Mic_Effekt_In, J25 AUX_Send_3, J26 AUX_Send_2, J27 Mic_Effekt_Out, J28 AUX_RET_3, J29 Pegel_Out, J3 L_Phono_In, J30 Conn_02x07_Odd_Even, J31 Conn_02x07_Odd_Even, J32 Pegel_Out, J33 Pegel_In, J34 VU_Meter_Out, J35 Pegel_In, J36 Pegel_In, J37 LED_Out, J38 LED_In, J39 VCC_IN, J4 Phono/Line_Out, J40 Conn_02x07_Odd_Even, J41 Conn_02x07_Odd_Even, J42 Pegel_In, J43 VCC_OUT, J5 Phono/Line_In, J6 Kick_Out, J7 R_Line_In, J8 L_Line_In, J9 Mic_In, SW1 SW_SPDT, SW10 SW_SPDT, SW11 SW_Rotary_1x4, SW12 SW_DPST, SW2 SW_SPDT, SW3 SW_SPDT, SW4 SW_SPDT, SW5 SW_SPDT, SW6 SW_SPDT, SW7 SW_SPDT, SW8 SW_SPDT, SW9 SW_SPDT, U1 TL074, U10 TL074, U11 TL074, U12 TL074, U13 TL074, U14 TL074, U15 TL074, U16 TL074, U17 TL074, U18 TL074, U19 TL074, U2 TL074, U20 TL074, U21 TL074, U22 TL074, U23 TL074, U24 TL074, U25 REC10K-2409, U26 REC10K-2415, U3 TL074, U4 TL074, U5 TL074, U6 TL074, U7 TL074, U8 TL074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

Commit message: Mitten update
Parts:
- C26, C27, C28, C29: value 13n6 -> 1n5
- R50, R51: value 10k -> 90k
- R59, R60: value 20k -> 180k
Changed lines of the file:
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@@
 			)
 		)
-		(property "Value" "13n6"
+		(property "Value" "1n5"
 			(at 692.1563 182.88 90)
 			(show_name no)
@@
 			)
 		)
-		(property "Value" "13n6"
+		(property "Value" "1n5"
 			(at 661.6763 182.88 90)
 			(show_name no)
@@
 			)
 		)
-		(property "Value" "13n6"
+		(property "Value" "1n5"
 			(at 708.6663 182.88 90)
 			(show_name no)
@@
 			)
 		)
-		(property "Value" "20k"
+		(property "Value" "180k"
 			(at 716.28 194.3099 0)
 			(show_name no)
@@
 			)
 		)
-		(property "Value" "20k"
+		(property "Value" "180k"
 			(at 670.56 194.3099 0)
 			(show_name no)
@@
 			)
 		)
-		(property "Value" "13n6"
+		(property "Value" "1n5"
 			(at 646.4363 182.88 90)
 			(show_name no)
@@
 			)
 		)
-		(property "Value" "10k"
+		(property "Value" "90k"
 			(at 655.32 181.6099 0)
 			(show_name no)
@@
 			)
 		)
-		(property "Value" "10k"
+		(property "Value" "90k"
 			(at 701.04 181.6099 0)
 			(show_name no)

Commit message: Höhen Update
Parts:
- added R161, R162: 10k, Resistor_SMD:R_0805_2012Metric_Pad1.20x1.40mm_HandSolder, symbol Device:R
- C38, C39, C40, C41: value 130n -> 3n
- C42, C45: value 130n -> 2n2
- C43: value 130n -> 6n8
- C46: value 130n -> 1n
- R81, R82: value 6k8 -> 7k5
- R86, R87: value 6k8 -> 15k
- R94, R95: value 22k -> 3k9
- R96, R97: value 22k -> 3k3
- Z114, Z197: value (none) -> 1u
- Z120, Z200: value (none) -> 100k
- Z126, Z127, Z128, Z129, Z130, Z131, Z217, Z231: value (none) -> 0R
- Z133, Z138: value (none) -> 820k
Connections:
- net at R160.1, R66.1, R92.1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: now also R162.1
- net at R152.1, R153.2, U7.13 (-): now also R161.2, R162.2
- net at R159.1, R62.1, R89.1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: now also R161.1
Other:
- moved on the sheet: J21, J32, R153, Z218, Z231, Z233, Z234, Z235, Z236

Commit message: Finales Update Ausgangsstufe
Parts:
- added R163, R164, R165, R166: 1k, Resistor_SMD:R_0805_2012Metric_Pad1.20x1.40mm_HandSolder, symbol Device:R
- Z183, Z208, Z209: value (none) -> 1u
- Z186, Z222: value (none) -> 100k
- Z220: value (none) -> 100K
Connections:
- net at R38.1, RV5.2, SW3.2 (B)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: now also R164.1; no longer RV5.3
- net at R85.1, RV14.2, SW5.2 (B)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: now also R166.1; no longer RV14.3
- net at R13.1, RV1.2, SW1.2 (B)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: now also R163.1; no longer RV1.3
- net at R56.1, RV8.2, SW4.2 (B)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: now also R165.1; no longer RV8.3
- new net: R163.2, RV1.3
- new net: R164.2, RV5.3
- new net: R166.2, RV14.3
- new net: R165.2, RV8.3
Other:
- moved on the sheet: J18, J25, J26, RV1, RV14, RV5, RV8, SW1, SW3, SW4, SW5

Commit message: Pegel Update
Parts:
- R142: value 80k -> 20k
- R150: value 12k -> 100R
- R151: value 3k -> 3k3
- Z237, Z244, Z249, Z259: value (none) -> 2u2
- Z240, Z248, Z254, Z262: value (none) -> 100k
- Z250, Z251, Z257: value (none) -> 0R
Connections:
- net GND_M: now also Z245.1; no longer Z245.2
- net at Z242.2, Z243.1: now also Z245.2; no longer Z245.1
Other:
- moved on the sheet: R150
Changed lines of the file:
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@@
 	)
 	(junction
-		(at 511.81 537.21)
-		(diameter 0)
-		(color 0 0 0 0)
-	)
-	(junction
 		(at 652.78 186.69)
 		(diameter 0)
@@
 	)
 	(junction
+		(at 511.81 537.21)
+		(diameter 0)
+		(color 0 0 0 0)
+	)
+	(junction
 		(at 786.13 250.19)
 		(diameter 0)
@@
 	(wire
 		(pts
-			(xy 505.46 537.21) (xy 511.81 537.21)
+			(xy 492.76 537.21) (xy 511.81 537.21)
 		)
 		(stroke
@@
 	(wire
 		(pts
-			(xy 505.46 539.75) (xy 505.46 537.21)
+			(xy 492.76 539.75) (xy 492.76 537.21)
 		)
 		(stroke
@@
 	(wire
 		(pts
-			(xy 505.46 549.91) (xy 505.46 547.37)
+			(xy 492.76 549.91) (xy 492.76 547.37)
 		)
 		(stroke
@@
 		(dnp no)
 		(property "Reference" "Z244"
-			(at 377.19 506.222 90)
+			(at 377.19 504.952 90)
 			(show_name no)
 			(do_not_autoplace no)
@@
 			)
 		)
-		(property "Value" ""
-			(at 377.19 505.46 90)
-			(hide yes)
+		(property "Value" "2u2"
+			(at 377.19 506.984 90)
 			(show_name no)
 			(do_not_autoplace no)
@@
 		(dnp no)
 		(property "Reference" "Z259"
-			(at 377.19 549.402 90)
+			(at 377.19 548.132 90)
 			(show_name no)
 			(do_not_autoplace no)
@@
 			)
 		)
-		(property "Value" ""
-			(at 377.19 548.64 90)
-			(hide yes)
+		(property "Value" "2u2"
+			(at 377.19 550.164 90)
 			(show_name no)
 			(do_not_autoplace no)
@@
 		(dnp no)
 		(property "Reference" "Z262"
-			(at 385.318 558.8 90)
+			(at 386.588 557.784 0)
 			(show_name no)
 			(do_not_autoplace no)
@@
 			)
 		)
-		(property "Value" ""
-			(at 386.08 558.8 90)
-			(hide yes)
+		(property "Value" "100k"
+			(at 386.588 560.07 0)
 			(show_name no)
 			(do_not_autoplace no)
@@
 	(symbol
 		(lib_id "Device:R")
-		(at 505.46 543.56 180)
+		(at 492.76 543.56 0)
+		(mirror x)
 		(unit 1)
 		(body_style 1)
@@
 		(in_pos_files yes)
 		(dnp no)
-		(fields_autoplaced yes)
 		(property "Reference" "R150"
-			(at 502.92 544.8301 0)
+			(at 495.808 542.544 0)
 			(show_name no)
 			(do_not_autoplace no)
@@
 			)
 		)
-		(property "Value" "12k"
-			(at 502.92 542.2901 0)
+		(property "Value" "100R"
+			(at 495.554 544.8301 0)
 			(show_name no)
 			(do_not_autoplace no)
@@
 		)
 		(property "Footprint" "Resistor_SMD:R_0805_2012Metric_Pad1.20x1.40mm_HandSolder"
-			(at 507.238 543.56 90)
+			(at 490.982 543.56 90)
 			(hide yes)
 			(show_name no)
@@
 		)
 		(property "Datasheet" ""
-			(at 505.46 543.56 0)
+			(at 492.76 543.56 0)
 			(hide yes)
 			(show_name no)
@@
 		)
 		(property "Description" "Resistor"
-			(at 505.46 543.56 0)
+			(at 492.76 543.56 0)
 			(hide yes)
 			(show_name no)
@@
 		)
 		(property "Height" ""
-			(at 505.46 543.56 0)
+			(at 492.76 543.56 0)
 			(hide yes)
 			(show_name no)
@@
 		)
 		(property "Manufacturer_Name" ""
-			(at 505.46 543.56 0)
+			(at 492.76 543.56 0)
 			(hide yes)
 			(show_name no)
@@
 		)
 		(property "Manufacturer_Part_Number" ""
-			(at 505.46 543.56 0)
+			(at 492.76 543.56 0)
 			(hide yes)
 			(show_name no)
@@
 		)
 		(property "Mouser Part Number" ""
-			(at 505.46 543.56 0)
+			(at 492.76 543.56 0)
 			(hide yes)
 			(show_name no)
@@
 		)
 		(property "Mouser Price/Stock" ""
-			(at 505.46 543.56 0)
+			(at 492.76 543.56 0)
 			(hide yes)
 			(show_name no)
@@
 		)
 		(property "Mouser-Teilenr." ""
-			(at 505.46 543.56 0)
+			(at 492.76 543.56 0)
 			(hide yes)
 			(show_name no)
@@
 		)
 		(property "Gegenstück Mouser Teilenr." ""
-			(at 505.46 543.56 0)
+			(at 492.76 543.56 0)
 			(hide yes)
 			(show_name no)
@@
 		(lib_id "Device:R")
 		(at 543.56 511.81 0)
-		(mirror y)
+		(mirror x)
 		(unit 1)
 		(body_style 1)
@@
 		(dnp no)
 		(property "Reference" "Z245"
-			(at 540.512 511.81 90)
+			(at 546.608 511.81 90)
 			(show_name no)
 			(do_not_autoplace no)
@@
 		)
 		(property "Value" ""
-			(at 539.75 511.81 90)
+			(at 547.37 511.81 90)
 			(hide yes)
 			(show_name no)
@@
 		)
 		(property "Footprint" "Resistor_SMD:R_0805_2012Metric_Pad1.20x1.40mm_HandSolder"
-			(at 545.338 511.81 90)
+			(at 541.782 511.81 90)
 			(hide yes)
 			(show_name no)
@@
 			)
 		)
-		(property "Value" "80k"
+		(property "Value" "20k"
 			(at 504.19 499.11 90)
 			(show_name no)
@@
 		(dnp no)
 		(property "Reference" "Z250"
-			(at 538.48 531.622 90)
+			(at 538.48 528.574 90)
 			(show_name no)
 			(do_not_autoplace no)
@@
 			)
 		)
-		(property "Value" ""
+		(property "Value" "0R"
 			(at 538.48 530.86 90)
-			(hide yes)
 			(show_name no)
 			(do_not_autoplace no)
@@
 		(dnp no)
 		(property "Reference" "Z251"
-			(at 548.64 531.622 90)
+			(at 548.64 528.32 90)
 			(show_name no)
 			(do_not_autoplace no)
@@
 			)
 		)
-		(property "Value" ""
+		(property "Value" "0R"
 			(at 548.64 530.86 90)
-			(hide yes)
 			(show_name no)
 			(do_not_autoplace no)
@@
 			)
 		)
-		(property "Value" "3k"
+		(property "Value" "3k3"
 			(at 514.35 544.8299 0)
 			(show_name no)
@@
 		(dnp no)
 		(property "Reference" "Z248"
-			(at 385.318 515.62 90)
+			(at 386.334 514.35 0)
 			(show_name no)
 			(do_not_autoplace no)
@@
 			)
 		)
-		(property "Value" ""
-			(at 386.08 515.62 90)
-			(hide yes)
+		(property "Value" "100k"
+			(at 386.334 516.636 0)
 			(show_name no)
 			(do_not_autoplace no)
@@
 		(dnp no)
 		(property "Reference" "Z249"
-			(at 377.19 527.812 90)
+			(at 377.19 526.542 90)
 			(show_name no)
 			(do_not_autoplace no)
@@
 			)
 		)
-		(property "Value" ""
-			(at 377.19 527.05 90)
-			(hide yes)
+		(property "Value" "2u2"
+			(at 377.19 528.574 90)
 			(show_name no)
 			(do_not_autoplace no)
@@
 		(dnp no)
 		(property "Reference" "Z240"
-			(at 385.318 494.03 90)
+			(at 386.334 492.76 0)
 			(show_name no)
 			(do_not_autoplace no)
@@
 			)
 		)
-		(property "Value" ""
-			(at 386.08 494.03 90)
-			(hide yes)
+		(property "Value" "100k"
+			(at 386.334 495.046 0)
 			(show_name no)
 			(do_not_autoplace no)
@@
 		(dnp no)
 		(property "Reference" "Z257"
-			(at 580.898 543.56 90)
+			(at 583.184 542.29 0)
 			(show_name no)
 			(do_not_autoplace no)
@@
 			)
 		)
-		(property "Value" ""
-			(at 581.66 543.56 90)
-			(hide yes)
+		(property "Value" "0R"
+			(at 583.184 545.084 0)
 			(show_name no)
 			(do_not_autoplace no)
@@
 		(dnp no)
 		(property "Reference" "Z254"
-			(at 385.318 537.21 90)
+			(at 386.334 535.94 0)
 			(show_name no)
 			(do_not_autoplace no)
@@
 			)
 		)
-		(property "Value" ""
-			(at 386.08 537.21 90)
-			(hide yes)
+		(property "Value" "100k"
+			(at 386.334 538.226 0)
 			(show_name no)
 			(do_not_autoplace no)
@@
 	(symbol
 		(lib_id "power:VCC")
-		(at 505.46 549.91 180)
+		(at 492.76 549.91 180)
 		(unit 1)
 		(body_style 1)
@@
 		(dnp no)
 		(property "Reference" "#PWR0350"
-			(at 505.46 546.1 0)
+			(at 492.76 546.1 0)
 			(hide yes)
 			(show_name no)
@@
 		)
 		(property "Value" "+15V_M"
-			(at 504.444 554.99 0)
+			(at 491.744 554.99 0)
 			(show_name no)
 			(do_not_autoplace no)
@@
 		)
 		(property "Footprint" ""
-			(at 505.46 549.91 0)
+			(at 492.76 549.91 0)
 			(hide yes)
 			(show_name no)
@@
 		)
 		(property "Datasheet" ""
-			(at 505.46 549.91 0)
+			(at 492.76 549.91 0)
 			(hide yes)
 			(show_name no)
@@
 		)
 		(property "Description" "Power symbol creates a global label with name \"VCC\""
-			(at 505.46 549.91 0)
+			(at 492.76 549.91 0)
 			(hide yes)
 			(show_name no)
@@
 		(dnp no)
 		(property "Reference" "Z237"
-			(at 377.19 484.632 90)
+			(at 377.19 483.362 90)
 			(show_name no)
 			(do_not_autoplace no)
@@
 			)
 		)
-		(property "Value" ""
-			(at 377.19 483.87 90)
-			(hide yes)
+		(property "Value" "2u2"
+			(at 377.19 485.394 90)
 			(show_name no)
 			(do_not_autoplace no)

Commit message: VU Test
Parts:
- R141, R142: value 20k -> 33k
- R143, R144: value 1k8 -> 2k2
- R147: value 10k -> 16k5
- Z238, Z242, Z243: value (none) -> 0R
Other:
- moved on the sheet: J33, Z238
Changed lines of the file:
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@@
 	)
 	(junction
-		(at 372.11 487.68)
-		(diameter 0)
-		(color 0 0 0 0)
-	)
-	(junction
 		(at 633.73 186.69)
 		(diameter 0)
@@
 	)
 	(junction
+		(at 372.11 487.68)
+		(diameter 0)
+		(color 0 0 0 0)
+	)
+	(junction
 		(at 36.83 350.52)
 		(diameter 0)
@@
 	(wire
 		(pts
-			(xy 361.95 487.68) (xy 372.11 487.68)
+			(xy 358.14 487.68) (xy 372.11 487.68)
 		)
 		(stroke
@@
 			)
 		)
-		(property "Value" "20k"
+		(property "Value" "33k"
 			(at 504.19 499.11 90)
 			(show_name no)
@@
 	(symbol
 		(lib_id "power:GNDREF")
-		(at 361.95 497.84 0)
+		(at 358.14 497.84 0)
 		(unit 1)
 		(body_style 1)
@@
 		(fields_autoplaced yes)
 		(property "Reference" "#PWR0273"
-			(at 361.95 504.19 0)
+			(at 358.14 504.19 0)
 			(hide yes)
 			(show_name no)
@@
 		)
 		(property "Value" "GND_M"
-			(at 361.95 502.92 0)
+			(at 358.14 502.92 0)
 			(show_name no)
 			(do_not_autoplace no)
@@
 		)
 		(property "Footprint" ""
-			(at 361.95 497.84 0)
+			(at 358.14 497.84 0)
 			(hide yes)
 			(show_name no)
@@
 		)
 		(property "Datasheet" ""
-			(at 361.95 497.84 0)
+			(at 358.14 497.84 0)
 			(hide yes)
 			(show_name no)
@@
 		)
 		(property "Description" "Power symbol creates a global label with name \"GNDREF\" , reference supply ground"
-			(at 361.95 497.84 0)
+			(at 358.14 497.84 0)
 			(hide yes)
 			(show_name no)
@@
 	(symbol
 		(lib_id "Device:R")
-		(at 361.95 494.03 0)
+		(at 358.14 494.03 0)
 		(unit 1)
 		(body_style 1)
@@
 		(dnp no)
 		(property "Reference" "Z238"
-			(at 364.998 494.03 90)
+			(at 363.22 492.506 0)
 			(show_name no)
 			(do_not_autoplace no)
@@
 			)
 		)
-		(property "Value" ""
-			(at 365.76 494.03 90)
-			(hide yes)
+		(property "Value" "0R"
+			(at 363.22 495.046 0)
 			(show_name no)
 			(do_not_autoplace no)
@@
 		)
 		(property "Footprint" "Resistor_SMD:R_0805_2012Metric_Pad1.20x1.40mm_HandSolder"
-			(at 360.172 494.03 90)
+			(at 356.362 494.03 90)
 			(hide yes)
 			(show_name no)
@@
 		)
 		(property "Datasheet" ""
-			(at 361.95 494.03 0)
+			(at 358.14 494.03 0)
 			(hide yes)
 			(show_name no)
@@
 		)
 		(property "Description" "Resistor"
-			(at 361.95 494.03 0)
+			(at 358.14 494.03 0)
 			(hide yes)
 			(show_name no)
@@
 		)
 		(property "Height" ""
-			(at 361.95 494.03 90)
+			(at 358.14 494.03 90)
 			(hide yes)
 			(show_name no)
@@
 		)
 		(property "Manufacturer_Name" ""
-			(at 361.95 494.03 90)
+			(at 358.14 494.03 90)
 			(hide yes)
 			(show_name no)
@@
 		)
 		(property "Manufacturer_Part_Number" ""
-			(at 361.95 494.03 90)
+			(at 358.14 494.03 90)
 			(hide yes)
 			(show_name no)
@@
 		)
 		(property "Mouser Part Number" ""
-			(at 361.95 494.03 90)
+			(at 358.14 494.03 90)
 			(hide yes)
 			(show_name no)
@@
 		)
 		(property "Mouser Price/Stock" ""
-			(at 361.95 494.03 90)
+			(at 358.14 494.03 90)
 			(hide yes)
 			(show_name no)
@@
 		)
 		(property "Mouser-Teilenr." ""
-			(at 361.95 494.03 90)
+			(at 358.14 494.03 90)
 			(hide yes)
 			(show_name no)
@@
 		)
 		(property "Gegenstück Mouser Teilenr." ""
-			(at 361.95 494.03 90)
+			(at 358.14 494.03 90)
 			(hide yes)
 			(show_name no)
@@
 			)
 		)
-		(property "Value" "1k8"
+		(property "Value" "2k2"
 			(at 580.39 513.0799 0)
 			(show_name no)
@@
 		(dnp no)
 		(property "Reference" "Z242"
-			(at 538.48 502.412 90)
+			(at 538.48 499.11 90)
 			(show_name no)
 			(do_not_autoplace no)
@@
 			)
 		)
-		(property "Value" ""
+		(property "Value" "0R"
 			(at 538.48 501.65 90)
-			(hide yes)
 			(show_name no)
 			(do_not_autoplace no)
@@
 		(dnp no)
 		(property "Reference" "Z243"
-			(at 548.64 502.412 90)
+			(at 548.64 499.11 90)
 			(show_name no)
 			(do_not_autoplace no)
@@
 			)
 		)
-		(property "Value" ""
+		(property "Value" "0R"
 			(at 548.64 501.65 90)
-			(hide yes)
 			(show_name no)
 			(do_not_autoplace no)
@@
 		(dnp no)
 		(property "Reference" "J35"
-			(at 356.87 502.92 0)
+			(at 350.266 505.46 0)
 			(show_name no)
 			(do_not_autoplace no)
@@
 	(symbol
 		(lib_id "Connector:Conn_01x02_Pin")
-		(at 356.87 487.68 0)
+		(at 353.06 487.68 0)
 		(unit 1)
 		(body_style 1)
@@
 		(dnp no)
 		(property "Reference" "J33"
-			(at 356.87 481.33 0)
+			(at 350.52 483.87 0)
 			(show_name no)
 			(do_not_autoplace no)
@@
 		)
 		(property "Footprint" "Connector_PinHeader_2.54mm_LongPads:PinHeader_1x02_P2.54mm_Vertical_LongPads"
-			(at 356.87 487.68 0)
+			(at 353.06 487.68 0)
 			(hide yes)
 			(show_name no)
@@
 		)
 		(property "Datasheet" ""
-			(at 356.87 487.68 0)
+			(at 353.06 487.68 0)
 			(hide yes)
 			(show_name no)
@@
 		)
 		(property "Description" "Generic connector, single row, 01x02, script generated"
-			(at 356.87 487.68 0)
+			(at 353.06 487.68 0)
 			(hide yes)
 			(show_name no)
@@
 		)
 		(property "Height" ""
-			(at 356.87 487.68 0)
+			(at 353.06 487.68 0)
 			(hide yes)
 			(show_name no)
@@
 		)
 		(property "Manufacturer_Name" ""
-			(at 356.87 487.68 0)
+			(at 353.06 487.68 0)
 			(hide yes)
 			(show_name no)
@@
 		)
 		(property "Manufacturer_Part_Number" ""
-			(at 356.87 487.68 0)
+			(at 353.06 487.68 0)
 			(hide yes)
 			(show_name no)
@@
 		)
 		(property "Mouser Part Number" ""
-			(at 356.87 487.68 0)
+			(at 353.06 487.68 0)
 			(hide yes)
 			(show_name no)
@@
 		)
 		(property "Mouser Price/Stock" ""
-			(at 356.87 487.68 0)
+			(at 353.06 487.68 0)
 			(hide yes)
 			(show_name no)
@@
 		)
 		(property "Mouser-Teilenr." ""
-			(at 356.87 487.68 0)
+			(at 353.06 487.68 0)
 			(hide yes)
 			(show_name no)
@@
 		)
 		(property "Gegenstück Mouser Teilenr." ""
-			(at 356.87 487.68 0)
+			(at 353.06 487.68 0)
 			(hide yes)
 			(show_name no)
@@
 			)
 		)
-		(property "Value" "20k"
+		(property "Value" "33k"
 			(at 486.41 499.11 90)
 			(show_name no)
@@
 			)
 		)
-		(property "Value" "1k8"
+		(property "Value" "2k2"
 			(at 558.8 501.65 90)
 			(show_name no)
@@
 			)
 		)
-		(property "Value" "10k"
+		(property "Value" "16k5"
 			(at 486.41 510.54 90)
 			(show_name no)
