File: KiCad/Input.kicad_sch (KiCad schematic)
At the start: 629 parts, among them J1 R_Phono_In, J10 VCC_IN, J11 VCC_OUT, J12 EMK_In, J13 EMK_Out, J14 EMK_Out, J15 Mic_Effekt_Out, J16 Mic_Effekt_Out, J17 Mic_Effekt_Out, J18 Mic_Effekt_Out, J19 Phono/Line_Out, J2 L_Phono_In, J20 Mic_Effekt_Out, J21 EMK_Out, J22 EMK_In, J23 EMK_In, J24 Mic_Effekt_In, J25 Mic_Effekt_In, J26 Phono/Line_In, J27 Mic_Effekt_In, J28 Pegel_Out, J29 Pegel_Out, J3 R_Line_In, J30 Pegel_In, J31 Pegel_In, J32 Pegel_In, J33 Pegel_In, J34 LED_Out, J35 LED_In, J36 VU_Meter_Out, J37 AUX_Send_3, J38 AUX_Send_1, J39 AUX_Send_2, J4 L_Line_In, J40 Bass_Out, J41 Kick_Out, J42 Mid_Out, J43 High_Out, J44 Line_Out_L, J45 Line_Out_R, J5 Mic_In, J6 Effekt_In, J7 AUX_RET_1, J8 AUX_RET_2, J9 AUX_RET_3, SW1 SW_DPST, SW10 SW_SPDT, SW11 SW_SPDT, SW12 SW_SPDT, SW2 SW_SPDT, SW3 SW_SPDT, SW4 SW_SPDT, SW5 SW_SPDT, SW6 SW_SPDT, SW7 SW_SPDT, SW8 SW_SPDT, SW9 Pegel_Selector, U1 TL074, U10 TL074, U11 TL074, U12 TL074, U13 TL074, U14 TL074, U15 TL074, U16 TL074, U17 TL074, U18 TL074, U19 TL074, U2 TL074, U20 TL074, U21 TL074, U22 TL074, U23 TL074, U24 TL074, U25 INA128U, U3 TL074, U4 TL074, U5 TL074, U6 REC10K-2409, U7 REC10K-2415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

Commit message: PCB Update
Parts:
- SW10, SW11, SW12, SW2, SW3, SW4, SW5, SW6, SW7, SW8: footprint Connector_PinSocket_2.54mm_LongPads:PinSocket_1x03_P2.54mm_Vertical_LongPads -> Connector_PinHeader_2.54mm_LongPads:PinHeader_1x03_P2.54mm_Vertical_LongPads
Connections:
- net at R13.2, Z62.1: now also U1.14; no longer U1.8
- net at C15.2, C21.1, R20.2: now also U1.9 (-); no longer U1.13 (-)
- net at R29.1, RV6.2, RV6.3: now also U2.9 (-); no longer U2.13 (-)
- net at Z52.1: now also U1.12 (+); no longer U1.10 (+)
- net at R13.1, R5.2, R6.2: now also U1.13 (-); no longer U1.9 (-)
- net at R28.1, RV6.1: now also U2.8; no longer U2.14
- net at Z53.1: now also U2.12 (+); no longer U2.10 (+)
- net at R14.2, Z63.1: now also U2.14; no longer U2.8
- net at R14.1, R7.2, R8.2: now also U2.13 (-); no longer U2.9 (-)
- net at SW2.2 (B): now also U2.10 (+); no longer U2.12 (+)
- net at C27.2, R22.1, Z74.1: now also U1.8; no longer U1.14
- net at Z68.2: now also U1.10 (+); no longer U1.12 (+)
Changed lines of the file:
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@@
 			)
 		)
-		(property "Footprint" "Connector_PinSocket_2.54mm_LongPads:PinSocket_1x03_P2.54mm_Vertical_LongPads"
+		(property "Footprint" "Connector_PinHeader_2.54mm_LongPads:PinHeader_1x03_P2.54mm_Vertical_LongPads"
 			(at 392.43 179.07 0)
 			(effects
@@
 			)
 		)
-		(property "Footprint" "Connector_PinSocket_2.54mm_LongPads:PinSocket_1x03_P2.54mm_Vertical_LongPads"
+		(property "Footprint" "Connector_PinHeader_2.54mm_LongPads:PinHeader_1x03_P2.54mm_Vertical_LongPads"
 			(at 392.43 245.11 0)
 			(effects
@@
 			)
 		)
-		(property "Footprint" "Connector_PinSocket_2.54mm_LongPads:PinSocket_1x03_P2.54mm_Vertical_LongPads"
+		(property "Footprint" "Connector_PinHeader_2.54mm_LongPads:PinHeader_1x03_P2.54mm_Vertical_LongPads"
 			(at 656.59 408.94 0)
 			(effects
@@
 			)
 		)
-		(property "Footprint" "Connector_PinSocket_2.54mm_LongPads:PinSocket_1x03_P2.54mm_Vertical_LongPads"
+		(property "Footprint" "Connector_PinHeader_2.54mm_LongPads:PinHeader_1x03_P2.54mm_Vertical_LongPads"
 			(at 393.7 388.62 0)
 			(effects
@@
 		(at 119.38 64.77 0)
 		(mirror x)
-		(unit 3)
+		(unit 4)
 		(exclude_from_sim no)
 		(in_bom yes)
@@
 				(path "/81a92cd6-862a-4567-ad33-f8a3bc120591"
 					(reference "U1")
-					(unit 3)
+					(unit 4)
 				)
 			)
@@
 		(at 119.38 133.35 0)
 		(mirror x)
-		(unit 3)
+		(unit 4)
 		(exclude_from_sim no)
 		(in_bom yes)
@@
 				(path "/81a92cd6-862a-4567-ad33-f8a3bc120591"
 					(reference "U2")
-					(unit 3)
+					(unit 4)
 				)
 			)
@@
 			)
 		)
-		(property "Footprint" "Connector_PinSocket_2.54mm_LongPads:PinSocket_1x03_P2.54mm_Vertical_LongPads"
+		(property "Footprint" "Connector_PinHeader_2.54mm_LongPads:PinHeader_1x03_P2.54mm_Vertical_LongPads"
 			(at 161.29 109.22 0)
 			(effects
@@
 			)
 		)
-		(property "Footprint" "Connector_PinSocket_2.54mm_LongPads:PinSocket_1x03_P2.54mm_Vertical_LongPads"
+		(property "Footprint" "Connector_PinHeader_2.54mm_LongPads:PinHeader_1x03_P2.54mm_Vertical_LongPads"
 			(at 393.7 55.88 0)
 			(effects
@@
 		(lib_id "Amplifier_Operational:TL074")
 		(at 177.8 111.76 0)
-		(unit 4)
+		(unit 3)
 		(exclude_from_sim no)
 		(in_bom yes)
@@
 				(path "/81a92cd6-862a-4567-ad33-f8a3bc120591"
 					(reference "U2")
-					(unit 4)
+					(unit 3)
 				)
 			)
@@
 			)
 		)
-		(property "Footprint" "Connector_PinSocket_2.54mm_LongPads:PinSocket_1x03_P2.54mm_Vertical_LongPads"
+		(property "Footprint" "Connector_PinHeader_2.54mm_LongPads:PinHeader_1x03_P2.54mm_Vertical_LongPads"
 			(at 656.59 354.33 0)
 			(effects
@@
 		(at 172.72 62.23 0)
 		(mirror x)
-		(unit 4)
+		(unit 3)
 		(exclude_from_sim no)
 		(in_bom yes)
@@
 				(path "/81a92cd6-862a-4567-ad33-f8a3bc120591"
 					(reference "U1")
-					(unit 4)
+					(unit 3)
 				)
 			)
@@
 			)
 		)
-		(property "Footprint" "Connector_PinSocket_2.54mm_LongPads:PinSocket_1x03_P2.54mm_Vertical_LongPads"
+		(property "Footprint" "Connector_PinHeader_2.54mm_LongPads:PinHeader_1x03_P2.54mm_Vertical_LongPads"
 			(at 393.7 334.01 0)
 			(effects
@@
 			)
 		)
-		(property "Footprint" "Connector_PinSocket_2.54mm_LongPads:PinSocket_1x03_P2.54mm_Vertical_LongPads"
+		(property "Footprint" "Connector_PinHeader_2.54mm_LongPads:PinHeader_1x03_P2.54mm_Vertical_LongPads"
 			(at 393.7 123.19 0)
 			(effects
@@
 			)
 		)
-		(property "Footprint" "Connector_PinSocket_2.54mm_LongPads:PinSocket_1x03_P2.54mm_Vertical_LongPads"
+		(property "Footprint" "Connector_PinHeader_2.54mm_LongPads:PinHeader_1x03_P2.54mm_Vertical_LongPads"
 			(at 529.59 408.94 0)
 			(effects

Commit message: PCB Update
Connections:
- net at R29.2, R31.2: now also U3.5 (+); no longer U3.3 (+)
- net at R32.2, Z84.1, Z89.1: now also U3.7; no longer U3.1
- net at RV1.2: now also U3.10 (+); no longer U3.12 (+)
- net at C30.1, RV5.1, RV5.2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: now also U3.12 (+); no longer U3.10 (+)
- net at R30.2, RV4.3, Z78.1: now also U3.14; no longer U3.8
- net at R23.2, R30.1: now also U3.13 (-); no longer U3.9 (-)
- net at RV4.2: now also U3.3 (+); no longer U3.5 (+)
- net at R28.2, R32.1: now also U3.6 (-); no longer U3.2 (-)
- new net: C22.2, U3.1, U3.2 (-)
- new net: C1.2, U3.8, U3.9 (-)
Changed lines of the file:
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@@
 		(at 204.47 213.36 0)
 		(mirror x)
-		(unit 3)
+		(unit 4)
 		(exclude_from_sim no)
 		(in_bom yes)
@@
 				(path "/81a92cd6-862a-4567-ad33-f8a3bc120591"
 					(reference "U3")
-					(unit 3)
+					(unit 4)
 				)
 			)
@@
 		(lib_id "Amplifier_Operational:TL074")
 		(at 152.4 242.57 0)
-		(unit 2)
+		(unit 1)
 		(exclude_from_sim no)
 		(in_bom yes)
@@
 				(path "/81a92cd6-862a-4567-ad33-f8a3bc120591"
 					(reference "U3")
-					(unit 2)
+					(unit 1)
 				)
 			)
@@
 		(lib_id "Amplifier_Operational:TL074")
 		(at 49.53 328.93 0)
-		(unit 4)
+		(unit 3)
 		(exclude_from_sim no)
 		(in_bom yes)
@@
 				(path "/81a92cd6-862a-4567-ad33-f8a3bc120591"
 					(reference "U3")
-					(unit 4)
+					(unit 3)
 				)
 			)
@@
 		(at 223.52 127 0)
 		(mirror x)
-		(unit 1)
+		(unit 2)
 		(exclude_from_sim no)
 		(in_bom yes)
@@
 				(path "/81a92cd6-862a-4567-ad33-f8a3bc120591"
 					(reference "U3")
-					(unit 1)
+					(unit 2)
 				)
 			)

Commit message: PCB Update
Parts:
- C7, C8: value 0.1uF -> 100n
Connections:
- net at R16.2, R17.2, R19.1: now also U4.6 (-); no longer U4.9 (-)
- net at R19.2, Z71.1: now also U4.7; no longer U4.8
- net at Z76.2, Z81.1, Z82.1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: now also U4.3 (+); no longer U4.5 (+)
- net at Z80.1, Z85.1: now also U4.1, U4.2 (-); no longer U4.6 (-), U4.7
- net at R12.2, RV1.3, Z56.1: now also U4.8; no longer U4.1
- net at Z12.2, Z22.1: now also U5.3 (+); no longer U5.10 (+)
- net at Z70.1: now also U4.5 (+); no longer U4.10 (+)
- net at C3.1, RV3.1, RV3.2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: now also U4.10 (+); no longer U4.3 (+)
- net at R12.1, R3.2: now also U4.9 (-); no longer U4.2 (-)
- net at Z14.2, Z24.1: now also U5.10 (+); no longer U5.3 (+)
- new net: U5.1, U5.2 (-), Z31.1
- new net: U5.8, U5.9 (-), Z33.1
Changed lines of the file:
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@@
 		(lib_id "Amplifier_Operational:TL074")
 		(at 208.28 302.26 0)
-		(unit 2)
+		(unit 1)
 		(exclude_from_sim no)
 		(in_bom yes)
@@
 				(path "/81a92cd6-862a-4567-ad33-f8a3bc120591"
 					(reference "U4")
-					(unit 2)
+					(unit 1)
 				)
 			)
@@
 			)
 		)
-		(property "Value" "0.1uF"
+		(property "Value" "100n"
 			(at 96.5136 224.79 90)
 			(effects
@@
 			)
 		)
-		(property "Value" "0.1uF"
+		(property "Value" "100n"
 			(at 96.5136 191.77 90)
 			(effects
@@
 		(at 101.6 299.72 0)
 		(mirror x)
-		(unit 1)
+		(unit 3)
 		(exclude_from_sim no)
 		(in_bom yes)
@@
 				(path "/81a92cd6-862a-4567-ad33-f8a3bc120591"
 					(reference "U4")
-					(unit 1)
+					(unit 3)
 				)
 			)
@@
 		(at 161.29 313.69 0)
 		(mirror x)
-		(unit 3)
+		(unit 2)
 		(exclude_from_sim no)
 		(in_bom yes)
@@
 				(path "/81a92cd6-862a-4567-ad33-f8a3bc120591"
 					(reference "U4")
-					(unit 3)
+					(unit 2)
 				)
 			)
@@
 		(lib_id "Amplifier_Operational:TL074")
 		(at 64.77 387.35 0)
-		(unit 3)
+		(unit 1)
 		(exclude_from_sim no)
 		(in_bom yes)
@@
 				(path "/81a92cd6-862a-4567-ad33-f8a3bc120591"
 					(reference "U5")
-					(unit 3)
+					(unit 1)
 				)
 			)
@@
 		(lib_id "Amplifier_Operational:TL074")
 		(at 66.04 450.85 0)
-		(unit 1)
+		(unit 3)
 		(exclude_from_sim no)
 		(in_bom yes)
@@
 				(path "/81a92cd6-862a-4567-ad33-f8a3bc120591"
 					(reference "U5")
-					(unit 1)
+					(unit 3)
 				)
 			)
