File: KiCad/Input.kicad_sch (KiCad schematic)
At the start: 633 parts, among them J1 R_Phono_In, J10 VCC_IN, J11 VCC_OUT, J12 EMK_In, J13 EMK_Out, J14 EMK_Out, J15 Mic_Effekt_Out, J16 Mic_Effekt_Out, J17 Mic_Effekt_Out, J18 Mic_Effekt_Out, J19 Phono/Line_Out, J2 L_Phono_In, J20 Mic_Effekt_Out, J21 EMK_Out, J22 EMK_In, J23 EMK_In, J24 Mic_Effekt_In, J25 Mic_Effekt_In, J26 Phono/Line_In, J27 Mic_Effekt_In, J28 Pegel_Out, J29 Pegel_Out, J3 R_Line_In, J30 Pegel_In, J31 Pegel_In, J32 Pegel_In, J33 Pegel_In, J34 LED_Out, J35 LED_In, J36 VU_Meter_Out, J37 AUX_Send_3, J38 AUX_Send_1, J39 AUX_Send_2, J4 L_Line_In, J40 Bass_Out, J41 Kick_Out, J42 Mid_Out, J43 High_Out, J44 Line_Out_L, J45 Line_Out_R, J5 Mic_In, J6 Effekt_In, J7 AUX_RET_1, J8 AUX_RET_2, J9 AUX_RET_3, SW1 SW_DPST, SW10 SW_SPDT, SW11 SW_SPDT, SW12 SW_SPDT, SW2 SW_SPDT, SW3 SW_SPDT, SW4 SW_SPDT, SW5 SW_SPDT, SW6 SW_SPDT, SW7 SW_SPDT, SW8 SW_SPDT, SW9 SW_Rotary_1x4, U1 TL074, U10 TL074, U11 TL074, U12 TL074, U13 TL074, U14 TL074, U15 TL074, U16 TL074, U17 TL074, U18 TL074, U19 TL074, U2 TL074, U20 TL074, U21 TL074, U22 TL074, U23 TL074, U24 TL074, U25 INA128U, U3 TL074, U4 TL074, U5 TL074, U6 REC10K-2409, U7 REC10K-2415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

Commit message: PCB Update
Parts:
- removed J13, J14: EMK_Out, Connector_PinSocket_2.54mm_LongPads:PinSocket_1x05_P2.54mm_Vertical_LongPads, symbol Connector:Conn_01x05_Socket
Connections:
- net +15V: no longer C13.2, C16.2, C28.2, C31.2, C33.2, C7.2, J12.5 (Pin_5), U1.4 (V+), U2.4 (V+), U25.7 (V+), U3.4 (V+), U4.4 (V+), U5.4 (V+)
- net +9V: no longer J12.2 (Pin_2)
- net -15V: no longer C14.2, C17.2, C29.2, C32.2, C34.2, C8.2, J12.3 (Pin_3), U1.11 (V-), U2.11 (V-), U25.4 (V-), U3.11 (V-), U4.11 (V-), U5.11 (V-)
- net 9V_GND: no longer J12.1 (Pin_1)
- net GND: no longer C112.1, C112.2, C113.1, C113.2, C114.1, C114.2, C115.1, C115.2, C13.1, C14.1, C16.1, C17.1, C28.1, C29.1, C3.2, C30.2, C31.1, C32.1, C33.1, C34.1, C7.1, C8.1, J1.2 (Pin_2), J12.4 (Pin_4), J2.2 (Pin_2), J3.2 (Pin_2), J4.2 (Pin_2), J5.1 (Pin_1), J6.2 (Pin_2), J7.2 (Pin_2), J8.2 (Pin_2), J9.2 (Pin_2), R18.1, R24.1, R31.1, R4.1, U25.5 (REF), Z1.2, Z10.2, Z100.2, Z2.2, Z21.2, Z22.2, Z23.2, Z24.2, Z25.2, Z26.2, Z27.2, Z28.2, Z29.2, Z3.2, Z30.2, Z38.2, Z39.2, Z4.2, Z40.2, Z41.2, Z42.2, Z43.2, Z44.2, Z5.2, Z52.2, Z53.2, Z54.2, Z57.2, Z58.2, Z6.2, Z60.2, Z66.2, Z67.2, Z7.2, Z70.2, Z72.2, Z73.2, Z77.2, Z8.2, Z80.2, Z81.2, Z82.2, Z83.2, Z84.2, Z9.2, Z90.2, Z91.2, Z92.2, Z93.2, Z94.2, Z95.2, Z96.2, Z97.2, Z98.2, Z99.2
- new net +15V_I: C13.2, C16.2, C28.2, C31.2, C33.2, C7.2, J12.5 (Pin_5), U1.4 (V+), U2.4 (V+), U25.7 (V+), U3.4 (V+), U4.4 (V+), U5.4 (V+)
- new net +9V_I: J12.2 (Pin_2)
- new net -15V_I: C14.2, C17.2, C29.2, C32.2, C34.2, C8.2, J12.3 (Pin_3), U1.11 (V-), U2.11 (V-), U25.4 (V-), U3.11 (V-), U4.11 (V-), U5.11 (V-)
- new net 9V_GND_I: J12.1 (Pin_1)
- new net GND_I: C112.1, C112.2, C113.1, C113.2, C114.1, C114.2, C115.1, C115.2, C13.1, C14.1, C16.1, C17.1, C28.1, C29.1, C3.2, C30.2, C31.1, C32.1, C33.1, C34.1, C7.1, C8.1, J1.2 (Pin_2), J12.4 (Pin_4), J2.2 (Pin_2), J3.2 (Pin_2), J4.2 (Pin_2), J5.1 (Pin_1), J6.2 (Pin_2), J7.2 (Pin_2), J8.2 (Pin_2), J9.2 (Pin_2), R18.1, R24.1, R31.1, R4.1, U25.5 (REF), Z1.2, Z10.2, Z100.2, Z2.2, Z21.2, Z22.2, Z23.2, Z24.2, Z25.2, Z26.2, Z27.2, Z28.2, Z29.2, Z3.2, Z30.2, Z38.2, Z39.2, Z4.2, Z40.2, Z41.2, Z42.2, Z43.2, Z44.2, Z5.2, Z52.2, Z53.2, Z54.2, Z57.2, Z58.2, Z6.2, Z60.2, Z66.2, Z67.2, Z7.2, Z70.2, Z72.2, Z73.2, Z77.2, Z8.2, Z80.2, Z81.2, Z82.2, Z83.2, Z84.2, Z9.2, Z90.2, Z91.2, Z92.2, Z93.2, Z94.2, Z95.2, Z96.2, Z97.2, Z98.2, Z99.2
Other:
- moved on the sheet: C115

Commit message: PCB Update
Parts:
- removed J21: EMK_Out, Connector_PinSocket_2.54mm_LongPads:PinSocket_1x05_P2.54mm_Vertical_LongPads, symbol Connector:Conn_01x05_Socket
- removed J23: EMK_In, Connector_PinHeader_2.54mm_LongPads:PinHeader_1x05_P2.54mm_Vertical_LongPads, symbol Connector:Conn_01x05_Pin
- removed L1: 470uF, 1.6A, WE-SL575:WE-SL575, symbol Device:L_Coupled
- removed SW10, SW11, SW12, SW3, SW4, SW5, SW6, SW7, SW8: SW_SPDT, Connector_PinHeader_2.54mm_LongPads:PinHeader_1x03_P2.54mm_Vertical_LongPads, symbol Switch:SW_SPDT
- removed Z185, Z193, Z198: ~, Resistor_SMD:R_0805_2012Metric_Pad1.20x1.40mm_HandSolder, symbol Device:R_Small
- added C116, C119: 10n, Capacitor_SMD:C_1210_3225Metric_Pad1.33x2.70mm_HandSolder, symbol Device:C_Small
- added C117, C118, C123: 10n, Capacitor_SMD:C_0805_2012Metric_Pad1.18x1.45mm_HandSolder, symbol Device:C_Small
- added C120, C121, C122: 100n, Capacitor_SMD:C_0805_2012Metric_Pad1.18x1.45mm_HandSolder, symbol Device:C_Small
- added H1, H10, H11, H12, H13, H14, H16, H2, H3, H4, H6, H7, H8: MountingHole, MountingHole:MountingHole_3.2mm_M3_Pad, symbol Mechanical:MountingHole
- added H15, H5, H9: MountingHole_Pad, MountingHole:MountingHole_3.2mm_M3_Pad, symbol Mechanical:MountingHole_Pad
- added J21: Conn_01x05_bridged, Connector_Bridged_2.54mm_LongPads:Bridge_2x05_P2.54mm_Vertical_LongPads, symbol conn_01x05_bridged:Conn_01x05_bridged
- added L1: ~, WE-SL575:WE-SL575, symbol Common_Mode_Choke:Common_Mode_Choke
- added SW10, SW11, SW12, SW3, SW4, SW5, SW6, SW7, SW8: SW_SPDT, Connector_PinHeader_2.54mm_LongPads:PinHeader_1x02_P2.54mm_Vertical_LongPads, symbol sw_spdt_2:SW_SPDT
- added Z185, Z193, Z198, Z257, Z258, Z259: ~, Resistor_SMD:R_0805_2012Metric_Pad1.20x1.40mm_HandSolder, symbol Device:R
- C12: now not fitted; now left out of the parts list
- C2, C5: footprint Capacitor_SMD:C_0805_2012Metric_Pad1.18x1.45mm_HandSolder -> Capacitor_SMD:C_1210_3225Metric_Pad1.33x2.70mm_HandSolder
- C25: value 1n -> 10n; footprint Capacitor_SMD:C_0805_2012Metric_Pad1.18x1.45mm_HandSolder -> Capacitor_SMD:C_1210_3225Metric_Pad1.33x2.70mm_HandSolder
- C4: value 10n -> 1n
- L2, L3, L4, L5: footprint Connector_PinSocket_2.54mm_LongPads:PinSocket_1x02_P2.54mm_Vertical_LongPads -> Inductor_SMD:L_1206_3216Metric
- RV16, RV17, RV20: footprint Connector_PinSocket_2.54mm_LongPads:PinSocket_1x06_P2.54mm_Vertical_LongPads -> Connector_PinSocket_2.54mm_LongPads:PinSocket_2x03_P2.54mm_Vertical_LongPads
- RV18, RV19: footprint Connector_PinSocket_2.54mm_LongPads:PinSocket_1x06_P2.54mm_Vertical_LongPads -> Connector_PinSocket_2.54mm_LongPads:PinSocket_2x03_P2.54mm_Vertical_LongPads_Mirrored
- renumbered U13 to U10, U12 to U10, U10 to U11, U22 to U11, U9 to U12, U8 to U12, U10 to U13, U12 to U13, U11 to U13, U16 to U14, U15 to U14, U16 to U15, U17 to U16, U18 to U16, U18 to U17, U20 to U18, U14 to U20, U21 to U20, U22 to U21, U13 to U22, U14 to U22, U24 to U23, U23 to U24, U9 to U8, U10 to U9, U11 to U9
Connections:
- net GND_I: now also C116.2
- net Pegel_Aux_Return: now also SW9.2, U24.1, U24.2 (-); no longer SW9.3, U24.8, U24.9 (-)
- net Pegel_Mic_Effekt: now also SW9.3; no longer SW9.2
- net Pegel_Post: now also SW9.1, U24.6 (-), U24.7; no longer SW9.4, U24.13 (-), U24.14
- net Pegel_Pre: now also SW9.4; no longer SW9.1
- net at R35.1, RV7.1, U9.1: now also SW3.1 (A)
- net at R36.1, RV7.2, RV7.3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: now also SW3.2 (B)
- net at R93.1, RV13.1: now also Z152.2; no longer Z153.2
- net at U18.5 (+), Z223.2: now also U18.10 (+); no longer U18.3 (+)
- net at C37.1, R85.1: now also U22.10 (+); no longer U22.5 (+)
- net at Z228.1, Z238.1: now also U19.8, U19.9 (-); no longer U19.1, U19.2 (-)
- net at Z133.2, Z137.1: now also U24.5 (+); no longer U24.12 (+)
- net at R64.2, R65.2, R66.2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: now also U11.6 (-); no longer U11.13 (-)
- net at C59.2, R118.2: now also U14.5 (+); no longer U14.3 (+)
- net at R83.1, Z175.1, Z176.1: now also U22.14; no longer U22.7
- net at C61.2, R120.2: now also U16.5 (+); no longer U16.3 (+)
- net at C11.2, C19.1, L4.2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: now also C4.2; no longer C25.2
- net at R37.1, RV8.1, U9.7: now also SW4.1 (A)
- net at R38.1, RV8.2, RV8.3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: now also SW4.2 (B)
- net at R40.2, R49.2: now also U8.12 (+); no longer U8.5 (+)
- net at R39.2, R55.1: now also U8.13 (-); no longer U8.6 (-)
- net at R55.2, Z140.1: now also U8.14; no longer U8.7
- net at R123.2, RV22.1, U20.8: now also SW12.1 (A)
- net at R124.2, RV22.2, RV22.3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: now also SW12.2 (B)
- net at C88.2, R139.2: now also U17.5 (+); no longer U17.12 (+)
- net at RV14.2: now also U13.3 (+); no longer U13.12 (+)
- net at D1.1 (K), R59.2, R60.1: now also U23.13 (-); no longer U23.2 (-)
- net at R58.1, Z143.1: now also U10.8; no longer U10.14
- net at C2.1, SW1.4: now also L1.1
- net at C11.1, C5.1, C9.1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: now also C117.2, C123.2, L1.2; no longer C4.2
- net at C2.2, SW1.2: now also L1.4
- net at C10.1, C12.1, C5.2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: now also C118.1, L1.3
- net at R76.1, Z163.1: now also U22.7; no longer U22.1
- net at R69.1, R70.1, R76.2: now also U22.6 (-); no longer U22.2 (-)
- net at Z158.1: now also U22.5 (+); no longer U22.3 (+)
- net at C45.1, RV20.1, RV20.2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: now also U13.10 (+); no longer U13.3 (+)
- net at C82.2, R141.2: now also U14.12 (+); no longer U14.5 (+)
- net at R61.2, R62.2, R63.2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: now also U11.2 (-); no longer U11.9 (-)
- net at R73.2, Z159.1: now also U11.1; no longer U11.8
- net at U8.3 (+), U9.3 (+), U9.5 (+)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: now also U10.3 (+), U8.5 (+); no longer U10.10 (+), U8.3 (+)
- net at Z236.1, Z246.1: now also U21.13 (-), U21.14; no longer U21.1, U21.2 (-)
- net at R104.2, RV15.3, Z184.1: now also U13.8; no longer U13.1
- net at U19.5 (+), Z221.2: now also U19.10 (+); no longer U19.3 (+)
- net at Z132.2, Z136.1: now also U24.3 (+); no longer U24.10 (+)
- net at D1.2 (A), D2.1 (K): now also U23.14; no longer U23.1
- net at C89.2, R140.2: now also U17.3 (+); no longer U17.12 (+)
- net at Z112.2, Z116.1: now also U10.5 (+); no longer U10.10 (+)
- net at R34.1, R45.2: now also U10.7, SW8.1 (A); no longer U10.8
- net at R34.2, R46.2: now also U10.6 (-), SW8.2 (B); no longer U10.9 (-)
- net at Z231.1, Z241.1: now also U18.8, U18.9 (-); no longer U18.1, U18.2 (-)
- net at R41.2, R56.1: now also U8.9 (-); no longer U8.6 (-)
- net at R56.2, Z141.1: now also U8.8; no longer U8.7
- net at Z229.1, Z239.1: now also U19.13 (-), U19.14; no longer U19.8, U19.9 (-)
- net at R67.2, R68.2, R71.1: now also U23.9 (-); no longer U23.6 (-)
- net at R71.2, U24.10 (+), U24.12 (+): now also U23.8; no longer U23.7
- net at R41.1, RV10.1: now also U8.7, SW6.1 (A); no longer U8.1
- net at R42.1, RV10.2, RV10.3: now also U8.6 (-), SW6.2 (B); no longer U8.2 (-)
- net at C63.2, R114.2: now also U15.5 (+); no longer U15.10 (+)
- net at R124.1, R126.1: now also U20.5 (+); no longer U20.12 (+)
- net at C53.2, R128.1: now also U15.6 (-), U15.7; no longer U15.8, U15.9 (-)
- net at R122.1, R125.1: now also U20.3 (+); no longer U20.5 (+)
- net at R42.2, R50.2: now also U8.10 (+); no longer U8.5 (+)
- net at R99.1, RV16.3, Z178.1: now also U22.8; no longer U22.7
- net at C84.2, R143.2: now also U16.12 (+); no longer U16.5 (+)
- net at C42.1, RV17.1, RV17.2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: now also U12.10 (+); no longer U12.12 (+)
- net at R131.1, Z205.1, Z207.1: now also U20.1; no longer U20.7
- net at R121.1, R131.2: now also U20.2 (-); no longer U20.6 (-)
- net at R123.1, R132.2: now also U20.6 (-); no longer U20.13 (-)
- net at R132.1, Z206.1, Z208.1: now also U20.7; no longer U20.14
- net at C65.2, R116.2: now also U17.12 (+); no longer U17.10 (+)
- net at R33.1, R43.2: now also U10.1, SW7.1 (A); no longer U10.8
- net at R33.2, R44.2: now also U10.2 (-), SW7.2 (B); no longer U10.9 (-)
- net at C44.1, RV19.1, RV19.2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: now also U13.12 (+); no longer U13.3 (+)
- net at R91.1, RV12.1: now also Z153.2; no longer Z152.2
- net at RV12.2: now also U12.5 (+); no longer U12.10 (+)
- net at R101.2, RV12.3, Z181.1: now also U12.8; no longer U12.14
- net at C76.2, Z214.1: now also U17.6 (-), U17.7; no longer U17.13 (-), U17.14
- net at C52.2, R127.1: now also U15.1, U15.2 (-); no longer U15.8, U15.9 (-)
- net at R100.1, R99.2: now also U22.9 (-); no longer U22.6 (-)
- net at Z235.1, Z245.1: now also U21.1, U21.2 (-); no longer U21.13 (-), U21.14
- net at R104.1, R97.2: now also U13.9 (-); no longer U13.2 (-)
- net at R103.1, R95.2: now also U13.13 (-); no longer U13.2 (-)
- net at C48.1: now also Z199.2; no longer Z197.2
- net at R101.1, R91.2: now also U12.9 (-); no longer U12.13 (-)
- net at R136.2, Z188.1: now also U16.8, U16.9 (-); no longer U16.6 (-), U16.7
- net at U20.10 (+), U22.3 (+), Z180.2: now also U20.12 (+); no longer U20.3 (+)
- net at C75.2, Z213.1: now also U15.8, U15.9 (-); no longer U15.13 (-), U15.14
- net at C77.2, Z215.1: now also U17.1, U17.2 (-); no longer U17.13 (-), U17.14
- net at R35.2, R53.1: now also U9.13 (-); no longer U9.6 (-)
- net at R53.2, Z138.1: now also U9.14; no longer U9.7
- net at R74.2, Z160.1: now also U11.7; no longer U11.14
- net at R46.1, R52.1: now also U10.10 (+); no longer U10.12 (+)
- net at Z156.1: now also U11.3 (+); no longer U11.10 (+)
- net at R45.1, R58.2: now also U10.9 (-); no longer U10.13 (-)
- net at C49.1: now also Z197.2; no longer Z199.2
- net at R122.2, RV21.2, RV21.3: now also U20.13 (-), SW11.2 (B); no longer U20.2 (-)
- net at R78.1, R80.1: now also U22.12 (+); no longer U22.5 (+)
- net at R77.1, R83.2: now also U22.13 (-); no longer U22.6 (-)
- net at Z233.1, Z243.1: now also U18.13 (-), U18.14; no longer U18.8, U18.9 (-)
- net at R103.2, RV14.3, Z183.1: now also U13.14; no longer U13.1
- net at R39.1, RV9.1, U8.1: now also SW5.1 (A)
- net at R40.1, RV9.2, RV9.3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: now also SW5.2 (B)
- net at C83.2, R142.2: now also U14.10 (+); no longer U14.5 (+)
- net at R134.2, Z186.1: now also U14.8, U14.9 (-); no longer U14.6 (-), U14.7
- net at C73.1, R112.2: now also U16.6 (-), U16.7; no longer U16.1, U16.2 (-)
- net at C62.2, R113.2: now also U15.3 (+); no longer U15.10 (+)
- net at C87.2, R138.2: now also U15.10 (+); no longer U15.12 (+)
- net at R105.1: now also Z198.2
- net at C55.2, R130.1: now also U17.13 (-), U17.14; no longer U17.8, U17.9 (-)
- net at C85.2, R144.2: now also U16.10 (+); no longer U16.5 (+)
- net at R135.2, Z187.1: now also U16.13 (-), U16.14; no longer U16.6 (-), U16.7
- net at C71.1, R110.2: now also U14.6 (-), U14.7; no longer U14.1, U14.2 (-)
- net at RV13.2: now also U12.3 (+); no longer U12.10 (+)
- net at R36.2, R47.2: now also U9.12 (+); no longer U9.5 (+)
- net at R121.2, RV21.1: now also U20.14, SW11.1 (A); no longer U20.1
- net at R77.2, RV11.1, U22.1: now also SW10.1 (A)
- net at R78.2, RV11.2, RV11.3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: now also SW10.2 (B)
- net at Z157.1: now also U11.5 (+); no longer U11.12 (+)
- net +15V renamed +15V_O
- net +15V_O: now also J22.5 (Pin_5); no longer C46.2, C56.2, J22.3 (Pin_3), R26.1, R72.1, U23.4 (V+), U24.4 (V+)
- removed net +9V: J22.1 (Pin_1), J36.3 (Pin_3), R25.1
- net -15V renamed -15V_O
- net -15V_O: now also J22.3 (Pin_3); no longer C47.2, C57.2, J22.4 (Pin_4), R27.1, U23.11 (V-), U24.11 (V-)
- net 9V_GND renamed 9V_GND_P
- net 9V_GND_P: now also J21.1 (Pin_1); no longer J22.2 (Pin_2), J36.4 (Pin_4)
- net FILT_GND renamed GND_15V_FILT
- net GND_15V_FILT: now also C123.1; no longer C23.1, C24.2, C25.1
- net GND renamed GND_O
- net GND_O: now also J22.4 (Pin_4), U11.10 (+), U11.12 (+), C119.2, C120.1, C120.2, C121.1, C121.2, C122.1, C122.2, Z193.2, Z258.2, Z259.2; no longer C19.2, C20.1, C36.2, C46.1, C47.1, C56.1, C57.1, D3.2 (A), J22.5 (Pin_5), J36.2 (Pin_2), R75.1, R86.1, U11.10 (+), U11.12 (+), U23.3 (+), U23.5 (+), U7.5 (COM), Z122.2, Z123.2, Z124.2, Z125.2, Z126.2, Z127.2, Z128.2, Z129.2, Z134.2, Z135.2, Z136.2, Z137.2, Z170.2, Z171.2, Z174.2
- new net: C40.2, U13.1, U13.2 (-)
- new net: C25.1, H5.1
- new net: C119.1, H9.1
- new net: U21.12 (+), U21.3 (+), Z226.2, Z257.2, Z259.1
- new net: U19.1, U19.2 (-), Z230.1
- new net: C39.2, U12.1, U12.2 (-)
- new net: U18.1, U18.2 (-), Z234.1
- new net: U18.12 (+), U18.3 (+), Z224.2
- new net: R133.2, U14.13 (-), U14.14, Z185.1
- new net: Z185.2, Z193.1, Z198.1
- new net: J29.1 (Pin_1), Z257.1, Z258.1
- new net: U11.13 (-), U11.14
- new net: U19.12 (+), U19.3 (+), Z222.2
- new net: C116.1, H15.1
- new net: C38.2, U12.6 (-), U12.7
- new net: U11.8, U11.9 (-)
- new net +15V_M: C46.2, C56.2, J21.6 (Pin_5), R72.1, U23.4 (V+), U24.4 (V+)
- new net +15V_P: J21.5 (Pin_5), R26.1
- new net +9V_M: J21.9 (Pin_2), J36.4 (Pin_4)
- new net +9V_O: J22.2 (Pin_2)
- new net +9V_P: J21.2 (Pin_2), R25.1
- new net -15V_M: C47.2, C57.2, J21.8 (Pin_3), U23.11 (V-), U24.11 (V-)
- new net -15V_P: J21.3 (Pin_3), R27.1
- new net 9V_GND_M: J21.10 (Pin_1), J36.3 (Pin_3)
- new net 9V_GND_O: J22.1 (Pin_1)
- new net GND_9V_FILT: C117.1, C118.2, C23.1, C24.2
- new net GND_M: C25.2, C36.2, C46.1, C47.1, C56.1, C57.1, D3.2 (A), J21.7 (Pin_4), J36.2 (Pin_2), R75.1, R86.1, U23.10 (+), U23.12 (+), Z122.2, Z123.2, Z124.2, Z125.2, Z126.2, Z127.2, Z128.2, Z129.2, Z134.2, Z135.2, Z136.2, Z137.2, Z170.2, Z171.2, Z174.2
- new net GND_P: C19.2, C20.1, J21.4 (Pin_4), U7.5 (COM)
- no-connect marks 12 -> 3
Other:
- moved on the sheet: C10, C11, C18, C19, C2, C20, C23, C24, C26, C38, C39, C42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

Commit message: PCB Update
Parts:
- removed C112, C113, C114, C115: 100n, Capacitor_SMD:C_0805_2012Metric_Pad1.18x1.45mm_HandSolder, symbol Device:C_Small
- removed unit 3 of U2
- removed U25: INA128U, INA128U:INA128U_L, symbol INA128U:INA128U
- added C124, C125: 100n, Capacitor_SMD:C_0805_2012Metric_Pad1.18x1.45mm_HandSolder, symbol Device:C_Small
- added R150, R151, R152, R153, R154: 10k, Resistor_SMD:R_0805_2012Metric_Pad1.20x1.40mm_HandSolder, symbol Device:R
- added unit 4 of U2
- added U25: TL074, Package_DIP:DIP-14_W7.62mm_Socket_LongPads, symbol Amplifier_Operational:TL074
- added unit 3 of U26
- added unit 1 of U26
- added unit 5 of U26
- added unit 4 of U26
- added unit 4 of U5
- R2: value 100R -> 10k
- RV18, RV19: footprint Connector_PinSocket_2.54mm_LongPads:PinSocket_2x03_P2.54mm_Vertical_LongPads_Mirrored -> Connector_PinSocket_2.54mm_LongPads:PinSocket_2x03_P2.54mm_Vertical_LongPads
- RV3: footprint Connector_PinSocket_2.54mm_LongPads:PinSocket_1x06_P2.54mm_Vertical_LongPads -> Connector_PinSocket_2.54mm_LongPads:PinSocket_2x03_P2.54mm_Vertical_LongPads
- RV5: footprint Connector_PinSocket_2.54mm_LongPads:PinSocket_1x06_P2.54mm_Vertical_LongPads -> Connector_PinSocket_2.54mm_LongPads:PinSocket_2x03_P2.54mm_Vertical_LongPads_Mirrored
- U4: footprint Package_DIP:DIP-14_W7.62mm_Socket_LongPads -> (none)
- renumbered U4 to U26, U5 to U4
Connections:
- net +15V_I: now also C7.1, C124.2, U25.4 (V+), U26.4 (V+); no longer C7.2
- net -15V_I: now also C125.2, U25.11 (V-), U26.11 (V-)
- net GND_I: now also C7.2, J5.2 (Pin_2), U4.10 (+), Z77.1, C124.1, C125.1, R152.1, U2.12 (+), U25.12 (+), U26.10 (+), U5.12 (+); no longer C7.1, J5.1 (Pin_1), Z77.2
- net at RV2.1: now also R2.2, U25.2 (-)
- net at RV2.2, RV2.3: now also R150.1, U25.6 (-); no longer R2.1
- net at R15.1, Z83.1, Z88.1: now also U5.8; no longer U5.7
- net at R10.1, R11.1, R15.2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: now also U5.9 (-); no longer U5.6 (-)
- net at R29.1, RV6.2, RV6.3: now also U26.2 (-)
- net at R29.2, R31.2: now also U26.13 (-); no longer U3.5 (+)
- net at Z11.2, Z21.1: now also U4.3 (+); no longer U4.12 (+)
- net at Z13.2, Z23.1: now also U5.3 (+); no longer U5.12 (+)
- net at R16.2, R17.2, R19.1: now also U4.13 (-); no longer U4.6 (-)
- net at R19.2, Z71.1: now also U4.14; no longer U4.7
- net at Z19.1, Z9.1: now also J5.1 (Pin_1); no longer J5.3 (Pin_3)
- net at Z76.2, Z81.1, Z82.1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: now also U26.5 (+); no longer U26.3 (+)
- net at Z80.1, Z85.1: now also U26.6 (-), U26.7; no longer U26.1, U26.2 (-)
- net at R32.2, Z84.1, Z89.1: now also U26.14; no longer U3.7
- net at Z20.2, Z30.1: now also U25.5 (+)
- net at R16.1: now also Z79.2; no longer Z61.2
- net at Z19.2, Z29.1: now also U25.3 (+)
- net at Z10.1, Z20.1: now also J5.3 (Pin_3); no longer J5.2 (Pin_2)
- net at R3.1, RV1.1: now also Z59.2; no longer Z79.2
- net at RV1.2: now also U3.5 (+); no longer U3.10 (+)
- net at R12.2, RV1.3, Z56.1: now also U3.8; no longer U4.8
- net at Z12.2, Z22.1: now also U4.5 (+); no longer U4.3 (+)
- net at Z70.1: now also U4.12 (+); no longer U4.5 (+)
- net at Z54.1: now also U5.10 (+); no longer U5.5 (+)
- net at R28.1, RV6.1: now also U26.1
- net at R23.1, RV4.1: now also Z61.2; no longer Z59.2
- net at C3.1, RV3.1, RV3.2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: now also U3.10 (+); no longer U4.10 (+)
- net at R12.1, R3.2: now also U3.9 (-); no longer U4.9 (-)
- net at Z55.1: now also R154.1, U25.8
- net at Z14.2, Z24.1: now also U5.5 (+); no longer U5.10 (+)
- net at Z53.1: now also U2.10 (+); no longer U2.12 (+)
- net at R14.1, R7.2, R8.2: now also U2.9 (-); no longer U2.13 (-)
- net at R14.2, Z63.1: now also U2.8; no longer U2.14
- net at SW2.2 (B): now also U26.3 (+)
- net at Z78.2, Z79.1: now also Z77.2; no longer Z77.1
- net at R28.2, R32.1: now also U26.12 (+); no longer U3.6 (-)
- new net: U5.1, U5.2 (-), Z32.1
- new net: R151.1, R2.1, U25.1
- new net: R151.2, R152.2, U25.10 (+)
- new net: U4.1, U4.2 (-), Z31.1
- new net: U2.13 (-), U2.14
- new net: U26.8, U26.9 (-)
- new net: C1.2, U3.6 (-), U3.7
- new net: U5.13 (-), U5.14
- new net: U4.6 (-), U4.7, Z65.2
- new net: R153.2, R154.2, U25.9 (-)
- new net: U4.8, U4.9 (-)
- new net: U25.13 (-), U25.14
- new net: R150.2, R153.1, U25.7
- new net: U5.6 (-), U5.7, Z33.1
Other:
- moved on the sheet: C1, C13, C14, C16, C17, C22, C28, C29, C3, C30, C31, C32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

Commit message: PCB Update
Connections:
- net GND_I: now also U26.12 (+); no longer U26.10 (+), U4.10 (+), U5.12 (+)
- net at R29.1, RV6.2, RV6.3: now also U26.6 (-); no longer U26.2 (-)
- net at R29.2, R31.2: now also U26.10 (+); no longer U26.13 (-)
- net at Z80.1, Z85.1: now also U26.1, U26.2 (-); no longer U26.6 (-), U26.7
- net at R32.2, Z84.1, Z89.1: now also U26.8; no longer U26.14
- net at R28.1, RV6.1: now also U26.7; no longer U26.1
- net at U5.13 (-), U5.14: now also Z81.1, Z86.1
- net at SW2.2 (B): now also U26.5 (+); no longer U26.3 (+)
- net at U4.8, U4.9 (-): now also Z82.1, Z87.1
- net at R28.2, R32.1: now also U26.9 (-); no longer U26.12 (+)
- new net: U26.3 (+), U4.10 (+), U5.12 (+), Z76.2
- new net: U26.13 (-), U26.14
Other:
- moved on the sheet: U25D, U26D, U2D, U4C, U5D

Commit message: PCB Update
Other:
- moved on the sheet: R31
Changed lines of the file:
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@@
 	(symbol
 		(lib_id "Device:R")
-		(at 210.82 135.89 180)
+		(at 210.82 135.89 0)
+		(mirror x)
 		(unit 1)
 		(exclude_from_sim no)
@@
 		(on_board yes)
 		(dnp no)
-		(fields_autoplaced yes)
 		(property "Reference" "R31"
-			(at 213.36 134.6199 0)
+			(at 208.28 134.6199 0)
 			(effects
 				(font
@@
 		)
 		(property "Value" "1k"
-			(at 213.36 137.1599 0)
+			(at 208.28 137.1599 0)
 			(effects
 				(font
@@
 		)
 		(property "Footprint" "Resistor_SMD:R_0805_2012Metric_Pad1.20x1.40mm_HandSolder"
-			(at 212.598 135.89 90)
+			(at 209.042 135.89 90)
 			(effects
 				(font
@@
 		(lib_id "Device:R")
 		(at 223.52 219.71 0)
+		(mirror y)
 		(unit 1)
 		(exclude_from_sim no)
@@
 		(dnp no)
 		(property "Reference" "Z58"
-			(at 226.568 219.71 90)
+			(at 220.472 219.71 90)
 			(effects
 				(font
@@
 		)
 		(property "Value" "~"
-			(at 227.33 219.71 90)
+			(at 219.71 219.71 90)
 			(effects
 				(font
@@
 		)
 		(property "Footprint" "Resistor_SMD:R_0805_2012Metric_Pad1.20x1.40mm_HandSolder"
-			(at 221.742 219.71 90)
+			(at 225.298 219.71 90)
 			(effects
 				(font

Commit message: PCB Final Update
Parts:
- removed J12: EMK_In, Connector_PinHeader_2.54mm_LongPads:PinHeader_1x05_P2.54mm_Vertical_LongPads, symbol Connector:Conn_01x05_Pin
- added J12: Conn_02x07_Odd_Even, Connector_PinHeader_2.54mm:PinHeader_2x07_P2.54mm_Vertical, symbol Connector_Generic:Conn_02x07_Odd_Even
Connections:
- net +15V_I: now also J12.13 (Pin_13), J12.14 (Pin_14)
- net +9V_I: now also J12.5 (Pin_5), J12.6 (Pin_6)
- net -15V_I: now also J12.7 (Pin_7), J12.8 (Pin_8)
- net 9V_GND_I: now also J12.1 (Pin_1), J12.2 (Pin_2), J12.3 (Pin_3), J12.4 (Pin_4)
- net GND_I: now also J12.10 (Pin_10), J12.11 (Pin_11), J12.12 (Pin_12), J12.9 (Pin_9)
Other:
- moved on the sheet: C124, C125, C13, C14, C16, C17, C28, C29, C31, C32, C33, C34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

Commit message: final PCB Update
Parts:
- removed C117, C118, C123: 10n, Capacitor_SMD:C_0805_2012Metric_Pad1.18x1.45mm_HandSolder, symbol Device:C_Small
- removed C120, C121, C122: 100n, Capacitor_SMD:C_0805_2012Metric_Pad1.18x1.45mm_HandSolder, symbol Device:C_Small
- removed C25: 10n, Capacitor_SMD:C_1210_3225Metric_Pad1.33x2.70mm_HandSolder, symbol Device:C_Small
- removed C4: 1n, Capacitor_SMD:C_0805_2012Metric_Pad1.18x1.45mm_HandSolder, symbol Device:C_Small
- removed J21: Conn_01x05_bridged, Connector_Bridged_2.54mm_LongPads:Bridge_2x05_P2.54mm_Vertical_LongPads, symbol conn_01x05_bridged:Conn_01x05_bridged
- removed J22: EMK_In, Connector_PinHeader_2.54mm_LongPads:PinHeader_1x05_P2.54mm_Vertical_LongPads, symbol Connector:Conn_01x05_Pin
- removed R25, R26, R27: 22R, Resistor_SMD:R_0805_2012Metric_Pad1.20x1.40mm_HandSolder, symbol Device:R
- removed unit 5 of U10
- removed unit 5 of U11
- removed unit 5 of U12
- removed unit 5 of U13
- added C100, C112, C89: 10n, Capacitor_SMD:C_0805_2012Metric_Pad1.18x1.45mm_HandSolder, symbol Device:C_Small
- added C111: 1n, Capacitor_SMD:C_0805_2012Metric_Pad1.18x1.45mm_HandSolder, symbol Device:C_Small
- added C114, C118, C91: 10u, Capacitor_THT:CP_Radial_D5.0mm_P2.50mm, symbol Device:C_Polarized_Small
- added C85: 10n, Capacitor_SMD:C_1210_3225Metric_Pad1.33x2.70mm_HandSolder, symbol Device:C_Small
- added J31, J40, J41: Conn_02x07_Odd_Even, Connector_PinHeader_2.54mm:PinHeader_2x07_P2.54mm_Vertical, symbol Connector_Generic:Conn_02x07_Odd_Even
- added unit 5 of U18
- added unit 5 of U2
- added unit 5 of U5
- added unit 5 of U7
- added Z241, Z255, Z258: ~, Resistor_SMD:R_0805_2012Metric_Pad1.20x1.40mm_HandSolder, symbol Device:R
- RV10: renamed from RV19; footprint Connector_PinSocket_2.54mm_LongPads:PinSocket_2x03_P2.54mm_Vertical_LongPads -> Connector_PinSocket_2.54mm_LongPads:PinSocket_2x03_P2.54mm_Vertical_LongPads_Mirrored
- RV2: renamed from RV18; footprint Connector_PinSocket_2.54mm_LongPads:PinSocket_2x03_P2.54mm_Vertical_LongPads -> Connector_PinSocket_2.54mm_LongPads:PinSocket_2x03_P2.54mm_Vertical_LongPads_Mirrored
- renumbered C21 to C1, C52 to C10, C36 to C101, C24 to C102, C10 to C103, C67 to C104, C79 to C105, C97 to C106, C101 to C107, C105 to C108, C74 to C11, C11 to C110, C19 to C113, C2 to C115, C5 to C116, C20 to C117, C6 to C119, C43 to C12, C26 to C120, C12 to C121, C62 to C13, C86 to C14, C39 to C15, C49 to C16, C59 to C17, C71 to C18, C83 to C19, C27 to C2, C53 to C20, C75 to C21, C42 to C22, C63 to C23, C87 to C24, C38 to C25, C50 to C26, C60 to C27, C72 to C28, C84 to C29, C116 to C3, C54 to C30, C76 to C31, C44 to C32, C3 to C33, C64 to C34, C88 to C35, C40 to C36, C1 to C37, C51 to C38, C61 to C39, C119 to C4, C73 to C40, C85 to C41, C55 to C42, C77 to C43, C45 to C44, C65 to C45, C89 to C46, C41 to C47, C30 to C48, C22 to C49, C48 to C5, C35 to C50, C37 to C51, C7 to C52, C124 to C53, C13 to C54, C16 to C55, C31 to C56, C33 to C57, C28 to C58, C8 to C59, C58 to C6, C125 to C60, C14 to C61, C17 to C62, C32 to C63, C34 to C64, C29 to C65, C110 to C66, C68 to C67, C80 to C68, C92 to C69, C70 to C7, C111 to C70, C69 to C71, C81 to C72, C93 to C73, C90 to C74, C94 to C75, C98 to C76, C102 to C77, C106 to C78, C91 to C79, C82 to C8, C95 to C80, C99 to C81, C103 to C82, C107 to C83, C9 to C84, C23 to C86, C46 to C87, C56 to C88, C15 to C9, C18 to C90, C47 to C92, C57 to C93, C66 to C94, C78 to C95, C100 to C97, C104 to C98, C108 to C99, D2 to D1, D1 to D2, D4 to D3, D3 to D4, H16 to H1, H4 to H10, H8 to H11, H5 to H12, H2 to H13, H3 to H14, H6 to H15, H7 to H16, H12 to H2, H15 to H3, H9 to H4, H11 to H5, H14 to H6, H13 to H7, H10 to H8, H1 to H9, J40 to J1, J42 to J10, J43 to J11, J20 to J12, J27 to J13, J16 to J14, J24 to J15, J15 to J16, J7 to J17, J38 to J18, J44 to J19, J1 to J2, J6 to J20, J45 to J21, J8 to J22, J17 to J23, J25 to J24, J37 to J25, J39 to J26, J18 to J27, J9 to J28, J28 to J29, J2 to J3, J12 to J30, J29 to J32, J30 to J33, J36 to J34, J31 to J35, J32 to J36, J34 to J37, J35 to J38, J10 to J39, J19 to J4, J33 to J42, J11 to J43, J26 to J5, J41 to J6, J3 to J7, J4 to J8, J5 to J9, L2 to L1, L3 to L2, L4 to L3, L1 to L4, R39 to R1, R117 to R10, R98 to R100, R23 to R101, R16 to R102, R19 to R103, R17 to R104, R21 to R105, R24 to R106, R43 to R107, R57 to R108, R145 to R109, R141 to R11, R33 to R110, R69 to R111, R76 to R112, R44 to R113, R121 to R114, R131 to R115, R79 to R116, R85 to R117, R99 to R118, R51 to R119, R93 to R12, R70 to R120, R100 to R121, R125 to R123, R45 to R124, R58 to R125, R9 to R126, R34 to R127, R46 to R128, R77 to R129, R40 to R13, R83 to R130, R123 to R131, R52 to R133, R10 to R134, R15 to R135, R78 to R136, R124 to R137, R80 to R138, R126 to R139, R49 to R14, R11 to R140, R67 to R141, R71 to R142, R81 to R143, R86 to R144, R59 to R145, R60 to R146, R68 to R147, R82 to R148, R84 to R149, R18 to R15, R72 to R150, R75 to R151, R6 to R16, R105 to R17, R113 to R18, R127 to R19, R55 to R2, R137 to R20, R146 to R21, R88 to R22, R94 to R23, R28 to R24, R32 to R25, R41 to R26, R56 to R27, R110 to R28, R134 to R29, R20 to R3, R14 to R30, R101 to R31, R29 to R32, R7 to R33, R118 to R34, R142 to R35, R31 to R36, R91 to R37, R42 to R38, R50 to R39, R22 to R4, R106 to R40, R114 to R41, R128 to R42, R138 to R43, R147 to R44, R8 to R45, R87 to R46, R92 to R47, R35 to R48, R53 to R49, R109 to R5, R111 to R50, R135 to R51, R153 to R52, R154 to R53, R61 to R54, R103 to R55, R36 to R56, R150 to R57, R12 to R58, R119 to R59, R133 to R6, R143 to R60, R47 to R61, R73 to R63, R95 to R64, R3 to R65, R63 to R66, R2 to R67, R107 to R68, R115 to R69, R13 to R7, R129 to R70, R139 to R71, R148 to R72, R89 to R73, R96 to R74, R151 to R75, R1 to R76, R4 to R77, R37 to R78, R54 to R79, R102 to R8, R152 to R80, R112 to R81, R136 to R82, R64 to R83, R104 to R84, R38 to R85, R120 to R86, R144 to R87, R48 to R88, R65 to R89, R5 to R9, R74 to R90, R97 to R91, R66 to R92, R30 to R93, R108 to R94, R116 to R95, R130 to R96, R140 to R97, R149 to R98, R90 to R99, RV9 to RV1, RV3 to RV11, RV14 to RV12, RV1 to RV13, RV8 to RV14, RV20 to RV15, RV15 to RV16, RV5 to RV17, RV4 to RV18, RV16 to RV19, RV21 to RV20, RV11 to RV21, RV13 to RV3, RV6 to RV4, RV10 to RV5, RV17 to RV6, RV12 to RV7, RV7 to RV8, RV2 to RV9, SW5 to SW1, SW12 to SW10, SW9 to SW11, SW1 to SW12, SW6 to SW3, SW3 to SW4, SW4 to SW5, SW7 to SW6, SW11 to SW7, SW10 to SW9, U8 to U1, U9 to U10, U25 to U11, U16 to U12, U18 to U13, U13 to U14, U3 to U15, U17 to U16, U4 to U17, U10 to U18, U5 to U19, U14 to U2, U21 to U20, U22 to U21, U20 to U22, U6 to U25, U7 to U26, U19 to U3, U1 to U4, U12 to U5, U15 to U6, U11 to U7, U26 to U8, U2 to U9, Z238 to Z1, Z68 to Z10, Z58 to Z100, Z214 to Z101, Z223 to Z102, Z187 to Z103, Z203 to Z104, Z232 to Z105, Z252 to Z106, Z156 to Z107, Z218 to Z108, Z19 to Z109, Z5 to Z11, Z195 to Z110, Z242 to Z111, Z9 to Z112, Z29 to Z113, Z243 to Z114, Z139 to Z115, Z151 to Z116, Z184 to Z117, Z201 to Z118, Z233 to Z119, Z25 to Z12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
Connections:
- net +15V_M: now also J41.13 (Pin_13), J41.14 (Pin_14)
- net +15V_O: now also J31.13 (Pin_13), J31.14 (Pin_14), U18.4 (V+), U2.4 (V+), U5.4 (V+), U7.4 (V+)
- net +15V_P: now also C114.1, J40.13 (Pin_13), J40.14 (Pin_14), Z255.2
- net +9V_M: now also J41.5 (Pin_5), J41.6 (Pin_6)
- net +9V_O: now also J31.5 (Pin_5), J31.6 (Pin_6)
- net +9V_P: now also C91.1, J40.5 (Pin_5), J40.6 (Pin_6), Z241.2
- net -15V_M: now also J41.7 (Pin_7), J41.8 (Pin_8)
- net -15V_O: now also J31.7 (Pin_7), J31.8 (Pin_8), U18.11 (V-), U2.11 (V-), U5.11 (V-), U7.11 (V-)
- net -15V_P: now also C118.2, J40.7 (Pin_7), J40.8 (Pin_8), Z258.2
- net 9V_GND_M: now also J41.1 (Pin_1), J41.2 (Pin_2), J41.3 (Pin_3), J41.4 (Pin_4)
- net 9V_GND_O: now also J31.1 (Pin_1), J31.2 (Pin_2), J31.3 (Pin_3), J31.4 (Pin_4)
- net 9V_GND_P: now also C91.2, J40.1 (Pin_1), J40.2 (Pin_2), J40.3 (Pin_3), J40.4 (Pin_4)
- net GND_15V_FILT: now also C111.1, C112.1
- net GND_9V_FILT: now also C100.2, C89.1
- net GND_M: now also C85.2, J41.10 (Pin_10), J41.11 (Pin_11), J41.12 (Pin_12), J41.9 (Pin_9)
- net GND_O: now also J31.10 (Pin_10), J31.11 (Pin_11), J31.12 (Pin_12), J31.9 (Pin_9)
- net GND_P: now also C114.2, C118.1, J40.10 (Pin_10), J40.11 (Pin_11), J40.12 (Pin_12), J40.9 (Pin_9)
- net at C117.2, C120.1, C121.2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: now also Z258.1
- net at H12.1: now also C85.1
- net at C110.2, C113.1, L3.2: now also C111.2, Z255.1
- net at C103.1, C116.2, C119.1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: now also C100.1
- net at C110.1, C116.1, C84.1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: now also C112.2, C89.2
- net at C84.2, C86.2, C90.1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: now also Z241.1
Other:
- moved on the sheet: C1, C10, C101, C102, C103, C104, C105, C106, C107, C108, C109, C11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
