File: KiCad/Input.kicad_pcb (KiCad board)
At the start: 4 copper layers, 150 x 75 mm, 177 parts, among them J1 R_Phono_In, J12 EMK_In, J15 Mic_Effekt_Out, J16 Mic_Effekt_Out, J17 Mic_Effekt_Out, J18 Mic_Effekt_Out, J19 Phono/Line_Out, J2 L_Phono_In, J20 Mic_Effekt_Out, J3 R_Line_In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

Commit message: PCB Update
Parts:
- SW2: footprint Connector_PinSocket_2.54mm_LongPads:PinSocket_1x03_P2.54mm_Vertical_LongPads -> Connector_PinHeader_2.54mm_LongPads:PinHeader_1x03_P2.54mm_Vertical_LongPads
- moved SW2 329.6 mm to (58.4, 96.5)
- moved RV6 326.3 mm to (58.4, 86.4)
- moved C16 316.8 mm to (68.6, 109.2)
- moved C13 310.2 mm to (68.6, 73.7)
- moved C17 298.8 mm to (86.4, 109.2), turned to 180 degrees
- moved C21 297.0 mm to (86.4, 83.8)
- moved Z51 294.1 mm to (68.6, 119.4)
- moved C14 292.6 mm to (86.4, 73.7), turned to 180 degrees
- moved C15 292.5 mm to (86.4, 78.7), turned to 180 degrees
- moved Z50 292.3 mm to (68.6, 101.6)
- moved C27 291.9 mm to (91.4, 83.8)
- moved Z41 291.7 mm to (63.5, 68.6), turned to 180 degrees
- moved Z43 291.6 mm to (63.5, 104.1), turned to 180 degrees
- moved Z37 289.5 mm to (68.6, 116.8), turned to 180 degrees
- moved Z48 288.9 mm to (68.6, 66.0)
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Connections:
- C15 pad 2: Net-(U1D--) -> Net-(U1C--)
- C21 pad 1: Net-(U1D--) -> Net-(U1C--)
- R13 pad 1: Net-(U1C--) -> Net-(U1D--)
- R14 pad 1: Net-(U2C--) -> Net-(U2D--)
- R20 pad 2: Net-(U1D--) -> Net-(U1C--)
- R29 pad 1: Net-(U2D--) -> Net-(U2C--)
- R5 pad 2: Net-(U1C--) -> Net-(U1D--)
- R6 pad 2: Net-(U1C--) -> Net-(U1D--)
- R7 pad 2: Net-(U2C--) -> Net-(U2D--)
- R8 pad 2: Net-(U2C--) -> Net-(U2D--)
- RV6 pad 2: Net-(U2D--) -> Net-(U2C--)
- RV6 pad 3: Net-(U2D--) -> Net-(U2C--)
- U1 pad 14: Net-(C27-Pad2) -> Net-(R13-Pad2)
- U1 pad 8: Net-(R13-Pad2) -> Net-(C27-Pad2)
- U2 pad 10: Net-(U2C-+) -> Net-(SW2-B)
- U2 pad 12: Net-(SW2-B) -> Net-(U2D-+)
- U2 pad 14: Net-(R28-Pad1) -> Net-(R14-Pad2)
- U2 pad 8: Net-(R14-Pad2) -> Net-(R28-Pad1)
- Z52 pad 1: Net-(U1C-+) -> Net-(U1D-+)
- Z53 pad 1: Net-(U2C-+) -> Net-(U2D-+)
- Z68 pad 2: Net-(U1D-+) -> Net-(U1C-+)
Routing:
- net Net-(SW2-B): track 0.00 -> 55.8 mm
- net Net-(U1D--): track 0.00 -> 38.0 mm
- net Net-(U2D--): track 0.00 -> 37.8 mm
- net Net-(SW2-C): track 0.00 -> 32.3 mm, vias 0 -> 1
- net Net-(SW2-A): track 0.00 -> 30.1 mm
- net Net-(C27-Pad2): track 0.00 -> 19.8 mm
- net Net-(Z62-Pad2): track 0.00 -> 11.8 mm
- net Net-(U2B-+): track 0.00 -> 10.4 mm
- net Net-(U2A-+): track 0.00 -> 10.4 mm
- net Net-(R13-Pad2): track 0.00 -> 9.57 mm
- net Net-(R14-Pad2): track 0.00 -> 9.57 mm
- net Net-(U1C--): track 0.00 -> 9.15 mm
- net Net-(C21-Pad2): track 0.00 -> 8.19 mm
- net -15V: track 0.00 -> 8.09 mm
- net +15V: track 0.00 -> 8.08 mm
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
Commit message: PCB Update
Parts:
- moved J5 333.1 mm to (58.4, 61.0)
- moved C31 297.0 mm to (101.6, 109.2)
- moved C8 285.3 mm to (101.6, 96.5)
- moved U25 281.5 mm to (110.5, 94.6)
- moved Z89 280.7 mm to (106.7, 121.9)
- moved C32 279.0 mm to (119.4, 109.2), turned to 180 degrees
- moved Z84 276.6 mm to (101.6, 119.4)
- moved Z94 270.4 mm to (114.3, 121.9)
- moved U4 268.7 mm to (106.7, 66.0)
- moved C7 267.6 mm to (119.4, 94.0), turned to 180 degrees
- moved Z30 261.1 mm to (96.5, 94.0), turned to 180 degrees
- moved Z29 256.2 mm to (101.6, 94.0), turned to 180 degrees
- moved Z20 256.0 mm to (96.5, 91.4)
- moved RV2 252.3 mm to (129.5, 86.4)
- moved Z10 251.4 mm to (96.5, 88.9)
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Connections:
- C1 pad 2: Net-(U3D--) -> Net-(U3C--)
- C22 pad 2: Net-(U3B--) -> Net-(U3A--)
- C30 pad 1: Net-(U3C-+) -> Net-(U3D-+)
- R23 pad 2: Net-(U3C--) -> Net-(U3D--)
- R28 pad 2: Net-(U3A--) -> Net-(U3B--)
- R29 pad 2: Net-(U3A-+) -> Net-(U3B-+)
- R30 pad 1: Net-(U3C--) -> Net-(U3D--)
- R31 pad 2: Net-(U3A-+) -> Net-(U3B-+)
- R32 pad 1: Net-(U3A--) -> Net-(U3B--)
- RV1 pad 2: Net-(U3D-+) -> Net-(U3C-+)
- RV4 pad 2: Net-(U3B-+) -> Net-(U3A-+)
- RV5 pad 1: Net-(U3C-+) -> Net-(U3D-+)
- RV5 pad 2: Net-(U3C-+) -> Net-(U3D-+)
- RV5 pad 5: Net-(U3C-+) -> Net-(U3D-+)
- RV5 pad 6: Net-(U3C-+) -> Net-(U3D-+)
- U3 pad 1: Net-(R32-Pad2) -> Net-(U3A--)
- U3 pad 14: Net-(U3D--) -> Net-(R30-Pad2)
- U3 pad 7: Net-(U3B--) -> Net-(R32-Pad2)
- U3 pad 8: Net-(R30-Pad2) -> Net-(U3C--)
Routing:
- net Net-(J19-Pin_1): track 0.00 -> 92.6 mm, vias 0 -> 1
- net Net-(R28-Pad1): track 0.00 -> 84.8 mm
- net Net-(U2C--): track 0.00 -> 79.7 mm
- net Net-(RV2-Pad1): track 0.00 -> 24.3 mm
- net Net-(R32-Pad2): track 0.00 -> 16.9 mm
- net Net-(SW2-B): track 55.8 -> 42.0 mm
- net Net-(U25-IN+): track 0.00 -> 13.4 mm
- net Net-(R2-Pad1): track 0.00 -> 11.7 mm
- net Net-(U3B-+): track 0.00 -> 10.2 mm
- net +15V: track 8.08 -> 17.4 mm
- net -15V: track 8.09 -> 17.4 mm
- net Net-(U25-IN-): track 0.00 -> 7.80 mm
- net Net-(U3B--): track 0.00 -> 6.62 mm
- net Net-(R2-Pad2): track 0.00 -> 5.79 mm
- net Net-(J19-Pin_2): track 0.00 -> 4.08 mm
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
Commit message: PCB Update
Parts:
- C7, C8: value 0.1uF -> 100n
- moved C33 293.8 mm to (101.6, 73.7)
- moved C34 276.0 mm to (119.4, 73.7), turned to 180 degrees
- moved C30 275.4 mm to (124.5, 111.8), turned to 180 degrees
- moved Z76 274.7 mm to (101.6, 68.6)
- moved C22 274.5 mm to (119.4, 114.3), turned to 180 degrees
- moved C1 271.9 mm to (119.4, 116.8), turned to 180 degrees
- moved RV5 271.8 mm to (129.5, 106.7)
- moved Z73 271.1 mm to (101.6, 66.0)
- moved RV3 270.6 mm to (129.5, 58.4)
- moved Z71 270.3 mm to (101.6, 71.1), turned to 180 degrees
- moved Z70 270.0 mm to (101.6, 76.2), turned to 180 degrees
- moved RV4 255.7 mm to (129.5, 96.5)
- moved C3 251.2 mm to (134.6, 61.0)
- moved RV1 249.4 mm to (129.5, 76.2)
- moved C28 247.8 mm to (144.8, 109.2)
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Connections:
- C3 pad 1: Net-(U4A-+) -> Net-(U4C-+)
- R12 pad 1: Net-(U4A--) -> Net-(U4C--)
- R16 pad 2: Net-(U4C--) -> Net-(U4B--)
- R17 pad 2: Net-(U4C--) -> Net-(U4B--)
- R19 pad 1: Net-(U4C--) -> Net-(U4B--)
- R3 pad 2: Net-(U4A--) -> Net-(U4C--)
- RV3 pad 1: Net-(U4A-+) -> Net-(U4C-+)
- RV3 pad 2: Net-(U4A-+) -> Net-(U4C-+)
- RV3 pad 5: Net-(U4A-+) -> Net-(U4C-+)
- RV3 pad 6: Net-(U4A-+) -> Net-(U4C-+)
- U4 pad 1: Net-(R12-Pad2) -> Net-(U4A--)
- U4 pad 7: Net-(U4B--) -> Net-(R19-Pad2)
- U4 pad 8: Net-(R19-Pad2) -> Net-(R12-Pad2)
- Z12 pad 2: Net-(U5C-+) -> Net-(U5A-+)
- Z14 pad 2: Net-(U5A-+) -> Net-(U5C-+)
- Z22 pad 1: Net-(U5C-+) -> Net-(U5A-+)
- Z24 pad 1: Net-(U5A-+) -> Net-(U5C-+)
- Z31 pad 1: Net-(U5C--) -> Net-(U5A--)
- Z33 pad 1: Net-(U5A--) -> Net-(U5C--)
- Z70 pad 1: Net-(U4C-+) -> Net-(U4B-+)
- Z76 pad 2: Net-(U4B-+) -> Net-(U4A-+)
- Z80 pad 1: Net-(U4B--) -> Net-(U4A--)
- Z81 pad 1: Net-(U4B-+) -> Net-(U4A-+)
- Z82 pad 1: Net-(U4B-+) -> Net-(U4A-+)
- Z85 pad 1: Net-(U4B--) -> Net-(U4A--)
- Z86 pad 1: Net-(U4B-+) -> Net-(U4A-+)
- Z87 pad 1: Net-(U4B-+) -> Net-(U4A-+)
Routing:
- net Net-(J19-Pin_1): track 92.6 -> 0.00 mm, vias 1 -> 0
- net Net-(J5-Pin_3): track 2.54 -> 67.9 mm, vias 0 -> 1
- net Net-(J5-Pin_2): track 2.54 -> 65.3 mm, vias 0 -> 1
- net Net-(R1-Pad2): track 0.00 -> 61.6 mm, vias 0 -> 1
- net Net-(U3C-+): track 0.00 -> 47.4 mm
- net Net-(R30-Pad2): track 0.00 -> 43.7 mm
- net Net-(U5B--): track 0.00 -> 39.1 mm
- net Net-(U3D-+): track 0.00 -> 37.2 mm
- net Net-(J6-Pin_1): track 0.00 -> 36.2 mm
- net Net-(U4C-+): track 0.00 -> 36.2 mm
- net Net-(U3A-+): track 0.00 -> 33.3 mm
- net Net-(J8-Pin_1): track 0.00 -> 30.9 mm
- net Net-(U4B--): track 0.00 -> 24.9 mm
- net Net-(J7-Pin_1): track 0.00 -> 23.5 mm
- net Net-(R19-Pad2): track 0.00 -> 23.0 mm
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
Commit message: PCB Update
Parts:
- moved Z64 129.2 mm to (127.0, 61.0)
- moved Z85 124.7 mm to (109.2, 68.6), turned to 180 degrees
- moved Z65 124.2 mm to (132.1, 63.5), turned to 180 degrees
- moved Z90 120.9 mm to (109.2, 71.1)
- moved Z80 120.1 mm to (109.2, 66.0), turned to 180 degrees
- moved Z60 119.3 mm to (127.0, 58.4), turned to 180 degrees
- moved Z94 111.7 mm to (147.3, 111.8)
- moved R17 110.7 mm to (127.0, 86.4)
- moved Z99 110.7 mm to (147.3, 119.4)
- moved J19 110.3 mm to (152.4, 114.3)
- moved J17 109.5 mm to (152.4, 76.2)
- moved J18 109.5 mm to (152.4, 83.8)
- moved Z89 103.9 mm to (147.3, 114.3)
- moved Z83 101.1 mm to (157.5, 71.1), turned to 180 degrees
- moved Z88 100.2 mm to (157.5, 73.7), turned to 180 degrees
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Routing:
- net +15V: track 25.4 -> 680.9 mm, vias 0 -> 1
- net -15V: track 25.4 -> 444.8 mm, vias 0 -> 1
- net Net-(U4A-+): track 7.67 -> 105.1 mm
- net Net-(J20-Pin_1): track 0.00 -> 57.3 mm, vias 0 -> 1
- net Net-(R15-Pad1): track 9.83 -> 55.1 mm, vias 0 -> 1
- net Net-(R32-Pad2): track 4.08 -> 34.6 mm
- net Net-(R17-Pad1): track 0.00 -> 26.7 mm
- net GND: track 0.00 -> 18.7 mm
- net Net-(U25-IN-): track 7.80 -> 21.7 mm
- net Net-(U4A--): track 2.54 -> 14.2 mm
- net Net-(R19-Pad2): track 23.0 -> 13.2 mm
- net Net-(Z60-Pad1): track 0.00 -> 9.57 mm
- net Net-(J7-Pin_1): track 23.5 -> 14.8 mm
- net Net-(J9-Pin_1): track 6.62 -> 15.1 mm
- net Net-(J6-Pin_1): track 36.2 -> 28.6 mm
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
Commit message: PCB Update
Parts:
- moved C1 10.2 mm to (121.9, 116.8)
- moved C22 10.2 mm to (121.9, 114.3)
- moved C32 10.2 mm to (121.9, 109.2)
- moved C34 10.2 mm to (121.9, 73.7)
- moved C7 10.2 mm to (121.9, 94.0)
- moved R13 10.2 mm to (83.8, 61.0)
- moved R14 10.2 mm to (83.8, 96.5)
- moved R16 10.2 mm to (121.9, 88.9)
- moved R2 10.2 mm to (121.9, 91.4)
- moved R21 10.2 mm to (121.9, 111.8)
- moved Z1 10.2 mm to (121.9, 66.0)
- moved Z11 10.2 mm to (121.9, 71.1)
- moved Z21 10.2 mm to (121.9, 68.6)
- moved Z55 10.2 mm to (121.9, 96.5)
- moved Z58 10.2 mm to (121.9, 86.4)
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Routing:
- net GND: track 18.7 -> 155.4 mm, vias 0 -> 74
- net Net-(U3D--): track 5.08 -> 27.5 mm, vias 0 -> 2
- net +15V: track 680.9 -> 695.4 mm
- net Net-(R15-Pad1): track 55.1 -> 61.3 mm
- net Net-(J19-Pin_1): track 3.37 -> 7.45 mm
- net Net-(J15-Pin_1): track 2.54 -> 6.62 mm
- net -15V: track 444.8 -> 440.9 mm
- net Net-(J9-Pin_1): track 15.1 -> 18.0 mm
- net Net-(R30-Pad2): track 46.0 -> 45.3 mm
- net Net-(U5D-+): track 17.8 -> 17.1 mm
- net Net-(J5-Pin_3): track 70.7 -> 70.0 mm
- net Net-(J20-Pin_1): track 57.3 -> 56.5 mm
- net Net-(U3A-+): track 32.8 -> 33.3 mm
- added copper zone on B.Cu, net GND
Other:
- board size 150 x 75 mm -> 150 x 90 mm

Commit message: PCB Update
Parts:
- moved C28 5.08 mm to (152.4, 109.2)
- moved C29 5.08 mm to (170.2, 109.2)
- moved C3 5.08 mm to (142.2, 61.0)
- moved C30 5.08 mm to (132.1, 111.8)
- moved R1 5.08 mm to (132.1, 116.8)
- moved R10 5.08 mm to (170.2, 106.7)
- moved R11 5.08 mm to (170.2, 111.8)
- moved R12 5.08 mm to (132.1, 78.7)
- moved R13 5.08 mm to (88.9, 61.0)
- moved R14 5.08 mm to (88.9, 96.5)
- moved R15 5.08 mm to (152.4, 114.3)
- moved R23 5.08 mm to (142.2, 96.5)
- moved R24 5.08 mm to (132.1, 114.3)
- moved R3 5.08 mm to (132.1, 76.2)
- moved R30 5.08 mm to (142.2, 99.1)
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Routing:
- net +15V: track 695.4 -> 25.4 mm, vias 1 -> 3
- net -15V: track 440.9 -> 25.7 mm, vias 1 -> 3
- net Net-(SW2-B): track 42.0 -> 47.9 mm
- net Net-(J5-Pin_2): track 64.1 -> 66.2 mm
- net Net-(R28-Pad1): track 91.4 -> 89.9 mm
- net GND: track 155.4 -> 154.7 mm
- added copper zone on B.Cu, net (none)
- added copper zone on F.Cu, net (none)
- added copper zone on In1.Cu, net (none)
- added copper zone on In2.Cu, net (none)
- added copper zone on In2.Cu, net +15V
- added copper zone on In2.Cu, net -15V
Other:
- board size 150 x 90 mm -> 150 x 85.2 mm
- board text added: "DiKo-Elektrotechnik Eingangsstufe"

Commit message: PCB Update Power Supply VU Amp
Routing:
- net GND: track 154.7 -> 157.6 mm
Changed lines of the file:
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@@
 	)
 	(segment
+		(start 124.46 85.09)
+		(end 125.73 86.36)
+		(width 0.6)
+		(layer "F.Cu")
+		(net 3)
+	)
+	(segment
 		(start 101.6 78.74)
 		(end 100.06 78.74)
@@
 	)
 	(segment
-		(start 128.0375 73.66)
-		(end 128.27 73.66)
+		(start 124.46 83.82)
+		(end 124.46 85.09)
 		(width 0.6)
 		(layer "F.Cu")
@@
 	)
 	(segment
-		(start 105.14 88.9)
-		(end 106.68 88.9)
+		(start 128.0375 73.66)
+		(end 128.27 73.66)
 		(width 0.6)
 		(layer "F.Cu")
@@
 	)
 	(segment
-		(start 126 86.36)
-		(end 124.46 86.36)
-		(width 0.6)
-		(layer "F.Cu")
-		(net 3)
-	)
-	(segment
 		(start 128.524 109.22)
 		(end 128.0375 109.22)
@@
 	)
 	(segment
+		(start 129.54 95.25)
+		(end 128.27 93.98)
+		(width 0.6)
+		(layer "F.Cu")
+		(net 3)
+	)
+	(segment
+		(start 125.73 86.36)
+		(end 126 86.36)
+		(width 0.6)
+		(layer "F.Cu")
+		(net 3)
+	)
+	(segment
 		(start 151.13 111.76)
 		(end 149.86 110.49)
@@
 	)
 	(segment
-		(start 129.54 93.98)
-		(end 128.0375 93.98)
-		(width 0.6)
-		(layer "F.Cu")
-		(net 3)
-	)
-	(segment
 		(start 131.064 110.236)
 		(end 131.064 111.7385)
@@
 	)
 	(segment
+		(start 105.41 88.9)
+		(end 106.68 90.17)
+		(width 0.6)
+		(layer "F.Cu")
+		(net 3)
+	)
+	(segment
 		(start 151.4 101.6)
 		(end 149.86 101.6)
@@
 	)
 	(segment
+		(start 105.14 88.9)
+		(end 105.41 88.9)
+		(width 0.6)
+		(layer "F.Cu")
+		(net 3)
+	)
+	(segment
 		(start 105.41 71.12)
 		(end 106.68 69.85)
@@
 	)
 	(segment
+		(start 128.27 93.98)
+		(end 128.0375 93.98)
+		(width 0.6)
+		(layer "F.Cu")
+		(net 3)
+	)
+	(segment
 		(start 95.0175 109.22)
 		(end 95.25 109.22)
@@
 	)
 	(via
-		(at 106.68 88.9)
+		(at 106.68 90.17)
 		(size 0.6)
 		(drill 0.3)
@@
 	)
 	(via
-		(at 129.54 93.98)
+		(at 129.54 95.25)
 		(size 0.6)
 		(drill 0.3)
@@
 	)
 	(via
-		(at 124.46 86.36)
+		(at 124.46 83.82)
 		(size 0.6)
 		(drill 0.3)
@@
 	)
 	(segment
-		(start 111.76 101.6)
-		(end 111.76 105.41)
+		(start 135.89 100.33)
+		(end 113.03 100.33)
 		(width 0.4)
 		(layer "F.Cu")
@@
 	)
 	(segment
-		(start 111.76 105.41)
-		(end 113.03 106.68)
+		(start 113.03 100.33)
+		(end 111.76 101.6)
 		(width 0.4)
 		(layer "F.Cu")
@@
 	)
 	(segment
-		(start 113.03 100.33)
-		(end 111.76 101.6)
+		(start 111.76 105.41)
+		(end 113.03 106.68)
 		(width 0.4)
 		(layer "F.Cu")
@@
 	)
 	(segment
-		(start 137.16 99.06)
-		(end 135.89 100.33)
+		(start 113.03 106.68)
+		(end 114.3 106.68)
 		(width 0.4)
 		(layer "F.Cu")
@@
 	)
 	(segment
-		(start 135.89 100.33)
-		(end 113.03 100.33)
+		(start 111.76 101.6)
+		(end 111.76 105.41)
 		(width 0.4)
 		(layer "F.Cu")
@@
 	)
 	(segment
-		(start 113.03 106.68)
-		(end 114.3 106.68)
+		(start 137.16 99.06)
+		(end 135.89 100.33)
 		(width 0.4)
 		(layer "F.Cu")
@@
 		(priority 1)
 		(connect_pads yes
-			(clearance 0.5)
+			(clearance 1)
 		)
 		(min_thickness 0.25)
@@
 				(xy 79.502 104.394) (xy 79.502 117.856) (xy 81.026 119.38) (xy 105.156 119.38) (xy 107.442 117.094)
 				(xy 107.442 110.998) (xy 108.966 109.474) (xy 110.998 109.474) (xy 112.268 110.744) (xy 112.268 117.602)
-				(xy 114.3 119.634) (xy 122.936 119.634) (xy 124.206 118.364) (xy 124.206 101.092) (xy 123.444 100.33)
-				(xy 123.444 95.758) (xy 125.984 93.218) (xy 130.302 93.218) (xy 132.08 94.996) (xy 132.08 110.998)
-				(xy 135.382 114.3) (xy 135.382 119.888) (xy 136.398 120.904) (xy 138.43 120.904) (xy 138.938 120.396)
-				(xy 138.938 117.348) (xy 140.462 115.824) (xy 144.526 115.824) (xy 145.542 116.84) (xy 145.542 118.618)
-				(xy 145.796 118.872) (xy 149.098 118.872) (xy 149.606 118.364) (xy 149.606 113.538) (xy 148.844 112.776)
-				(xy 144.78 112.776) (xy 143.764 111.76) (xy 143.764 108.966) (xy 144.78 107.95) (xy 148.844 107.95)
-				(xy 149.86 107.188) (xy 149.86 105.41) (xy 149.098 104.648) (xy 146.304 104.648) (xy 145.034 103.378)
-				(xy 145.034 101.346) (xy 146.05 100.33) (xy 153.924 100.33) (xy 155.448 101.854) (xy 155.448 117.094)
-				(xy 156.464 118.11) (xy 166.624 118.11) (xy 167.132 117.348) (xy 167.132 100.33) (xy 166.37 99.568)
-				(xy 155.956 99.568) (xy 153.924 97.536) (xy 144.018 97.536) (xy 141.478 94.996) (xy 134.874 94.996)
-				(xy 131.826 91.948) (xy 123.19 91.948) (xy 121.412 93.472) (xy 121.412 94.742) (xy 121.412 99.568)
-				(xy 120.142 100.838) (xy 120.142 107.95) (xy 120.142 108.966) (xy 119.126 109.982) (xy 117.602 109.982)
-				(xy 116.586 108.966) (xy 116.586 96.52) (xy 115.824 95.504) (xy 111.98225 95.504) (xy 111.506 96.139)
-				(xy 111.506 104.938286) (xy 103.886 112.014) (xy 93.472 112.014) (xy 90.678 109.22) (xy 90.678 105.41)
-				(xy 92.964 103.124) (xy 92.964 83.82) (xy 90.932 81.788) (xy 90.932 73.66) (xy 91.694 72.898) (xy 93.726 72.898)
-				(xy 96.012 75.184) (xy 103.886 75.184) (xy 105.664 73.406) (xy 108.712 73.406) (xy 111.252 75.946)
-				(xy 111.252 81.28) (xy 112.776 82.804) (xy 123.19 82.804) (xy 123.952 81.8896) (xy 123.952 65.278)
-				(xy 125.476 64.008) (xy 133.096 64.008) (xy 135.128 65.701334) (xy 135.128 81.8896) (xy 135.89 82.804)
-				(xy 138.176 82.804) (xy 139.192 81.788) (xy 139.192 69.088) (xy 139.192 61.214) (xy 140.97 59.436)
-				(xy 144.526 59.436) (xy 145.288 60.198) (xy 145.288 61.722) (xy 145.796 62.23) (xy 148.59 62.23)
-				(xy 149.352 62.992) (xy 149.352 64.516) (xy 148.336 65.532) (xy 146.05 65.532) (xy 145.288 66.294)
-				(xy 145.288 86.614) (xy 146.304 87.63) (xy 149.098 87.63) (xy 149.86 86.868) (xy 149.86 73.66) (xy 149.098 72.898)
-				(xy 149.098 71.12) (xy 149.86 70.358) (xy 153.162 70.358) (xy 154.178 71.374) (xy 154.178 74.168)
-				(xy 155.702 75.692) (xy 155.702 83.312) (xy 159.648066 87.122) (xy 163.322 87.122) (xy 171.45 95.25)
-				(xy 171.45 99.06) (xy 172.72 100.33) (xy 176.784 100.33) (xy 177.8 99.314) (xy 177.8 88.392) (xy 175.514 86.106)
+				(xy 114.3 119.634) (xy 121.92 119.634) (xy 123.825 118.364) (xy 123.825 100.33) (xy 123.825 96.729177)
+				(xy 125.73 94.488) (xy 130.33375 94.488) (xy 132.715 96.393) (xy 132.715 111.76) (xy 135.382 114.3)
+				(xy 135.382 120.523) (xy 135.763 120.904) (xy 138.43 120.904) (xy 138.938 120.396) (xy 138.938 117.348)
+				(xy 140.462 115.824) (xy 144.526 115.824) (xy 145.542 116.84) (xy 145.542 117.729) (xy 146.177 118.364)
+				(xy 148.717 118.364) (xy 149.225 117.856) (xy 149.225 113.157) (xy 148.844 112.776) (xy 144.78 112.776)
+				(xy 143.764 111.76) (xy 143.764 108.966) (xy 144.78 107.95) (xy 148.844 107.95) (xy 149.352 107.569)
+				(xy 149.352 105.791) (xy 148.717 105.156) (xy 146.812 105.156) (xy 145.034 103.378) (xy 145.034 101.346)
+				(xy 146.05 100.33) (xy 153.924 100.33) (xy 155.448 101.854) (xy 155.448 117.094) (xy 156.464 118.11)
+				(xy 166.624 118.11) (xy 167.132 117.348) (xy 167.132 100.33) (xy 166.37 99.568) (xy 155.956 99.568)
+				(xy 153.924 97.536) (xy 144.018 97.536) (xy 141.478 94.996) (xy 134.874 94.996) (xy 130.81 91.948)
+				(xy 123.19 91.948) (xy 121.412 93.472) (xy 121.412 94.742) (xy 121.412 99.568) (xy 120.142 100.838)
+				(xy 120.142 107.95) (xy 120.142 108.966) (xy 119.126 109.982) (xy 117.602 109.982) (xy 116.586 108.966)
+				(xy 116.586 96.52) (xy 115.824 95.504) (xy 111.98225 95.504) (xy 111.506 96.139) (xy 111.506 104.938286)
+				(xy 103.886 112.014) (xy 93.472 112.014) (xy 90.678 109.22) (xy 90.678 105.41) (xy 92.964 103.124)
+				(xy 92.964 83.82) (xy 90.932 81.788) (xy 90.932 74.93) (xy 91.694 74.168) (xy 93.726 74.168) (xy 94.742 75.184)
+				(xy 103.886 75.184) (xy 105.664 73.406) (xy 108.712 73.406) (xy 111.252 75.946) (xy 111.252 81.28)
+				(xy 112.776 82.804) (xy 123.19 82.804) (xy 123.952 81.8896) (xy 123.952 65.278) (xy 125.476 64.008)
+				(xy 133.096 64.008) (xy 135.128 65.701334) (xy 135.128 81.8896) (xy 135.89 82.804) (xy 138.176 82.804)
+				(xy 139.192 81.788) (xy 139.192 69.088) (xy 139.192 61.214) (xy 140.97 59.436) (xy 144.526 59.436)
+				(xy 145.288 60.198) (xy 145.288 61.722) (xy 145.796 62.23) (xy 148.59 62.23) (xy 149.352 62.992)
+				(xy 149.352 64.516) (xy 148.336 65.532) (xy 146.05 65.532) (xy 145.288 66.294) (xy 145.288 86.614)
+				(xy 146.304 87.63) (xy 149.098 87.63) (xy 149.86 86.868) (xy 149.86 73.66) (xy 149.098 72.898) (xy 149.098 71.12)
+				(xy 149.86 70.358) (xy 153.162 70.358) (xy 154.178 71.374) (xy 154.178 74.168) (xy 155.702 75.692)
+				(xy 155.702 83.312) (xy 159.648066 87.122) (xy 163.322 87.122) (xy 171.45 95.25) (xy 171.45 99.06)
+				(xy 172.72 100.33) (xy 177.419 100.33) (xy 178.435 99.314) (xy 178.435 87.757) (xy 176.784 86.106)
 				(xy 166.37 86.106) (xy 159.512 79.248) (xy 159.512 61.722) (xy 154.432 56.642) (xy 135.636 56.642)
 				(xy 133.604 59.436) (xy 121.92 59.436) (xy 114.723331 59.436) (xy 112.268 61.540572) (xy 112.268 69.596)
@@
 			(pts
 				(xy 135.89 90.17) (xy 135.255 89.535) (xy 135.255 88.392) (xy 135.763 87.884) (xy 135.255 87.376)
-				(xy 135.255 85.725) (xy 126.746 85.725) (xy 125.095 87.376) (xy 103.759 87.376) (xy 102.616 86.233)
-				(xy 92.837 86.233) (xy 92.202 86.233) (xy 92.202 95.758) (xy 92.202 95.504) (xy 99.314 95.504) (xy 100.457 94.361)
-				(xy 100.457 93.472) (xy 99.441 92.456) (xy 99.441 89.662) (xy 100.33 88.773) (xy 104.775 88.773)
-				(xy 105.537 88.011) (xy 131.445 88.011) (xy 134.747 91.313) (xy 135.255 91.313) (xy 135.382 91.186)
+				(xy 135.255 85.725) (xy 126.746 85.725) (xy 92.202 85.725) (xy 92.202 95.504) (xy 99.314 95.504)
+				(xy 100.457 94.361) (xy 100.457 93.472) (xy 99.441 92.456) (xy 99.441 89.662) (xy 100.33 88.773)
+				(xy 104.775 88.773) (xy 131.445 88.9) (xy 134.747 91.313) (xy 135.255 91.313) (xy 135.382 91.186)
 				(xy 135.382 90.678)
 			)

Commit message: PCB Update
Routing:
- net -15V: track 25.7 -> 54.5 mm
- net +15V: track 25.4 -> 54.2 mm
- net Net-(J5-Pin_2): track 66.2 -> 64.9 mm
- net Net-(SW2-B): track 47.9 -> 46.7 mm
