File: KiCad/Input.kicad_pcb (KiCad board)
At the start: 4 copper layers, 150 x 85.2 mm, 177 parts, among them J1 R_Phono_In, J12 EMK_In, J15 Mic_Effekt_Out, J16 Mic_Effekt_Out, J17 Mic_Effekt_Out, J18 Mic_Effekt_Out, J19 Phono/Line_Out, J2 L_Phono_In, J20 Mic_Effekt_Out, J3 R_Line_In, J4 L_Line_In, J5 Mic_In, J6 Effekt_In, J7 AUX_RET_1, J8 AUX_RET_2, J9 AUX_RET_3, SW2 SW_SPDT, U1 TL074, U2 TL074, U25 INA128U, U3 TL074, U4 TL074, U5 TL074

Commit message: PCB Update
Parts:
- added C112: 100n, Capacitor_SMD:C_0805_2012Metric_Pad1.18x1.45mm_HandSolder, B.Cu at (71.1, 83.8)
- added C113: 100n, Capacitor_SMD:C_0805_2012Metric_Pad1.18x1.45mm_HandSolder, B.Cu at (101.0, 74.7)
- added C114: 100n, Capacitor_SMD:C_0805_2012Metric_Pad1.18x1.45mm_HandSolder, B.Cu at (111.8, 87.6)
- added C115: 100n, Capacitor_SMD:C_0805_2012Metric_Pad1.18x1.45mm_HandSolder, B.Cu at (100.3, 119.4)
Connections:
- J12 pad 1: +9V -> 9V_GND
- J12 pad 2: 9V_GND -> +9V
- J12 pad 3: +15V -> -15V
- J12 pad 4: -15V -> GND
- J12 pad 5: GND -> +15V
Routing:
- net Net-(J20-Pin_1): track 56.5 -> 76.9 mm
- net -15V: track 54.5 -> 40.9 mm
- net +15V: track 54.2 -> 40.7 mm
- net Net-(R1-Pad2): track 62.4 -> 75.5 mm
- net GND: track 157.6 -> 168.5 mm, vias 74 -> 69
- net Net-(U3C-+): track 47.4 -> 49.6 mm
- net Net-(U2C--): track 81.2 -> 83.3 mm
- net Net-(J5-Pin_3): track 70.1 -> 71.6 mm
- net Net-(SW2-B): track 46.7 -> 48.2 mm
- net Net-(R28-Pad1): track 89.9 -> 91.4 mm
- net Net-(J5-Pin_2): track 64.9 -> 66.2 mm
- net Net-(J9-Pin_1): track 18.0 -> 19.0 mm
- net Net-(U3D--): track 27.5 -> 28.3 mm
- net Net-(U5C-+): track 18.9 -> 19.6 mm
- net Net-(U2D--): track 36.6 -> 37.3 mm
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- added copper zone on In1.Cu, net GND
- removed copper zone on B.Cu, net (none)
- removed copper zone on F.Cu, net (none)
- removed copper zone on In1.Cu, net (none)
- removed copper zone on In2.Cu, net (none)
- removed copper zone on B.Cu, net GND

Commit message: PCB Update
Routing:
- net Net-(J6-Pin_1): track 29.4 -> 37.7 mm
- net GND: track 168.5 -> 175.2 mm, vias 69 -> 67
- net Net-(J16-Pin_1): track 10.6 -> 4.87 mm
- net Net-(U4C-+): track 36.2 -> 40.2 mm
- net Net-(U4A-+): track 104.6 -> 106.2 mm
- added copper zone on F.Cu, net Net-(J16-Pin_1)

Commit message: PCB Update
Parts:
- added C116: 10n, Capacitor_SMD:C_1210_3225Metric_Pad1.33x2.70mm_HandSolder, F.Cu at (185.4, 64.5)
- added H13: MountingHole, MountingHole:MountingHole_3.2mm_M3_Pad, F.Cu at (50.8, 53.3)
- added H14: MountingHole, MountingHole:MountingHole_3.2mm_M3_Pad, F.Cu at (50.8, 124.5)
- added H15: MountingHole_Pad, MountingHole:MountingHole_3.2mm_M3_Pad, F.Cu at (185.4, 53.3)
- added H16: MountingHole, MountingHole:MountingHole_3.2mm_M3_Pad, F.Cu at (185.4, 124.5)
- moved J12 15.2 mm to (175.3, 106.7)
Connections:
- net +15V renamed +15V_I
- net +9V renamed +9V_I
- net -15V renamed -15V_I
- net 9V_GND renamed 9V_GND_I
- net GND renamed GND_I
Routing:
- net -15V_I: track 40.9 -> 57.6 mm
- net +15V_I: track 40.7 -> 49.7 mm
- net Net-(J5-Pin_3): track 71.6 -> 64.9 mm
- net GND_I: track 175.2 -> 172.7 mm, vias 67 -> 69
- net Net-(R30-Pad2): track 45.6 -> 47.5 mm
- net Net-(R28-Pad1): track 91.4 -> 92.9 mm
- net Net-(J17-Pin_1): track 17.8 -> 19.3 mm
- net Net-(SW2-B): track 48.2 -> 48.9 mm
- net Net-(J5-Pin_2): track 66.2 -> 67.0 mm
- net Net-(U3C-+): track 49.6 -> 50.4 mm
- net Net-(R15-Pad1): track 61.3 -> 62.1 mm
- net Net-(U2C--): track 83.3 -> 83.8 mm
- added copper zone on F.Cu, net GND_I
- added copper zone on F.Cu, net Net-(C116-Pad1)
- added copper zone on B.Cu, net Net-(J17-Pin_1)
- added copper zone on B.Cu, net Net-(R15-Pad1)
- added copper zone on B.Cu, net Net-(R28-Pad1)
- added copper zone on B.Cu, net Net-(SW2-B)
- added copper zone on B.Cu, net Net-(U2C--)
- added copper zone on B.Cu, net Net-(U3C-+)

Commit message: PCB Update
Parts:
- removed C112, C113, C114, C115: 100n, Capacitor_SMD:C_0805_2012Metric_Pad1.18x1.45mm_HandSolder
- added C124: 100n, Capacitor_SMD:C_0805_2012Metric_Pad1.18x1.45mm_HandSolder, F.Cu at (256.0, 105.0)
- added C125: 100n, Capacitor_SMD:C_0805_2012Metric_Pad1.18x1.45mm_HandSolder, F.Cu at (256.0, 108.0)
- added R150: 10k, Resistor_SMD:R_0805_2012Metric_Pad1.20x1.40mm_HandSolder, B.Cu at (71.1, 67.3)
- added R151: 10k, Resistor_SMD:R_0805_2012Metric_Pad1.20x1.40mm_HandSolder, B.Cu at (71.1, 59.7)
- added R152: 10k, Resistor_SMD:R_0805_2012Metric_Pad1.20x1.40mm_HandSolder, B.Cu at (78.7, 64.8)
- added R153: 10k, Resistor_SMD:R_0805_2012Metric_Pad1.20x1.40mm_HandSolder, B.Cu at (71.1, 69.8)
- added R154: 10k, Resistor_SMD:R_0805_2012Metric_Pad1.20x1.40mm_HandSolder, B.Cu at (78.7, 67.3)
- added U26: TL074, Package_DIP:DIP-14_W7.62mm_Socket_LongPads, F.Cu at (250.8, 77.2)
- C1, C13, C14, C15, C16, C17, C21, C22, C27, C28, C29, C3, C30, C31, C32, C33, C34, C7, C8, R1, R10, R11, R12, R13, R14, R15, R16, R17, R18, R19, R20, R21, R22, R23, R24, R3, R30, R4, R5, R6, R7, R8, R9, Z1, Z10, Z11, Z12, Z13, Z14, Z15, Z16, Z17, Z18, Z19, Z2, Z20, Z21, Z22, Z23, Z24, Z25, Z26, Z27, Z28, Z29, Z3, Z30, Z31, Z32, Z33, Z34, Z35, Z36, Z37, Z38, Z39, Z4, Z40, Z41, Z42, Z43, Z44, Z45, Z46, Z47, Z48, Z49, Z5, Z50, Z51, Z52, Z53, Z55, Z56, Z57, Z58, Z59, Z6, Z60, Z61, Z62, Z63, Z64, Z65, Z66, Z67, Z68, Z69, Z7, Z70, Z72, Z74, Z75, Z77, Z78, Z79, Z8, Z9: moved to B.Cu
- R2: value 100R -> 10k; moved to B.Cu
- RV3: footprint Connector_PinSocket_2.54mm_LongPads:PinSocket_1x06_P2.54mm_Vertical_LongPads -> Connector_PinSocket_2.54mm_LongPads:PinSocket_2x03_P2.54mm_Vertical_LongPads
- RV5: footprint Connector_PinSocket_2.54mm_LongPads:PinSocket_1x06_P2.54mm_Vertical_LongPads -> Connector_PinSocket_2.54mm_LongPads:PinSocket_2x03_P2.54mm_Vertical_LongPads_Mirrored
- U25: value INA128U -> TL074; footprint INA128U:INA128U_L -> Package_DIP:DIP-14_W7.62mm_Socket_LongPads
- moved RV6 161.9 mm to (227.3, 101.0)
- moved H14 152.3 mm to (185.4, 53.3)
- moved Z90 139.0 mm to (241.6, 91.3)
- moved Z85 137.7 mm to (241.6, 76.5), turned to 0 degrees
- moved H16 134.6 mm to (50.8, 121.9)
- moved Z80 134.1 mm to (236.9, 85.4), turned to 0 degrees
- moved R31 131.4 mm to (232.1, 79.5)
- moved Z71 127.9 mm to (236.9, 76.5)
- moved R29 127.9 mm to (232.1, 76.5)
- moved Z76 127.7 mm to (236.9, 82.4), turned to 0 degrees
- moved Z73 127.7 mm to (236.9, 79.5), turned to 0 degrees
- moved R32 127.6 mm to (232.1, 82.4)
- moved R28 119.4 mm to (227.4, 97.2)
- moved Z94 109.0 mm to (246.4, 79.5)
- moved J19 107.8 mm to (245.7, 70.2)
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Connections:
- C1 pad 2: Net-(U3C--) -> Net-(U3B--)
- C3 pad 1: Net-(U4C-+) -> Net-(U3C-+)
- C7 pad 1: GND_I -> +15V_I
- C7 pad 2: +15V_I -> GND_I
- J5 pad 1: GND_I -> Net-(J5-Pin_1)
- J5 pad 2: Net-(J5-Pin_2) -> GND_I
- R10 pad 1: Net-(U5B--) -> Net-(U5C--)
- R11 pad 1: Net-(U5B--) -> Net-(U5C--)
- R12 pad 1: Net-(U4C--) -> Net-(U3C--)
- R14 pad 1: Net-(U2D--) -> Net-(U2C--)
- R15 pad 2: Net-(U5B--) -> Net-(U5C--)
- R16 pad 2: Net-(U4B--) -> Net-(U4D--)
- R17 pad 2: Net-(U4B--) -> Net-(U4D--)
- R19 pad 1: Net-(U4B--) -> Net-(U4D--)
- R2 pad 1: Net-(R2-Pad1) -> Net-(R151-Pad1)
- R2 pad 2: Net-(R2-Pad2) -> Net-(U25A--)
- R28 pad 2: Net-(U3B--) -> Net-(U26D-+)
- R29 pad 1: Net-(U2C--) -> Net-(U26A--)
- R29 pad 2: Net-(U3B-+) -> Net-(U26D--)
- R3 pad 2: Net-(U4C--) -> Net-(U3C--)
- R31 pad 2: Net-(U3B-+) -> Net-(U26D--)
- R32 pad 1: Net-(U3B--) -> Net-(U26D-+)
- R7 pad 2: Net-(U2D--) -> Net-(U2C--)
- R8 pad 2: Net-(U2D--) -> Net-(U2C--)
- R9 pad 1: Net-(U5B--) -> Net-(U5C--)
- RV1 pad 2: Net-(U3C-+) -> Net-(U3B-+)
- RV2 pad 1: Net-(RV2-Pad1) -> Net-(U25A--)
- RV2 pad 2: Net-(R2-Pad1) -> Net-(U25B--)
- RV2 pad 3: Net-(R2-Pad1) -> Net-(U25B--)
- RV3 pad 1: Net-(U4C-+) -> Net-(U3C-+)
- RV3 pad 2: Net-(U4C-+) -> Net-(U3C-+)
- RV3 pad 5: Net-(U4C-+) -> Net-(U3C-+)
- RV3 pad 6: Net-(U4C-+) -> Net-(U3C-+)
- RV6 pad 2: Net-(U2C--) -> Net-(U26A--)
- RV6 pad 3: Net-(U2C--) -> Net-(U26A--)
- U2 pad 10: Net-(SW2-B) -> Net-(U2C-+)
- U2 pad 12: Net-(U2D-+) -> GND_I
- U2 pad 14: Net-(R14-Pad2) -> Net-(U2D--)
- U2 pad 8: Net-(R28-Pad1) -> Net-(R14-Pad2)
- U25 pad 1: Net-(RV2-Pad1) -> Net-(R151-Pad1)
- U25 pad 2: Net-(U25-IN-) -> Net-(U25A--)
- U25 pad 3: Net-(U25-IN+) -> Net-(U25A-+)
- U25 pad 4: -15V_I -> +15V_I
- U25 pad 5: GND_I -> Net-(U25B-+)
- U25 pad 6: Net-(U25-Pad6) -> Net-(U25B--)
- U25 pad 7: +15V_I -> Net-(R150-Pad2)
- U25 pad 8: Net-(R2-Pad2) -> Net-(R154-Pad1)
- U3 pad 7: Net-(R32-Pad2) -> Net-(U3B--)
- U3 pad 8: Net-(U3C--) -> Net-(R12-Pad2)
- U4 pad 10: Net-(U4C-+) -> GND_I
- U4 pad 14: Net-(U4D--) -> Net-(R19-Pad2)
- U4 pad 7: Net-(R19-Pad2) -> Net-(U4B--)
- U4 pad 8: Net-(R12-Pad2) -> Net-(U4C--)
- U5 pad 12: Net-(U5D-+) -> GND_I
- U5 pad 7: Net-(R15-Pad1) -> Net-(U5B--)
- U5 pad 8: Net-(U5C--) -> Net-(R15-Pad1)
- Z10 pad 1: Net-(J5-Pin_2) -> Net-(J5-Pin_3)
- Z11 pad 2: Net-(U4D-+) -> Net-(U4A-+)
- Z12 pad 2: Net-(U5A-+) -> Net-(U4B-+)
- Z13 pad 2: Net-(U5D-+) -> Net-(U5A-+)
- Z14 pad 2: Net-(U5C-+) -> Net-(U5B-+)
- Z19 pad 1: Net-(J5-Pin_3) -> Net-(J5-Pin_1)
- Z19 pad 2: Net-(U25-IN-) -> Net-(U25A-+)
- Z20 pad 1: Net-(J5-Pin_2) -> Net-(J5-Pin_3)
- Z20 pad 2: Net-(U25-IN+) -> Net-(U25B-+)
- Z21 pad 1: Net-(U4D-+) -> Net-(U4A-+)
- Z22 pad 1: Net-(U5A-+) -> Net-(U4B-+)
- Z23 pad 1: Net-(U5D-+) -> Net-(U5A-+)
- Z24 pad 1: Net-(U5C-+) -> Net-(U5B-+)
- Z29 pad 1: Net-(U25-IN-) -> Net-(U25A-+)
- Z30 pad 1: Net-(U25-IN+) -> Net-(U25B-+)
- Z31 pad 1: Net-(U5A--) -> Net-(U4A--)
- Z32 pad 1: Net-(U5D--) -> Net-(U5A--)
- Z33 pad 1: Net-(U5C--) -> Net-(U5B--)
- Z53 pad 1: Net-(U2D-+) -> Net-(U2C-+)
- Z54 pad 1: Net-(U5B-+) -> Net-(U5C-+)
- Z55 pad 1: Net-(U25-Pad6) -> Net-(R154-Pad1)
- Z59 pad 2: Net-(R23-Pad1) -> Net-(R3-Pad1)
- Z61 pad 2: Net-(R16-Pad1) -> Net-(R23-Pad1)
- Z65 pad 2: Net-(U4D--) -> Net-(U4B--)
- Z70 pad 1: Net-(U4B-+) -> Net-(U4D-+)
- Z76 pad 2: Net-(U4A-+) -> Net-(U26B-+)
- Z77 pad 1: Net-(Z77-Pad1) -> GND_I
- Z77 pad 2: GND_I -> Net-(Z77-Pad2)
- Z78 pad 2: Net-(Z77-Pad1) -> Net-(Z77-Pad2)
- Z79 pad 1: Net-(Z77-Pad1) -> Net-(Z77-Pad2)
- Z79 pad 2: Net-(R3-Pad1) -> Net-(R16-Pad1)
- Z80 pad 1: Net-(U4A--) -> Net-(U26B--)
- Z81 pad 1: Net-(U4A-+) -> Net-(U26B-+)
- Z82 pad 1: Net-(U4A-+) -> Net-(U26B-+)
- Z85 pad 1: Net-(U4A--) -> Net-(U26B--)
- Z86 pad 1: Net-(U4A-+) -> Net-(U26B-+)
- Z87 pad 1: Net-(U4A-+) -> Net-(U26B-+)
- Z9 pad 1: Net-(J5-Pin_3) -> Net-(J5-Pin_1)
Routing:
- net GND_I: track 172.7 -> 63.0 mm, vias 69 -> 3
- net Net-(U4A-+): track 106.2 -> 5.35 mm
- net Net-(R28-Pad1): track 92.9 -> 0.00 mm
- net Net-(J20-Pin_1): track 76.9 -> 0.00 mm, vias 1 -> 0
- net Net-(U2C--): track 83.8 -> 13.2 mm
- net Net-(J5-Pin_2): track 67.0 -> 0.00 mm, vias 1 -> 0
- net Net-(R1-Pad2): track 75.5 -> 10.6 mm, vias 1 -> 0
- net Net-(R15-Pad1): track 62.1 -> 2.81 mm, vias 1 -> 0
- net Net-(J5-Pin_3): track 64.9 -> 7.77 mm, vias 1 -> 0
- net Net-(SW2-B): track 48.9 -> 0.00 mm
- net Net-(R23-Pad1): track 8.16 -> 57.0 mm, vias 0 -> 1
- net Net-(U3C-+): track 50.4 -> 2.77 mm
- net -15V_I: track 57.6 -> 16.6 mm, vias 3 -> 0
- net Net-(U4C-+): track 40.2 -> 0.00 mm
- net Net-(U25B--): track 0.00 -> 37.2 mm
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- added copper zone on F.Cu, net Net-(R12-Pad2)
- added copper zone on F.Cu, net Net-(R30-Pad2)
- added copper zone on F.Cu, net Net-(U3C-+)
- added copper zone on F.Cu, net Net-(U3D-+)
- removed copper zone on In2.Cu, net +15V_I
- removed copper zone on In2.Cu, net -15V_I
- removed copper zone on F.Cu, net GND_I
- removed copper zone on In1.Cu, net GND_I
- removed copper zone on F.Cu, net Net-(C116-Pad1)
- removed copper zone on F.Cu, net Net-(J16-Pin_1)
- removed copper zone on B.Cu, net Net-(J17-Pin_1)
- removed copper zone on B.Cu, net Net-(R15-Pad1)
- removed copper zone on B.Cu, net Net-(R28-Pad1)
- removed copper zone on B.Cu, net Net-(SW2-B)
- removed copper zone on B.Cu, net Net-(U2C--)
- removed copper zone on B.Cu, net Net-(U3C-+)
Other:
- board text added: "."
- board text added: "16 25 34"
- board text added: "34 25 16"
- board text removed: "DiKo-Elektrotechnik Eingangsstufe"

Commit message: PCB Update
Parts:
- C124, C125, R28, R29, R31, R32, Z100, Z54, Z71, Z73, Z76, Z80, Z81, Z82, Z83, Z84, Z85, Z86, Z87, Z88, Z89, Z90, Z91, Z92, Z93, Z94, Z95, Z96, Z97, Z98, Z99: moved to B.Cu
- moved C124 122.8 mm to (133.3, 111.8)
- moved U26 116.8 mm to (137.2, 104.1)
- moved Z54 113.9 mm to (121.9, 114.3)
- moved Z73 110.7 mm to (129.5, 106.7), turned to 180 degrees
- moved Z71 107.8 mm to (133.3, 106.7), turned to 180 degrees
- moved C125 107.4 mm to (148.6, 111.8), turned to 180 degrees
- moved Z76 106.9 mm to (133.3, 109.2)
- moved R29 99.7 mm to (141.0, 116.8)
- moved Z94 97.6 mm to (156.2, 116.8), turned to 180 degrees
- moved J19 96.4 mm to (160.0, 114.3)
- moved RV6 95.8 mm to (133.3, 119.4), turned to 180 degrees
- moved Z93 94.7 mm to (156.2, 105.4), turned to 180 degrees
- moved Z92 94.6 mm to (156.2, 56.5), turned to 180 degrees
- moved Z99 93.6 mm to (156.2, 119.4), turned to 180 degrees
- moved Z95 93.1 mm to (156.2, 59.1), turned to 180 degrees
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Connections:
- R28 pad 2: Net-(U26D-+) -> Net-(U26C--)
- R29 pad 1: Net-(U26A--) -> Net-(U26B--)
- R29 pad 2: Net-(U26D--) -> Net-(U26C-+)
- R31 pad 2: Net-(U26D--) -> Net-(U26C-+)
- R32 pad 1: Net-(U26D-+) -> Net-(U26C--)
- RV6 pad 2: Net-(U26A--) -> Net-(U26B--)
- RV6 pad 3: Net-(U26A--) -> Net-(U26B--)
- U26 pad 1: Net-(R28-Pad1) -> Net-(U26A--)
- U26 pad 10: unconnected-(U26C-+-Pad10) -> Net-(U26C-+)
- U26 pad 12: Net-(U26D-+) -> GND_I
- U26 pad 14: Net-(R32-Pad2) -> Net-(U26D--)
- U26 pad 3: Net-(SW2-B) -> Net-(U26A-+)
- U26 pad 5: Net-(U26B-+) -> Net-(SW2-B)
- U26 pad 7: Net-(U26B--) -> Net-(R28-Pad1)
- U26 pad 8: unconnected-(U26-Pad8) -> Net-(R32-Pad2)
- U26 pad 9: unconnected-(U26C---Pad9) -> Net-(U26C--)
- U4 pad 10: GND_I -> Net-(U26A-+)
- U5 pad 12: GND_I -> Net-(U26A-+)
- Z76 pad 2: Net-(U26B-+) -> Net-(U26A-+)
- Z80 pad 1: Net-(U26B--) -> Net-(U26A--)
- Z81 pad 1: Net-(U26B-+) -> Net-(U5D--)
- Z82 pad 1: Net-(U26B-+) -> Net-(U4C--)
- Z85 pad 1: Net-(U26B--) -> Net-(U26A--)
- Z86 pad 1: Net-(U26B-+) -> Net-(U5D--)
- Z87 pad 1: Net-(U26B-+) -> Net-(U4C--)
Routing:
- net GND_I: track 63.0 -> 246.5 mm, vias 3 -> 34
- net Net-(SW2-B): track 0.00 -> 129.5 mm
- net Net-(U5D--): track 2.54 -> 76.8 mm, vias 0 -> 1
- net Net-(U4C--): track 2.54 -> 75.8 mm, vias 0 -> 1
- net Net-(R15-Pad1): track 2.81 -> 66.7 mm, vias 0 -> 1
- net Net-(U26A--): track 0.00 -> 51.8 mm
- net Net-(R19-Pad2): track 2.81 -> 52.5 mm
- net Net-(U26A-+): track 0.00 -> 47.0 mm
- net +15V_I: track 13.9 -> 41.0 mm
- net -15V_I: track 16.6 -> 39.7 mm
- net Net-(R32-Pad2): track 0.00 -> 21.1 mm
- net Net-(U26C--): track 0.00 -> 10.6 mm
- net Net-(U26B--): track 0.00 -> 9.16 mm
- net Net-(U1C-+): track 8.63 -> 15.4 mm, vias 0 -> 1
- net Net-(U26C-+): track 0.00 -> 6.67 mm
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- added copper zone on In2.Cu, net +15V_I
- added copper zone on In2.Cu, net -15V_I
- added copper zone on In1.Cu, net GND_I
Other:
- board size 150 x 85.2 mm -> 150 x 92.8 mm

Commit message: PCB Update
Parts:
- moved C116 65.9 mm to (170.2, 121.9), turned to 180 degrees
- turned Z83 to 180 degrees
Routing:
- net GND_I: track 246.5 -> 309.0 mm, vias 34 -> 37
- net Net-(J17-Pin_1): track 6.62 -> 20.4 mm
- net Net-(U25B--): track 37.6 -> 44.1 mm
- net Net-(C116-Pad1): track 0.00 -> 5.89 mm
- net Net-(R16-Pad1): track 38.4 -> 41.3 mm
- net Net-(R4-Pad2): track 0.00 -> 2.81 mm
- net Net-(R11-Pad2): track 0.00 -> 2.81 mm
- net Net-(U26D--): track 0.27 -> 2.81 mm
- net Net-(R10-Pad2): track 0.00 -> 2.54 mm
- net Net-(R15-Pad1): track 66.7 -> 67.9 mm
- net Net-(SW2-B): track 129.5 -> 130.6 mm
- added copper zone on B.Cu, net GND_I
- added copper zone on F.Cu, net GND_I
- added copper zone on F.Cu, net Net-(C116-Pad1)

Commit message: PCB Final Update
Parts:
- J12: value EMK_In -> Conn_02x07_Odd_Even; footprint Connector_PinHeader_2.54mm_LongPads:PinHeader_1x05_P2.54mm_Vertical_LongPads -> Connector_PinHeader_2.54mm:PinHeader_2x07_P2.54mm_Vertical
- moved J12 5.08 mm to (170.2, 101.6)
- moved C116 1.27 mm to (171.4, 121.9)
Connections:
- J12 pad 2: +9V_I -> 9V_GND_I
- J12 pad 3: -15V_I -> 9V_GND_I
- J12 pad 4: GND_I -> 9V_GND_I
- J12 pad 5: +15V_I -> +9V_I
Routing:
- net GND_I: track 309.0 -> 321.1 mm
- net +15V_I: track 41.0 -> 44.8 mm
- net -15V_I: track 39.7 -> 42.9 mm
- net +9V_I: track 0.00 -> 2.54 mm
- added copper zone on F.Cu, net 9V_GND_I

Commit message: final PCB Update
Parts:
- renumbered C21 to C1, C27 to C2, C116 to C3, C3 to C33, C1 to C37, C30 to C48, C22 to C49, C7 to C52, C124 to C53, C13 to C54, C16 to C55, C31 to C56, C33 to C57, C28 to C58, C8 to C59, C125 to C60, C14 to C61, C17 to C62, C32 to C63, C34 to C64, C29 to C65, C15 to C9, H16 to H1, H15 to H3, H14 to H6, H13 to H7, J20 to J12, J16 to J14, J15 to J16, J7 to J17, J1 to J2, J6 to J20, J8 to J22, J17 to J23, J18 to J27, J9 to J28, J2 to J3, J12 to J30, J19 to J4, J3 to J7, J4 to J8, J5 to J9, R23 to R101, R16 to R102, R19 to R103, R17 to R104, R21 to R105, R24 to R106, R9 to R126, R10 to R134, R15 to R135, R11 to R140, R18 to R15, R6 to R16, R28 to R24, R32 to R25, R20 to R3, R14 to R30, R29 to R32, R7 to R33, R31 to R36, R22 to R4, R8 to R45, R153 to R52, R154 to R53, R150 to R57, R12 to R58, R3 to R65, R2 to R67, R13 to R7, R151 to R75, R1 to R76, R4 to R77, R152 to R80, R5 to R9, R30 to R93, RV3 to RV11, RV1 to RV13, RV5 to RV17, RV4 to RV18, RV6 to RV4, RV2 to RV9, U25 to U11, U3 to U15, U4 to U17, U5 to U19, U1 to U4, U26 to U8, U2 to U9, Z68 to Z10, Z58 to Z100, Z19 to Z109, Z5 to Z11, Z9 to Z112, Z29 to Z113, Z25 to Z12, Z78 to Z134, Z79 to Z135, Z71 to Z136, Z76 to Z137, Z41 to Z14, Z85 to Z140, Z73 to Z142, Z77 to Z143, Z80 to Z144, Z90 to Z145, Z100 to Z146, Z74 to Z15, Z64 to Z150, Z70 to Z151, Z86 to Z152, Z60 to Z154, Z65 to Z155, Z81 to Z156, Z91 to Z157, Z96 to Z158, Z66 to Z16, Z87 to Z175, Z12 to Z176, Z82 to Z177, Z92 to Z178, Z95 to Z179, Z2 to Z180, Z22 to Z181, Z11 to Z189, Z52 to Z19, Z31 to Z190, Z45 to Z191, Z1 to Z192, Z21 to Z193, Z38 to Z194, Z15 to Z2, Z13 to Z201, Z32 to Z202, Z46 to Z203, Z88 to Z204, Z3 to Z206, Z23 to Z207, Z72 to Z21, Z39 to Z210, Z83 to Z211, Z93 to Z212, Z97 to Z213, Z75 to Z22, Z54 to Z224, Z14 to Z225, Z33 to Z226, Z47 to Z227, Z98 to Z228, Z4 to Z229, Z16 to Z23, Z24 to Z230, Z40 to Z232, Z35 to Z26, Z49 to Z27, Z6 to Z32, Z26 to Z33, Z42 to Z35, Z89 to Z38, Z84 to Z40, Z94 to Z41, Z99 to Z42, Z17 to Z49, Z34 to Z5, Z36 to Z50, Z50 to Z51, Z63 to Z54, Z69 to Z55, Z7 to Z57, Z27 to Z58, Z43 to Z59, Z48 to Z6, Z67 to Z62, Z53 to Z63, Z18 to Z67, Z37 to Z72, Z51 to Z73, Z8 to Z75, Z28 to Z76, Z44 to Z79, Z20 to Z80, Z10 to Z86, Z30 to Z87, Z62 to Z9, Z55 to Z94, Z59 to Z95, Z56 to Z97, Z61 to Z98, Z57 to Z99
Routing:
- net GND_I: track 321.1 -> 253.8 mm
- net +15V_I: track 44.8 -> 19.4 mm
- net -15V_I: track 42.9 -> 19.4 mm
