File: KiCad/Input.kicad_pcb (KiCad board)
At the start: 4 copper layers, 150 x 92.8 mm, 190 parts, among them J12 Mic_Effekt_Out, J14 Mic_Effekt_Out, J16 Mic_Effekt_Out, J17 AUX_RET_1, J2 R_Phono_In, J20 Effekt_In, J22 AUX_RET_2, J23 Mic_Effekt_Out, J27 Mic_Effekt_Out, J28 AUX_RET_3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

Commit message: DRC Update
Routing:
- net Net-(R102-Pad1): track 41.3 -> 38.1 mm

Commit message: Gerber Update
Routing:
- net GND_I: track 253.8 -> 242.8 mm, vias 37 -> 40
- net Net-(U11B--): track 44.1 -> 37.2 mm
- net Net-(C3-Pad1): track 5.89 -> 0.00 mm
- net Net-(R58-Pad2): track 13.5 -> 7.66 mm
- net Net-(U4C-+): track 15.1 -> 16.6 mm
- net Net-(U19C--): track 46.8 -> 45.5 mm

Commit message: Gerber Update
Parts:
- moved C1 0.64 mm to (91.4, 95.9)
- moved C3 0.64 mm to (171.4, 122.6)
- moved C33 0.64 mm to (129.5, 62.9)
- moved C37 0.64 mm to (110.3, 70.5)
- moved C9 0.64 mm to (91.4, 90.8)
- moved H1 0.64 mm to (50.8, 122.6)
- moved H3 0.64 mm to (185.4, 122.6)
- moved J12 0.64 mm to (160.0, 77.5)
- moved J14 0.64 mm to (160.0, 66.0)
- moved J17 0.64 mm to (102.9, 90.8)
- moved J27 0.64 mm to (160.0, 92.1)
- moved J3 0.64 mm to (72.4, 90.8)
- moved J30 0.64 mm to (170.2, 102.2)
- moved J4 0.64 mm to (160.0, 114.9)
- moved R102 0.64 mm to (125.7, 78.1)
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Other:
- board size 150 x 92.8 mm -> 150 x 95 mm
- board text added: "Eingangsstufe"
