File: KiCad/Power_Supply_Meter_Amp.kicad_pcb (KiCad board)
At the start: 4 copper layers, 150 x 85.2 mm, 83 parts, among them J10 VCC_IN, J11 VCC_OUT, J13 EMK_Out, J14 EMK_Out, J21 EMK_Out, J23 EMK_In, J30 Pegel_In, J31 Pegel_In, J32 Pegel_In, J33 Pegel_In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

Commit message: PCB Update
Parts:
- C4, C6: moved to B.Cu
- moved C10 127.0 mm to (127.0, 53.3)
- moved C12 116.6 mm to (127.0, 88.9)
- moved C9 115.2 mm to (127.0, 83.8)
- moved C11 113.3 mm to (127.0, 119.4)
- moved U7 92.5 mm to (127.0, 104.1)
- moved U6 92.5 mm to (127.0, 68.6)
- moved C6 22.0 mm to (123.0, 66.0)
- moved C4 20.5 mm to (123.0, 71.1), turned to 180 degrees
- moved C5 7.24 mm to (109.2, 68.6), turned to 90 degrees
- moved J10 1.27 mm to (53.3, 55.9)
- moved J11 1.27 mm to (53.3, 63.5)
- moved SW1 1.27 mm to (58.4, 55.9)
- moved C2 0.28 mm to (63.5, 60.0)
Routing:
- net Net-(U6-+VIN): track 0.00 -> 83.7 mm
- net Net-(U6--VIN): track 0.00 -> 83.7 mm

Commit message: PCB Update
Parts:
- removed J23: EMK_In, Connector_PinHeader_2.54mm_LongPads:PinHeader_1x05_P2.54mm_Vertical_LongPads
- added C112: 10n, Capacitor_SMD:C_0805_2012Metric_Pad1.18x1.45mm_HandSolder, B.Cu at (68.3, 61.0)
- added C113: 10n, Capacitor_SMD:C_0805_2012Metric_Pad1.18x1.45mm_HandSolder, B.Cu at (68.3, 66.0)
- C23, C24, C25, C26: moved to B.Cu
- J21: value EMK_Out -> Conn_01x05_bridged; footprint Connector_PinSocket_2.54mm_LongPads:PinSocket_1x05_P2.54mm_Vertical_LongPads -> Connector_Bridged_2.54mm_LongPads:Bridge_2x05_P2.54mm_Vertical_LongPads
- L1: value Choke_Wurth_WE-CNSW_744232090 -> ~; footprint Inductor_THT:L_CommonMode_Wuerth_WE-CMB-M -> WE-SL575:WE-SL575
- L2, L3, L4, L5: footprint Connector_PinSocket_2.54mm_LongPads:PinSocket_1x02_P2.54mm_Vertical_LongPads -> Inductor_SMD:L_1206_3216Metric
- moved C24 168.9 mm to (86.6, 58.4), turned to 180 degrees
- moved C23 164.8 mm to (86.6, 68.6)
- moved L5 164.6 mm to (89.9, 88.9)
- moved J21 163.9 mm to (106.7, 55.9)
- moved L3 162.9 mm to (89.9, 53.3)
- moved C26 160.8 mm to (86.6, 95.2), turned to 180 degrees
- moved C25 159.3 mm to (86.6, 102.9)
- moved L4 159.3 mm to (89.9, 109.2)
- moved C18 159.1 mm to (91.4, 63.5), turned to 90 degrees
- moved J14 157.0 mm to (106.7, 96.5)
- moved C20 154.4 mm to (91.4, 95.0), turned to 90 degrees
- moved L2 153.2 mm to (89.9, 73.7)
- moved J13 152.3 mm to (106.7, 76.2)
- moved C19 150.1 mm to (91.4, 103.1), turned to 90 degrees
- moved R26 144.8 mm to (96.2, 104.1), turned to 180 degrees
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Connections:
- C10 pad 2: 9V_GND -> 9V_GND_P
- C18 pad 2: 9V_GND -> 9V_GND_P
- C19 pad 2: GND -> GND_P
- C20 pad 1: GND -> GND_P
- C23 pad 1: FILT_GND -> GND_9V_FILT
- C24 pad 1: 9V_GND -> 9V_GND_P
- C24 pad 2: FILT_GND -> GND_9V_FILT
- C25 pad 1: FILT_GND -> GND_15V_FILT
- C26 pad 2: FILT_GND -> GND_15V_FILT
- C36 pad 2: GND -> GND_M
- C4 pad 1: FILT_GND -> GND_15V_FILT
- C46 pad 2: +15V -> +15V_M
- C47 pad 2: -15V -> -15V_M
- C56 pad 2: +15V -> +15V_M
- C57 pad 2: -15V -> -15V_M
- C6 pad 2: FILT_GND -> GND_15V_FILT
- D3 pad 2: GND -> GND_M
- J13 pad 1: +9V -> +9V_P
- J13 pad 2: 9V_GND -> 9V_GND_P
- J13 pad 3: +15V -> +15V_P
- J13 pad 4: -15V -> -15V_P
- J13 pad 5: GND -> GND_P
- J14 pad 1: +9V -> +9V_P
- J14 pad 2: 9V_GND -> 9V_GND_P
- J14 pad 3: +15V -> +15V_P
- J14 pad 4: -15V -> -15V_P
- J14 pad 5: GND -> GND_P
- J21 pad 1: +9V -> +9V_P
- J21 pad 2: 9V_GND -> 9V_GND_P
- J21 pad 3: +15V -> +15V_P
- J21 pad 4: -15V -> -15V_P
- J21 pad 5: GND -> GND_P
- J36 pad 2: GND -> GND_M
- J36 pad 3: +9V -> +9V_M
- J36 pad 4: 9V_GND -> 9V_GND_M
- L3 pad 2: 9V_GND -> 9V_GND_P
- R25 pad 1: +9V -> +9V_P
- R26 pad 1: +15V -> +15V_P
- R27 pad 1: -15V -> -15V_P
- R75 pad 1: GND -> GND_M
- R86 pad 1: GND -> GND_M
- U23 pad 11: -15V -> -15V_M
- U23 pad 4: +15V -> +15V_M
- U24 pad 11: -15V -> -15V_M
- U24 pad 3: GND -> GND_M
- U24 pad 4: +15V -> +15V_M
- U24 pad 5: GND -> GND_M
- U7 pad 5: GND -> GND_P
- Z122 pad 2: GND -> GND_M
- Z123 pad 2: GND -> GND_M
- Z124 pad 2: GND -> GND_M
- Z125 pad 2: GND -> GND_M
- Z126 pad 2: GND -> GND_M
- Z127 pad 2: GND -> GND_M
- Z128 pad 2: GND -> GND_M
- Z129 pad 2: GND -> GND_M
- Z134 pad 2: GND -> GND_M
- Z135 pad 2: GND -> GND_M
- Z136 pad 2: GND -> GND_M
- Z137 pad 2: GND -> GND_M
- Z170 pad 2: GND -> GND_M
- Z171 pad 2: GND -> GND_M
- Z174 pad 2: GND -> GND_M
Routing:
- net Net-(C18-Pad1): track 0.00 -> 40.8 mm, vias 0 -> 1
- net 9V_GND_P: track 0.00 -> 38.3 mm, vias 0 -> 1
- net Net-(C12-Pad2): track 0.00 -> 36.4 mm, vias 0 -> 1
- net Net-(C11-Pad2): track 0.00 -> 36.4 mm, vias 0 -> 1
- net Net-(U6--VIN): track 83.7 -> 107.8 mm
- net Net-(U6-+VIN): track 83.7 -> 102.1 mm
- net Net-(J10-Pin_2): track 17.0 -> 33.4 mm
- net Net-(C2-Pad1): track 6.29 -> 21.9 mm
- net GND_P: track 0.00 -> 14.9 mm
- net Net-(C2-Pad2): track 5.08 -> 16.8 mm
- net Net-(J10-Pin_1): track 13.5 -> 22.4 mm
- net Net-(U7--VOUT): track 0.00 -> 5.74 mm
- net Net-(U7-+VOUT): track 0.00 -> 5.74 mm
- net Net-(U6--VOUT): track 0.00 -> 5.74 mm
- net Net-(U6-+VOUT): track 0.00 -> 5.74 mm
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- added copper zone on B.Cu, net GND_15V_FILT
- added copper zone on B.Cu, net GND_9V_FILT

Commit message: PCB Update
Parts:
- moved J13 1.27 mm to (105.4, 76.2)
- moved J14 1.27 mm to (105.4, 96.5)
- moved J21 1.27 mm to (105.4, 55.9)
- moved C25 1.27 mm to (86.6, 104.1)
- moved C26 1.27 mm to (86.6, 94.0)
- moved R26 1.27 mm to (95.0, 104.1)
- moved R27 1.27 mm to (95.0, 94.0)
Routing:
- net +9V_P: track 0.00 -> 58.0 mm
- net 9V_GND_P: track 38.3 -> 92.5 mm
- net +15V_P: track 3.08 -> 50.4 mm, vias 1 -> 0
- net Net-(C12-Pad2): track 36.4 -> 33.8 mm
- net Net-(C11-Pad2): track 36.4 -> 33.8 mm
- net -15V_P: track 1.81 -> 0.00 mm
Changed lines of the file:
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@@
 	(footprint "Connector_Bridged_2.54mm_LongPads:Bridge_2x05_P2.54mm_Vertical_LongPads"
 		(layer "F.Cu")
-		(at 106.68 55.88)
+		(at 105.41 55.88)
 		(descr "Through hole straight socket strip, 1x05, 2.54mm pitch, single row (from Kicad 4.0.7), script generated")
 		(tags "Through hole socket strip THT 1x05 2.54mm single row")
@@
 	(footprint "Connector_PinSocket_2.54mm_LongPads:PinSocket_1x05_P2.54mm_Vertical_LongPads"
 		(layer "F.Cu")
-		(at 106.68 76.2)
+		(at 105.41 76.2)
 		(descr "Through hole straight socket strip, 1x05, 2.54mm pitch, single row (from Kicad 4.0.7), script generated")
 		(tags "Through hole socket strip THT 1x05 2.54mm single row")
@@
 	(footprint "Connector_PinSocket_2.54mm_LongPads:PinSocket_1x05_P2.54mm_Vertical_LongPads"
 		(layer "F.Cu")
-		(at 106.68 96.52)
+		(at 105.41 96.52)
 		(descr "Through hole straight socket strip, 1x05, 2.54mm pitch, single row (from Kicad 4.0.7), script generated")
 		(tags "Through hole socket strip THT 1x05 2.54mm single row")
@@
 	(footprint "Resistor_SMD:R_0805_2012Metric_Pad1.20x1.40mm_HandSolder"
 		(layer "F.Cu")
-		(at 96.25 93.98 180)
+		(at 94.98 93.98 180)
 		(descr "Resistor SMD 0805 (2012 Metric), square (rectangular) end terminal, IPC-7351 nominal with elongated pad for handsoldering. (Body size source: IPC-SM-782 page 72, https://www.pcb-3d.com/wordpress/wp-content/uploads/ipc-sm-782a_amendment_1_and_2.pdf), generated with kicad-footprint-generator")
 		(tags "resistor handsolder")
@@
 	(footprint "Resistor_SMD:R_0805_2012Metric_Pad1.20x1.40mm_HandSolder"
 		(layer "F.Cu")
-		(at 96.25 104.14 180)
+		(at 94.98 104.14 180)
 		(descr "Resistor SMD 0805 (2012 Metric), square (rectangular) end terminal, IPC-7351 nominal with elongated pad for handsoldering. (Body size source: IPC-SM-782 page 72, https://www.pcb-3d.com/wordpress/wp-content/uploads/ipc-sm-782a_amendment_1_and_2.pdf), generated with kicad-footprint-generator")
 		(tags "resistor handsolder")
@@
 	(footprint "Capacitor_SMD:C_0805_2012Metric_Pad1.18x1.45mm_HandSolder"
 		(layer "B.Cu")
-		(at 86.5925 102.87)
+		(at 86.5925 104.14)
 		(descr "Capacitor SMD 0805 (2012 Metric), square (rectangular) end terminal, IPC-7351 nominal with elongated pad for handsoldering. (Body size source: IPC-SM-782 page 76, https://www.pcb-3d.com/wordpress/wp-content/uploads/ipc-sm-782a_amendment_1_and_2.pdf, https://docs.google.com/spreadsheets/d/1BsfQQcO9C6DZCsRaXUlFlo91Tg2WpOkGARC1WS5S8t0/edit?usp=sharing), generated with kicad-footprint-generator")
 		(tags "capacitor handsolder")
@@
 	(footprint "Capacitor_SMD:C_0805_2012Metric_Pad1.18x1.45mm_HandSolder"
 		(layer "B.Cu")
-		(at 86.5925 95.25 180)
+		(at 86.5925 93.98 180)
 		(descr "Capacitor SMD 0805 (2012 Metric), square (rectangular) end terminal, IPC-7351 nominal with elongated pad for handsoldering. (Body size source: IPC-SM-782 page 76, https://www.pcb-3d.com/wordpress/wp-content/uploads/ipc-sm-782a_amendment_1_and_2.pdf, https://docs.google.com/spreadsheets/d/1BsfQQcO9C6DZCsRaXUlFlo91Tg2WpOkGARC1WS5S8t0/edit?usp=sharing), generated with kicad-footprint-generator")
 		(tags "capacitor handsolder")
@@
 	)
 	(segment
-		(start 89.535 104.14)
-		(end 89.535 102.87)
+		(start 80.01 104.14)
+		(end 73.4275 110.7225)
 		(width 0.4)
 		(layer "F.Cu")
@@
 	)
 	(segment
-		(start 95.25 104.14)
+		(start 93.98 104.14)
 		(end 91.44 104.14)
 		(width 0.4)
@@
 		(net 2)
 	)
-	(segment
-		(start 80.01 104.14)
-		(end 73.4275 110.7225)
-		(width 0.4)
-		(layer "F.Cu")
-		(net 2)
-	)
 	(via
-		(at 89.535 102.87)
+		(at 89.535 104.14)
 		(size 0.6)
 		(drill 0.3)
@@
 	)
 	(segment
-		(start 89.535 102.87)
-		(end 87.63 102.87)
+		(start 87.63 104.14)
+		(end 89.535 104.14)
 		(width 0.4)
 		(layer "B.Cu")
@@
 	)
 	(segment
-		(start 89.535 93.98)
-		(end 89.535 95.25)
+		(start 93.98 93.98)
+		(end 91.44 93.98)
 		(width 0.4)
 		(layer "F.Cu")
@@
 	)
 	(segment
-		(start 95.25 93.98)
-		(end 91.44 93.98)
-		(width 0.4)
-		(layer "F.Cu")
-		(net 3)
-	)
-	(segment
 		(start 80.01 93.98)
 		(end 73.4275 87.3975)
@@
 	)
 	(via
-		(at 89.535 95.25)
+		(at 89.535 93.98)
 		(size 0.6)
 		(drill 0.3)
@@
 	)
 	(segment
-		(start 89.535 95.25)
-		(end 87.63 95.25)
+		(start 87.63 93.98)
+		(end 89.535 93.98)
 		(width 0.4)
 		(layer "B.Cu")
@@
 	)
 	(segment
+		(start 100.33 80.01)
+		(end 100.33 97.79)
+		(width 0.4)
+		(layer "In1.Cu")
+		(net 53)
+	)
+	(segment
+		(start 100.33 77.47)
+		(end 101.6 78.74)
+		(width 0.4)
+		(layer "In1.Cu")
+		(net 53)
+	)
+	(segment
+		(start 101.6 99.06)
+		(end 105.41 99.06)
+		(width 0.4)
+		(layer "In1.Cu")
+		(net 53)
+	)
+	(segment
+		(start 100.33 59.69)
+		(end 100.33 77.47)
+		(width 0.4)
+		(layer "In1.Cu")
+		(net 53)
+	)
+	(segment
+		(start 101.6 78.74)
+		(end 100.33 80.01)
+		(width 0.4)
+		(layer "In1.Cu")
+		(net 53)
+	)
+	(segment
+		(start 100.33 97.79)
+		(end 101.6 99.06)
+		(width 0.4)
+		(layer "In1.Cu")
+		(net 53)
+	)
+	(segment
+		(start 101.6 78.74)
+		(end 105.41 78.74)
+		(width 0.4)
+		(layer "In1.Cu")
+		(net 53)
+	)
+	(segment
+		(start 105.41 58.42)
+		(end 101.6 58.42)
+		(width 0.4)
+		(layer "In1.Cu")
+		(net 53)
+	)
+	(segment
+		(start 101.6 58.42)
+		(end 100.33 59.69)
+		(width 0.4)
+		(layer "In1.Cu")
+		(net 53)
+	)
+	(segment
 		(start 91.44 96.055)
 		(end 91.44 99.06)
@@
 	)
 	(segment
-		(start 97.25 104.14)
-		(end 99.06 104.14)
+		(start 105.41 60.96)
+		(end 102.87 60.96)
 		(width 0.4)
-		(layer "F.Cu")
+		(layer "In2.Cu")
 		(net 59)
 	)
-	(via
-		(at 99.06 104.14)
-		(size 0.6)
-		(drill 0.3)
-		(layers "F.Cu" "B.Cu")
+	(segment
+		(start 101.6 82.55)
+		(end 101.6 100.33)
+		(width 0.4)
+		(layer "In2.Cu")
 		(net 59)
 	)
 	(segment
-		(start 105.41 60.96)
-		(end 106.68 60.96)
+		(start 101.6 100.33)
+		(end 102.87 101.6)
+		(width 0.4)
+		(layer "In2.Cu")
+		(net 59)
+	)
+	(segment
+		(start 102.87 101.6)
+		(end 105.41 101.6)
+		(width 0.4)
+		(layer "In2.Cu")
+		(net 59)
+	)
+	(segment
+		(start 101.6 62.23)
+		(end 101.6 80.01)
+		(width 0.4)
+		(layer "In2.Cu")
+		(net 59)
+	)
+	(segment
+		(start 102.87 81.28)
+		(end 105.41 81.28)
+		(width 0.4)
+		(layer "In2.Cu")
+		(net 59)
+	)
+	(segment
+		(start 102.87 60.96)
+		(end 101.6 62.23)
+		(width 0.4)
+		(layer "In2.Cu")
+		(net 59)
+	)
+	(segment
+		(start 102.87 81.28)
+		(end 101.6 82.55)
+		(width 0.4)
+		(layer "In2.Cu")
+		(net 59)
+	)
+	(segment
+		(start 101.6 80.01)
+		(end 102.87 81.28)
 		(width 0.4)
 		(layer "In2.Cu")
@@
 	)
 	(segment
-		(start 97.25 93.98)
-		(end 99.06 93.98)
+		(start 100.33 76.2)
+		(end 99.06 74.93)
+		(width 0.4)
+		(layer "F.Cu")
+		(net 61)
+	)
+	(segment
+		(start 99.06 57.15)
+		(end 100.33 55.88)
+		(width 0.4)
+		(layer "F.Cu")
+		(net 61)
+	)
+	(segment
+		(start 99.06 74.93)
+		(end 99.06 57.15)
+		(width 0.4)
+		(layer "F.Cu")
+		(net 61)
+	)
+	(segment
+		(start 105.41 76.2)
+		(end 100.33 76.2)
+		(width 0.4)
+		(layer "F.Cu")
+		(net 61)
+	)
+	(segment
+		(start 100.33 76.2)
+		(end 99.06 77.47)
+		(width 0.4)
+		(layer "F.Cu")
+		(net 61)
+	)
+	(segment
+		(start 100.33 55.88)
+		(end 105.41 55.88)
+		(width 0.4)
+		(layer "F.Cu")
+		(net 61)
+	)
+	(segment
+		(start 99.06 77.47)
+		(end 99.06 95.25)
+		(width 0.4)
+		(layer "F.Cu")
+		(net 61)
+	)
+	(segment
+		(start 100.33 96.52)
+		(end 105.41 96.52)
+		(width 0.4)
+		(layer "F.Cu")
+		(net 61)
+	)
+	(segment
+		(start 99.06 95.25)
+		(end 100.33 96.52)
 		(width 0.4)
 		(layer "F.Cu")
-		(net 60)
+		(net 61)
 	)
 	(zone

Commit message: PCB Update
Parts:
- moved J13 40.7 mm to (146.1, 74.9)
- moved J14 40.7 mm to (146.1, 95.2)
- moved J21 40.7 mm to (146.1, 54.6)
- moved C10 3.81 mm to (76.2, 48.3)
- moved C11 3.81 mm to (76.2, 114.3)
- moved C112 3.81 mm to (72.2, 61.0)
- moved C113 3.81 mm to (72.2, 66.0)
- moved C12 3.81 mm to (76.2, 83.8)
- moved C18 3.81 mm to (95.2, 63.5)
- moved C19 3.81 mm to (95.2, 103.1)
- moved C2 3.81 mm to (54.6, 90.2)
- moved C20 3.81 mm to (95.2, 95.0)
- moved C23 3.81 mm to (90.4, 68.6)
- moved C24 3.81 mm to (90.4, 58.4)
- moved C25 3.81 mm to (90.4, 104.1)
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Routing:
- net +9V_P: track 58.0 -> 0.00 mm
- net 9V_GND_P: track 92.5 -> 38.3 mm
- net +15V_P: track 50.4 -> 0.00 mm
- net Net-(U6--VIN): track 107.8 -> 80.8 mm
- net Net-(U6-+VIN): track 102.1 -> 80.8 mm
- net Net-(C2-Pad1): track 21.9 -> 5.16 mm
- net Net-(C2-Pad2): track 16.8 -> 5.16 mm
- net Net-(J10-Pin_2): track 33.4 -> 31.9 mm
- net Net-(J10-Pin_1): track 22.4 -> 23.5 mm
- added copper zone on F.Cu, net Net-(C2-Pad1)
- added copper zone on F.Cu, net Net-(C2-Pad2)
- added copper zone on F.Cu, net Net-(U6-+VIN)
- added copper zone on F.Cu, net Net-(U6--VIN)

Commit message: PCB Update
Parts:
- moved J33 101.4 mm to (148.6, 78.7)
- moved J32 97.5 mm to (148.6, 86.4)
- moved SW9 97.0 mm to (148.6, 63.5)
- moved J31 94.3 mm to (148.6, 94.0)
- moved J30 91.8 mm to (148.6, 101.6)
- moved Z127 91.6 mm to (133.2, 71.1)
- moved Z131 91.6 mm to (137.9, 56.4)
- moved Z135 91.6 mm to (137.9, 68.2)
- moved Z134 76.4 mm to (155.2, 61.0), turned to 180 degrees
- moved U24 74.4 mm to (165.6, 93.7)
- moved Z130 72.6 mm to (155.2, 63.5)
- moved Z126 71.2 mm to (155.2, 66.0), turned to 180 degrees
- moved J21 56.7 mm to (130.8, 109.2)
- moved U23 52.0 mm to (165.1, 58.4)
- moved J13 45.9 mm to (115.6, 109.2)
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Connections:
- J13 pad 1: +9V_P -> 9V_GND_P
- J13 pad 2: 9V_GND_P -> +9V_P
- J13 pad 3: +15V_P -> -15V_P
- J13 pad 4: -15V_P -> GND_P
- J13 pad 5: GND_P -> +15V_P
- J14 pad 1: +9V_P -> 9V_GND_P
- J14 pad 2: 9V_GND_P -> +9V_P
- J14 pad 3: +15V_P -> -15V_P
- J14 pad 4: -15V_P -> GND_P
- J14 pad 5: GND_P -> +15V_P
- J21 pad 1: +9V_P -> 9V_GND_P
- J21 pad 10: +9V_M -> 9V_GND_M
- J21 pad 2: 9V_GND_P -> +9V_P
- J21 pad 3: +15V_P -> -15V_P
- J21 pad 4: -15V_P -> GND_P
- J21 pad 5: GND_P -> +15V_P
- J21 pad 6: GND_M -> +15V_M
- J21 pad 7: -15V_M -> GND_M
- J21 pad 8: +15V_M -> -15V_M
- J21 pad 9: 9V_GND_M -> +9V_M
Routing:
- net +9V_P: track 0.00 -> 67.6 mm
- net 9V_GND_P: track 38.3 -> 89.8 mm
- net -15V_P: track 0.00 -> 46.6 mm
- net +15V_P: track 0.00 -> 36.4 mm
- net GND_P: track 14.9 -> 42.9 mm
- net Net-(C18-Pad1): track 40.8 -> 26.0 mm
- net Net-(C12-Pad2): track 33.8 -> 23.0 mm
- net Net-(C11-Pad2): track 33.8 -> 23.0 mm
- net Net-(J30-Pin_1): track 0.00 -> 3.37 mm
- net Net-(U23A-+): track 0.00 -> 2.54 mm
- net /Pegel_Pre: track 0.00 -> 2.54 mm
- net /Pegel_Post: track 0.00 -> 2.54 mm
- net /Pegel_Mic_Effekt: track 0.00 -> 2.54 mm
- net /Pegel_Aux_Return: track 0.00 -> 2.54 mm
- net Net-(U6-+VIN): track 80.8 -> 82.3 mm
- added copper zone on F.Cu, net 9V_GND_P
- added copper zone on F.Cu, net GND_P
- added copper zone on F.Cu, net Net-(C11-Pad2)
- added copper zone on F.Cu, net Net-(C12-Pad2)
- added copper zone on F.Cu, net Net-(C18-Pad1)

Commit message: PCB Update
Parts:
- moved C46 86.9 mm to (160.3, 66.0)
- moved C56 85.2 mm to (160.3, 90.2)
- moved Z128 76.9 mm to (160.3, 82.5)
- moved Z136 75.5 mm to (160.3, 87.6), turned to 180 degrees
- moved Z137 74.3 mm to (160.3, 92.7), turned to 180 degrees
- moved C47 70.8 mm to (177.6, 66.0), turned to 180 degrees
- moved Z132 70.5 mm to (160.3, 85.1)
- moved C57 67.9 mm to (177.6, 90.2), turned to 180 degrees
- moved Z133 67.2 mm to (160.3, 95.2)
- moved Z129 62.6 mm to (160.3, 97.8)
- moved Z127 27.2 mm to (160.3, 73.7)
- moved Z131 26.8 mm to (160.3, 71.1)
- moved Z135 22.4 mm to (160.3, 68.6), turned to 180 degrees
- moved U24 11.2 mm to (165.1, 82.5)
- moved Z126 9.16 mm to (160.3, 58.4), turned to 0 degrees
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Connections:
- R67 pad 2: Net-(U24B--) -> Net-(U23D--)
- R68 pad 2: Net-(U24B--) -> Net-(U23D--)
- R71 pad 1: Net-(U24B--) -> Net-(U23D--)
- U23 pad 10: Net-(U23C-+) -> GND_M
- U23 pad 12: Net-(U23D-+) -> GND_M
- U23 pad 13: /Pegel_Post -> Net-(U23D--)
- U23 pad 14: /Pegel_Post -> Net-(U24C-+)
- U23 pad 8: /Pegel_Aux_Return -> Net-(D1-A)
- U23 pad 9: /Pegel_Aux_Return -> Net-(D1-K)
- U24 pad 1: Net-(D1-A) -> /Pegel_Aux_Return
- U24 pad 2: Net-(D1-K) -> /Pegel_Aux_Return
- U24 pad 3: GND_M -> Net-(U24A-+)
- U24 pad 5: GND_M -> Net-(U24B-+)
- U24 pad 6: Net-(U24B--) -> /Pegel_Post
- U24 pad 7: Net-(U24C-+) -> /Pegel_Post
- Z132 pad 2: Net-(U23C-+) -> Net-(U24A-+)
- Z133 pad 2: Net-(U23D-+) -> Net-(U24B-+)
- Z136 pad 1: Net-(U23C-+) -> Net-(U24A-+)
- Z137 pad 1: Net-(U23D-+) -> Net-(U24B-+)
Routing:
- net -15V_M: track 0.00 -> 7.62 mm
- net +15V_M: track 0.00 -> 7.62 mm
- net Net-(U24B-+): track 0.00 -> 6.35 mm
- net Net-(U23B-+): track 0.00 -> 6.35 mm
- net Net-(U24A-+): track 0.00 -> 6.35 mm
- net Net-(U23A-+): track 2.54 -> 6.35 mm
- net Net-(U24D--): track 0.00 -> 2.54 mm
- net Net-(J33-Pin_1): track 0.00 -> 2.54 mm
- net Net-(J32-Pin_1): track 0.00 -> 2.54 mm
- net /Pegel_Aux_Return: track 2.54 -> 5.08 mm
- net Net-(U24C-+): track 0.00 -> 2.54 mm
- net Net-(J31-Pin_1): track 0.00 -> 2.54 mm
- net Net-(J30-Pin_1): track 3.37 -> 2.54 mm

Commit message: PCB Update
Parts:
- moved Z122 79.8 mm to (153.4, 68.6)
- moved D2 76.0 mm to (176.3, 66.0)
- moved Z123 74.2 mm to (153.4, 81.3)
- moved Z171 70.3 mm to (170.4, 116.8), turned to 180 degrees
- moved D1 69.4 mm to (181.9, 68.6), turned to 180 degrees
- moved Z173 68.7 mm to (170.4, 119.4)
- moved Z124 68.6 mm to (153.4, 96.5)
- moved R67 65.7 mm to (153.4, 63.5)
- moved Z125 65.5 mm to (153.4, 109.2)
- moved R59 65.0 mm to (153.4, 61.0)
- moved Z168 64.4 mm to (176.3, 109.2)
- moved R82 46.8 mm to (176.3, 119.4), turned to 180 degrees
- moved R72 44.1 mm to (176.3, 104.1), turned to 180 degrees
- moved R75 44.0 mm to (176.3, 106.7), turned to 180 degrees
- moved R71 41.1 mm to (176.3, 81.3), turned to 180 degrees
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Connections:
- R67 pad 2: Net-(U23D--) -> Net-(U23C--)
- R68 pad 2: Net-(U23D--) -> Net-(U23C--)
- R71 pad 1: Net-(U23D--) -> Net-(U23C--)
- R72 pad 1: +15V -> +15V_M
- SW9 pad 1: /Pegel_Pre -> /Pegel_Post
- SW9 pad 2: /Pegel_Mic_Effekt -> /Pegel_Aux_Return
- SW9 pad 3: /Pegel_Aux_Return -> /Pegel_Mic_Effekt
- SW9 pad 4: /Pegel_Post -> /Pegel_Pre
- U23 pad 13: Net-(U23D--) -> Net-(D1-K)
- U23 pad 14: Net-(U24C-+) -> Net-(D1-A)
- U23 pad 8: Net-(D1-A) -> Net-(U24C-+)
- U23 pad 9: Net-(D1-K) -> Net-(U23C--)
Routing:
- net +15V_M: track 7.62 -> 124.0 mm, vias 0 -> 1
- net -15V_M: track 7.62 -> 110.5 mm
- net /Pegel_Post: track 2.54 -> 80.1 mm
- net /Pegel_Aux_Return: track 5.08 -> 63.1 mm
- net /Pegel_Mic_Effekt: track 2.54 -> 42.7 mm
- net Net-(D1-K): track 0.00 -> 38.1 mm
- net Net-(U23C--): track 0.00 -> 37.6 mm
- net Net-(U24C-+): track 2.54 -> 25.2 mm
- net /Pegel_Pre: track 2.54 -> 23.9 mm
- net Net-(D2-A): track 0.00 -> 17.9 mm, vias 0 -> 2
- net Net-(Z168-Pad2): track 0.00 -> 13.4 mm
- net Net-(D1-A): track 0.00 -> 9.63 mm
- net Net-(J31-Pin_1): track 2.54 -> 12.0 mm
- net Net-(J30-Pin_1): track 2.54 -> 12.0 mm
- net Net-(J33-Pin_1): track 2.54 -> 12.0 mm
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
Commit message: PCB Update
Parts:
- moved J36 82.6 mm to (172.7, 101.6)
- moved J34 81.1 mm to (172.7, 114.3)
- moved C36 74.5 mm to (172.7, 96.5), turned to 180 degrees
- moved Z167 69.5 mm to (166.1, 96.5)
- moved Z170 68.4 mm to (166.1, 99.1), turned to 180 degrees
- moved D3 66.7 mm to (166.1, 116.8), turned to 180 degrees
- moved Z174 66.5 mm to (172.7, 121.9)
- moved Z172 66.0 mm to (166.1, 94.0), turned to 180 degrees
- moved R86 52.4 mm to (172.7, 94.0)
- moved R84 44.9 mm to (166.1, 121.9), turned to 180 degrees
- moved R81 44.6 mm to (172.7, 91.4)
- moved Z122 11.1 mm to (143.5, 73.7)
- moved Z123 11.1 mm to (143.5, 86.4)
- moved Z124 11.1 mm to (143.5, 101.6)
- moved C47 10.5 mm to (166.1, 76.2)
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Connections:
- C46 pad 1: GND -> GND_M
- C47 pad 1: GND -> GND_M
- C56 pad 1: GND -> GND_M
- C57 pad 1: GND -> GND_M
Routing:
- net GND_M: track 0.00 -> 52.1 mm, vias 0 -> 14
- net +9V_M: track 0.00 -> 40.0 mm
- net 9V_GND_M: track 0.00 -> 31.3 mm
- net Net-(J34-Pin_1): track 0.00 -> 11.0 mm
- net Net-(J36-Pin_1): track 0.00 -> 10.6 mm
- net Net-(D1-K): track 38.1 -> 27.6 mm
- net Net-(U23C--): track 37.6 -> 28.8 mm
- net -15V_M: track 110.5 -> 119.0 mm
- net Net-(R81-Pad1): track 0.00 -> 8.45 mm
- net +15V_M: track 124.0 -> 117.8 mm
- net Net-(D3-K): track 0.00 -> 6.00 mm
- net Net-(R59-Pad1): track 6.35 -> 12.2 mm
- net Net-(J34-Pin_2): track 0.00 -> 5.49 mm
- net /Pegel_Pre: track 23.9 -> 18.8 mm
- net Net-(Z167-Pad2): track 0.00 -> 5.08 mm
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- added copper zone on In2.Cu, net +15V_M
- added copper zone on B.Cu, net GND_M
- added copper zone on F.Cu, net Net-(D1-K)
- added copper zone on F.Cu, net Net-(D2-A)
Other:
- board text added: "J21"
