File: KiCad/Power_Supply_Meter_Amp.kicad_pcb (KiCad board)
At the start: 4 copper layers, 150 x 85.2 mm, 84 parts, among them J10 VCC_IN, J11 VCC_OUT, J13 EMK_Out, J14 EMK_Out, J21 Conn_01x05_bridged, J30 Pegel_In, J31 Pegel_In, J32 Pegel_In, J33 Pegel_In, J34 LED_Out, J36 VU_Meter_Out, SW1 SW_DPST, SW9 SW_Rotary_1x4, U23 TL074, U24 TL074, U6 REC10K-2409, U7 REC10K-2415

Commit message: PCB Update
Parts:
- removed J13, J14: EMK_Out, Connector_PinSocket_2.54mm_LongPads:PinSocket_1x05_P2.54mm_Vertical_LongPads
- added C115: 10n, Capacitor_SMD:C_1210_3225Metric_Pad1.33x2.70mm_HandSolder, F.Cu at (173.6, 50.8)
- added H1: MountingHole, MountingHole:MountingHole_3.2mm_M3_Pad, F.Cu at (43.2, 50.8)
- added H2: MountingHole, MountingHole:MountingHole_3.2mm_M3_Pad, F.Cu at (121.9, 50.8)
- added H3: MountingHole, MountingHole:MountingHole_3.2mm_M3_Pad, F.Cu at (43.2, 125.7)
- added H4: MountingHole, MountingHole:MountingHole_3.2mm_M3_Pad, F.Cu at (121.9, 125.7)
- added H5: MountingHole_Pad, MountingHole:MountingHole_3.2mm_M3_Pad, F.Cu at (182.9, 50.8)
- added H6: MountingHole, MountingHole:MountingHole_3.2mm_M3_Pad, F.Cu at (182.9, 125.7)
- added H7: MountingHole, MountingHole:MountingHole_3.2mm_M3_Pad, F.Cu at (137.2, 125.7)
- added H8: MountingHole, MountingHole:MountingHole_3.2mm_M3_Pad, F.Cu at (137.2, 50.8)
- moved J21 15.2 mm to (115.6, 114.3)
Routing:
- net +9V_P: track 67.6 -> 52.4 mm
- net GND_P: track 42.9 -> 27.6 mm
- net 9V_GND_P: track 91.3 -> 76.1 mm
- net -15V_P: track 46.6 -> 31.3 mm
- net +15V_P: track 36.4 -> 21.2 mm
- net Net-(D2-A): track 22.7 -> 22.1 mm
- net GND_M: vias 18 -> 20
- added copper zone on F.Cu, net Net-(C115-Pad1)

Commit message: PCB Update
Routing:
- net Net-(J34-Pin_1): track 11.8 -> 5.08 mm
- added copper zone on F.Cu, net Net-(J34-Pin_1)
Changed lines of the file:
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@@
-	)
-	(segment
-		(start 167.1 121.92)
-		(end 168.275 121.92)
-		(width 0.6)
-		(layer "F.Cu")
-		(net 20)
-	)
-	(segment
-		(start 172.72 114.3)
-		(end 170.815 114.3)
-		(width 0.6)
-		(layer "F.Cu")
-		(net 20)
-	)
-	(segment
-		(start 168.275 121.92)
-		(end 169.545 120.65)
-		(width 0.6)
-		(layer "F.Cu")
-		(net 20)
-	)
-	(segment
-		(start 169.545 115.57)
-		(end 170.815 114.3)
-		(width 0.6)
-		(layer "F.Cu")
-		(net 20)
 	)
 	(segment
@@
 	)
 	(zone
+		(net 20)
+		(net_name "Net-(J34-Pin_1)")
+		(layer "F.Cu")
+		(hatch edge 0.5)
+		(priority 8)
+		(connect_pads yes
+			(clearance 0.5)
+		)
+		(min_thickness 0.25)
+		(filled_areas_thickness no)
+		(fill yes
+			(thermal_gap 0.5)
+			(thermal_bridge_width 0.5)
+			(smoothing chamfer)
+			(radius 0.5)
+		)
+		(polygon
+			(pts
+				(xy 167.005 122.428) (xy 169.8498 122.428) (xy 169.8498 120.396) (xy 169.291 120.396) (xy 168.275 121.412)
+				(xy 167.005 121.412)
+			)
+		)
+	)
+	(zone
 		(net 54)
 		(net_name "GND_M")
@@
 			)
 		)
+	)
+	(zone
+		(net 20)
+		(net_name "Net-(J34-Pin_1)")
+		(layer "F.Cu")
+		(hatch edge 0.5)
+		(priority 8)
+		(connect_pads yes
+			(clearance 0.5)
+		)
+		(min_thickness 0.25)
+		(filled_areas_thickness no)
+		(fill yes
+			(thermal_gap 0.5)
+			(thermal_bridge_width 0.5)
+			(smoothing chamfer)
+			(radius 0.5)
+		)
+		(polygon
+			(pts
+				(xy 172.085 113.792) (xy 169.2402 113.792) (xy 169.2402 115.824) (xy 169.799 115.824) (xy 170.815 114.808)
+				(xy 172.085 114.808)
+			)
+		)

Commit message: PCB Update
Parts:
- moved R72 2.54 mm to (166.1, 106.7)
- moved R75 2.54 mm to (166.1, 104.1)
- turned Z174 to 180 degrees
Routing:
- net -15V_M: track 152.9 -> 18.3 mm
- net +15V_M: track 123.0 -> 28.4 mm
- net GND_M: track 49.6 -> 32.2 mm, vias 20 -> 21
- net Net-(D2-A): track 22.1 -> 34.1 mm, vias 2 -> 0
- added copper zone on In2.Cu, net +15V_M
- added copper zone on In2.Cu, net -15V_M

Commit message: PCB Update
Parts:
- removed R25, R26, R27: 22R, Resistor_SMD:R_0805_2012Metric_Pad1.20x1.40mm_HandSolder
- added C114: 10u, Capacitor_THT:CP_Radial_D5.0mm_P2.50mm, F.Cu at (112.5, 93.3)
- added C116: 10u, Capacitor_THT:CP_Radial_D5.0mm_P2.50mm, F.Cu at (104.2, 116.2)
- added C117: 10u, Capacitor_THT:CP_Radial_D5.0mm_P2.50mm, F.Cu at (106.7, 104.8)
- added Z257: ~, Resistor_SMD:R_0805_2012Metric_Pad1.20x1.40mm_HandSolder, F.Cu at (103.1, 111.8)
- added Z258: ~, Resistor_SMD:R_0805_2012Metric_Pad1.20x1.40mm_HandSolder, F.Cu at (103.1, 96.5)
- added Z259: ~, Resistor_SMD:R_0805_2012Metric_Pad1.20x1.40mm_HandSolder, F.Cu at (103.1, 73.7)
Routing:
- net GND_P: track 27.6 -> 34.1 mm

Commit message: PCB Final Update
Parts:
- added J13: Conn_02x07_Odd_Even, Connector_PinHeader_2.54mm:PinHeader_2x07_P2.54mm_Vertical, F.Cu at (139.7, 108.0)
- J21: value Conn_01x05_bridged -> Conn_02x07_Odd_Even; footprint Connector_Bridged_2.54mm_LongPads:Bridge_2x05_P2.54mm_Vertical_LongPads -> Connector_PinHeader_2.54mm:PinHeader_2x07_P2.54mm_Vertical
- moved H7 26.7 mm to (137.2, 99.1)
- moved C114 18.7 mm to (112.0, 74.7)
- moved J21 7.29 mm to (112.0, 108.0)
- moved C10 4.45 mm to (75.2, 49.5)
- moved C11 4.45 mm to (75.2, 115.6)
- moved C12 4.45 mm to (75.2, 85.1)
- moved C2 4.45 mm to (53.6, 91.4)
- moved C23 4.45 mm to (89.4, 69.8)
- moved C24 4.45 mm to (89.4, 59.7)
- moved C25 4.45 mm to (89.4, 105.4)
- moved C26 4.45 mm to (89.4, 95.2)
- moved C5 4.45 mm to (53.6, 73.7)
- moved J10 4.45 mm to (53.6, 110.5)
- moved J11 4.45 mm to (53.6, 118.1)
- moved L1 4.45 mm to (53.6, 82.5)
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Connections:
- J21 pad 10: 9V_GND_M -> GND_P
- J21 pad 2: +9V_P -> 9V_GND_P
- J21 pad 3: -15V_P -> 9V_GND_P
- J21 pad 4: GND_P -> 9V_GND_P
- J21 pad 5: +15V_P -> +9V_P
- J21 pad 6: +15V_M -> +9V_P
- J21 pad 7: GND_M -> -15V_P
- J21 pad 8: -15V_M -> -15V_P
- J21 pad 9: +9V_M -> GND_P
Routing:
- net GND_M: track 32.2 -> 59.1 mm
- net 9V_GND_M: track 32.4 -> 50.5 mm
- net +9V_M: track 32.4 -> 39.3 mm
- net +9V_P: track 51.9 -> 57.4 mm
- net +15V_P: track 21.5 -> 25.8 mm
- net 9V_GND_P: track 76.1 -> 72.5 mm
- net +15V_M: track 28.4 -> 31.4 mm
- net -15V_M: track 18.3 -> 20.7 mm
- net -15V_P: track 30.9 -> 32.7 mm
- net GND_P: track 34.1 -> 34.6 mm
- added copper zone on B.Cu, net 9V_GND_M

Commit message: common mode chocke Update
Parts:
- moved C5 4.71 mm to (50.8, 69.8)
- moved C2 3.05 mm to (50.8, 92.7)
- moved J10 2.77 mm to (50.8, 110.5)
- moved J11 2.77 mm to (50.8, 118.1)
- moved L1 2.77 mm to (50.8, 82.5)
- moved SW1 2.77 mm to (50.8, 97.8)
Routing:
- net Net-(U6-+VIN): track 85.2 -> 92.5 mm
- net Net-(U6--VIN): track 83.8 -> 86.5 mm
Changed lines of the file:
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@@
 	(footprint "Connector_PinHeader_2.54mm_LongPads:PinHeader_1x02_P2.54mm_Vertical_LongPads"
 		(layer "F.Cu")
-		(at 53.5725 110.49)
+		(at 50.8 110.49)
 		(descr "Through hole straight pin header, 1x02, 2.54mm pitch, single row")
 		(tags "Through hole pin header THT 1x02 2.54mm single row")
@@
 	(footprint "Connector_PinHeader_2.54mm_LongPads:PinHeader_1x02_P2.54mm_Vertical_LongPads"
 		(layer "F.Cu")
-		(at 53.5725 118.11)
+		(at 50.8 118.11)
 		(descr "Through hole straight pin header, 1x02, 2.54mm pitch, single row")
 		(tags "Through hole pin header THT 1x02 2.54mm single row")
@@
 	(footprint "Capacitor_SMD:C_1210_3225Metric_Pad1.33x2.70mm_HandSolder"
 		(layer "F.Cu")
-		(at 53.5725 91.44 180)
+		(at 50.8 92.71 180)
 		(descr "Capacitor SMD 1210 (3225 Metric), square (rectangular) end terminal, IPC-7351 nominal with elongated pad for handsoldering. (Body size source: IPC-SM-782 page 76, https://www.pcb-3d.com/wordpress/wp-content/uploads/ipc-sm-782a_amendment_1_and_2.pdf), generated with kicad-footprint-generator")
 		(tags "capacitor handsolder")
@@
 	(footprint "WE-SL575:WE-SL575"
 		(layer "F.Cu")
-		(at 53.5725 82.55 -90)
+		(at 50.8 82.55 -90)
 		(descr "WE-SL575")
 		(tags "Inductor")
@@
 		)
 		(fp_text user "${REFERENCE}"
-			(at -6.985 3.81 180)
+			(at -6.985 3.81 0)
 			(layer "F.Fab")
 			(effects
@@
 			)
 		)
-		(pad "1" smd rect
-			(at 3.81 -3.11)
-			(size 2.7 2.7)
-			(layers "F.Cu" "F.Mask" "F.Paste")
+		(pad "1" thru_hole rect
+			(at 3.81 -3.175 270)
+			(size 3 3)
+			(drill oval 0.9 1.8)
+			(layers "*.Cu" "*.Mask")
+			(remove_unused_layers no)
 			(net 46 "Net-(C2-Pad1)")
 			(pintype "passive")
 		)
+		(pad "2" thru_hole oval
+			(at -6.19 -3.175 270)
+			(size 2 3)
+			(drill oval 0.9 1.8)
+			(layers "*.Cu" "*.Mask")
+			(remove_unused_layers no)
+			(net 48 "Net-(U6-+VIN)")
+			(pintype "passive")
+		)
 		(pad "2" smd rect
 			(at -3.81 -3.11)
@@
 			(pintype "passive")
 		)
+		(pad "3" thru_hole oval
+			(at -6.19 9.325 270)
+			(size 2 3)
+			(drill oval 0.9 1.8)
+			(layers "*.Cu" "*.Mask")
+			(remove_unused_layers no)
+			(net 49 "Net-(U6--VIN)")
+			(pintype "passive")
+		)
 		(pad "3" smd rect
 			(at -3.81 3.11)
@@
 			(pintype "passive")
 		)
+		(pad "4" thru_hole oval
+			(at 3.81 9.325 270)
+			(size 2 3)
+			(drill oval 0.9 1.8)
+			(layers "*.Cu" "*.Mask")
+			(remove_unused_layers no)
+			(net 47 "Net-(C2-Pad2)")
+			(pintype "passive")
+		)
 		(embedded_fonts no)
 		(model "${KIPRJMOD}/Components/3dmodels/744272471.3dshapes/744272471.stp"
@@
 	(footprint "Capacitor_SMD:C_1210_3225Metric_Pad1.33x2.70mm_HandSolder"
 		(layer "F.Cu")
-		(at 53.5725 73.66 180)
+		(at 50.8 69.85 180)
 		(descr "Capacitor SMD 1210 (3225 Metric), square (rectangular) end terminal, IPC-7351 nominal with elongated pad for handsoldering. (Body size source: IPC-SM-782 page 76, https://www.pcb-3d.com/wordpress/wp-content/uploads/ipc-sm-782a_amendment_1_and_2.pdf), generated with kicad-footprint-generator")
 		(tags "capacitor handsolder")
@@
 	(footprint "Connector_PinSocket_2.54mm_LongPads:PinSocket_1x04_P2.54mm_Vertical_LongPdas"
 		(layer "F.Cu")
-		(at 53.5725 97.79)
+		(at 50.8 97.79)
 		(descr "Through hole straight socket strip, 1x04, 2.54mm pitch, single row (from Kicad 4.0.7), script generated")
 		(tags "Through hole socket strip THT 1x04 2.54mm single row")
@@
 	)
 	(segment
-		(start 52.9375 113.03)
-		(end 53.5725 113.03)
+		(start 50.165 113.03)
+		(end 50.8 113.03)
 		(width 0.4)
 		(layer "F.Cu")
@@
 	)
 	(segment
-		(start 51.0325 119.63)
-		(end 51.0325 114.3)
+		(start 48.0275 114.5325)
+		(end 49.53 113.03)
 		(width 1)
 		(layer "F.Cu")
@@
 	)
 	(segment
-		(start 52.3025 113.03)
-		(end 53.5725 113.03)
-		(width 1.6)
+		(start 48.0275 119.3975)
+		(end 48.0275 114.5325)
+		(width 1)
 		(layer "F.Cu")
 		(net 9)
 	)
 	(segment
-		(start 52.0525 120.65)
-		(end 51.0325 119.63)
-		(width 1)
+		(start 49.53 113.03)
+		(end 50.8 113.03)
+		(width 1.6)
 		(layer "F.Cu")
 		(net 9)
 	)
 	(segment
-		(start 51.0325 114.3)
-		(end 52.3025 113.03)
+		(start 49.28 120.65)
+		(end 48.0275 119.3975)
 		(width 1)
 		(layer "F.Cu")
@@
 	)
 	(segment
-		(start 53.5725 120.65)
-		(end 52.0525 120.65)
+		(start 50.8 120.65)
+		(end 49.28 120.65)
 		(width 1.6)
 		(layer "F.Cu")
@@
 	)
 	(segment
-		(start 57.3825 100.33)
-		(end 57.3825 110.49)
+		(start 54.3775 110.7225)
+		(end 52.07 113.03)
 		(width 1)
 		(layer "In2.Cu")
@@
 	)
 	(segment
-		(start 54.8425 97.79)
-		(end 57.3825 100.33)
+		(start 52.07 97.79)
+		(end 54.3775 100.0975)
 		(width 1)
 		(layer "In2.Cu")
@@
 	)
 	(segment
-		(start 53.5725 97.79)
-		(end 54.8425 97.79)
+		(start 50.8 97.79)
+		(end 52.07 97.79)
 		(width 1.6)
 		(layer "In2.Cu")
@@
 	)
 	(segment
-		(start 54.8425 113.03)
-		(end 53.5725 113.03)
+		(start 52.07 113.03)
+		(end 50.8 113.03)
 		(width 1.6)
 		(layer "In2.Cu")
@@
 	)
 	(segment
-		(start 57.3825 110.49)
-		(end 54.8425 113.03)
+		(start 54.3775 100.0975)
+		(end 54.3775 110.7225)
 		(width 1)
 		(layer "In2.Cu")
@@
 	)
 	(segment
-		(start 54.8425 118.11)
-		(end 53.5725 118.11)
-		(width 1.6)
+		(start 52.07 110.49)
+		(end 54.3775 112.7975)
+		(width 1)
 		(layer "F.Cu")
 		(net 10)
 	)
 	(segment
-		(start 57.3825 113.03)
-		(end 57.3825 115.57)
+		(start 54.3775 112.7975)
+		(end 54.3775 115.8025)
 		(width 1)
 		(layer "F.Cu")
@@
 	)
 	(segment
-		(start 53.5725 110.49)
-		(end 54.8425 110.49)
+		(start 52.07 118.11)
+		(end 50.8 118.11)
 		(width 1.6)
 		(layer "F.Cu")
@@
 	)
 	(segment
-		(start 54.8425 110.49)
-		(end 57.3825 113.03)
+		(start 54.3775 115.8025)
+		(end 52.07 118.11)
 		(width 1)
 		(layer "F.Cu")
@@
 	)
 	(segment
-		(start 57.3825 115.57)
-		(end 54.8425 118.11)
-		(width 1)
+		(start 50.8 110.49)
+		(end 52.07 110.49)
+		(width 1.6)
 		(layer "F.Cu")
 		(net 10)
 	)
 	(segment
-		(start 51.0325 104.14)
-		(end 51.0325 109.22)
+		(start 48.0275 108.9875)
+		(end 49.53 110.49)
 		(width 1)
 		(layer "In2.Cu")
@@
 	)
 	(segment
-		(start 52.3025 102.87)
-		(end 51.0325 104.14)
+		(start 49.53 102.87)
+		(end 48.0275 104.3725)
 		(width 1)
 		(layer "In2.Cu")
@@
 	)
 	(segment
-		(start 52.3025 110.49)
-		(end 53.5725 110.49)
+		(start 49.53 110.49)
+		(end 50.8 110.49)
 		(width 1.6)
 		(layer "In2.Cu")
@@
 	)
 	(segment
-		(start 51.0325 109.22)
-		(end 52.3025 110.49)
-		(width 1)
+		(start 50.8 102.87)
+		(end 49.53 102.87)
+		(width 1.6)
 		(layer "In2.Cu")
 		(net 10)
 	)
 	(segment
-		(start 53.5725 102.87)
-		(end 52.3025 102.87)
-		(width 1.6)
+		(start 48.0275 104.3725)
+		(end 48.0275 108.9875)
+		(width 1)
 		(layer "In2.Cu")
 		(net 10)
@@
 	)
 	(segment
-		(start 53.5725 105.41)
-		(end 56.1125 105.41)
+		(start 50.8 105.41)
+		(end 53.34 105.41)
 		(width 1.6)
 		(layer "F.Cu")
@@
 	)
 	(segment
-		(start 53.5725 105.41)
-		(end 53.8265 105.41)
+		(start 50.8 105.41)
+		(end 51.054 105.41)
 		(width 0.4)
 		(layer "F.Cu")
@@
 	)
 	(segment
-		(start 53.5725 100.33)
-		(end 51.0325 100.33)
+		(start 50.8 100.33)
+		(end 48.26 100.33)
 		(width 1.6)
 		(layer "F.Cu")
@@
 	)
 	(segment
-		(start 53.5725 100.33)
-		(end 53.3185 100.33)
+		(start 50.8 100.33)
+		(end 50.546 100.33)
 		(width 0.4)
 		(layer "F.Cu")
@@
 	)
 	(segment
+		(start 53.975 78.675)
+		(end 53.91 78.74)
+		(width 0.6)
+		(layer "F.Cu")
+		(net 48)
+	)
+	(segment
 		(start 74.125 80.01)
 		(end 74.125 73.8925)
@@
 	)
 	(segment
+		(start 53.975 76.36)
+		(end 53.975 78.675)
+		(width 1.2)
+		(layer "F.Cu")
+		(net 48)
+	)
+	(segment
 		(start 67.5425 102.87)
 		(end 65.0025 102.87)
@@
 	)
 	(segment
+		(start 65.0025 67.31)
+		(end 62.23 67.31)
+		(width 1.2)
+		(layer "F.Cu")
+		(net 48)
+	)
+	(segment
+		(start 53.975 74.295)
+		(end 53.975 76.36)
+		(width 1.2)
+		(layer "F.Cu")
+		(net 48)
+	)
+	(segment
 		(start 67.5425 67.31)
 		(end 65.0025 67.31)
@@
 	)
 	(segment
+		(start 65.0025 62.23)
+		(end 62.23 62.23)
+		(width 1.2)
+		(layer "F.Cu")
+		(net 49)
+	)
+	(segment
 		(start 74.125 91.2075)
 		(end 67.5425 97.79)
@@
 		(polygon
 			(pts
-				(xy 59.2875 78.994) (xy 54.2075 78.994) (xy 54.2075 67.945) (xy 55.4775 66.675) (xy 56.7475 65.405)
-				(xy 65.3835 65.405) (xy 65.3835 69.215) (xy 59.2875 69.215)
+				(xy 56.515 78.994) (xy 51.435 78.994) (xy 51.435 67.945) (xy 52.705 66.675) (xy 53.975 65.405) (xy 63.5 65.405)
+				(xy 64.516 66.04) (xy 64.516 68.58) (xy 63.5 69.215) (xy 56.515 69.215)
 			)
 		)
@@
 		(polygon
 			(pts
-				(xy 47.8575 86.106) (xy 52.9375 86.106) (xy 52.9375 95.885) (xy 51.6675 95.885) (xy 51.6675 99.06)
-				(xy 54.8425 99.06) (xy 54.8425 101.6) (xy 47.8575 101.6)
+				(xy 45.085 90.805) (xy 40.64 88.265) (xy 40.64 84.836) (xy 50.165 84.836) (xy 50.165 95.885) (xy 48.895 95.885)
+				(xy 48.895 99.06) (xy 52.07 99.06) (xy 52.07 101.6) (xy 45.085 101.6)
 			)
 		)
@@
 		(polygon
 			(pts
-				(xy 53.3185 78.994) (xy 53.3185 67.31) (xy 56.3665 64.262) (xy 63.3515 64.262) (xy 65.0025 62.611)
-				(xy 65.0025 61.849) (xy 63.3515 60.198) (xy 52.6835 60.198) (xy 47.8575 65.024) (xy 47.8575 78.994)
+				(xy 42.545 77.724) (xy 43.815 78.994) (xy 50.546 78.994) (xy 50.546 67.31) (xy 53.594 64.262) (xy 63.5 64.262)
+				(xy 64.77 62.611) (xy 64.77 61.849) (xy 63.5 60.198) (xy 49.911 60.198) (xy 45.085 65.024) (xy 45.085 72.39)
+				(xy 40.64 74.295) (xy 40.64 77.724)
 			)
 		)
@@
 		(polygon
 			(pts
-				(xy 59.2875 86.106) (xy 54.2075 86.106) (xy 54.2075 95.885) (xy 55.4775 95.885) (xy 55.4775 104.14)
-				(xy 52.3025 104.14) (xy 52.3025 106.68) (xy 59.2875 106.68)
+				(xy 56.515 86.106) (xy 51.435 86.106) (xy 51.435 95.885) (xy 52.705 95.885) (xy 52.705 104.14) (xy 49.53 104.14)
+				(xy 49.53 106.68) (xy 56.515 106.68)
 			)
 		)

Commit message: final PCB Update
Parts:
- removed the C116 at (101.9, 112.4)
- removed the Z257 at (100.8, 108.0)
- removed the Z259 at (100.8, 69.8)
- added C114: 10u, Capacitor_THT:CP_Radial_D5.0mm_P2.50mm, F.Cu at (101.9, 113.0)
- added Z241: ~, Resistor_SMD:R_0805_2012Metric_Pad1.20x1.40mm_HandSolder, F.Cu at (100.8, 69.8)
- added Z255: ~, Resistor_SMD:R_0805_2012Metric_Pad1.20x1.40mm_HandSolder, F.Cu at (100.8, 108.0)
- renumbered C112 to C100, C36 to C101, C24 to C102, C10 to C103, C11 to C110, C25 to C111, C4 to C112, C19 to C113, C2 to C115, C5 to C116, C20 to C117, C117 to C118, C6 to C119, C26 to C120, C12 to C121, C9 to C84, C115 to C85, C23 to C86, C46 to C87, C56 to C88, C113 to C89, C18 to C90, C114 to C91, C47 to C92, C57 to C93, D2 to D1, D1 to D2, D3 to D4, H4 to H10, H8 to H11, H5 to H12, H2 to H13, H3 to H14, H6 to H15, H7 to H16, H1 to H9, J30 to J33, J36 to J34, J31 to J35, J32 to J36, J34 to J37, J10 to J39, J21 to J40, J13 to J41, J33 to J42, J11 to J43, L2 to L1, L3 to L2, L4 to L3, L1 to L4, R67 to R141, R71 to R142, R81 to R143, R86 to R144, R59 to R145, R60 to R146, R68 to R147, R82 to R148, R84 to R149, R72 to R150, R75 to R151, SW9 to SW11, SW1 to SW12, U6 to U25, U7 to U26, Z130 to Z237, Z122 to Z238, Z126 to Z239, Z134 to Z240, Z167 to Z242, Z172 to Z243, Z131 to Z244, Z170 to Z245, Z123 to Z246, Z127 to Z247, Z135 to Z248, Z132 to Z249, Z168 to Z250, Z173 to Z251, Z124 to Z252, Z128 to Z253, Z136 to Z254, Z171 to Z256, Z174 to Z257, Z133 to Z259, Z125 to Z260, Z129 to Z261, Z137 to Z262
Routing:
- net GND_M: track 59.1 -> 32.2 mm
- net 9V_GND_M: track 50.5 -> 36.7 mm
- net +15V_M: track 31.4 -> 20.0 mm
- net -15V_M: track 20.7 -> 9.42 mm
- net Net-(R141-Pad1): track 3.81 -> 0.00 mm
