File: KiCad/Power_Supply_Meter_Amp.kicad_sch (KiCad schematic)
At the start: 629 parts, among them J1 R_Phono_In, J10 VCC_IN, J11 VCC_OUT, J12 EMK_In, J13 EMK_Out, J14 EMK_Out, J15 Mic_Effekt_Out, J16 Mic_Effekt_Out, J17 Mic_Effekt_Out, J18 Mic_Effekt_Out, J19 Phono/Line_Out, J2 L_Phono_In, J20 Mic_Effekt_Out, J21 EMK_Out, J22 EMK_In, J23 EMK_In, J24 Mic_Effekt_In, J25 Mic_Effekt_In, J26 Phono/Line_In, J27 Mic_Effekt_In, J28 Pegel_Out, J29 Pegel_Out, J3 R_Line_In, J30 Pegel_In, J31 Pegel_In, J32 Pegel_In, J33 Pegel_In, J34 LED_Out, J35 LED_In, J36 VU_Meter_Out, J37 AUX_Send_3, J38 AUX_Send_1, J39 AUX_Send_2, J4 L_Line_In, J40 Bass_Out, J41 Kick_Out, J42 Mid_Out, J43 High_Out, J44 Line_Out_L, J45 Line_Out_R, J5 Mic_In, J6 Effekt_In, J7 AUX_RET_1, J8 AUX_RET_2, J9 AUX_RET_3, SW1 SW_DPST, SW10 SW_SPDT, SW11 SW_SPDT, SW12 SW_SPDT, SW2 SW_SPDT, SW3 SW_SPDT, SW4 SW_SPDT, SW5 SW_SPDT, SW6 SW_SPDT, SW7 SW_SPDT, SW8 SW_SPDT, SW9 SW_Rotary_1x4, U1 TL074, U10 TL074, U11 TL074, U12 TL074, U13 TL074, U14 TL074, U15 TL074, U16 TL074, U17 TL074, U18 TL074, U19 TL074, U2 TL074, U20 TL074, U21 TL074, U22 TL074, U23 TL074, U24 TL074, U25 INA128U, U3 TL074, U4 TL074, U5 TL074, U6 REC10K-2409, U7 REC10K-2415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

Commit message: PCB Update Power Supply VU Amp
Parts:
- removed L1: 470uF, 1.6A, WE-SL575:WE-SL575, symbol Device:L_Coupled
- added L1: Choke_Wurth_WE-CNSW_744232090, Inductor_THT:L_CommonMode_Wuerth_WE-CMB-M, symbol Filter:Choke_Wurth_WE-CNSW_744232090
- C1, C13, C14, C15, C16, C17, C21, C22, C27, C28, C29, C3, C30, C31, C32, C33, C34, C7, C8, J1, J12, J15, J16, J17, J18, J19, J2, J20, J3, J4, J5, J6, J7, J8, J9, R1, R10, R11, R12, R13, R14, R15, R16, R17, R18, R19, R2, R20, R21, R22, R23, R24, R28, R29, R3, R30, R31, R32, R4, R5, R6, R7, R8, R9, RV1, RV2, RV3, RV4, RV5, RV6, SW2, U1, U2, U25, U3, U4, U5, Z1, Z10, Z100, Z11, Z12, Z13, Z14, Z15, Z16, Z17, Z18, Z19, Z2, Z20, Z21, Z22, Z23, Z24, Z25, Z26, Z27, Z28, Z29, Z3, Z30, Z31, Z32, Z33, Z34, Z35, Z36, Z37, Z38, Z39, Z4, Z40, Z41, Z42, Z43, Z44, Z45, Z46, Z47, Z48, Z49, Z5, Z50, Z51, Z52, Z53, Z54, Z55, Z56, Z57, Z58, Z59, Z6, Z60, Z61, Z62, Z63, Z64, Z65, Z66, Z67, Z68, Z69, Z7, Z70, Z71, Z72, Z73, Z74, Z75, Z76, Z77, Z78, Z79, Z8, Z80, Z81, Z82, Z83, Z84, Z85, Z86, Z87, Z88, Z89, Z9, Z90, Z91, Z92, Z93, Z94, Z95, Z96, Z97, Z98, Z99: now not fitted; now left out of the parts list
- C10, C11, C18, C19, C20, C23, C24, C25, C26, C36, C4, C46, C47, C56, C57, C6, C9, D1, D2, D3, J10, J11, J13, J14, J21, J30, J31, J32, J33, J34, J36, L2, L3, L4, L5, R25, R26, R27, R59, R60, R67, R68, R71, R72, R75, R81, R82, R84, R86, SW1, SW9, U23, U24, U6, U7, Z122, Z123, Z124, Z125, Z126, Z127, Z128, Z129, Z130, Z131, Z132, Z133, Z134, Z135, Z136, Z137, Z167, Z168, Z170, Z171, Z172, Z173, Z174: now fitted; now in the parts list
- C2, C5: footprint Capacitor_SMD:C_0805_2012Metric_Pad1.18x1.45mm_HandSolder -> Capacitor_SMD:C_1210_3225Metric_Pad1.33x2.70mm_HandSolder; now fitted; now in the parts list
Connections:
- net at C2.1, SW1.4: now also L1.1
- net at C11.1, C4.2, C5.1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: now also L1.2
- net at C2.2, SW1.2: now also L1.4
- net at C10.1, C12.1, C5.2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: now also L1.3

Commit message: PCB Update
Parts:
- removed J21: EMK_Out, Connector_PinSocket_2.54mm_LongPads:PinSocket_1x05_P2.54mm_Vertical_LongPads, symbol Connector:Conn_01x05_Socket
- removed J23: EMK_In, Connector_PinHeader_2.54mm_LongPads:PinHeader_1x05_P2.54mm_Vertical_LongPads, symbol Connector:Conn_01x05_Pin
- removed L1: Choke_Wurth_WE-CNSW_744232090, Inductor_THT:L_CommonMode_Wuerth_WE-CMB-M, symbol Filter:Choke_Wurth_WE-CNSW_744232090
- added C112, C113: 10n, Capacitor_SMD:C_0805_2012Metric_Pad1.18x1.45mm_HandSolder, symbol Device:C_Small
- added J21: Conn_01x05_bridged, Connector_Bridged_2.54mm_LongPads:Bridge_2x05_P2.54mm_Vertical_LongPads, symbol conn_01x05_bridged:Conn_01x05_bridged
- added L1: ~, WE-SL575:WE-SL575, symbol Common_Mode_Choke:Common_Mode_Choke
- L2, L3, L4, L5: footprint Connector_PinSocket_2.54mm_LongPads:PinSocket_1x02_P2.54mm_Vertical_LongPads -> Inductor_SMD:L_1206_3216Metric
Connections:
- net +15V: no longer C46.2, C56.2, J13.3 (Pin_3), J14.3 (Pin_3), R26.1, U23.4 (V+), U24.4 (V+)
- net +9V: no longer J13.1 (Pin_1), J14.1 (Pin_1), J36.3 (Pin_3), R25.1
- net -15V: no longer C47.2, C57.2, J13.4 (Pin_4), J14.4 (Pin_4), R27.1, U23.11 (V-), U24.11 (V-)
- net 9V_GND: no longer C10.2, C18.2, C24.1, J13.2 (Pin_2), J14.2 (Pin_2), J36.4 (Pin_4), L3.2
- net GND: no longer C19.2, C20.1, C36.2, D3.2 (A), J13.5 (Pin_5), J14.5 (Pin_5), J36.2 (Pin_2), R75.1, R86.1, U24.3 (+), U24.5 (+), U7.5 (COM), Z122.2, Z123.2, Z124.2, Z125.2, Z126.2, Z127.2, Z128.2, Z129.2, Z134.2, Z135.2, Z136.2, Z137.2, Z170.2, Z171.2, Z174.2
- net at C10.1, C12.1, C5.2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: now also C112.1, L1.3
- net at C2.1, SW1.4: now also L1.1
- net at C2.2, SW1.2: now also L1.4
- net at C11.1, C4.2, C5.1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: now also C113.2, L1.2
- net FILT_GND renamed GND_15V_FILT
- net GND_15V_FILT: no longer C23.1, C24.2
- new net +15V_M: C46.2, C56.2, J21.8 (Pin_3), U23.4 (V+), U24.4 (V+)
- new net +15V_P: J13.3 (Pin_3), J14.3 (Pin_3), J21.3 (Pin_3), R26.1
- new net +9V_M: J21.10 (Pin_1), J36.3 (Pin_3)
- new net +9V_P: J13.1 (Pin_1), J14.1 (Pin_1), J21.1 (Pin_1), R25.1
- new net -15V_M: C47.2, C57.2, J21.7 (Pin_4), U23.11 (V-), U24.11 (V-)
- new net -15V_P: J13.4 (Pin_4), J14.4 (Pin_4), J21.4 (Pin_4), R27.1
- new net 9V_GND_M: J21.9 (Pin_2), J36.4 (Pin_4)
- new net 9V_GND_P: C10.2, C18.2, C24.1, J13.2 (Pin_2), J14.2 (Pin_2), J21.2 (Pin_2), L3.2
- new net GND_9V_FILT: C112.2, C113.1, C23.1, C24.2
- new net GND_M: C36.2, D3.2 (A), J21.6 (Pin_5), J36.2 (Pin_2), R75.1, R86.1, U24.3 (+), U24.5 (+), Z122.2, Z123.2, Z124.2, Z125.2, Z126.2, Z127.2, Z128.2, Z129.2, Z134.2, Z135.2, Z136.2, Z137.2, Z170.2, Z171.2, Z174.2
- new net GND_P: C19.2, C20.1, J13.5 (Pin_5), J14.5 (Pin_5), J21.5 (Pin_5), U7.5 (COM)
Other:
- moved on the sheet: C2, C24, C25, C26, C4, C5, C6, J10, J11, SW1

Commit message: PCB Update
Connections:
- net +15V: now also J12.5 (Pin_5), J22.5 (Pin_5); no longer J12.3 (Pin_3), J22.3 (Pin_3)
- net +15V_M: now also J21.6 (Pin_5); no longer J21.8 (Pin_3)
- net +15V_P: now also J13.5 (Pin_5), J14.5 (Pin_5), J21.5 (Pin_5); no longer J13.3 (Pin_3), J14.3 (Pin_3), J21.3 (Pin_3)
- net +9V: now also J12.2 (Pin_2), J22.2 (Pin_2); no longer J12.1 (Pin_1), J22.1 (Pin_1)
- net +9V_M: now also J21.9 (Pin_2); no longer J21.10 (Pin_1)
- net +9V_P: now also J13.2 (Pin_2), J14.2 (Pin_2), J21.2 (Pin_2); no longer J13.1 (Pin_1), J14.1 (Pin_1), J21.1 (Pin_1)
- net -15V: now also J12.3 (Pin_3), J22.3 (Pin_3); no longer J12.4 (Pin_4), J22.4 (Pin_4)
- net -15V_M: now also J21.8 (Pin_3); no longer J21.7 (Pin_4)
- net -15V_P: now also J13.3 (Pin_3), J14.3 (Pin_3), J21.3 (Pin_3); no longer J13.4 (Pin_4), J14.4 (Pin_4), J21.4 (Pin_4)
- net 9V_GND: now also J12.1 (Pin_1), J22.1 (Pin_1); no longer J12.2 (Pin_2), J22.2 (Pin_2)
- net 9V_GND_M: now also J21.10 (Pin_1); no longer J21.9 (Pin_2)
- net 9V_GND_P: now also J13.1 (Pin_1), J14.1 (Pin_1), J21.1 (Pin_1); no longer J13.2 (Pin_2), J14.2 (Pin_2), J21.2 (Pin_2)
- net GND: now also J12.4 (Pin_4), J22.4 (Pin_4); no longer J12.5 (Pin_5), J22.5 (Pin_5)
- net GND_M: now also J21.7 (Pin_4); no longer J21.6 (Pin_5)
- net GND_P: now also J13.4 (Pin_4), J14.4 (Pin_4), J21.4 (Pin_4); no longer J13.5 (Pin_5), J14.5 (Pin_5), J21.5 (Pin_5)

Commit message: PCB Update
Parts:
- renumbered U24 to U23, U23 to U24
Connections:
- net GND_M: now also U23.10 (+), U23.12 (+); no longer U23.3 (+), U23.5 (+)
- net Pegel_Aux_Return: now also U24.1, U24.2 (-); no longer U24.8, U24.9 (-)
- net Pegel_Post: now also U24.6 (-), U24.7; no longer U24.13 (-), U24.14
- net at Z133.2, Z137.1: now also U24.5 (+); no longer U24.12 (+)
- net at D1.1 (K), R59.2, R60.1: now also U23.9 (-); no longer U23.2 (-)
- net at Z132.2, Z136.1: now also U24.3 (+); no longer U24.10 (+)
- net at D1.2 (A), D2.1 (K): now also U23.8; no longer U23.1
- net at R67.2, R68.2, R71.1: now also U23.13 (-); no longer U23.6 (-)
- net at R71.2, U24.10 (+), U24.12 (+): now also U23.14; no longer U23.7
Changed lines of the file:
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@@
 		(lib_id "Amplifier_Operational:TL074")
 		(at 438.15 541.02 0)
-		(unit 3)
+		(unit 1)
 		(exclude_from_sim no)
 		(in_bom yes)
 		(on_board yes)
 		(dnp no)
-		(property "Reference" "U23"
+		(property "Reference" "U24"
 			(at 438.15 530.86 0)
 			(effects
@@
 			(project ""
 				(path "/81a92cd6-862a-4567-ad33-f8a3bc120591"
-					(reference "U23")
-					(unit 3)
+					(reference "U24")
+					(unit 1)
 				)
 			)
@@
 		(at 509.27 544.83 0)
 		(mirror x)
-		(unit 1)
+		(unit 3)
 		(exclude_from_sim no)
 		(in_bom yes)
 		(on_board yes)
 		(dnp no)
-		(property "Reference" "U24"
+		(property "Reference" "U23"
 			(at 509.27 534.67 0)
 			(effects
@@
 			(project ""
 				(path "/81a92cd6-862a-4567-ad33-f8a3bc120591"
-					(reference "U24")
-					(unit 1)
+					(reference "U23")
+					(unit 3)
 				)
 			)
@@
 		(lib_id "Amplifier_Operational:TL074")
 		(at 438.15 562.61 0)
-		(unit 4)
+		(unit 2)
 		(exclude_from_sim no)
 		(in_bom yes)
@@
 		(dnp no)
 		(fields_autoplaced yes)
-		(property "Reference" "U23"
+		(property "Reference" "U24"
 			(at 438.15 552.45 0)
 			(effects
@@
 			(project "DiKo_PreAmp"
 				(path "/81a92cd6-862a-4567-ad33-f8a3bc120591"
-					(reference "U23")
-					(unit 4)
+					(reference "U24")
+					(unit 2)
 				)
 			)
@@
 		(at 544.83 524.51 0)
 		(mirror x)
-		(unit 2)
+		(unit 4)
 		(exclude_from_sim no)
 		(in_bom yes)
 		(on_board yes)
 		(dnp no)
-		(property "Reference" "U24"
+		(property "Reference" "U23"
 			(at 544.83 534.67 0)
 			(effects
@@
 			(project ""
 				(path "/81a92cd6-862a-4567-ad33-f8a3bc120591"
-					(reference "U24")
-					(unit 2)
+					(reference "U23")
+					(unit 4)
 				)
 			)

Commit message: PCB Update
Connections:
- net +15V: no longer R72.1
- net +15V_M: now also R72.1
- net GND_M: now also U23.10 (+), U23.12 (+); no longer U23.10 (+), U23.12 (+)
- net Pegel_Aux_Return: now also SW9.2; no longer SW9.3
- net Pegel_Mic_Effekt: now also SW9.3; no longer SW9.2
- net Pegel_Post: now also SW9.1; no longer SW9.4
- net Pegel_Pre: now also SW9.4; no longer SW9.1
- net at D1.1 (K), R59.2, R60.1: now also U23.13 (-); no longer U23.9 (-)
- net at D1.2 (A), D2.1 (K): now also U23.14; no longer U23.8
- net at R67.2, R68.2, R71.1: now also U23.9 (-); no longer U23.13 (-)
- net at R71.2, U24.10 (+), U24.12 (+): now also U23.8; no longer U23.14
Changed lines of the file:
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@@
 		(on_board yes)
 		(dnp no)
-		(fields_autoplaced yes)
 		(property "Reference" "#PWR0176"
 			(at 552.45 563.88 0)
@@
 		)
 		(property "Value" "GND_M"
-			(at 552.45 562.61 0)
+			(at 552.958 562.61 0)
 			(effects
 				(font
@@
 		(at 509.27 544.83 0)
 		(mirror x)
-		(unit 3)
+		(unit 4)
 		(exclude_from_sim no)
 		(in_bom yes)
@@
 				(path "/81a92cd6-862a-4567-ad33-f8a3bc120591"
 					(reference "U23")
-					(unit 3)
+					(unit 4)
 				)
 			)
@@
 		(on_board yes)
 		(dnp no)
-		(fields_autoplaced yes)
 		(property "Reference" "#PWR0174"
 			(at 546.1 553.72 0)
@@
 			)
 		)
-		(property "Value" "+15V"
-			(at 546.1 562.61 0)
+		(property "Value" "+15V_M"
+			(at 545.084 562.61 0)
 			(effects
 				(font
@@
 		(at 544.83 524.51 0)
 		(mirror x)
-		(unit 4)
+		(unit 3)
 		(exclude_from_sim no)
 		(in_bom yes)
@@
 				(path "/81a92cd6-862a-4567-ad33-f8a3bc120591"
 					(reference "U23")
-					(unit 4)
+					(unit 3)
 				)
 			)

Commit message: PCB Update
Connections:
- net GND: no longer C46.1, C47.1, C56.1, C57.1
- net GND_M: now also C46.1, C47.1, C56.1, C57.1
Changed lines of the file:
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@@
 			)
 		)
-		(property "Value" "GND"
+		(property "Value" "GND_M"
 			(at 708.66 541.02 0)
 			(effects
@@
 			)
 		)
-		(property "Value" "GND"
+		(property "Value" "GND_M"
 			(at 690.88 541.02 0)
 			(effects

Commit message: PCB Update
Connections:
- net +9V_M: now also J36.4 (Pin_4); no longer J36.3 (Pin_3)
- net 9V_GND_M: now also J36.3 (Pin_3); no longer J36.4 (Pin_4)
Other:
- moved on the sheet: J36
Changed lines of the file:
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@@
 	(wire
 		(pts
-			(xy 637.54 525.78) (xy 637.54 520.7)
+			(xy 637.54 518.16) (xy 637.54 525.78)
 		)
 		(stroke
@@
 	(wire
 		(pts
-			(xy 637.54 520.7) (xy 641.35 520.7)
-		)
-		(stroke
-			(width 0)
-			(type default)
-		)
-	)
-	(wire
-		(pts
 			(xy 368.3 238.76) (xy 365.76 238.76)
 		)
@@
 	(wire
 		(pts
+			(xy 637.54 518.16) (xy 650.24 518.16)
+		)
+		(stroke
+			(width 0)
+			(type default)
+		)
+	)
+	(wire
+		(pts
 			(xy 487.68 283.21) (xy 490.22 283.21)
 		)
@@
 	(wire
 		(pts
-			(xy 618.49 513.08) (xy 641.35 513.08)
+			(xy 618.49 513.08) (xy 650.24 513.08)
 		)
 		(stroke
@@
 	(wire
 		(pts
-			(xy 628.65 515.62) (xy 641.35 515.62)
+			(xy 628.65 515.62) (xy 650.24 515.62)
 		)
 		(stroke
@@
 	(symbol
 		(lib_id "Connector:Conn_01x04_Socket")
-		(at 646.43 515.62 0)
+		(at 655.32 515.62 0)
 		(unit 1)
 		(exclude_from_sim no)
@@
 		(dnp no)
 		(property "Reference" "J36"
-			(at 640.334 506.984 0)
+			(at 649.224 506.984 0)
 			(effects
 				(font
@@
 		)
 		(property "Value" "VU_Meter_Out"
-			(at 640.334 509.524 0)
+			(at 649.224 509.524 0)
 			(effects
 				(font
@@
 		)
 		(property "Footprint" "Connector_PinSocket_2.54mm_LongPads:PinSocket_1x04_P2.54mm_Vertical_LongPdas"
-			(at 646.43 515.62 0)
+			(at 655.32 515.62 0)
 			(effects
 				(font
@@
 		)
 		(property "Datasheet" "~"
-			(at 646.43 515.62 0)
+			(at 655.32 515.62 0)
 			(effects
 				(font
@@
 		)
 		(property "Description" "Generic connector, single row, 01x04, script generated"
-			(at 646.43 515.62 0)
+			(at 655.32 515.62 0)
 			(effects
 				(font
@@
 	(symbol
 		(lib_id "power:VCC")
-		(at 641.35 518.16 90)
+		(at 650.24 520.7 90)
 		(unit 1)
 		(exclude_from_sim no)
@@
 		(fields_autoplaced yes)
 		(property "Reference" "#PWR0197"
-			(at 645.16 518.16 0)
+			(at 654.05 520.7 0)
 			(effects
 				(font
@@
 		)
 		(property "Value" "+9V_M"
-			(at 637.54 518.1599 90)
+			(at 646.43 520.6999 90)
 			(effects
 				(font
@@
 		)
 		(property "Footprint" ""
-			(at 641.35 518.16 0)
+			(at 650.24 520.7 0)
 			(effects
 				(font
@@
 		)
 		(property "Datasheet" ""
-			(at 641.35 518.16 0)
+			(at 650.24 520.7 0)
 			(effects
 				(font
@@
 		)
 		(property "Description" "Power symbol creates a global label with name \"VCC\""
-			(at 641.35 518.16 0)
+			(at 650.24 520.7 0)
 			(effects
 				(font

Commit message: PCB Update
Parts:
- removed J12, J22: EMK_In, Connector_PinHeader_2.54mm_LongPads:PinHeader_1x05_P2.54mm_Vertical_LongPads, symbol Connector:Conn_01x05_Pin
- removed J13, J14: EMK_Out, Connector_PinSocket_2.54mm_LongPads:PinSocket_1x05_P2.54mm_Vertical_LongPads, symbol Connector:Conn_01x05_Socket
- added C115: 10n, Capacitor_SMD:C_1210_3225Metric_Pad1.33x2.70mm_HandSolder, symbol Device:C_Small
- added H1, H2, H3, H4, H6, H7, H8: MountingHole, MountingHole:MountingHole_3.2mm_M3_Pad, symbol Mechanical:MountingHole
- added H5: MountingHole_Pad, MountingHole:MountingHole_3.2mm_M3_Pad, symbol Mechanical:MountingHole_Pad
Connections:
- net GND_M: now also C115.2
- new net: C115.1, H5.1
