File: KiCad/Power_Supply_Meter_Amp.kicad_sch (KiCad schematic)
At the start: 635 parts, among them J1 R_Phono_In, J10 VCC_IN, J11 VCC_OUT, J15 Mic_Effekt_Out, J16 Mic_Effekt_Out, J17 Mic_Effekt_Out, J18 Mic_Effekt_Out, J19 Phono/Line_Out, J2 L_Phono_In, J20 Mic_Effekt_Out, J21 Conn_01x05_bridged, J24 Mic_Effekt_In, J25 Mic_Effekt_In, J26 Phono/Line_In, J27 Mic_Effekt_In, J28 Pegel_Out, J29 Pegel_Out, J3 R_Line_In, J30 Pegel_In, J31 Pegel_In, J32 Pegel_In, J33 Pegel_In, J34 LED_Out, J35 LED_In, J36 VU_Meter_Out, J37 AUX_Send_3, J38 AUX_Send_1, J39 AUX_Send_2, J4 L_Line_In, J40 Bass_Out, J41 Kick_Out, J42 Mid_Out, J43 High_Out, J44 Line_Out_L, J45 Line_Out_R, J5 Mic_In, J6 Effekt_In, J7 AUX_RET_1, J8 AUX_RET_2, J9 AUX_RET_3, SW1 SW_DPST, SW10 SW_SPDT, SW11 SW_SPDT, SW12 SW_SPDT, SW2 SW_SPDT, SW3 SW_SPDT, SW4 SW_SPDT, SW5 SW_SPDT, SW6 SW_SPDT, SW7 SW_SPDT, SW8 SW_SPDT, SW9 SW_Rotary_1x4, U1 TL074, U10 TL074, U11 TL074, U12 TL074, U13 TL074, U14 TL074, U15 TL074, U16 TL074, U17 TL074, U18 TL074, U19 TL074, U2 TL074, U20 TL074, U21 TL074, U22 TL074, U23 TL074, U24 TL074, U25 INA128U, U3 TL074, U4 TL074, U5 TL074, U6 REC10K-2409, U7 REC10K-2415, U8 TL074, U9 TL074

Commit message: PCB Update
Parts:
- added J12, J22: EMK_In, Connector_PinHeader_2.54mm_LongPads:PinHeader_1x05_P2.54mm_Vertical_LongPads, symbol Connector:Conn_01x05_Pin
Connections:
- net +15V: now also J22.5 (Pin_5)
- net -15V: now also J22.3 (Pin_3)
- net GND: now also J22.4 (Pin_4)
- new net +15V_I: J12.5 (Pin_5)
- new net +9V: J22.2 (Pin_2)
- new net +9V_I: J12.2 (Pin_2)
- new net -15V_I: J12.3 (Pin_3)
- new net 9V_GND: J22.1 (Pin_1)
- new net 9V_GND_I: J12.1 (Pin_1)
- new net GND_I: J12.4 (Pin_4)
Other:
- moved on the sheet: R25

Commit message: PCB Update
Changed lines of the file:
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@@
 	(wire
 		(pts
+			(xy 637.54 518.16) (xy 650.24 518.16)
+		)
+		(stroke
+			(width 0)
+			(type default)
+		)
+	)
+	(wire
+		(pts
 			(xy 781.05 105.41) (xy 781.05 104.14)
 		)
@@
 	(wire
 		(pts
-			(xy 637.54 518.16) (xy 650.24 518.16)
-		)
-		(stroke
-			(width 0)
-			(type default)
-		)
-	)
-	(wire
-		(pts
 			(xy 487.68 283.21) (xy 490.22 283.21)
 		)
@@
 		(lib_id "Device:R")
 		(at 584.2 519.43 0)
+		(mirror y)
 		(unit 1)
 		(exclude_from_sim no)
@@
 		(dnp no)
 		(property "Reference" "Z170"
-			(at 587.248 519.43 90)
+			(at 581.152 519.43 90)
 			(effects
 				(font
@@
 		)
 		(property "Value" "~"
-			(at 588.01 519.43 90)
+			(at 580.39 519.43 90)
 			(effects
 				(font
@@
 		)
 		(property "Footprint" "Resistor_SMD:R_0805_2012Metric_Pad1.20x1.40mm_HandSolder"
-			(at 582.422 519.43 90)
+			(at 585.978 519.43 90)
 			(effects
 				(font
@@
 		(on_board yes)
 		(dnp no)
-		(fields_autoplaced yes)
 		(property "Reference" "R75"
 			(at 554.99 549.9099 0)

Commit message: PCB Update
Parts:
- removed R25, R26, R27: 22R, Resistor_SMD:R_0805_2012Metric_Pad1.20x1.40mm_HandSolder, symbol Device:R
- added C114, C116, C117: 10u, Capacitor_THT:CP_Radial_D5.0mm_P2.50mm, symbol Device:C_Polarized_Small
- added J13: Conn_02x07_Pin, symbol conn_02x07:Conn_02x07_Pin
- added Z257, Z258, Z259: ~, Resistor_SMD:R_0805_2012Metric_Pad1.20x1.40mm_HandSolder, symbol Device:R
Connections:
- net +15V_P: now also C116.1, Z257.2
- net +9V_P: now also C114.1, Z259.2
- net -15V_P: now also C117.2, Z258.2
- net 9V_GND_P: now also C114.2
- net GND_P: now also C116.2, C117.1
- net at C12.2, C20.2, C26.1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: now also Z258.1
- net at C11.2, C19.1, C25.2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: now also Z257.1
- net at C18.1, C23.2, C9.2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: now also Z259.1
Other:
- moved on the sheet: C23, C24, C25, C26

Commit message: PCB Final Update
Parts:
- removed J13: Conn_02x07_Pin, symbol conn_02x07:Conn_02x07_Pin
- removed J21: Conn_01x05_bridged, Connector_Bridged_2.54mm_LongPads:Bridge_2x05_P2.54mm_Vertical_LongPads, symbol conn_01x05_bridged:Conn_01x05_bridged
- added J13, J21: Conn_02x07_Odd_Even, Connector_PinHeader_2.54mm:PinHeader_2x07_P2.54mm_Vertical, symbol Connector_Generic:Conn_02x07_Odd_Even
- U25: footprint INA128U:INA128U_L -> D0008A_N
Connections:
- net +15V_M: now also J13.13 (Pin_13), J13.14 (Pin_14)
- net +15V_P: now also J21.13 (Pin_13), J21.14 (Pin_14)
- net +9V_M: now also J13.5 (Pin_5), J13.6 (Pin_6)
- net +9V_P: now also J21.5 (Pin_5), J21.6 (Pin_6)
- net -15V_M: now also J13.7 (Pin_7), J13.8 (Pin_8)
- net -15V_P: now also J21.7 (Pin_7), J21.8 (Pin_8)
- net 9V_GND_M: now also J13.1 (Pin_1), J13.2 (Pin_2), J13.3 (Pin_3), J13.4 (Pin_4)
- net 9V_GND_P: now also J21.1 (Pin_1), J21.2 (Pin_2), J21.3 (Pin_3), J21.4 (Pin_4)
- net GND_M: now also J13.10 (Pin_10), J13.11 (Pin_11), J13.12 (Pin_12), J13.9 (Pin_9)
- net GND_P: now also J21.10 (Pin_10), J21.11 (Pin_11), J21.12 (Pin_12), J21.9 (Pin_9)
Other:
- moved on the sheet: C46, C56, U23E, U24E

Commit message: final PCB Update
Parts:
- removed C116: 10u, Capacitor_THT:CP_Radial_D5.0mm_P2.50mm, symbol Device:C_Polarized_Small
- removed C7, C8: 100n, Capacitor_SMD:C_0805_2012Metric_Pad1.18x1.45mm_HandSolder, symbol Device:C_Small
- removed J12, J22: EMK_In, Connector_PinHeader_2.54mm_LongPads:PinHeader_1x05_P2.54mm_Vertical_LongPads, symbol Connector:Conn_01x05_Pin
- removed R2: 100R, Resistor_SMD:R_0805_2012Metric_Pad1.20x1.40mm_HandSolder, symbol Device:R
- removed SW10, SW11, SW12, SW3, SW4, SW5, SW6, SW7, SW8: SW_SPDT, Connector_PinHeader_2.54mm_LongPads:PinHeader_1x03_P2.54mm_Vertical_LongPads, symbol Switch:SW_SPDT
- removed unit 5 of U10
- removed unit 5 of U12
- removed unit 5 of U13
- removed unit 3 of U2
- removed U25: INA128U, D0008A_N, symbol INA128U:INA128U
- removed unit 3 of U4
- removed Z185, Z193, Z198: ~, Resistor_SMD:R_0805_2012Metric_Pad1.20x1.40mm_HandSolder, symbol Device:R_Small
- removed Z257, Z259: ~, Resistor_SMD:R_0805_2012Metric_Pad1.20x1.40mm_HandSolder, symbol Device:R
- added C114: 10u, Capacitor_THT:CP_Radial_D5.0mm_P2.50mm, symbol Device:C_Polarized_Small
- added C3, C4: 10n, Capacitor_SMD:C_1210_3225Metric_Pad1.33x2.70mm_HandSolder, symbol Device:C_Small
- added C52, C53, C59, C60: 100n, Capacitor_SMD:C_0805_2012Metric_Pad1.18x1.45mm_HandSolder, symbol Device:C_Small
- added H1, H2, H5, H6, H7, H8: MountingHole, MountingHole:MountingHole_3.2mm_M3_Pad, symbol Mechanical:MountingHole
- added H3, H4: MountingHole_Pad, MountingHole:MountingHole_3.2mm_M3_Pad, symbol Mechanical:MountingHole_Pad
- added J30, J31: Conn_02x07_Odd_Even, Connector_PinHeader_2.54mm:PinHeader_2x07_P2.54mm_Vertical, symbol Connector_Generic:Conn_02x07_Odd_Even
- added R52, R53, R57, R67, R75, R80: 10k, Resistor_SMD:R_0805_2012Metric_Pad1.20x1.40mm_HandSolder, symbol Device:R
- added SW1, SW10, SW3, SW4, SW5, SW6, SW7, SW8, SW9: SW_SPDT, Connector_PinHeader_2.54mm_LongPads:PinHeader_1x02_P2.54mm_Vertical_LongPads, symbol sw_spdt_2:SW_SPDT
- added unit 1 of U11
- added unit 3 of U11
- added unit 4 of U11
- added unit 2 of U11
- added unit 3 of U17
- added unit 5 of U18
- added unit 4 of U19
- added unit 5 of U2
- added unit 5 of U5
- added unit 5 of U7
- added unit 4 of U8
- added unit 2 of U8
- added unit 5 of U8
- added unit 3 of U8
- added unit 4 of U9
- added Z231, Z234, Z235, Z241, Z255, Z28, Z29, Z36: ~, Resistor_SMD:R_0805_2012Metric_Pad1.20x1.40mm_HandSolder, symbol Device:R
- H10: renamed from H4; now in the parts list
- H11: renamed from H8; now in the parts list
- H12: renamed from H5; now in the parts list
- H13: renamed from H2; now in the parts list
- H14: renamed from H3; now in the parts list
- H15: renamed from H6; now in the parts list
- H16: renamed from H7; now in the parts list
- H9: renamed from H1; now in the parts list
- RV10: renamed from RV19; footprint Connector_PinSocket_2.54mm_LongPads:PinSocket_1x06_P2.54mm_Vertical_LongPads -> Connector_PinSocket_2.54mm_LongPads:PinSocket_2x03_P2.54mm_Vertical_LongPads_Mirrored
- RV11: renamed from RV3; footprint Connector_PinSocket_2.54mm_LongPads:PinSocket_1x06_P2.54mm_Vertical_LongPads -> Connector_PinSocket_2.54mm_LongPads:PinSocket_2x03_P2.54mm_Vertical_LongPads
- RV15: renamed from RV20; footprint Connector_PinSocket_2.54mm_LongPads:PinSocket_1x06_P2.54mm_Vertical_LongPads -> Connector_PinSocket_2.54mm_LongPads:PinSocket_2x03_P2.54mm_Vertical_LongPads
- RV17: renamed from RV5; footprint Connector_PinSocket_2.54mm_LongPads:PinSocket_1x06_P2.54mm_Vertical_LongPads -> Connector_PinSocket_2.54mm_LongPads:PinSocket_2x03_P2.54mm_Vertical_LongPads_Mirrored
- RV19: renamed from RV16; footprint Connector_PinSocket_2.54mm_LongPads:PinSocket_1x06_P2.54mm_Vertical_LongPads -> Connector_PinSocket_2.54mm_LongPads:PinSocket_2x03_P2.54mm_Vertical_LongPads
- RV2: renamed from RV18; footprint Connector_PinSocket_2.54mm_LongPads:PinSocket_1x06_P2.54mm_Vertical_LongPads -> Connector_PinSocket_2.54mm_LongPads:PinSocket_2x03_P2.54mm_Vertical_LongPads_Mirrored
- RV6: renamed from RV17; footprint Connector_PinSocket_2.54mm_LongPads:PinSocket_1x06_P2.54mm_Vertical_LongPads -> Connector_PinSocket_2.54mm_LongPads:PinSocket_2x03_P2.54mm_Vertical_LongPads
- renumbered C21 to C1, C52 to C10, C112 to C100, C36 to C101, C24 to C102, C10 to C103, C67 to C104, C79 to C105, C97 to C106, C101 to C107, C105 to C108, C74 to C11, C11 to C110, C25 to C111, C4 to C112, C19 to C113, C2 to C115, C5 to C116, C20 to C117, C117 to C118, C6 to C119, C43 to C12, C26 to C120, C12 to C121, C62 to C13, C86 to C14, C39 to C15, C49 to C16, C59 to C17, C71 to C18, C83 to C19, C27 to C2, C53 to C20, C75 to C21, C42 to C22, C63 to C23, C87 to C24, C38 to C25, C50 to C26, C60 to C27, C72 to C28, C84 to C29, C54 to C30, C76 to C31, C44 to C32, C3 to C33, C64 to C34, C88 to C35, C40 to C36, C1 to C37, C51 to C38, C61 to C39, C73 to C40, C85 to C41, C55 to C42, C77 to C43, C45 to C44, C65 to C45, C89 to C46, C41 to C47, C30 to C48, C22 to C49, C48 to C5, C35 to C50, C37 to C51, C13 to C54, C16 to C55, C31 to C56, C33 to C57, C28 to C58, C58 to C6, C14 to C61, C17 to C62, C32 to C63, C34 to C64, C29 to C65, C110 to C66, C68 to C67, C80 to C68, C92 to C69, C70 to C7, C111 to C70, C69 to C71, C81 to C72, C93 to C73, C90 to C74, C94 to C75, C98 to C76, C102 to C77, C106 to C78, C91 to C79, C82 to C8, C95 to C80, C99 to C81, C103 to C82, C107 to C83, C9 to C84, C115 to C85, C23 to C86, C46 to C87, C56 to C88, C113 to C89, C15 to C9, C18 to C90, C114 to C91, C47 to C92, C57 to C93, C66 to C94, C78 to C95, C100 to C97, C104 to C98, C108 to C99, D2 to D1, D1 to D2, D4 to D3, D3 to D4, J40 to J1, J42 to J10, J43 to J11, J20 to J12, J27 to J13, J16 to J14, J24 to J15, J15 to J16, J7 to J17, J38 to J18, J44 to J19, J1 to J2, J6 to J20, J45 to J21, J8 to J22, J17 to J23, J25 to J24, J37 to J25, J39 to J26, J18 to J27, J9 to J28, J28 to J29, J2 to J3, J29 to J32, J30 to J33, J36 to J34, J31 to J35, J32 to J36, J34 to J37, J35 to J38, J10 to J39, J19 to J4, J21 to J40, J13 to J41, J33 to J42, J11 to J43, J26 to J5, J41 to J6, J3 to J7, J4 to J8, J5 to J9, L2 to L1, L3 to L2, L4 to L3, L1 to L4, R39 to R1, R117 to R10, R98 to R100, R23 to R101, R16 to R102, R19 to R103, R17 to R104, R21 to R105, R24 to R106, R43 to R107, R57 to R108, R145 to R109, R141 to R11, R33 to R110, R69 to R111, R76 to R112, R44 to R113, R121 to R114, R131 to R115, R79 to R116, R85 to R117, R99 to R118, R51 to R119, R93 to R12, R70 to R120, R100 to R121, R125 to R123, R45 to R124, R58 to R125, R9 to R126, R34 to R127, R46 to R128, R77 to R129, R40 to R13, R83 to R130, R123 to R131, R52 to R133, R10 to R134, R15 to R135, R78 to R136, R124 to R137, R80 to R138, R126 to R139, R49 to R14, R11 to R140, R67 to R141, R71 to R142, R81 to R143, R86 to R144, R59 to R145, R60 to R146, R68 to R147, R82 to R148, R84 to R149, R18 to R15, R72 to R150, R75 to R151, R6 to R16, R105 to R17, R113 to R18, R127 to R19, R55 to R2, R137 to R20, R146 to R21, R88 to R22, R94 to R23, R28 to R24, R32 to R25, R41 to R26, R56 to R27, R110 to R28, R134 to R29, R20 to R3, R14 to R30, R101 to R31, R29 to R32, R7 to R33, R118 to R34, R142 to R35, R31 to R36, R91 to R37, R42 to R38, R50 to R39, R22 to R4, R106 to R40, R114 to R41, R128 to R42, R138 to R43, R147 to R44, R8 to R45, R87 to R46, R92 to R47, R35 to R48, R53 to R49, R109 to R5, R111 to R50, R135 to R51, R61 to R54, R103 to R55, R36 to R56, R12 to R58, R119 to R59, R133 to R6, R143 to R60, R47 to R61, R73 to R63, R95 to R64, R3 to R65, R63 to R66, R107 to R68, R115 to R69, R13 to R7, R129 to R70, R139 to R71, R148 to R72, R89 to R73, R96 to R74, R1 to R76, R4 to R77, R37 to R78, R54 to R79, R102 to R8, R112 to R81, R136 to R82, R64 to R83, R104 to R84, R38 to R85, R120 to R86, R144 to R87, R48 to R88, R65 to R89, R5 to R9, R74 to R90, R97 to R91, R66 to R92, R30 to R93, R108 to R94, R116 to R95, R130 to R96, R140 to R97, R149 to R98, R90 to R99, RV9 to RV1, RV14 to RV12, RV1 to RV13, RV8 to RV14, RV15 to RV16, RV4 to RV18, RV21 to RV20, RV11 to RV21, RV13 to RV3, RV6 to RV4, RV10 to RV5, RV12 to RV7, RV7 to RV8, RV2 to RV9, SW9 to SW11, SW1 to SW12, U8 to U1, U9 to U1, U11 to U10, U9 to U10, U17 to U12, U18 to U12, U16 to U12, U20 to U13, U18 to U13, U10 to U14, U12 to U14, U11 to U14, U3 to U15, U17 to U16, U18 to U16, U4 to U17, U5 to U17, U13 to U18, U12 to U18, U5 to U19, U16 to U2, U15 to U2, U21 to U20, U22 to U20, U13 to U21, U22 to U21, U14 to U21, U14 to U22, U21 to U22, U20 to U22, U6 to U25, U7 to U26, U19 to U3, U1 to U4, U9 to U5, U8 to U5, U15 to U6, U16 to U6, U10 to U7, U22 to U7, U11 to U7, U4 to U8, U2 to U9, Z238 to Z1, Z68 to Z10, Z58 to Z100, Z214 to Z101, Z223 to Z102, Z187 to Z103, Z203 to Z104, Z232 to Z105, Z252 to Z106, Z156 to Z107, Z218 to Z108, Z19 to Z109, Z5 to Z11, Z195 to Z110, Z242 to Z111, Z9 to Z112, Z29 to Z113, Z243 to Z114, Z139 to Z115, Z151 to Z116, Z184 to Z117, Z201 to Z118, Z233 to Z119, Z25 to Z12, Z253 to Z120, Z145 to Z121, Z192 to Z122, Z160 to Z123, Z165 to Z124, Z162 to Z125, Z215 to Z126, Z224 to Z127, Z188 to Z128, Z204 to Z129, Z190 to Z13, Z234 to Z130, Z254 to Z131, Z157 to Z132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
Connections:
- net +15V_I: now also C54.2, C55.2, C56.2, C57.2, C58.2, U11.4 (V+), U15.4 (V+), U17.4 (V+), U19.4 (V+), U4.4 (V+), U9.4 (V+), C52.1, C53.2, J30.13 (Pin_13), J30.14 (Pin_14), U8.4 (V+)
- net +15V_P: now also C114.1, Z255.2
- net +9V_I: now also J30.5 (Pin_5), J30.6 (Pin_6)
- net +9V_P: now also Z241.2
- net -15V_I: now also C61.2, C62.2, C63.2, C64.2, C65.2, U11.11 (V-), U15.11 (V-), U17.11 (V-), U19.11 (V-), U4.11 (V-), U9.11 (V-), C59.2, C60.2, J30.7 (Pin_7), J30.8 (Pin_8), U8.11 (V-)
- net 9V_GND_I: now also J30.1 (Pin_1), J30.2 (Pin_2), J30.3 (Pin_3), J30.4 (Pin_4)
- net GND_I: now also C33.2, C48.2, C54.1, C55.1, C56.1, C57.1, C58.1, C61.1, C62.1, C63.1, C64.1, C65.1, J17.2 (Pin_2), J2.2 (Pin_2), J20.2 (Pin_2), J22.2 (Pin_2), J28.2 (Pin_2), J3.2 (Pin_2), J7.2 (Pin_2), J8.2 (Pin_2), J9.2 (Pin_2), R106.1, R15.1, R36.1, R77.1, Z100.2, Z11.2, Z112.2, Z113.2, Z12.2, Z14.2, Z142.2, Z143.1, Z144.2, Z145.2, Z146.2, Z151.2, Z154.2, Z156.2, Z157.2, Z158.2, Z16.2, Z177.2, Z178.2, Z179.2, Z180.2, Z181.2, Z19.2, Z192.2, Z193.2, Z194.2, Z206.2, Z207.2, Z21.2, Z210.2, Z211.2, Z212.2, Z213.2, Z224.2, Z228.2, Z229.2, Z230.2, Z232.2, Z32.2, Z33.2, Z35.2, Z40.2, Z41.2, Z42.2, Z57.2, Z58.2, Z59.2, Z62.2, Z63.2, Z75.2, Z76.2, Z79.2, Z86.2, Z87.2, Z99.2, C3.2, C52.2, C53.1, C59.1, C60.1, J30.10 (Pin_10), J30.11 (Pin_11), J30.12 (Pin_12), J30.9 (Pin_9), R80.1, U11.12 (+), U8.12 (+), U9.12 (+)
- net GND_P: now also C114.2
- net at R48.1, RV8.1, U10.1: now also SW4.1 (A)
- net at R56.1, RV8.2, RV8.3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: now also SW4.2 (B)
- net at R12.1, RV3.1: now also Z18.2; no longer Z61.2
- net at U13.5 (+), Z102.2: now also U13.10 (+); no longer U13.3 (+)
- net at C51.1, R117.1: now also U21.10 (+); no longer U21.5 (+)
- net at RV9.1: now also R67.2, U11.2 (-)
- net at RV9.2, RV9.3: now also R57.1, U11.6 (-)
- net at R135.1, Z204.1, Z211.1: now also U19.8; no longer U19.7
- net at R126.1, R134.1, R135.2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: now also U19.9 (-); no longer U19.6 (-)
- net at Z1.1, Z7.1: now also U3.8, U3.9 (-); no longer U3.1, U3.2 (-)
- net at R32.1, RV4.2, RV4.3: now also U8.6 (-)
- net at R32.2, R36.2: now also U8.10 (+); no longer U15.5 (+)
- net at R83.2, R89.2, R90.1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: now also U7.6 (-); no longer U7.13 (-)
- net at C17.2, R34.2: now also U2.5 (+); no longer U2.3 (+)
- net at Z189.2, Z193.1: now also U17.3 (+); no longer U17.12 (+)
- net at R130.1, Z208.1, Z219.1: now also U21.14; no longer U21.7
- net at C39.2, R86.2: now also U12.5 (+); no longer U12.3 (+)
- net at R78.1, RV14.1, U10.7: now also SW5.1 (A)
- net at R85.1, RV14.2, RV14.3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: now also SW5.2 (B)
- net at R13.2, R14.2: now also U1.12 (+); no longer U1.5 (+)
- net at R1.2, R2.1: now also U1.13 (-); no longer U1.6 (-)
- net at R2.2, Z17.1: now also U1.14; no longer U1.7
- net at R131.2, RV22.1, U22.8: now also SW10.1 (A)
- net at R137.2, RV22.2, RV22.3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: now also SW10.2 (B)
- net at Z201.2, Z207.1: now also U19.3 (+); no longer U19.12 (+)
- net at R102.2, R103.1, R104.2: now also U17.13 (-); no longer U17.6 (-)
- net at R103.2, Z136.1: now also U17.14; no longer U17.7
- net at C35.2, R71.2: now also U16.5 (+); no longer U16.12 (+)
- net at RV12.2: now also U14.3 (+); no longer U14.12 (+)
- net at R125.1, Z195.1: now also U18.8; no longer U18.14
- net at R112.1, Z164.1: now also U21.7; no longer U21.1
- net at R111.1, R112.2, R120.1: now also U21.6 (-); no longer U21.2 (-)
- net at Z182.1: now also U21.5 (+); no longer U21.3 (+)
- net at C44.1, RV15.1, RV15.2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: now also U14.10 (+); no longer U14.3 (+)
- net at C8.2, R11.2: now also U2.12 (+); no longer U2.5 (+)
- net at Z109.1, Z112.1: now also J9.1 (Pin_1); no longer J9.3 (Pin_3)
- net at R54.2, R62.2, R63.1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: now also U7.2 (-); no longer U7.9 (-)
- net at R63.2, Z92.1: now also U7.1; no longer U7.8
- net at U1.3 (+), U10.3 (+), U10.5 (+)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: now also U1.5 (+), U18.3 (+); no longer U1.3 (+), U18.10 (+)
- net at Z197.1, Z199.1: now also U20.13 (-), U20.14; no longer U20.1, U20.2 (-)
- net at R84.2, RV16.3, Z117.1: now also U14.8; no longer U14.1
- net at U3.5 (+), Z25.2: now also U3.10 (+); no longer U3.3 (+)
- net at R25.2, Z38.1, Z40.1: now also U8.8; no longer U15.7
- net at Z80.2, Z87.1: now also U11.5 (+)
- net at C46.2, R97.2: now also U16.3 (+); no longer U16.12 (+)
- net at R102.1: now also Z135.2; no longer Z98.2
- net at Z153.2, Z161.1: now also U18.5 (+); no longer U18.10 (+)
- net at R124.2, R127.1: now also U18.7, SW8.1 (A); no longer U18.8
- net at R127.2, R128.2: now also U18.6 (-), SW8.2 (B); no longer U18.9 (-)
- net at Z109.2, Z113.1: now also U11.3 (+)
- net at Z80.1, Z86.1: now also J9.3 (Pin_3); no longer J9.2 (Pin_2)
- net at Z81.1, Z88.1: now also U13.8, U13.9 (-); no longer U13.1, U13.2 (-)
- net at R65.1, RV13.1: now also Z95.2; no longer Z135.2
- net at RV13.2: now also U15.5 (+); no longer U15.10 (+)
- net at R58.2, RV13.3, Z97.1: now also U15.8
- net at Z176.2, Z181.1: now also U17.5 (+); no longer U17.3 (+)
- net at R26.2, R27.1: now also U1.9 (-); no longer U1.6 (-)
- net at R27.2, Z60.1: now also U1.8; no longer U1.7
- net at Z46.1, Z52.1: now also U3.13 (-), U3.14; no longer U3.8, U3.9 (-)
- net at R26.1, RV5.1: now also U1.7, SW3.1 (A); no longer U1.1
- net at R38.1, RV5.2, RV5.3: now also U1.6 (-), SW3.2 (B); no longer U1.2 (-)
- net at C23.2, R41.2: now also U6.5 (+); no longer U6.10 (+)
- net at R137.1, R139.1: now also U22.5 (+); no longer U22.12 (+)
- net at C20.2, R42.1: now also U6.6 (-), U6.7; no longer U6.8, U6.9 (-)
- net at C84.2, C86.2, C90.1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: now also Z241.1
- net at Z151.1: now also U17.12 (+); no longer U17.5 (+)
- net at R122.1, R123.1: now also U22.3 (+); no longer U22.5 (+)
- net at C110.2, C111.2, C113.1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: now also Z255.1
- net at R38.2, R39.2: now also U1.10 (+); no longer U1.5 (+)
- net at R118.1, RV19.3, Z167.1: now also U21.8; no longer U21.7
- net at C29.2, R60.2: now also U12.12 (+); no longer U12.5 (+)
- net at C22.1, RV6.1, RV6.2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: now also U5.10 (+); no longer U5.12 (+)
- net at R115.1, Z183.1, Z185.1: now also U22.1; no longer U22.7
- net at R114.1, R115.2: now also U22.2 (-); no longer U22.6 (-)
- net at R131.1, R132.2: now also U22.6 (-); no longer U22.13 (-)
- net at R132.1, Z209.1, Z221.1: now also U22.7; no longer U22.14
- net at Z224.1: now also U19.10 (+); no longer U19.5 (+)
- net at C45.2, R95.2: now also U16.12 (+); no longer U16.10 (+)
- net at R107.2, R110.1: now also U18.1, SW6.1 (A); no longer U18.8
- net at R110.2, R113.2: now also U18.2 (-), SW6.2 (B); no longer U18.9 (-)
- net at C32.1, RV10.1, RV10.2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: now also U14.12 (+); no longer U14.3 (+)
- net at R37.1, RV7.1: now also Z61.2; no longer Z18.2
- net at RV7.2: now also U5.5 (+); no longer U5.10 (+)
- net at R31.2, RV7.3, Z47.1: now also U5.8; no longer U5.14
- net at R24.1, RV4.1: now also U8.7
- net at C31.2, Z101.1: now also U16.6 (-), U16.7; no longer U16.13 (-), U16.14
- net at R101.1, RV18.1: now also Z98.2; no longer Z95.2
- net at C10.2, R19.1: now also U6.1, U6.2 (-); no longer U6.8, U6.9 (-)
- net at R118.2, R121.1: now also U21.9 (-); no longer U21.6 (-)
- net at Z184.1, Z187.1: now also U20.1, U20.2 (-); no longer U20.13 (-), U20.14
- net at R84.1, R91.2: now also U14.9 (-); no longer U14.2 (-)
- net at R55.1, R64.2: now also U14.13 (-); no longer U14.2 (-)
- net at C33.1, RV11.1, RV11.2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: now also U15.10 (+)
- net at R58.1, R65.2: now also U15.9 (-)
- net at C5.1: now also Z4.2; no longer Z48.2
- net at R31.1, R37.2: now also U5.9 (-); no longer U5.13 (-)
- net at R82.2, Z128.1: now also U12.8, U12.9 (-); no longer U12.6 (-), U12.7
- net at U21.3 (+), U22.10 (+), Z168.2: now also U22.12 (+); no longer U22.3 (+)
- net at C21.2, Z65.1: now also U6.8, U6.9 (-); no longer U6.13 (-), U6.14
- net at C43.2, Z126.1: now also U16.1, U16.2 (-); no longer U16.13 (-), U16.14
- net at Z94.1: now also R53.1, U11.8
- net at R48.2, R49.1: now also U10.13 (-); no longer U10.6 (-)
- net at R49.2, Z82.1: now also U10.14; no longer U10.7
- net at Z225.2, Z230.1: now also U19.5 (+); no longer U19.10 (+)
- net at R90.2, Z123.1: now also U7.7; no longer U7.14
- net at Z63.1: now also U9.10 (+); no longer U9.12 (+)
- net at R30.1, R33.2, R45.2: now also U9.9 (-); no longer U9.13 (-)
- net at R30.2, Z54.1: now also U9.8; no longer U9.14
- net at R128.1, R133.1: now also U18.10 (+); no longer U18.12 (+)
- net at Z107.1: now also U7.3 (+); no longer U7.10 (+)
- net at R124.1, R125.2: now also U18.9 (-); no longer U18.13 (-)
- net at SW2.2 (B): now also U8.5 (+)
- net at C16.1: now also Z48.2; no longer Z4.2
- net at R122.2, RV20.2, RV20.3: now also U22.13 (-), SW7.2 (B); no longer U22.2 (-)
- net at R136.1, R138.1: now also U21.12 (+); no longer U21.5 (+)
- net at R129.1, R130.2: now also U21.13 (-); no longer U21.6 (-)
- net at Z134.2, Z135.1: now also Z143.2; no longer Z143.1
- net at Z114.1, Z119.1: now also U13.13 (-), U13.14; no longer U13.8, U13.9 (-)
- net at R55.2, RV12.3, Z84.1: now also U14.14; no longer U14.1
- net at R1.1, RV1.1, U1.1: now also SW1.1 (A)
- net at R13.1, RV1.2, RV1.3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: now also SW1.2 (B)
- net at C19.2, R35.2: now also U2.10 (+); no longer U2.5 (+)
- net at R29.2, Z68.1: now also U2.8, U2.9 (-); no longer U2.6 (-), U2.7
- net at C40.1, R81.2: now also U12.6 (-), U12.7; no longer U12.1, U12.2 (-)
- net at C13.2, R18.2: now also U6.3 (+); no longer U6.10 (+)
- net at C24.2, R43.2: now also U6.10 (+); no longer U6.12 (+)
- net at R17.1: now also Z29.2
- net at C42.2, R96.1: now also U16.13 (-), U16.14; no longer U16.8, U16.9 (-)
- net at C41.2, R87.2: now also U12.10 (+); no longer U12.5 (+)
- net at R51.2, Z103.1: now also U12.13 (-), U12.14; no longer U12.6 (-), U12.7
- net at C18.1, R28.2: now also U2.6 (-), U2.7; no longer U2.1, U2.2 (-)
- net at RV3.2: now also U5.3 (+); no longer U5.10 (+)
- net at R56.2, R61.2: now also U10.12 (+); no longer U10.5 (+)
- net at R114.2, RV20.1: now also U22.14, SW7.1 (A); no longer U22.1
- net at R129.2, RV21.1, U21.1: now also SW9.1 (A)
- net at R136.2, RV21.2, RV21.3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: now also SW9.2 (B)
- net at Z132.1: now also U7.5 (+); no longer U7.12 (+)
- net at R24.2, R25.1: now also U8.9 (-); no longer U15.6 (-)
- net +15V renamed +15V_O
- net +15V_O: now also J31.13 (Pin_13), J31.14 (Pin_14), U18.4 (V+), U2.4 (V+), U5.4 (V+), U7.4 (V+); no longer C54.2, C55.2, C56.2, C57.2, C58.2, U11.4 (V+), U15.4 (V+), U17.4 (V+), U19.4 (V+), U4.4 (V+), U9.4 (V+)
- net -15V renamed -15V_O
- net -15V_O: now also J31.7 (Pin_7), J31.8 (Pin_8), U18.11 (V-), U2.11 (V-), U5.11 (V-), U7.11 (V-); no longer C61.2, C62.2, C63.2, C64.2, C65.2, U11.11 (V-), U15.11 (V-), U17.11 (V-), U19.11 (V-), U4.11 (V-), U9.11 (V-)
- net GND renamed GND_O
- net GND_O: now also U7.10 (+), U7.12 (+), C4.2, J31.10 (Pin_10), J31.11 (Pin_11), J31.12 (Pin_12), J31.9 (Pin_9), Z234.2, Z235.2, Z36.2; no longer C33.2, C48.2, C54.1, C55.1, C56.1, C57.1, C58.1, C61.1, C62.1, C63.1, C64.1, C65.1, J17.2 (Pin_2), J2.2 (Pin_2), J20.2 (Pin_2), J22.2 (Pin_2), J28.2 (Pin_2), J3.2 (Pin_2), J7.2 (Pin_2), J8.2 (Pin_2), J9.1 (Pin_1), R106.1, R15.1, R36.1, R77.1, U7.10 (+), U7.12 (+), Z100.2, Z11.2, Z112.2, Z113.2, Z12.2, Z14.2, Z142.2, Z143.2, Z144.2, Z145.2, Z146.2, Z151.2, Z154.2, Z156.2, Z157.2, Z158.2, Z16.2, Z177.2, Z178.2, Z179.2, Z180.2, Z181.2, Z19.2, Z192.2, Z193.2, Z194.2, Z206.2, Z207.2, Z21.2, Z210.2, Z211.2, Z212.2, Z213.2, Z224.2, Z228.2, Z229.2, Z230.2, Z232.2, Z32.2, Z33.2, Z35.2, Z40.2, Z41.2, Z42.2, Z57.2, Z58.2, Z59.2, Z62.2, Z63.2, Z75.2, Z76.2, Z79.2, Z86.2, Z87.2, Z99.2
- new net: C36.2, U14.1, U14.2 (-)
- new net: U19.1, U19.2 (-), Z202.1
- new net: C4.1, H4.1
- new net: U20.12 (+), U20.3 (+), Z174.2, Z231.2, Z235.1
- new net: U3.1, U3.2 (-), Z70.1
- new net: R67.1, R75.1, U11.1
- new net: R75.2, R80.2, U11.10 (+)
- new net: U17.1, U17.2 (-), Z190.1
- new net: U17.10 (+), U19.12 (+), U8.3 (+), Z137.2
- new net: C15.2, U5.1, U5.2 (-)
- new net: U13.1, U13.2 (-), Z130.1
- new net: U9.13 (-), U9.14
- new net: U8.13 (-), U8.14
- new net: C37.2, U15.6 (-), U15.7
- new net: U13.12 (+), U13.3 (+), Z127.2
- new net: U19.13 (-), U19.14, Z152.1, Z156.1
- new net: U17.6 (-), U17.7, Z155.2
- new net: R6.2, U2.13 (-), U2.14, Z28.1
- new net: Z28.2, Z29.1, Z36.1
- new net: J32.1 (Pin_1), Z231.1, Z234.1
- new net: U17.8, U17.9 (-), Z175.1, Z177.1
- new net: U7.13 (-), U7.14
- new net: R52.2, R53.2, U11.9 (-)
- new net: U11.13 (-), U11.14
- new net: U3.12 (+), U3.3 (+), Z66.2
- new net: C3.1, H3.1
- new net: R52.1, R57.2, U11.7
- new net: U19.6 (-), U19.7, Z226.1
- new net: C25.2, U5.6 (-), U5.7
- new net: U7.8, U7.9 (-)
- new net +9V_O: J31.5 (Pin_5), J31.6 (Pin_6)
- new net 9V_GND_O: J31.1 (Pin_1), J31.2 (Pin_2), J31.3 (Pin_3), J31.4 (Pin_4)
- no-connect marks 12 -> 3
Other:
- moved on the sheet: C1, C10, C100, C101, C102, C103, C104, C106, C11, C110, C111, C112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
