File: KiCad/Output.kicad_pcb (KiCad board)
At the start: 4 copper layers, 150 x 85.2 mm, 84 parts, among them J10 VCC_IN, J11 VCC_OUT, J13 EMK_Out, J14 EMK_Out, J21 Conn_01x05_bridged, J30 Pegel_In, J31 Pegel_In, J32 Pegel_In, J33 Pegel_In, J34 LED_Out, J36 VU_Meter_Out, SW1 SW_DPST, SW9 SW_Rotary_1x4, U23 TL074, U24 TL074, U6 REC10K-2409, U7 REC10K-2415

Commit message: PCB Update
Routing:
- net Net-(J36-Pin_1): track 5.10 -> 10.6 mm
- net Net-(J34-Pin_2): track 0.00 -> 5.49 mm
- removed copper zone on F.Cu, net Net-(J34-Pin_2)
- removed copper zone on F.Cu, net Net-(J36-Pin_1)

Commit message: PCB Update
Parts:
- removed C10, C11, C12, C9: 470p, Capacitor_SMD:C_0805_2012Metric_Pad1.18x1.45mm_HandSolder
- removed C112, C113, C4, C6: 10n, Capacitor_SMD:C_0805_2012Metric_Pad1.18x1.45mm_HandSolder
- removed C18, C19, C20, C46, C47, C56, C57: 100n, Capacitor_SMD:C_0805_2012Metric_Pad1.18x1.45mm_HandSolder
- removed C2, C5: 10u, Capacitor_SMD:C_1210_3225Metric_Pad1.33x2.70mm_HandSolder
- removed C23, C24, C25, C26: 1n, Capacitor_SMD:C_0805_2012Metric_Pad1.18x1.45mm_HandSolder
- removed C36: 4u7, Capacitor_SMD:C_0805_2012Metric_Pad1.18x1.45mm_HandSolder
- removed D1, D2, D3: D, Diode_SMD:D_0805_2012Metric_Pad1.15x1.40mm_HandSolder
- removed J10: VCC_IN, Connector_PinHeader_2.54mm_LongPads:PinHeader_1x02_P2.54mm_Vertical_LongPads
- removed J11: VCC_OUT, Connector_PinHeader_2.54mm_LongPads:PinHeader_1x02_P2.54mm_Vertical_LongPads
- removed J13, J14: EMK_Out, Connector_PinSocket_2.54mm_LongPads:PinSocket_1x05_P2.54mm_Vertical_LongPads
- removed J21: Conn_01x05_bridged, Connector_Bridged_2.54mm_LongPads:Bridge_2x05_P2.54mm_Vertical_LongPads
- removed J30, J31, J32, J33: Pegel_In, Connector_PinHeader_2.54mm_LongPads:PinHeader_1x02_P2.54mm_Vertical_LongPads
- removed J34: LED_Out, Connector_PinSocket_2.54mm_LongPads:PinSocket_1x02_P2.54mm_Vertical_LongPads
- removed J36: VU_Meter_Out, Connector_PinSocket_2.54mm_LongPads:PinSocket_1x04_P2.54mm_Vertical_LongPdas
- removed L1: ~, WE-SL575:WE-SL575
- removed L2, L3, L4, L5: Dämpfungsperle, 220 Ohm @ 100MHz, 0.5A, Inductor_SMD:L_1206_3216Metric
- removed R25, R26, R27: 22R, Resistor_SMD:R_0805_2012Metric_Pad1.20x1.40mm_HandSolder
- removed R59, R60, R84: 1k, Resistor_SMD:R_0805_2012Metric_Pad1.20x1.40mm_HandSolder
- removed R67: 20k, Resistor_SMD:R_0805_2012Metric_Pad1.20x1.40mm_HandSolder
- removed R68, R82: 10k, Resistor_SMD:R_0805_2012Metric_Pad1.20x1.40mm_HandSolder
- removed R71: 80k, Resistor_SMD:R_0805_2012Metric_Pad1.20x1.40mm_HandSolder
- removed R72: 12k, Resistor_SMD:R_0805_2012Metric_Pad1.20x1.40mm_HandSolder
- removed R75: 3k, Resistor_SMD:R_0805_2012Metric_Pad1.20x1.40mm_HandSolder
- removed R81, R86: 1k8, Resistor_SMD:R_0805_2012Metric_Pad1.20x1.40mm_HandSolder
- removed SW1: SW_DPST, Connector_PinSocket_2.54mm_LongPads:PinSocket_1x04_P2.54mm_Vertical_LongPdas
- removed SW9: SW_Rotary_1x4, Connector_PinHeader_2.54mm_LongPads:PinHeader_1x05_P2.54mm_Vertical_LongPads
- removed U23, U24: TL074, Package_DIP:DIP-14_W7.62mm_Socket_LongPads
- removed U6: REC10K-2409, REC10K-2409SAW_H2:CONV_REC10K-2409SAW_H2
- removed U7: REC10K-2415, REC10K-2415DAW_H2:CONV_REC10K-2415DAW_H2
- removed Z122, Z123, Z124, Z125, Z126, Z127, Z128, Z129, Z130, Z131, Z132, Z133, Z134, Z135, Z136, Z137, Z167, Z168, Z170, Z171, Z172, Z173, Z174: ~, Resistor_SMD:R_0805_2012Metric_Pad1.20x1.40mm_HandSolder
- added C100: 100n, Capacitor_SMD:C_0805_2012Metric_Pad1.18x1.45mm_HandSolder, B.Cu at (379.6, 114.1)
- added C101: 100n, Capacitor_SMD:C_0805_2012Metric_Pad1.18x1.45mm_HandSolder, B.Cu at (359.3, 118.8)
- added C102: 100n, Capacitor_SMD:C_0805_2012Metric_Pad1.18x1.45mm_HandSolder, B.Cu at (359.3, 121.8)
- added C103: 100n, Capacitor_SMD:C_0805_2012Metric_Pad1.18x1.45mm_HandSolder, B.Cu at (359.3, 124.8)
- added C104: 100n, Capacitor_SMD:C_0805_2012Metric_Pad1.18x1.45mm_HandSolder, B.Cu at (359.3, 127.8)
- added C105: 100n, Capacitor_SMD:C_0805_2012Metric_Pad1.18x1.45mm_HandSolder, B.Cu at (359.3, 130.8)
- added C106: 100n, Capacitor_SMD:C_0805_2012Metric_Pad1.18x1.45mm_HandSolder, B.Cu at (359.3, 133.8)
- added C107: 100n, Capacitor_SMD:C_0805_2012Metric_Pad1.18x1.45mm_HandSolder, B.Cu at (359.3, 136.8)
- added C108: 100n, Capacitor_SMD:C_0805_2012Metric_Pad1.18x1.45mm_HandSolder, B.Cu at (359.3, 139.8)
- added C109: 100n, Capacitor_SMD:C_0805_2012Metric_Pad1.18x1.45mm_HandSolder, B.Cu at (359.3, 142.8)
- added C110: 100n, Capacitor_SMD:C_0805_2012Metric_Pad1.18x1.45mm_HandSolder, B.Cu at (359.3, 145.9)
- added C111: 100n, Capacitor_SMD:C_0805_2012Metric_Pad1.18x1.45mm_HandSolder, B.Cu at (359.3, 148.9)
- added C35: 6n8, Capacitor_SMD:C_0805_2012Metric_Pad1.18x1.45mm_HandSolder, B.Cu at (379.6, 99.0)
- added C37: 6n8, Capacitor_SMD:C_0805_2012Metric_Pad1.18x1.45mm_HandSolder, B.Cu at (383.4, 118.8)
- added C38: 3n, Capacitor_SMD:C_0805_2012Metric_Pad1.18x1.45mm_HandSolder, B.Cu at (383.4, 121.8)
- added C39: 3n, Capacitor_SMD:C_0805_2012Metric_Pad1.18x1.45mm_HandSolder, B.Cu at (383.4, 124.8)
- added C40: 3n, Capacitor_SMD:C_0805_2012Metric_Pad1.18x1.45mm_HandSolder, B.Cu at (383.4, 127.8)
- added C41: 3n, Capacitor_SMD:C_0805_2012Metric_Pad1.18x1.45mm_HandSolder, B.Cu at (383.4, 130.8)
- added C42: 470p, Capacitor_SMD:C_0805_2012Metric_Pad1.18x1.45mm_HandSolder, B.Cu at (383.4, 133.8)
- added C43: 470p, Capacitor_SMD:C_0805_2012Metric_Pad1.18x1.45mm_HandSolder, B.Cu at (383.4, 136.8)
- added C44: 470p, Capacitor_SMD:C_0805_2012Metric_Pad1.18x1.45mm_HandSolder, B.Cu at (383.4, 139.8)
- added C45: 470p, Capacitor_SMD:C_0805_2012Metric_Pad1.18x1.45mm_HandSolder, B.Cu at (383.4, 142.8)
- added C48: 130n, Capacitor_SMD:C_0805_2012Metric_Pad1.18x1.45mm_HandSolder, B.Cu at (383.4, 145.9)
- added C49: 130n, Capacitor_SMD:C_0805_2012Metric_Pad1.18x1.45mm_HandSolder, B.Cu at (383.4, 148.9)
- added C50: 130n, Capacitor_SMD:C_0805_2012Metric_Pad1.18x1.45mm_HandSolder, B.Cu at (379.6, 102.0)
- added C51: 130n, Capacitor_SMD:C_0805_2012Metric_Pad1.18x1.45mm_HandSolder, B.Cu at (378.6, 118.8)
- added C52: 130n, Capacitor_SMD:C_0805_2012Metric_Pad1.18x1.45mm_HandSolder, B.Cu at (378.6, 121.8)
- added C53: 130n, Capacitor_SMD:C_0805_2012Metric_Pad1.18x1.45mm_HandSolder, B.Cu at (378.6, 124.8)
- added C54: 130n, Capacitor_SMD:C_0805_2012Metric_Pad1.18x1.45mm_HandSolder, B.Cu at (378.6, 127.8)
- added C55: 130n, Capacitor_SMD:C_0805_2012Metric_Pad1.18x1.45mm_HandSolder, B.Cu at (378.6, 130.8)
- added C58: 130n, Capacitor_SMD:C_0805_2012Metric_Pad1.18x1.45mm_HandSolder, B.Cu at (378.6, 133.8)
- added C59: 130n, Capacitor_SMD:C_0805_2012Metric_Pad1.18x1.45mm_HandSolder, B.Cu at (378.6, 136.8)
- added C60: 130n, Capacitor_SMD:C_0805_2012Metric_Pad1.18x1.45mm_HandSolder, B.Cu at (378.6, 139.8)
- added C61: 130n, Capacitor_SMD:C_0805_2012Metric_Pad1.18x1.45mm_HandSolder, B.Cu at (378.6, 142.8)
- added C62: 130n, Capacitor_SMD:C_0805_2012Metric_Pad1.18x1.45mm_HandSolder, B.Cu at (378.6, 145.9)
- added C63: 130n, Capacitor_SMD:C_0805_2012Metric_Pad1.18x1.45mm_HandSolder, B.Cu at (378.6, 148.9)
- added C64: 130n, Capacitor_SMD:C_0805_2012Metric_Pad1.18x1.45mm_HandSolder, B.Cu at (379.6, 105.0)
- added C65: 130n, Capacitor_SMD:C_0805_2012Metric_Pad1.18x1.45mm_HandSolder, B.Cu at (373.7, 118.8)
- added C66: 100n, Capacitor_SMD:C_0805_2012Metric_Pad1.18x1.45mm_HandSolder, B.Cu at (373.7, 121.8)
- added C67: 100n, Capacitor_SMD:C_0805_2012Metric_Pad1.18x1.45mm_HandSolder, B.Cu at (373.7, 124.8)
- added C68: 100n, Capacitor_SMD:C_0805_2012Metric_Pad1.18x1.45mm_HandSolder, B.Cu at (373.7, 127.8)
- added C69: 100n, Capacitor_SMD:C_0805_2012Metric_Pad1.18x1.45mm_HandSolder, B.Cu at (373.7, 130.8)
- added C70: 130n, Capacitor_SMD:C_0805_2012Metric_Pad1.18x1.45mm_HandSolder, B.Cu at (373.7, 133.8)
- added C71: 130n, Capacitor_SMD:C_0805_2012Metric_Pad1.18x1.45mm_HandSolder, B.Cu at (373.7, 136.8)
- added C72: 130n, Capacitor_SMD:C_0805_2012Metric_Pad1.18x1.45mm_HandSolder, B.Cu at (373.7, 139.8)
- added C73: 130n, Capacitor_SMD:C_0805_2012Metric_Pad1.18x1.45mm_HandSolder, B.Cu at (373.7, 142.8)
- added C74: 130n, Capacitor_SMD:C_0805_2012Metric_Pad1.18x1.45mm_HandSolder, B.Cu at (373.7, 145.9)
- added C75: 130n, Capacitor_SMD:C_0805_2012Metric_Pad1.18x1.45mm_HandSolder, B.Cu at (373.7, 148.9)
- added C76: 130n, Capacitor_SMD:C_0805_2012Metric_Pad1.18x1.45mm_HandSolder, B.Cu at (379.6, 108.0)
- added C77: 130n, Capacitor_SMD:C_0805_2012Metric_Pad1.18x1.45mm_HandSolder, B.Cu at (368.9, 118.8)
- added C78: 100n, Capacitor_SMD:C_0805_2012Metric_Pad1.18x1.45mm_HandSolder, B.Cu at (368.9, 121.8)
- added C79: 100n, Capacitor_SMD:C_0805_2012Metric_Pad1.18x1.45mm_HandSolder, B.Cu at (368.9, 124.8)
- added C80: 100n, Capacitor_SMD:C_0805_2012Metric_Pad1.18x1.45mm_HandSolder, B.Cu at (368.9, 127.8)
- added C81: 100n, Capacitor_SMD:C_0805_2012Metric_Pad1.18x1.45mm_HandSolder, B.Cu at (368.9, 130.8)
- added C82: 130n, Capacitor_SMD:C_0805_2012Metric_Pad1.18x1.45mm_HandSolder, B.Cu at (368.9, 133.8)
- added C83: 130n, Capacitor_SMD:C_0805_2012Metric_Pad1.18x1.45mm_HandSolder, B.Cu at (368.9, 136.8)
- added C84: 130n, Capacitor_SMD:C_0805_2012Metric_Pad1.18x1.45mm_HandSolder, B.Cu at (368.9, 139.8)
- added C85: 130n, Capacitor_SMD:C_0805_2012Metric_Pad1.18x1.45mm_HandSolder, B.Cu at (368.9, 142.8)
- added C86: 130n, Capacitor_SMD:C_0805_2012Metric_Pad1.18x1.45mm_HandSolder, B.Cu at (368.9, 145.9)
- added C87: 130n, Capacitor_SMD:C_0805_2012Metric_Pad1.18x1.45mm_HandSolder, B.Cu at (368.9, 148.9)
- added C88: 130n, Capacitor_SMD:C_0805_2012Metric_Pad1.18x1.45mm_HandSolder, B.Cu at (379.6, 111.0)
- added C89: 130n, Capacitor_SMD:C_0805_2012Metric_Pad1.18x1.45mm_HandSolder, B.Cu at (364.1, 118.8)
- added C90: 100n, Capacitor_SMD:C_0805_2012Metric_Pad1.18x1.45mm_HandSolder, B.Cu at (364.1, 121.8)
- added C91: 100n, Capacitor_SMD:C_0805_2012Metric_Pad1.18x1.45mm_HandSolder, B.Cu at (364.1, 124.8)
- added C92: 100n, Capacitor_SMD:C_0805_2012Metric_Pad1.18x1.45mm_HandSolder, B.Cu at (364.1, 127.8)
- added C93: 100n, Capacitor_SMD:C_0805_2012Metric_Pad1.18x1.45mm_HandSolder, B.Cu at (364.1, 130.8)
- added C94: 100n, Capacitor_SMD:C_0805_2012Metric_Pad1.18x1.45mm_HandSolder, B.Cu at (364.1, 133.8)
- added C95: 100n, Capacitor_SMD:C_0805_2012Metric_Pad1.18x1.45mm_HandSolder, B.Cu at (364.1, 136.8)
- added C96: 100n, Capacitor_SMD:C_0805_2012Metric_Pad1.18x1.45mm_HandSolder, B.Cu at (364.1, 139.8)
- added C97: 100n, Capacitor_SMD:C_0805_2012Metric_Pad1.18x1.45mm_HandSolder, B.Cu at (364.1, 142.8)
- added C98: 100n, Capacitor_SMD:C_0805_2012Metric_Pad1.18x1.45mm_HandSolder, B.Cu at (364.1, 145.9)
- added C99: 100n, Capacitor_SMD:C_0805_2012Metric_Pad1.18x1.45mm_HandSolder, B.Cu at (364.1, 148.9)
- added J22: EMK_In, Connector_PinHeader_2.54mm_LongPads:PinHeader_1x05_P2.54mm_Vertical_LongPads, F.Cu at (399.6, 42.2)
- added J24: Mic_Effekt_In, Connector_PinHeader_2.54mm_LongPads:PinHeader_1x02_P2.54mm_Vertical_LongPads, F.Cu at (369.5, 59.5)
- added J25: Mic_Effekt_In, Connector_PinHeader_2.54mm_LongPads:PinHeader_1x02_P2.54mm_Vertical_LongPads, F.Cu at (374.1, 59.5)
- added J26: Phono/Line_In, Connector_PinHeader_2.54mm_LongPads:PinHeader_1x02_P2.54mm_Vertical_LongPads, F.Cu at (378.7, 59.5)
- added J27: Mic_Effekt_In, Connector_PinHeader_2.54mm_LongPads:PinHeader_1x02_P2.54mm_Vertical_LongPads, F.Cu at (383.3, 59.5)
- added J28: Pegel_Out, Connector_PinSocket_2.54mm_LongPads:PinSocket_1x02_P2.54mm_Vertical_LongPads, F.Cu at (369.6, 27.9)
- added J29: Pegel_Out, Connector_PinSocket_2.54mm_LongPads:PinSocket_1x02_P2.54mm_Vertical_LongPads, F.Cu at (374.2, 27.9)
- added J37: AUX_Send_3, Connector_PinSocket_2.54mm_LongPads:PinSocket_1x02_P2.54mm_Vertical_LongPads, F.Cu at (378.8, 27.9)
- added J38: AUX_Send_1, Connector_PinSocket_2.54mm_LongPads:PinSocket_1x02_P2.54mm_Vertical_LongPads, F.Cu at (383.4, 27.9)
- added J39: AUX_Send_2, Connector_PinSocket_2.54mm_LongPads:PinSocket_1x02_P2.54mm_Vertical_LongPads, F.Cu at (388.0, 27.9)
- added J40: Bass_Out, Connector_PinSocket_2.54mm_LongPads:PinSocket_1x02_P2.54mm_Vertical_LongPads, F.Cu at (392.6, 27.9)
- added J41: Kick_Out, Connector_PinSocket_2.54mm_LongPads:PinSocket_1x02_P2.54mm_Vertical_LongPads, F.Cu at (369.6, 35.1)
- added J42: Mid_Out, Connector_PinSocket_2.54mm_LongPads:PinSocket_1x02_P2.54mm_Vertical_LongPads, F.Cu at (374.2, 35.1)
- added J43: High_Out, Connector_PinSocket_2.54mm_LongPads:PinSocket_1x02_P2.54mm_Vertical_LongPads, F.Cu at (378.8, 35.1)
- added J44: Line_Out_L, Connector_PinSocket_2.54mm_LongPads:PinSocket_1x02_P2.54mm_Vertical_LongPads, F.Cu at (383.4, 35.1)
- added J45: Line_Out_R, Connector_PinSocket_2.54mm_LongPads:PinSocket_1x02_P2.54mm_Vertical_LongPads, F.Cu at (388.0, 35.1)
- added R100: 10k, Resistor_SMD:R_0805_2012Metric_Pad1.20x1.40mm_HandSolder, B.Cu at (430.9, 143.6)
- added R101: 22k, Resistor_SMD:R_0805_2012Metric_Pad1.20x1.40mm_HandSolder, B.Cu at (430.9, 146.5)
- added R102: 22k, Resistor_SMD:R_0805_2012Metric_Pad1.20x1.40mm_HandSolder, B.Cu at (430.9, 149.5)
- added R103: 22k, Resistor_SMD:R_0805_2012Metric_Pad1.20x1.40mm_HandSolder, B.Cu at (430.9, 152.4)
- added R104: 22k, Resistor_SMD:R_0805_2012Metric_Pad1.20x1.40mm_HandSolder, B.Cu at (426.1, 96.4)
- added R105: 22k, Resistor_SMD:R_0805_2012Metric_Pad1.20x1.40mm_HandSolder, B.Cu at (426.1, 99.3)
- added R106: 22k, Resistor_SMD:R_0805_2012Metric_Pad1.20x1.40mm_HandSolder, B.Cu at (426.1, 102.3)
- added R107: 22k, Resistor_SMD:R_0805_2012Metric_Pad1.20x1.40mm_HandSolder, B.Cu at (426.1, 105.2)
- added R108: 22k, Resistor_SMD:R_0805_2012Metric_Pad1.20x1.40mm_HandSolder, B.Cu at (426.1, 108.2)
- added R109: 6k8, Resistor_SMD:R_0805_2012Metric_Pad1.20x1.40mm_HandSolder, B.Cu at (426.1, 111.1)
- added R110: 6k8, Resistor_SMD:R_0805_2012Metric_Pad1.20x1.40mm_HandSolder, B.Cu at (426.1, 114.1)
- added R111: 6k8, Resistor_SMD:R_0805_2012Metric_Pad1.20x1.40mm_HandSolder, B.Cu at (426.1, 117.0)
- added R112: 6k8, Resistor_SMD:R_0805_2012Metric_Pad1.20x1.40mm_HandSolder, B.Cu at (426.1, 120.0)
- added R113: 22k, Resistor_SMD:R_0805_2012Metric_Pad1.20x1.40mm_HandSolder, B.Cu at (426.1, 122.9)
- added R114: 22k, Resistor_SMD:R_0805_2012Metric_Pad1.20x1.40mm_HandSolder, B.Cu at (426.1, 125.9)
- added R115: 22k, Resistor_SMD:R_0805_2012Metric_Pad1.20x1.40mm_HandSolder, B.Cu at (426.1, 128.8)
- added R116: 22k, Resistor_SMD:R_0805_2012Metric_Pad1.20x1.40mm_HandSolder, B.Cu at (426.1, 131.8)
- added R117: 6k8, Resistor_SMD:R_0805_2012Metric_Pad1.20x1.40mm_HandSolder, B.Cu at (426.1, 134.7)
- added R118: 6k8, Resistor_SMD:R_0805_2012Metric_Pad1.20x1.40mm_HandSolder, B.Cu at (426.1, 137.7)
- added R119: 6k8, Resistor_SMD:R_0805_2012Metric_Pad1.20x1.40mm_HandSolder, B.Cu at (426.1, 140.6)
- added R120: 6k8, Resistor_SMD:R_0805_2012Metric_Pad1.20x1.40mm_HandSolder, B.Cu at (426.1, 143.6)
- added R121: 4k7, Resistor_SMD:R_0805_2012Metric_Pad1.20x1.40mm_HandSolder, B.Cu at (426.1, 146.5)
- added R122: 470R, Resistor_SMD:R_0805_2012Metric_Pad1.20x1.40mm_HandSolder, B.Cu at (426.1, 149.5)
- added R123: 4k7, Resistor_SMD:R_0805_2012Metric_Pad1.20x1.40mm_HandSolder, B.Cu at (426.1, 152.4)
- added R124: 470R, Resistor_SMD:R_0805_2012Metric_Pad1.20x1.40mm_HandSolder, B.Cu at (421.4, 96.4)
- added R125: 1k, Resistor_SMD:R_0805_2012Metric_Pad1.20x1.40mm_HandSolder, B.Cu at (421.4, 99.3)
- added R126: 1k, Resistor_SMD:R_0805_2012Metric_Pad1.20x1.40mm_HandSolder, B.Cu at (421.4, 102.3)
- added R127: 22k, Resistor_SMD:R_0805_2012Metric_Pad1.20x1.40mm_HandSolder, B.Cu at (421.4, 105.2)
- added R128: 22k, Resistor_SMD:R_0805_2012Metric_Pad1.20x1.40mm_HandSolder, B.Cu at (421.4, 108.2)
- added R129: 22k, Resistor_SMD:R_0805_2012Metric_Pad1.20x1.40mm_HandSolder, B.Cu at (421.4, 111.1)
- added R130: 22k, Resistor_SMD:R_0805_2012Metric_Pad1.20x1.40mm_HandSolder, B.Cu at (421.4, 114.1)
- added R131: 10k, Resistor_SMD:R_0805_2012Metric_Pad1.20x1.40mm_HandSolder, B.Cu at (421.4, 117.0)
- added R132: 10k, Resistor_SMD:R_0805_2012Metric_Pad1.20x1.40mm_HandSolder, B.Cu at (421.4, 120.0)
- added R133: 6k8, Resistor_SMD:R_0805_2012Metric_Pad1.20x1.40mm_HandSolder, B.Cu at (421.4, 122.9)
- added R134: 6k8, Resistor_SMD:R_0805_2012Metric_Pad1.20x1.40mm_HandSolder, B.Cu at (421.4, 125.9)
- added R135: 6k8, Resistor_SMD:R_0805_2012Metric_Pad1.20x1.40mm_HandSolder, B.Cu at (421.4, 128.8)
- added R136: 6k8, Resistor_SMD:R_0805_2012Metric_Pad1.20x1.40mm_HandSolder, B.Cu at (421.4, 131.8)
- added R137: 22k, Resistor_SMD:R_0805_2012Metric_Pad1.20x1.40mm_HandSolder, B.Cu at (421.4, 134.7)
- added R138: 22k, Resistor_SMD:R_0805_2012Metric_Pad1.20x1.40mm_HandSolder, B.Cu at (421.4, 137.7)
- added R139: 22k, Resistor_SMD:R_0805_2012Metric_Pad1.20x1.40mm_HandSolder, B.Cu at (421.4, 140.6)
- added R140: 22k, Resistor_SMD:R_0805_2012Metric_Pad1.20x1.40mm_HandSolder, B.Cu at (421.4, 143.6)
- added R141: 6k8, Resistor_SMD:R_0805_2012Metric_Pad1.20x1.40mm_HandSolder, B.Cu at (421.4, 146.5)
- added R142: 6k8, Resistor_SMD:R_0805_2012Metric_Pad1.20x1.40mm_HandSolder, B.Cu at (421.4, 149.5)
- added R143: 6k8, Resistor_SMD:R_0805_2012Metric_Pad1.20x1.40mm_HandSolder, B.Cu at (421.4, 152.4)
- added R144: 6k8, Resistor_SMD:R_0805_2012Metric_Pad1.20x1.40mm_HandSolder, B.Cu at (416.6, 96.4)
- added R145: 10k, Resistor_SMD:R_0805_2012Metric_Pad1.20x1.40mm_HandSolder, B.Cu at (416.6, 99.3)
- added R146: 10k, Resistor_SMD:R_0805_2012Metric_Pad1.20x1.40mm_HandSolder, B.Cu at (416.6, 102.3)
- added R147: 10k, Resistor_SMD:R_0805_2012Metric_Pad1.20x1.40mm_HandSolder, B.Cu at (416.6, 105.2)
- added R148: 10k, Resistor_SMD:R_0805_2012Metric_Pad1.20x1.40mm_HandSolder, B.Cu at (416.6, 108.2)
- added R149: 10k, Resistor_SMD:R_0805_2012Metric_Pad1.20x1.40mm_HandSolder, B.Cu at (416.6, 111.1)
- added R33: 5k, Resistor_SMD:R_0805_2012Metric_Pad1.20x1.40mm_HandSolder, B.Cu at (434.8, 91.4)
- added R34: 5k, Resistor_SMD:R_0805_2012Metric_Pad1.20x1.40mm_HandSolder, B.Cu at (440.4, 99.3)
- added R35: 4k7, Resistor_SMD:R_0805_2012Metric_Pad1.20x1.40mm_HandSolder, B.Cu at (440.4, 102.3)
- added R36: 470R, Resistor_SMD:R_0805_2012Metric_Pad1.20x1.40mm_HandSolder, B.Cu at (440.4, 105.2)
- added R37: 4k7, Resistor_SMD:R_0805_2012Metric_Pad1.20x1.40mm_HandSolder, B.Cu at (440.4, 108.2)
- added R38: 470R, Resistor_SMD:R_0805_2012Metric_Pad1.20x1.40mm_HandSolder, B.Cu at (440.4, 111.1)
- added R39: 4k7, Resistor_SMD:R_0805_2012Metric_Pad1.20x1.40mm_HandSolder, B.Cu at (440.4, 114.1)
- added R40: 470R, Resistor_SMD:R_0805_2012Metric_Pad1.20x1.40mm_HandSolder, B.Cu at (440.4, 117.0)
- added R41: 4k7, Resistor_SMD:R_0805_2012Metric_Pad1.20x1.40mm_HandSolder, B.Cu at (440.4, 120.0)
- added R42: 470R, Resistor_SMD:R_0805_2012Metric_Pad1.20x1.40mm_HandSolder, B.Cu at (440.4, 122.9)
- added R43: 10k, Resistor_SMD:R_0805_2012Metric_Pad1.20x1.40mm_HandSolder, B.Cu at (440.4, 125.9)
- added R44: 5k, Resistor_SMD:R_0805_2012Metric_Pad1.20x1.40mm_HandSolder, B.Cu at (440.4, 128.8)
- added R45: 10k, Resistor_SMD:R_0805_2012Metric_Pad1.20x1.40mm_HandSolder, B.Cu at (440.4, 131.8)
- added R46: 5k, Resistor_SMD:R_0805_2012Metric_Pad1.20x1.40mm_HandSolder, B.Cu at (440.4, 134.7)
- added R47: 1k, Resistor_SMD:R_0805_2012Metric_Pad1.20x1.40mm_HandSolder, B.Cu at (440.4, 137.7)
- added R48: 1k, Resistor_SMD:R_0805_2012Metric_Pad1.20x1.40mm_HandSolder, B.Cu at (440.4, 140.6)
- added R49: 1k, Resistor_SMD:R_0805_2012Metric_Pad1.20x1.40mm_HandSolder, B.Cu at (440.4, 143.6)
- added R50: 1k, Resistor_SMD:R_0805_2012Metric_Pad1.20x1.40mm_HandSolder, B.Cu at (440.4, 146.5)
- added R51: 5k, Resistor_SMD:R_0805_2012Metric_Pad1.20x1.40mm_HandSolder, B.Cu at (440.4, 149.5)
- added R52: 5k, Resistor_SMD:R_0805_2012Metric_Pad1.20x1.40mm_HandSolder, B.Cu at (440.4, 152.4)
- added R53: 10k, Resistor_SMD:R_0805_2012Metric_Pad1.20x1.40mm_HandSolder, B.Cu at (441.1, 94.4)
- added R54: 10k, Resistor_SMD:R_0805_2012Metric_Pad1.20x1.40mm_HandSolder, B.Cu at (435.6, 99.3)
- added R55: 10k, Resistor_SMD:R_0805_2012Metric_Pad1.20x1.40mm_HandSolder, B.Cu at (435.6, 102.3)
- added R56: 10k, Resistor_SMD:R_0805_2012Metric_Pad1.20x1.40mm_HandSolder, B.Cu at (435.6, 105.2)
- added R57: 10k, Resistor_SMD:R_0805_2012Metric_Pad1.20x1.40mm_HandSolder, B.Cu at (435.6, 108.2)
- added R58: 10k, Resistor_SMD:R_0805_2012Metric_Pad1.20x1.40mm_HandSolder, B.Cu at (435.6, 111.1)
- added R61: 10k, Resistor_SMD:R_0805_2012Metric_Pad1.20x1.40mm_HandSolder, B.Cu at (435.6, 114.1)
- added R62: 10k, Resistor_SMD:R_0805_2012Metric_Pad1.20x1.40mm_HandSolder, B.Cu at (435.6, 117.0)
- added R63: 10k, Resistor_SMD:R_0805_2012Metric_Pad1.20x1.40mm_HandSolder, B.Cu at (435.6, 120.0)
- added R64: 10k, Resistor_SMD:R_0805_2012Metric_Pad1.20x1.40mm_HandSolder, B.Cu at (435.6, 122.9)
- added R65: 10k, Resistor_SMD:R_0805_2012Metric_Pad1.20x1.40mm_HandSolder, B.Cu at (435.6, 125.9)
- added R66: 10k, Resistor_SMD:R_0805_2012Metric_Pad1.20x1.40mm_HandSolder, B.Cu at (435.6, 128.8)
- added R69: 10k, Resistor_SMD:R_0805_2012Metric_Pad1.20x1.40mm_HandSolder, B.Cu at (435.6, 131.8)
- added R70: 10k, Resistor_SMD:R_0805_2012Metric_Pad1.20x1.40mm_HandSolder, B.Cu at (435.6, 134.7)
- added R73: 10k, Resistor_SMD:R_0805_2012Metric_Pad1.20x1.40mm_HandSolder, B.Cu at (435.6, 137.7)
- added R74: 10k, Resistor_SMD:R_0805_2012Metric_Pad1.20x1.40mm_HandSolder, B.Cu at (435.6, 140.6)
- added R76: 10k, Resistor_SMD:R_0805_2012Metric_Pad1.20x1.40mm_HandSolder, B.Cu at (435.6, 143.6)
- added R77: 4k7, Resistor_SMD:R_0805_2012Metric_Pad1.20x1.40mm_HandSolder, B.Cu at (435.6, 146.5)
- added R78: 470R, Resistor_SMD:R_0805_2012Metric_Pad1.20x1.40mm_HandSolder, B.Cu at (435.6, 149.5)
- added R79: 10k, Resistor_SMD:R_0805_2012Metric_Pad1.20x1.40mm_HandSolder, B.Cu at (435.6, 152.4)
- added R80: 1k, Resistor_SMD:R_0805_2012Metric_Pad1.20x1.40mm_HandSolder, B.Cu at (430.9, 96.4)
- added R83: 10k, Resistor_SMD:R_0805_2012Metric_Pad1.20x1.40mm_HandSolder, B.Cu at (430.9, 99.3)
- added R85: 10k, Resistor_SMD:R_0805_2012Metric_Pad1.20x1.40mm_HandSolder, B.Cu at (430.9, 102.3)
- added R87: 6k8, Resistor_SMD:R_0805_2012Metric_Pad1.20x1.40mm_HandSolder, B.Cu at (430.9, 105.2)
- added R88: 6k8, Resistor_SMD:R_0805_2012Metric_Pad1.20x1.40mm_HandSolder, B.Cu at (430.9, 108.2)
- added R89: 6k8, Resistor_SMD:R_0805_2012Metric_Pad1.20x1.40mm_HandSolder, B.Cu at (430.9, 111.1)
- added R90: 6k8, Resistor_SMD:R_0805_2012Metric_Pad1.20x1.40mm_HandSolder, B.Cu at (430.9, 114.1)
- added R91: 22k, Resistor_SMD:R_0805_2012Metric_Pad1.20x1.40mm_HandSolder, B.Cu at (430.9, 117.0)
- added R92: 6k8, Resistor_SMD:R_0805_2012Metric_Pad1.20x1.40mm_HandSolder, B.Cu at (430.9, 120.0)
- added R93: 22k, Resistor_SMD:R_0805_2012Metric_Pad1.20x1.40mm_HandSolder, B.Cu at (430.9, 122.9)
- added R94: 6k8, Resistor_SMD:R_0805_2012Metric_Pad1.20x1.40mm_HandSolder, B.Cu at (430.9, 125.9)
- added R95: 22k, Resistor_SMD:R_0805_2012Metric_Pad1.20x1.40mm_HandSolder, B.Cu at (430.9, 128.8)
- added R96: 6k8, Resistor_SMD:R_0805_2012Metric_Pad1.20x1.40mm_HandSolder, B.Cu at (430.9, 131.8)
- added R97: 22k, Resistor_SMD:R_0805_2012Metric_Pad1.20x1.40mm_HandSolder, B.Cu at (430.9, 134.7)
- added R98: 6k8, Resistor_SMD:R_0805_2012Metric_Pad1.20x1.40mm_HandSolder, B.Cu at (430.9, 137.7)
- added R99: 10k, Resistor_SMD:R_0805_2012Metric_Pad1.20x1.40mm_HandSolder, B.Cu at (430.9, 140.6)
- added RV10: 50k log, Connector_PinSocket_2.54mm_LongPads:PinSocket_1x03_P2.54mm_Vertical_LongPads, F.Cu at (423.0, 34.3)
- added RV11: 50k log, Connector_PinSocket_2.54mm_LongPads:PinSocket_1x03_P2.54mm_Vertical_LongPads, F.Cu at (427.6, 34.3)
- added RV12: 47k lin, Connector_PinSocket_2.54mm_LongPads:PinSocket_1x03_P2.54mm_Vertical_LongPads, F.Cu at (432.2, 34.3)
- added RV13: 47k lin, Connector_PinSocket_2.54mm_LongPads:PinSocket_1x03_P2.54mm_Vertical_LongPads, F.Cu at (436.8, 34.3)
- added RV14: 47k lin, Connector_PinSocket_2.54mm_LongPads:PinSocket_1x03_P2.54mm_Vertical_LongPads, F.Cu at (441.4, 34.3)
- added RV15: 47k lin, Connector_PinSocket_2.54mm_LongPads:PinSocket_1x03_P2.54mm_Vertical_LongPads, F.Cu at (446.0, 34.3)
- added RV16: 220k log, Connector_PinSocket_2.54mm_LongPads:PinSocket_1x06_P2.54mm_Vertical_LongPads, F.Cu at (395.0, 42.2)
- added RV17: 220k log, Connector_PinSocket_2.54mm_LongPads:PinSocket_1x06_P2.54mm_Vertical_LongPads, F.Cu at (374.2, 42.2)
- added RV18: 220k log, Connector_PinSocket_2.54mm_LongPads:PinSocket_1x06_P2.54mm_Vertical_LongPads, F.Cu at (378.8, 42.2)
- added RV19: 220k log, Connector_PinSocket_2.54mm_LongPads:PinSocket_1x06_P2.54mm_Vertical_LongPads, F.Cu at (383.4, 42.2)
- added RV20: 220k log, Connector_PinSocket_2.54mm_LongPads:PinSocket_1x06_P2.54mm_Vertical_LongPads, F.Cu at (388.0, 42.2)
- added RV21: 50k log, Connector_PinSocket_2.54mm_LongPads:PinSocket_1x03_P2.54mm_Vertical_LongPads, F.Cu at (450.6, 34.3)
- added RV22: 50k log, Connector_PinSocket_2.54mm_LongPads:PinSocket_1x03_P2.54mm_Vertical_LongPads, F.Cu at (455.2, 34.3)
- added RV7: 50k log, Connector_PinSocket_2.54mm_LongPads:PinSocket_1x03_P2.54mm_Vertical_LongPads, F.Cu at (409.2, 34.3)
- added RV8: 50k log, Connector_PinSocket_2.54mm_LongPads:PinSocket_1x03_P2.54mm_Vertical_LongPads, F.Cu at (413.8, 34.3)
- added RV9: 50k log, Connector_PinSocket_2.54mm_LongPads:PinSocket_1x03_P2.54mm_Vertical_LongPads, F.Cu at (418.4, 34.3)
- added SW10: SW_SPDT, Connector_PinHeader_2.54mm_LongPads:PinHeader_1x03_P2.54mm_Vertical_LongPads, F.Cu at (436.7, 44.0)
- added SW11: SW_SPDT, Connector_PinHeader_2.54mm_LongPads:PinHeader_1x03_P2.54mm_Vertical_LongPads, F.Cu at (441.3, 44.0)
- added SW12: SW_SPDT, Connector_PinHeader_2.54mm_LongPads:PinHeader_1x03_P2.54mm_Vertical_LongPads, F.Cu at (445.9, 44.0)
- added SW3: SW_SPDT, Connector_PinHeader_2.54mm_LongPads:PinHeader_1x03_P2.54mm_Vertical_LongPads, F.Cu at (409.1, 44.0)
- added SW4: SW_SPDT, Connector_PinHeader_2.54mm_LongPads:PinHeader_1x03_P2.54mm_Vertical_LongPads, F.Cu at (413.7, 44.0)
- added SW5: SW_SPDT, Connector_PinHeader_2.54mm_LongPads:PinHeader_1x03_P2.54mm_Vertical_LongPads, F.Cu at (418.3, 44.0)
- added SW6: SW_SPDT, Connector_PinHeader_2.54mm_LongPads:PinHeader_1x03_P2.54mm_Vertical_LongPads, F.Cu at (422.9, 44.0)
- added SW7: SW_SPDT, Connector_PinHeader_2.54mm_LongPads:PinHeader_1x03_P2.54mm_Vertical_LongPads, F.Cu at (427.5, 44.0)
- added SW8: SW_SPDT, Connector_PinHeader_2.54mm_LongPads:PinHeader_1x03_P2.54mm_Vertical_LongPads, F.Cu at (432.1, 44.0)
- added U10: TL074, Package_DIP:DIP-14_W7.62mm_Socket_LongPads, F.Cu at (109.2, 54.6)
- added U11: TL074, Package_DIP:DIP-14_W7.62mm_Socket_LongPads, F.Cu at (134.6, 54.6)
- added U12: TL074, Package_DIP:DIP-14_W7.62mm_Socket_LongPads, F.Cu at (160.0, 54.6)
- added U13: TL074, Package_DIP:DIP-14_W7.62mm_Socket_LongPads, F.Cu at (58.4, 81.3)
- added U14: TL074, Package_DIP:DIP-14_W7.62mm_Socket_LongPads, F.Cu at (83.8, 81.3)
- added U15: TL074, Package_DIP:DIP-14_W7.62mm_Socket_LongPads, F.Cu at (109.2, 81.3)
- added U16: TL074, Package_DIP:DIP-14_W7.62mm_Socket_LongPads, F.Cu at (134.6, 81.3)
- added U17: TL074, Package_DIP:DIP-14_W7.62mm_Socket_LongPads, F.Cu at (160.0, 81.3)
- added U18: TL074, Package_DIP:DIP-14_W7.62mm_Socket_LongPads, F.Cu at (58.4, 106.7)
- added U19: TL074, Package_DIP:DIP-14_W7.62mm_Socket_LongPads, F.Cu at (83.8, 106.7)
- added U20: TL074, Package_DIP:DIP-14_W7.62mm_Socket_LongPads, F.Cu at (109.2, 106.7)
- added U21: TL074, Package_DIP:DIP-14_W7.62mm_Socket_LongPads, F.Cu at (134.6, 106.7)
- added U22: TL074, Package_DIP:DIP-14_W7.62mm_Socket_LongPads, F.Cu at (160.0, 108.0)
- added U8: TL074, Package_DIP:DIP-14_W7.62mm_Socket_LongPads, F.Cu at (58.4, 54.6)
- added U9: TL074, Package_DIP:DIP-14_W7.62mm_Socket_LongPads, F.Cu at (83.8, 54.6)
- added Z101: ~, Resistor_SMD:R_0805_2012Metric_Pad1.20x1.40mm_HandSolder, B.Cu at (416.6, 114.1)
- added Z102: ~, Resistor_SMD:R_0805_2012Metric_Pad1.20x1.40mm_HandSolder, B.Cu at (416.6, 117.0)
- added Z103: ~, Resistor_SMD:R_0805_2012Metric_Pad1.20x1.40mm_HandSolder, B.Cu at (416.6, 120.0)
- added Z104: ~, Resistor_SMD:R_0805_2012Metric_Pad1.20x1.40mm_HandSolder, B.Cu at (416.6, 122.9)
- added Z105: ~, Resistor_SMD:R_0805_2012Metric_Pad1.20x1.40mm_HandSolder, B.Cu at (416.6, 125.9)
- added Z106: ~, Resistor_SMD:R_0805_2012Metric_Pad1.20x1.40mm_HandSolder, B.Cu at (416.6, 128.8)
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Routing:
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- removed copper zone on F.Cu, net 9V_GND_P
- removed copper zone on B.Cu, net GND_15V_FILT
- removed copper zone on B.Cu, net GND_9V_FILT
- removed copper zone on In1.Cu, net GND_M
- removed copper zone on F.Cu, net GND_P
- removed copper zone on F.Cu, net Net-(C11-Pad2)
- removed copper zone on F.Cu, net Net-(C12-Pad2)
- removed copper zone on F.Cu, net Net-(C18-Pad1)
- removed copper zone on F.Cu, net Net-(C2-Pad1)
- removed copper zone on F.Cu, net Net-(C2-Pad2)
- removed copper zone on F.Cu, net Net-(D1-K)
- removed copper zone on F.Cu, net Net-(D2-A)
- removed copper zone on F.Cu, net Net-(J30-Pin_2)
- removed copper zone on F.Cu, net Net-(J31-Pin_2)
- removed copper zone on F.Cu, net Net-(J32-Pin_2)
- removed copper zone on F.Cu, net Net-(R59-Pad1)
- removed copper zone on F.Cu, net Net-(U6-+VIN)
- removed copper zone on F.Cu, net Net-(U6--VIN)
Other:
- board text removed: "J21"

Commit message: PCB Update
Parts:
- moved U11 442.0 mm to (576.6, 58.4)
- moved U12 442.0 mm to (602.0, 58.4)
- moved U16 442.0 mm to (576.6, 85.1)
- moved U17 442.0 mm to (602.0, 85.1)
- moved U21 442.0 mm to (576.6, 110.5)
- moved U22 442.0 mm to (602.0, 111.8)
- moved U13 442.0 mm to (500.4, 85.1)
- moved U14 442.0 mm to (525.8, 85.1)
- moved U18 442.0 mm to (500.4, 110.5)
- moved U19 442.0 mm to (525.8, 110.5)
- moved U8 442.0 mm to (500.4, 58.4)
- moved U9 442.0 mm to (525.8, 58.4)
- moved U10 442.0 mm to (551.2, 58.4)
- moved U15 442.0 mm to (551.2, 85.1)
- moved U20 442.0 mm to (551.2, 110.5)
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Routing:
- net Net-(J26-Pin_1): track 0.00 -> 5.35 mm
- net Net-(J26-Pin_2): track 0.00 -> 2.81 mm
- net Net-(U10A-+): track 0.00 -> 2.54 mm

Commit message: PCB Update
Other:
- board size 150 x 85.2 mm -> 150 x 109.9 mm
Changed lines of the file:
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@@
 	)
 	(gr_rect
-		(start 37.73 45.08)
+		(start 37.73 20.315)
 		(end 187.73 130.254)
 		(stroke

Commit message: PCB Update
Parts:
- added Z257: ~, Resistor_SMD:R_0805_2012Metric_Pad1.20x1.40mm_HandSolder, B.Cu at (55.9, 38.1)
- added Z258: ~, Resistor_SMD:R_0805_2012Metric_Pad1.20x1.40mm_HandSolder, B.Cu at (55.9, 40.6)
- added Z259: ~, Resistor_SMD:R_0805_2012Metric_Pad1.20x1.40mm_HandSolder, B.Cu at (55.9, 35.6)
- moved Z113 370.0 mm to (55.9, 67.3)
- moved Z109 367.1 mm to (55.9, 69.8), turned to 0 degrees
- moved Z112 365.7 mm to (55.9, 86.4), turned to 0 degrees
- moved Z105 364.7 mm to (55.9, 72.4), turned to 0 degrees
- moved Z108 363.7 mm to (55.9, 88.9), turned to 0 degrees
- moved Z111 363.3 mm to (55.9, 100.3), turned to 0 degrees
- moved Z102 363.2 mm to (55.9, 74.9), turned to 0 degrees
- moved Z120 362.4 mm to (55.9, 43.2), turned to 0 degrees
- moved Z107 361.9 mm to (55.9, 102.9), turned to 0 degrees
- moved Z121 361.6 mm to (55.9, 50.8)
- moved Z101 361.5 mm to (55.9, 91.4), turned to 0 degrees
- moved Z104 361.2 mm to (55.9, 105.4), turned to 0 degrees
- moved Z119 360.2 mm to (55.9, 53.3)
- moved Z118 359.1 mm to (55.9, 58.4), turned to 0 degrees
- moved Z117 359.0 mm to (55.9, 55.9), turned to 0 degrees
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Connections:
- U21 pad 12: Net-(J29-Pin_1) -> Net-(U21D-+)
- U22 pad 3: Net-(J29-Pin_1) -> Net-(U21D-+)
- Z226 pad 2: Net-(J29-Pin_1) -> Net-(U21D-+)
Routing:
- net Net-(J27-Pin_1): track 0.00 -> 5.35 mm
- net Net-(J25-Pin_1): track 0.00 -> 5.35 mm
- net Net-(J24-Pin_1): track 0.00 -> 5.35 mm
- net Net-(J29-Pin_1): track 0.00 -> 5.35 mm
- net Net-(J28-Pin_1): track 0.00 -> 5.35 mm
- net Net-(J41-Pin_1): track 0.00 -> 5.35 mm
- net Net-(J40-Pin_1): track 0.00 -> 5.35 mm
- net Net-(J43-Pin_1): track 0.00 -> 5.35 mm
- net Net-(J42-Pin_1): track 0.00 -> 5.35 mm
- net Net-(J29-Pin_2): track 0.00 -> 2.81 mm
- net Net-(J28-Pin_2): track 0.00 -> 2.81 mm
- net Net-(J27-Pin_2): track 0.00 -> 2.81 mm
- net Net-(J25-Pin_2): track 0.00 -> 2.81 mm
- net Net-(J24-Pin_2): track 0.00 -> 2.81 mm
- net Net-(U20C--): track 0.00 -> 2.54 mm
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
Commit message: PCB Update
Parts:
- moved Z235 454.1 mm to (-54.9, 71.1)
- moved Z255 448.6 mm to (-54.9, 76.2), turned to 0 degrees
- moved J45 448.0 mm to (-54.9, 102.9)
- moved Z236 447.0 mm to (-51.1, 97.8)
- moved Z245 445.1 mm to (-54.9, 73.7)
- moved J44 444.0 mm to (-58.7, 76.2)
- moved Z256 441.7 mm to (-51.1, 102.9), turned to 0 degrees
- moved Z246 439.7 mm to (-51.1, 100.3)
- moved J24 171.3 mm to (-109.0, 30.5)
- moved Z101 171.3 mm to (-105.1, 33.0)
- moved Z108 171.3 mm to (-105.1, 30.5)
- moved Z112 171.3 mm to (-105.1, 27.9)
- moved Z116 171.3 mm to (-105.1, 25.4)
- moved J28 159.9 mm to (-104.4, 88.9)
- moved Z117 159.9 mm to (-100.6, 88.9)
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Routing:
- net Net-(J45-Pin_1): track 0.00 -> 5.35 mm
- net Net-(J44-Pin_1): track 0.00 -> 5.35 mm
- net Net-(U22A--): track 0.00 -> 2.54 mm
- net Net-(U21D--): track 0.00 -> 2.54 mm

Commit message: PCB Update
Parts:
- SW10, SW11, SW12, SW3, SW4, SW5, SW6, SW7, SW8: footprint Connector_PinHeader_2.54mm_LongPads:PinHeader_1x03_P2.54mm_Vertical_LongPads -> Connector_PinHeader_2.54mm_LongPads:PinHeader_1x02_P2.54mm_Vertical_LongPads
- moved U8 370.7 mm to (133.3, 110.5)
- moved RV10 311.0 mm to (125.7, 125.7), turned to 180 degrees
- moved SW6 304.6 mm to (129.5, 125.7), turned to 180 degrees
- moved R41 303.3 mm to (137.2, 125.7), turned to 0 degrees
- moved R39 303.3 mm to (137.2, 110.5), turned to 0 degrees
- moved R42 303.2 mm to (137.2, 120.7), turned to 0 degrees
- moved R40 303.2 mm to (137.2, 115.6), turned to 0 degrees
- moved RV9 302.4 mm to (125.7, 110.5)
- moved R49 296.9 mm to (144.8, 115.6)
- moved R50 296.7 mm to (144.8, 120.7)
- moved SW5 296.3 mm to (129.5, 110.5)
- moved R56 295.8 mm to (141.0, 130.8), turned to 0 degrees
- moved R55 294.7 mm to (141.0, 108.0), turned to 0 degrees
- moved Z146 269.1 mm to (144.8, 108.0)
- moved Z147 267.6 mm to (144.8, 128.3)
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Connections:
- C38 pad 2: Net-(U8C--) -> Net-(U9B--)
- C42 pad 1: Net-(U8D-+) -> Net-(U9A-+)
- R101 pad 1: Net-(U8D--) -> Net-(U9A--)
- R39 pad 2: Net-(U8B--) -> Net-(U8D--)
- R40 pad 2: Net-(U8B-+) -> Net-(U8D-+)
- R41 pad 2: Net-(U9B--) -> Net-(U8C--)
- R42 pad 2: Net-(U9B-+) -> Net-(U8C-+)
- R49 pad 2: Net-(U8B-+) -> Net-(U8D-+)
- R50 pad 2: Net-(U9B-+) -> Net-(U8C-+)
- R55 pad 1: Net-(U8B--) -> Net-(U8D--)
- R56 pad 1: Net-(U9B--) -> Net-(U8C--)
- R91 pad 2: Net-(U8D--) -> Net-(U9A--)
- RV12 pad 2: Net-(U8C-+) -> Net-(U9B-+)
- RV17 pad 1: Net-(U8D-+) -> Net-(U9A-+)
- RV17 pad 2: Net-(U8D-+) -> Net-(U9A-+)
- RV17 pad 5: Net-(U8D-+) -> Net-(U9A-+)
- RV17 pad 6: Net-(U8D-+) -> Net-(U9A-+)
- U8 pad 14: Net-(R101-Pad2) -> Net-(R55-Pad2)
- U8 pad 5: Net-(U8B-+) -> Net-(U10A-+)
- U8 pad 6: Net-(U8B--) -> Net-(SW6-B)
- U8 pad 7: Net-(R55-Pad2) -> Net-(SW6-A)
- U8 pad 8: Net-(U8C--) -> Net-(R56-Pad2)
- U9 pad 1: Net-(SW6-A) -> Net-(R101-Pad2)
- U9 pad 2: Net-(SW6-B) -> Net-(U9A--)
- U9 pad 3: Net-(U10A-+) -> Net-(U9A-+)
- U9 pad 7: Net-(R56-Pad2) -> Net-(U9B--)
Routing:
- net Net-(SW6-B): track 0.00 -> 14.6 mm
- net Net-(SW5-B): track 0.00 -> 14.6 mm
- net Net-(U8C--): track 0.00 -> 10.8 mm
- net Net-(SW6-A): track 0.00 -> 10.4 mm
- net Net-(SW5-A): track 0.00 -> 10.4 mm
- net Net-(U10A-+): track 5.08 -> 13.8 mm
- net Net-(R56-Pad2): track 0.00 -> 8.30 mm
- net Net-(U8D--): track 0.00 -> 8.27 mm
- net Net-(Z141-Pad2): track 0.00 -> 5.91 mm
- net Net-(Z140-Pad2): track 0.00 -> 5.91 mm
- net Net-(R55-Pad2): track 0.00 -> 5.76 mm
- net Net-(U8D-+): track 0.00 -> 5.62 mm
- net Net-(U8C-+): track 0.00 -> 2.81 mm
- net -15V: track 0.00 -> 2.77 mm
- net +15V: track 0.00 -> 2.77 mm
Other:
- board size 150 x 109.9 mm -> 150 x 113.7 mm
- board text added: "."

Commit message: PCB Update
Parts:
- added J21: Conn_01x05_bridged, Connector_Bridged_2.54mm_LongPads:Bridge_2x05_P2.54mm_Vertical_LongPads, F.Cu at (-122.8, 253.2)
- C100, C101, C102, C103, C104, C105, C106, C107, C108, C109, C110, C111, C35, C37, C38, C39, C40, C41, C42, C43, C44, C45, C48, C49, C50, C51, C52, C53, C54, C55, C58, C59, C60, C61, C62, C63, C64, C65, C68, C69, C70, C71, C72, C73, C74, C75, C76, C77, C80, C81, C82, C83, C84, C85, C86, C87, C88, C89, C90, C91, C92, C93, C94, C95, C96, C97, C98, C99, R100, R101, R102, R103, R104, R105, R106, R107, R108, R109, R110, R111, R112, R113, R114, R115, R116, R117, R118, R119, R120, R121, R122, R123, R124, R125, R126, R127, R128, R129, R130, R131, R132, R133, R134, R135, R136, R137, R138, R139, R140, R141, R142, R143, R144, R145, R146, R147, R148, R149, R33, R34, R43, R44, R45, R46, R51, R52, R57, R58, R61, R62, R63, R64, R65, R66, R69, R70, R73, R74, R76, R77, R78, R79, R80, R83, R85, R87, R88, R89, R90, R91, R92, R93, R94, R95, R96, R97, R98, R99, Z142, Z143, Z148, Z149, Z154, Z155, Z156, Z157, Z158, Z159, Z160, Z161, Z162, Z163, Z164, Z165, Z166, Z169, Z175, Z176, Z177, Z178, Z179, Z180, Z181, Z182, Z183, Z184, Z185, Z186, Z187, Z188, Z189, Z190, Z191, Z192, Z193, Z194, Z195, Z196, Z197, Z198, Z199, Z200, Z201, Z202, Z203, Z204, Z205, Z206, Z207, Z208, Z209, Z210, Z211, Z212, Z213, Z214, Z215, Z216, Z217, Z218, Z219, Z220, Z221, Z222, Z223, Z224, Z225, Z226, Z227, Z230, Z232, Z234, Z237, Z240, Z242, Z244, Z247, Z250, Z252, Z254: moved to F.Cu
- moved J22 650.4 mm to (-109.1, 284.8)
- moved R33 639.4 mm to (-175.1, 252.3), turned to 0 degrees
- moved R34 639.4 mm to (-175.1, 255.3), turned to 0 degrees
- moved R51 638.3 mm to (-175.1, 270.0), turned to 0 degrees
- moved R52 638.3 mm to (-175.1, 273.0), turned to 0 degrees
- moved R57 635.5 mm to (-175.1, 275.9), turned to 0 degrees
- moved R58 635.5 mm to (-175.1, 278.9), turned to 0 degrees
- moved R61 635.5 mm to (-175.1, 281.8), turned to 0 degrees
- moved R62 635.5 mm to (-175.1, 284.8), turned to 0 degrees
- moved R63 635.5 mm to (-175.1, 287.7), turned to 0 degrees
- moved R64 635.5 mm to (-175.1, 290.7), turned to 0 degrees
- moved R65 635.5 mm to (-175.1, 293.6), turned to 0 degrees
- moved R66 635.5 mm to (-175.1, 296.6), turned to 0 degrees
- moved R43 634.6 mm to (-175.1, 258.2), turned to 0 degrees
- moved R44 634.6 mm to (-175.1, 261.2), turned to 0 degrees
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Connections:
- net +15V renamed +15V_O
- net +9V renamed +9V_O
- net -15V renamed -15V_O
- net 9V_GND renamed 9V_GND_O
- net GND renamed GND_O
- C38 pad 2: Net-(U9B--) -> Net-(U10B--)
- C39 pad 2: Net-(U9C--) -> Net-(U11C--)
- C42 pad 1: Net-(U9A-+) -> Net-(U10A-+)
- C43 pad 1: Net-(U9D-+) -> Net-(U11B-+)
- R101 pad 1: Net-(U9A--) -> Net-(U10A--)
- R102 pad 1: Net-(U9D--) -> Net-(U11B--)
- R35 pad 2: Net-(U10B--) -> Net-(U9D--)
- R36 pad 2: Net-(U10B-+) -> Net-(U9D-+)
- R37 pad 2: Net-(U11C--) -> Net-(U9C--)
- R38 pad 2: Net-(U11C-+) -> Net-(U9C-+)
- R47 pad 2: Net-(U10B-+) -> Net-(U9D-+)
- R48 pad 2: Net-(U11C-+) -> Net-(U9C-+)
- R53 pad 1: Net-(U10B--) -> Net-(U9D--)
- R54 pad 1: Net-(U11C--) -> Net-(U9C--)
- R91 pad 2: Net-(U9A--) -> Net-(U10A--)
- R93 pad 2: Net-(U9D--) -> Net-(U11B--)
- RV12 pad 2: Net-(U9B-+) -> Net-(U10B-+)
- RV13 pad 2: Net-(U9C-+) -> Net-(U11C-+)
- RV17 pad 1: Net-(U9A-+) -> Net-(U10A-+)
- RV17 pad 2: Net-(U9A-+) -> Net-(U10A-+)
- RV17 pad 5: Net-(U9A-+) -> Net-(U10A-+)
- RV17 pad 6: Net-(U9A-+) -> Net-(U10A-+)
- RV18 pad 1: Net-(U9D-+) -> Net-(U11B-+)
- RV18 pad 2: Net-(U9D-+) -> Net-(U11B-+)
- RV18 pad 5: Net-(U9D-+) -> Net-(U11B-+)
- RV18 pad 6: Net-(U9D-+) -> Net-(U11B-+)
- U10 pad 1: Net-(SW3-A) -> Net-(R101-Pad2)
- U10 pad 2: Net-(SW3-B) -> Net-(U10A--)
- U10 pad 7: Net-(R53-Pad2) -> Net-(U10B--)
- U11 pad 5: Net-(U10A-+) -> Net-(U11B-+)
- U11 pad 6: Net-(SW4-B) -> Net-(U11B--)
- U11 pad 7: Net-(SW4-A) -> Net-(R102-Pad2)
- U11 pad 8: Net-(R54-Pad2) -> Net-(U11C--)
- U12 pad 10: Net-(U10A-+) -> Net-(U12C-+)
- U8 pad 3: Net-(U10A-+) -> Net-(U12C-+)
- U8 pad 5: Net-(U10A-+) -> Net-(U12C-+)
- U9 pad 1: Net-(R101-Pad2) -> Net-(SW3-A)
- U9 pad 14: Net-(R102-Pad2) -> Net-(R53-Pad2)
- U9 pad 2: Net-(U9A--) -> Net-(SW3-B)
- U9 pad 3: Net-(U9A-+) -> Net-(U12C-+)
- U9 pad 5: Net-(U9B-+) -> Net-(U12C-+)
- U9 pad 6: Net-(U9B--) -> Net-(SW4-B)
- U9 pad 7: Net-(U9B--) -> Net-(SW4-A)
- U9 pad 8: Net-(U9C--) -> Net-(R54-Pad2)
- Z110 pad 2: Net-(U10A-+) -> Net-(U12C-+)
- Z114 pad 1: Net-(U10A-+) -> Net-(U12C-+)
- Z119 pad 1: Net-(U10A-+) -> Net-(U12C-+)
- Z121 pad 1: Net-(U10A-+) -> Net-(U12C-+)
Routing:
- net Net-(U12C-+): track 0.00 -> 22.4 mm
- net Net-(SW5-B): track 14.6 -> 29.2 mm
- net Net-(SW6-B): track 14.6 -> 29.2 mm
- net Net-(U10A-+): track 13.8 -> 0.00 mm
- net Net-(U9D--): track 0.00 -> 11.0 mm
- net Net-(SW4-A): track 0.00 -> 10.4 mm
- net Net-(SW3-A): track 0.00 -> 10.4 mm
- net Net-(U9C--): track 0.00 -> 10.3 mm
- net Net-(R53-Pad2): track 0.00 -> 8.94 mm
- net Net-(R54-Pad2): track 0.00 -> 8.30 mm
- net Net-(Z139-Pad2): track 0.00 -> 5.91 mm
- net Net-(Z138-Pad2): track 0.00 -> 5.91 mm
- net Net-(U8D-+): track 5.62 -> 11.2 mm
- net Net-(U8C-+): track 2.81 -> 5.62 mm
- net -15V_O: track 2.77 -> 5.55 mm
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Other:
- board size 150 x 113.7 mm -> 150 x 136 mm
