File: KiCad/Output.kicad_pcb (KiCad board)
At the start: 4 copper layers, 150 x 136 mm, 371 parts, among them J21 Conn_01x05_bridged, J22 EMK_In, J24 Mic_Effekt_In, J25 Mic_Effekt_In, J26 Phono/Line_In, J27 Mic_Effekt_In, J28 Pegel_Out, J29 Pegel_Out, J37 AUX_Send_3, J38 AUX_Send_1, J39 AUX_Send_2, J40 Bass_Out, J41 Kick_Out, J42 Mid_Out, J43 High_Out, J44 Line_Out_L, J45 Line_Out_R, SW10 SW_SPDT, SW11 SW_SPDT, SW12 SW_SPDT, SW3 SW_SPDT, SW4 SW_SPDT, SW5 SW_SPDT, SW6 SW_SPDT, SW7 SW_SPDT, SW8 SW_SPDT, U10 TL074, U11 TL074, U12 TL074, U13 TL074, U14 TL074, U15 TL074, U16 TL074, U17 TL074, U18 TL074, U19 TL074, U20 TL074, U21 TL074, U22 TL074, U8 TL074, U9 TL074

Commit message: PCB Update
Parts:
- removed J21: Conn_01x05_bridged, Connector_Bridged_2.54mm_LongPads:Bridge_2x05_P2.54mm_Vertical_LongPads
- C90, C91, C94, C95, R33, R34, R43, R44, R45, R46, R51, R52, R57, R58, R61, R62, R63, R64, R65, R66, R73, R74, Z142, Z143, Z148, Z149, Z154, Z155, Z156, Z157, Z159, Z160, Z161, Z162, Z164, Z165: moved to B.Cu
- moved R57 399.9 mm to (171.4, 76.2), turned to 180 degrees
- moved R63 399.4 mm to (182.8, 110.5)
- moved R66 398.8 mm to (182.8, 120.7)
- moved R62 395.9 mm to (182.9, 115.6)
- moved R61 395.7 mm to (182.8, 113.0)
- moved R51 395.5 mm to (175.3, 86.4)
- moved R65 395.4 mm to (182.9, 125.7)
- moved R64 395.1 mm to (182.8, 123.2)
- moved R52 394.6 mm to (175.3, 91.4)
- moved R73 389.8 mm to (190.4, 110.5), turned to 180 degrees
- moved R58 389.2 mm to (171.4, 101.6), turned to 180 degrees
- moved Z154 388.2 mm to (175.3, 83.8)
- moved Z148 387.7 mm to (175.3, 78.7), turned to 180 degrees
- moved R46 387.4 mm to (167.6, 86.4), turned to 180 degrees
- moved R44 387.0 mm to (167.6, 81.3), turned to 180 degrees
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- renumbered R38 to R36, R36 to R38
Connections:
- C38 pad 2: Net-(U10B--) -> Net-(U12C--)
- C39 pad 2: Net-(U11C--) -> Net-(U22C--)
- C40 pad 2: Net-(U10D--) -> Net-(U13C--)
- C42 pad 1: Net-(U10A-+) -> Net-(U12D-+)
- C43 pad 1: Net-(U11B-+) -> Net-(U22D-+)
- C44 pad 1: Net-(U11A-+) -> Net-(U13D-+)
- R101 pad 1: Net-(U10A--) -> Net-(U12D--)
- R102 pad 1: Net-(U11B--) -> Net-(U22D--)
- R103 pad 1: Net-(U11A--) -> Net-(U13D--)
- R36 pad 1: Net-(SW4-B) -> Net-(SW3-B)
- R36 pad 2: Net-(U9C-+) -> Net-(U9D-+)
- R38 pad 1: Net-(SW3-B) -> Net-(SW4-B)
- R38 pad 2: Net-(U9D-+) -> Net-(U9C-+)
- R43 pad 1: Net-(U12D--) -> Net-(U10D--)
- R44 pad 1: Net-(U12D-+) -> Net-(U10D-+)
- R45 pad 1: Net-(U13D--) -> Net-(U10C--)
- R46 pad 1: Net-(U13D-+) -> Net-(U10C-+)
- R51 pad 1: Net-(U12D-+) -> Net-(U10D-+)
- R52 pad 1: Net-(U13D-+) -> Net-(U10C-+)
- R57 pad 2: Net-(U12D--) -> Net-(U10D--)
- R58 pad 2: Net-(U13D--) -> Net-(U10C--)
- R61 pad 2: Net-(U10C--) -> Net-(U11A--)
- R62 pad 2: Net-(U10C--) -> Net-(U11A--)
- R63 pad 2: Net-(U10C--) -> Net-(U11A--)
- R64 pad 2: Net-(U11D--) -> Net-(U11B--)
- R65 pad 2: Net-(U11D--) -> Net-(U11B--)
- R66 pad 2: Net-(U11D--) -> Net-(U11B--)
- R73 pad 1: Net-(U10C--) -> Net-(U11A--)
- R74 pad 1: Net-(U11D--) -> Net-(U11B--)
- R91 pad 2: Net-(U10A--) -> Net-(U12D--)
- R93 pad 2: Net-(U11B--) -> Net-(U22D--)
- R95 pad 2: Net-(U11A--) -> Net-(U13D--)
- RV12 pad 2: Net-(U10B-+) -> Net-(U12C-+)
- RV13 pad 2: Net-(U11C-+) -> Net-(U22C-+)
- RV14 pad 2: Net-(U10D-+) -> Net-(U13C-+)
- RV17 pad 1: Net-(U10A-+) -> Net-(U12D-+)
- RV17 pad 2: Net-(U10A-+) -> Net-(U12D-+)
- RV17 pad 5: Net-(U10A-+) -> Net-(U12D-+)
- RV17 pad 6: Net-(U10A-+) -> Net-(U12D-+)
- RV18 pad 1: Net-(U11B-+) -> Net-(U22D-+)
- RV18 pad 2: Net-(U11B-+) -> Net-(U22D-+)
- RV18 pad 5: Net-(U11B-+) -> Net-(U22D-+)
- RV18 pad 6: Net-(U11B-+) -> Net-(U22D-+)
- RV19 pad 1: Net-(U11A-+) -> Net-(U13D-+)
- RV19 pad 2: Net-(U11A-+) -> Net-(U13D-+)
- RV19 pad 5: Net-(U11A-+) -> Net-(U13D-+)
- RV19 pad 6: Net-(U11A-+) -> Net-(U13D-+)
- U10 pad 1: Net-(R101-Pad2) -> Net-(SW7-A)
- U10 pad 14: Net-(U10D--) -> Net-(R57-Pad1)
- U10 pad 2: Net-(U10A--) -> Net-(SW7-B)
- U10 pad 6: Net-(U10B--) -> Net-(SW8-B)
- U10 pad 7: Net-(U10B--) -> Net-(SW8-A)
- U10 pad 8: Net-(R73-Pad2) -> Net-(R58-Pad1)
- U11 pad 1: Net-(R103-Pad2) -> Net-(R73-Pad2)
- U11 pad 10: Net-(U11C-+) -> GND_O
- U11 pad 12: Net-(U11D-+) -> GND_O
- U11 pad 14: Net-(R74-Pad2) -> Net-(U11D--)
- U11 pad 7: Net-(R102-Pad2) -> Net-(R74-Pad2)
- U12 pad 14: Net-(R57-Pad1) -> Net-(R101-Pad2)
- U12 pad 8: Net-(SW7-A) -> Net-(U12C--)
- U12 pad 9: Net-(SW7-B) -> Net-(U12C--)
- U13 pad 14: Net-(R58-Pad1) -> Net-(R103-Pad2)
- U13 pad 8: Net-(SW8-A) -> Net-(U13C--)
- U13 pad 9: Net-(SW8-B) -> Net-(U13C--)
- U22 pad 10: GND_O -> Net-(U22C-+)
- U22 pad 12: GND_O -> Net-(U22D-+)
- U22 pad 14: Net-(U22D--) -> Net-(R102-Pad2)
- U8 pad 3: Net-(U12C-+) -> Net-(U10A-+)
- U8 pad 5: Net-(U12C-+) -> Net-(U10A-+)
- U9 pad 3: Net-(U12C-+) -> Net-(U10A-+)
- U9 pad 5: Net-(U12C-+) -> Net-(U10A-+)
- Z110 pad 2: Net-(U12C-+) -> Net-(U10A-+)
- Z112 pad 2: Net-(U13C-+) -> Net-(U10B-+)
- Z114 pad 1: Net-(U12C-+) -> Net-(U10A-+)
- Z116 pad 1: Net-(U13C-+) -> Net-(U10B-+)
- Z119 pad 1: Net-(U12C-+) -> Net-(U10A-+)
- Z121 pad 1: Net-(U12C-+) -> Net-(U10A-+)
- Z156 pad 1: Net-(U10C-+) -> Net-(U11A-+)
- Z157 pad 1: Net-(U11D-+) -> Net-(U11B-+)
Routing:
- net Net-(U10A-+): track 0.00 -> 94.4 mm
- net Net-(R62-Pad1): track 2.54 -> 50.3 mm, vias 0 -> 2
- net Net-(R63-Pad1): track 2.54 -> 49.6 mm, vias 0 -> 2
- net Net-(U12C-+): track 22.4 -> 0.00 mm
- net Net-(R74-Pad2): track 0.00 -> 16.4 mm
- net Net-(R73-Pad2): track 0.00 -> 16.4 mm
- net Net-(SW7-B): track 0.00 -> 15.0 mm
- net Net-(U11B--): track 0.00 -> 14.7 mm
- net Net-(U11A--): track 0.00 -> 14.6 mm
- net Net-(SW5-B): track 29.2 -> 14.6 mm
- net Net-(SW6-B): track 29.2 -> 14.6 mm
- net Net-(SW4-B): track 0.00 -> 14.6 mm
- net Net-(SW3-B): track 0.00 -> 14.6 mm
- net Net-(U10B-+): track 0.00 -> 14.0 mm, vias 0 -> 1
- net Net-(SW8-A): track 0.00 -> 13.4 mm
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
Commit message: PCB Update
Parts:
- C38, C39, C42, C43, C98, C99, R101, R102, R87, R88, R91, R92, R93, R94, Z181, Z182, Z189, Z190, Z197, Z199: moved to B.Cu
- moved C38 225.9 mm to (93.7, 54.0), turned to 180 degrees
- moved C39 225.9 mm to (93.7, 57.0), turned to 180 degrees
- moved C42 225.9 mm to (93.7, 66.0), turned to 180 degrees
- moved C43 225.9 mm to (93.7, 69.0), turned to 180 degrees
- moved R87 214.7 mm to (106.4, 43.8), turned to 180 degrees
- moved R92 214.7 mm to (106.4, 58.6), turned to 180 degrees
- moved R88 214.7 mm to (106.4, 46.8), turned to 180 degrees
- moved R91 214.7 mm to (106.4, 55.6), turned to 180 degrees
- moved R93 214.7 mm to (106.4, 61.5), turned to 180 degrees
- moved R94 214.7 mm to (106.4, 64.5), turned to 180 degrees
- moved R101 206.3 mm to (101.6, 37.9), turned to 180 degrees
- moved R102 206.3 mm to (101.6, 40.9), turned to 180 degrees
- moved RV13 196.1 mm to (41.9, 92.7)
- moved RV18 194.0 mm to (41.3, 105.4)
- moved C98 193.7 mm to (71.6, 60.5), turned to 180 degrees
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- renumbered U22 to U12, U12 to U22
Connections:
- C39 pad 2: Net-(U22C--) -> Net-(U12A--)
- C41 pad 2: Net-(U12B--) -> Net-(U22D--)
- C43 pad 1: Net-(U22D-+) -> Net-(U12B-+)
- C45 pad 1: Net-(U12A-+) -> Net-(U22C-+)
- R102 pad 1: Net-(U22D--) -> Net-(U12B--)
- R104 pad 1: Net-(U12A--) -> Net-(U22C--)
- R93 pad 2: Net-(U22D--) -> Net-(U12B--)
- R97 pad 2: Net-(U12A--) -> Net-(U22C--)
- RV13 pad 2: Net-(U22C-+) -> Net-(U12A-+)
- RV15 pad 2: Net-(U12B-+) -> Net-(U22D-+)
- RV18 pad 1: Net-(U22D-+) -> Net-(U12B-+)
- RV18 pad 2: Net-(U22D-+) -> Net-(U12B-+)
- RV18 pad 5: Net-(U22D-+) -> Net-(U12B-+)
- RV18 pad 6: Net-(U22D-+) -> Net-(U12B-+)
- RV20 pad 1: Net-(U12A-+) -> Net-(U22C-+)
- RV20 pad 2: Net-(U12A-+) -> Net-(U22C-+)
- RV20 pad 5: Net-(U12A-+) -> Net-(U22C-+)
- RV20 pad 6: Net-(U12A-+) -> Net-(U22C-+)
- U12 pad 1: Net-(U22A--) -> Net-(U12A--)
- U12 pad 10: Net-(U22C-+) -> Net-(U12C-+)
- U12 pad 12: Net-(U22D-+) -> Net-(U12D-+)
- U12 pad 13: Net-(U22D--) -> Net-(U12D--)
- U12 pad 14: Net-(R102-Pad2) -> Net-(R101-Pad2)
- U12 pad 2: Net-(U22A--) -> Net-(U12A--)
- U12 pad 3: Net-(U21D-+) -> Net-(U12A-+)
- U12 pad 5: GND_O -> Net-(U12B-+)
- U12 pad 6: Net-(U22B--) -> Net-(U12B--)
- U12 pad 7: Net-(U22B--) -> Net-(R102-Pad2)
- U12 pad 8: Net-(U22C--) -> Net-(U12C--)
- U12 pad 9: Net-(U22C--) -> Net-(U12C--)
- U22 pad 1: Net-(R104-Pad2) -> Net-(U22A--)
- U22 pad 10: Net-(U12C-+) -> Net-(U22C-+)
- U22 pad 12: Net-(U12D-+) -> Net-(U22D-+)
- U22 pad 13: Net-(U12D--) -> Net-(U22D--)
- U22 pad 14: Net-(R101-Pad2) -> Net-(U22D--)
- U22 pad 2: Net-(U12A--) -> Net-(U22A--)
- U22 pad 3: Net-(U12A-+) -> Net-(U21D-+)
- U22 pad 5: Net-(U12B-+) -> GND_O
- U22 pad 6: Net-(U12B--) -> Net-(U22B--)
- U22 pad 7: Net-(U12B--) -> Net-(U22B--)
- U22 pad 8: Net-(U12C--) -> Net-(R104-Pad2)
- U22 pad 9: Net-(U12C--) -> Net-(U22C--)
Routing:
- net Net-(R62-Pad1): track 50.3 -> 51.3 mm

Commit message: PCB Update
Parts:
- C102, C103, C40, C41, C44, C45, R103, R104, R89, R90, R95, R96, R97, R98, Z183, Z184, Z191, Z192, Z200, Z201: moved to B.Cu
- RV17, RV20: footprint Connector_PinSocket_2.54mm_LongPads:PinSocket_1x06_P2.54mm_Vertical_LongPads -> Connector_PinSocket_2.54mm_LongPads:PinSocket_2x03_P2.54mm_Vertical_LongPads
- RV18, RV19: footprint Connector_PinSocket_2.54mm_LongPads:PinSocket_1x06_P2.54mm_Vertical_LongPads -> Connector_PinSocket_2.54mm_LongPads:PinSocket_2x03_P2.54mm_Vertical_LongPads_Mirrored
- Z117, Z118, Z119, Z120, Z121, Z228, Z229, Z231, Z233, Z235, Z236, Z238, Z239, Z241, Z243, Z245, Z246, Z248, Z249, Z251, Z253, Z255, Z256, Z257, Z258, Z259: moved to F.Cu
- moved U15 269.7 mm to (133.3, 162.6)
- moved U16 258.6 mm to (133.3, 133.3)
- moved U17 251.0 mm to (133.3, 104.1)
- moved RV19 248.6 mm to (118.1, 138.4), turned to 180 degrees
- moved RV20 242.9 mm to (118.1, 143.5)
- moved U22 238.3 mm to (106.7, 76.2)
- moved RV14 231.5 mm to (102.9, 138.4), turned to 180 degrees
- moved U19 226.9 mm to (80.0, 104.1)
- moved RV15 225.8 mm to (102.9, 143.5)
- moved C44 225.5 mm to (125.7, 135.9)
- moved C45 223.4 mm to (125.7, 146.1)
- moved U13 219.4 mm to (106.7, 133.3)
- moved U21 215.8 mm to (80.0, 76.2)
- moved U18 213.6 mm to (106.7, 104.1)
- moved R96 213.0 mm to (125.7, 133.3), turned to 180 degrees
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Connections:
- C37 pad 1: Net-(U13B-+) -> Net-(U22C-+)
- C38 pad 2: Net-(U12C--) -> Net-(U12B--)
- C40 pad 2: Net-(U13C--) -> Net-(U13A--)
- C41 pad 2: Net-(U22D--) -> Net-(U13B--)
- C42 pad 1: Net-(U12D-+) -> Net-(U12C-+)
- C43 pad 1: Net-(U12B-+) -> Net-(U12D-+)
- C45 pad 1: Net-(U22C-+) -> Net-(U13C-+)
- R100 pad 1: Net-(U13B--) -> Net-(U22C--)
- R101 pad 1: Net-(U12D--) -> Net-(U12C--)
- R102 pad 1: Net-(U12B--) -> Net-(U12D--)
- R104 pad 1: Net-(U22C--) -> Net-(U13C--)
- R69 pad 1: Net-(U13A--) -> Net-(U22D--)
- R70 pad 1: Net-(U13A--) -> Net-(U22D--)
- R76 pad 2: Net-(U13A--) -> Net-(U22D--)
- R85 pad 1: Net-(U13B-+) -> Net-(U22C-+)
- R91 pad 2: Net-(U12D--) -> Net-(U12C--)
- R93 pad 2: Net-(U12B--) -> Net-(U12D--)
- R97 pad 2: Net-(U22C--) -> Net-(U13C--)
- R99 pad 2: Net-(U13B--) -> Net-(U22C--)
- RV12 pad 2: Net-(U12C-+) -> Net-(U12B-+)
- RV14 pad 2: Net-(U13C-+) -> Net-(U13A-+)
- RV15 pad 2: Net-(U22D-+) -> Net-(U13B-+)
- RV17 pad 1: Net-(U12D-+) -> Net-(U12C-+)
- RV17 pad 2: Net-(U12D-+) -> Net-(U12C-+)
- RV17 pad 5: Net-(U12D-+) -> Net-(U12C-+)
- RV17 pad 6: Net-(U12D-+) -> Net-(U12C-+)
- RV18 pad 1: Net-(U12B-+) -> Net-(U12D-+)
- RV18 pad 2: Net-(U12B-+) -> Net-(U12D-+)
- RV18 pad 5: Net-(U12B-+) -> Net-(U12D-+)
- RV18 pad 6: Net-(U12B-+) -> Net-(U12D-+)
- RV20 pad 1: Net-(U22C-+) -> Net-(U13C-+)
- RV20 pad 2: Net-(U22C-+) -> Net-(U13C-+)
- RV20 pad 5: Net-(U22C-+) -> Net-(U13C-+)
- RV20 pad 6: Net-(U22C-+) -> Net-(U13C-+)
- U12 pad 14: Net-(R101-Pad2) -> Net-(R102-Pad2)
- U12 pad 7: Net-(R102-Pad2) -> Net-(U12B--)
- U12 pad 8: Net-(U12C--) -> Net-(R101-Pad2)
- U13 pad 1: Net-(R76-Pad1) -> Net-(U13A--)
- U13 pad 7: Net-(R99-Pad1) -> Net-(U13B--)
- U13 pad 8: Net-(U13C--) -> Net-(R104-Pad2)
- U22 pad 14: Net-(U22D--) -> Net-(R76-Pad1)
- U22 pad 8: Net-(R104-Pad2) -> Net-(R99-Pad1)
- Z152 pad 2: Net-(R91-Pad1) -> Net-(R93-Pad1)
- Z153 pad 2: Net-(R93-Pad1) -> Net-(R91-Pad1)
- Z158 pad 1: Net-(U13A-+) -> Net-(U22D-+)
- Z197 pad 2: Net-(C48-Pad1) -> Net-(C49-Pad1)
- Z199 pad 2: Net-(C49-Pad1) -> Net-(C48-Pad1)
Routing:
- net Net-(R95-Pad1): track 0.00 -> 20.0 mm
- net Net-(R97-Pad1): track 0.00 -> 20.0 mm
- net Net-(R93-Pad1): track 0.00 -> 16.1 mm
- net Net-(R91-Pad1): track 0.00 -> 16.1 mm
- net Net-(U13D-+): track 0.00 -> 15.5 mm
- net Net-(U13C-+): track 0.00 -> 15.5 mm
- net Net-(U12D-+): track 0.00 -> 15.5 mm
- net Net-(U12C-+): track 0.00 -> 15.5 mm
- net Net-(R104-Pad2): track 0.00 -> 13.5 mm, vias 0 -> 1
- net Net-(R101-Pad2): track 0.00 -> 13.5 mm, vias 0 -> 1
- net Net-(R102-Pad2): track 0.00 -> 13.0 mm, vias 0 -> 1
- net Net-(R103-Pad2): track 0.00 -> 13.0 mm, vias 0 -> 1
- net Net-(R88-Pad2): track 0.00 -> 10.6 mm
- net Net-(R90-Pad2): track 0.00 -> 10.6 mm
- net Net-(R89-Pad2): track 0.00 -> 10.6 mm
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- added copper zone on F.Cu, net Net-(R101-Pad2)
- added copper zone on F.Cu, net Net-(R102-Pad2)
- added copper zone on F.Cu, net Net-(R103-Pad2)
- added copper zone on F.Cu, net Net-(R104-Pad2)
Other:
- board text added: "16 25 34"
- board text added: "34 25 16"

Commit message: PCB Update
Parts:
- C106, C107, C110, C111, C48, C49, C52, C53, C58, C59, C62, C63, C70, C71, C74, C75, C82, C83, C86, C87, R105, R106, R109, R110, R113, R114, R117, R118, R127, R128, R133, R134, R137, R138, R141, R142, Z185, Z186, Z193, Z194, Z198, Z202: moved to B.Cu
- moved R128 383.2 mm to (212.1, 143.8)
- moved R127 382.4 mm to (212.1, 128.3)
- moved R138 379.0 mm to (212.1, 138.4), turned to 180 degrees
- moved R137 378.8 mm to (212.1, 133.3), turned to 180 degrees
- moved R106 372.5 mm to (193.0, 141.0)
- moved R105 372.4 mm to (193.0, 133.3)
- moved R114 372.3 mm to (196.8, 138.4)
- moved R113 372.2 mm to (196.8, 133.3)
- moved R134 351.6 mm to (181.6, 141.0), turned to 180 degrees
- moved R133 351.6 mm to (181.7, 130.8), turned to 180 degrees
- moved R118 348.9 mm to (174.0, 138.4), turned to 180 degrees
- moved R117 348.8 mm to (174.0, 133.3), turned to 180 degrees
- moved Z186 347.4 mm to (189.2, 143.5), turned to 180 degrees
- moved Z185 346.3 mm to (189.2, 130.8), turned to 180 degrees
- moved Z193 345.8 mm to (189.2, 135.9)
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Connections:
- C52 pad 2: Net-(U15C--) -> Net-(U15A--)
- C53 pad 2: Net-(U16C--) -> Net-(U15B--)
- C58 pad 2: Net-(U15A-+) -> Net-(U14A-+)
- C59 pad 2: Net-(U16A-+) -> Net-(U14B-+)
- C62 pad 2: Net-(U15C-+) -> Net-(U15A-+)
- C63 pad 2: Net-(U16C-+) -> Net-(U15B-+)
- C70 pad 1: Net-(U15A--) -> Net-(U14A--)
- C71 pad 1: Net-(U16A--) -> Net-(U14B--)
- C75 pad 2: Net-(U16D--) -> Net-(U15C--)
- C82 pad 2: Net-(U15B-+) -> Net-(U14D-+)
- C83 pad 2: Net-(U16B-+) -> Net-(U14C-+)
- C87 pad 2: Net-(U16D-+) -> Net-(U15C-+)
- R109 pad 2: Net-(U15A--) -> Net-(U14A--)
- R110 pad 2: Net-(U16A--) -> Net-(U14B--)
- R113 pad 2: Net-(U15C-+) -> Net-(U15A-+)
- R114 pad 2: Net-(U16C-+) -> Net-(U15B-+)
- R117 pad 2: Net-(U15A-+) -> Net-(U14A-+)
- R118 pad 2: Net-(U16A-+) -> Net-(U14B-+)
- R123 pad 1: Net-(U14D--) -> Net-(U16D--)
- R124 pad 1: Net-(U14D-+) -> Net-(U16D-+)
- R126 pad 1: Net-(U14D-+) -> Net-(U16D-+)
- R127 pad 1: Net-(U15C--) -> Net-(U15A--)
- R128 pad 1: Net-(U16C--) -> Net-(U15B--)
- R132 pad 2: Net-(U14D--) -> Net-(U16D--)
- R133 pad 2: Net-(U15B--) -> Net-(U14D--)
- R134 pad 2: Net-(U16B--) -> Net-(U14C--)
- R138 pad 2: Net-(U16D-+) -> Net-(U15C-+)
- R141 pad 2: Net-(U15B-+) -> Net-(U14D-+)
- R142 pad 2: Net-(U16B-+) -> Net-(U14C-+)
- R77 pad 1: Net-(U14B--) -> Net-(U16B--)
- R78 pad 1: Net-(U14B-+) -> Net-(U16B-+)
- R80 pad 1: Net-(U14B-+) -> Net-(U16B-+)
- R83 pad 2: Net-(U14B--) -> Net-(U16B--)
- U14 pad 1: Net-(SW10-A) -> Net-(U14A--)
- U14 pad 10: Net-(U14A-+) -> Net-(U14C-+)
- U14 pad 14: Net-(R132-Pad1) -> Net-(U14D--)
- U14 pad 2: Net-(SW10-B) -> Net-(U14A--)
- U14 pad 7: Net-(R83-Pad1) -> Net-(U14B--)
- U14 pad 8: Net-(SW12-A) -> Net-(U14C--)
- U14 pad 9: Net-(SW12-B) -> Net-(U14C--)
- U16 pad 1: Net-(U16A--) -> Net-(SW10-A)
- U16 pad 10: Net-(U16C-+) -> Net-(U16A-+)
- U16 pad 14: Net-(U16D--) -> Net-(R132-Pad1)
- U16 pad 2: Net-(U16A--) -> Net-(SW10-B)
- U16 pad 7: Net-(U16B--) -> Net-(R83-Pad1)
- U16 pad 8: Net-(U16C--) -> Net-(SW12-A)
- U16 pad 9: Net-(U16C--) -> Net-(SW12-B)
- U21 pad 3: Net-(U14A-+) -> Net-(U16A-+)
- Z180 pad 2: Net-(U14A-+) -> Net-(U16A-+)
- Z185 pad 1: Net-(Z185-Pad1) -> Net-(U14D--)
- Z185 pad 2: Net-(U15B--) -> Net-(Z185-Pad2)
- Z186 pad 1: Net-(U16B--) -> Net-(U14C--)
- Z193 pad 1: GND_O -> Net-(Z185-Pad2)
- Z193 pad 2: Net-(Z185-Pad1) -> GND_O
- Z198 pad 1: Net-(R105-Pad1) -> Net-(Z185-Pad2)
- Z198 pad 2: Net-(Z185-Pad1) -> Net-(R105-Pad1)
- Z213 pad 1: Net-(U16D--) -> Net-(U15C--)
Routing:
- net Net-(U14D--): track 0.00 -> 25.5 mm, vias 0 -> 1
- net Net-(U14C--): track 0.00 -> 22.9 mm, vias 0 -> 1
- net Net-(U14B--): track 0.00 -> 19.2 mm
- net Net-(U14A--): track 0.00 -> 19.2 mm
- net Net-(U15A--): track 0.00 -> 19.2 mm
- net Net-(U15B--): track 0.00 -> 18.9 mm
- net Net-(U13D-+): track 15.5 -> 2.77 mm
- net Net-(U13C-+): track 15.5 -> 2.77 mm
- net Net-(U12D-+): track 15.5 -> 2.77 mm
- net Net-(U12C-+): track 15.5 -> 2.77 mm
- net Net-(U15C-+): track 0.00 -> 6.63 mm
- net Net-(U15A-+): track 0.00 -> 6.63 mm
- net Net-(U14D-+): track 0.00 -> 6.63 mm
- net Net-(U14C-+): track 0.00 -> 6.63 mm
- net Net-(C48-Pad1): track 0.00 -> 5.78 mm
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- added copper zone on F.Cu, net Net-(U12C-+)
- added copper zone on F.Cu, net Net-(U12D-+)
- added copper zone on F.Cu, net Net-(U13C-+)
- added copper zone on F.Cu, net Net-(U13D-+)
Other:
- board size 150 x 136 mm -> 150 x 119.5 mm

Commit message: PCB Update
Parts:
- C50, C51, C54, C55, C60, C61, C64, C65, C68, C69, C72, C73, C76, C77, C80, C81, C84, C85, C88, C89, R107, R108, R111, R112, R115, R116, R119, R120, R129, R130, R135, R136, R139, R140, R143, R144, Z117, Z118, Z119, Z120, Z121, Z175, Z176, Z177, Z187, Z188, Z195, Z196, Z203, Z204, Z205, Z206, Z207, Z208, Z209, Z210, Z212, Z213, Z214, Z215, Z216, Z217, Z218, Z219, Z221, Z222, Z223, Z224, Z228, Z229, Z231, Z233, Z238, Z239, Z241, Z243, Z248, Z249, Z251, Z253, Z257, Z258, Z259: moved to B.Cu
- moved R107 409.3 mm to (210.8, 80.0), turned to 180 degrees
- moved R116 398.3 mm to (206.9, 74.9), turned to 180 degrees
- moved R108 396.8 mm to (210.8, 72.4), turned to 180 degrees
- moved R115 396.2 mm to (206.9, 80.0), turned to 180 degrees
- moved R135 390.6 mm to (206.9, 101.6), turned to 180 degrees
- moved R119 385.8 mm to (199.3, 104.1), turned to 180 degrees
- moved R120 385.3 mm to (199.3, 109.2), turned to 180 degrees
- moved R130 380.6 mm to (191.7, 69.8), turned to 180 degrees
- moved Z203 378.5 mm to (210.8, 104.1)
- moved Z204 377.4 mm to (210.8, 111.8)
- moved R136 376.6 mm to (206.9, 111.8), turned to 180 degrees
- moved R129 375.6 mm to (191.7, 85.1), turned to 180 degrees
- moved Z196 375.4 mm to (210.8, 109.2)
- moved Z195 375.3 mm to (210.8, 106.7)
- moved R143 374.5 mm to (199.3, 101.6)
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Connections:
- C55 pad 2: Net-(U18C--) -> Net-(U17D--)
- C60 pad 2: Net-(U17A-+) -> Net-(U16A-+)
- C61 pad 2: Net-(U18A-+) -> Net-(U16B-+)
- C65 pad 2: Net-(U18C-+) -> Net-(U17D-+)
- C72 pad 1: Net-(U17A--) -> Net-(U16A--)
- C73 pad 1: Net-(U18A--) -> Net-(U16B--)
- C76 pad 2: Net-(U17D--) -> Net-(U17B--)
- C77 pad 2: Net-(U18D--) -> Net-(U17A--)
- C84 pad 2: Net-(U17B-+) -> Net-(U16D-+)
- C85 pad 2: Net-(U18B-+) -> Net-(U16C-+)
- C88 pad 2: Net-(U17D-+) -> Net-(U17B-+)
- C89 pad 2: Net-(U18D-+) -> Net-(U17A-+)
- R111 pad 2: Net-(U17A--) -> Net-(U16A--)
- R112 pad 2: Net-(U18A--) -> Net-(U16B--)
- R116 pad 2: Net-(U18C-+) -> Net-(U17D-+)
- R119 pad 2: Net-(U17A-+) -> Net-(U16A-+)
- R120 pad 2: Net-(U18A-+) -> Net-(U16B-+)
- R123 pad 1: Net-(U16D--) -> Net-(U20D--)
- R124 pad 1: Net-(U16D-+) -> Net-(U20D-+)
- R126 pad 1: Net-(U16D-+) -> Net-(U20D-+)
- R130 pad 1: Net-(U18C--) -> Net-(U17D--)
- R132 pad 2: Net-(U16D--) -> Net-(U20D--)
- R135 pad 2: Net-(U17B--) -> Net-(U16D--)
- R136 pad 2: Net-(U18B--) -> Net-(U16C--)
- R139 pad 2: Net-(U17D-+) -> Net-(U17B-+)
- R140 pad 2: Net-(U18D-+) -> Net-(U17A-+)
- R143 pad 2: Net-(U17B-+) -> Net-(U16D-+)
- R144 pad 2: Net-(U18B-+) -> Net-(U16C-+)
- R77 pad 1: Net-(U16B--) -> Net-(U20B--)
- R78 pad 1: Net-(U16B-+) -> Net-(U20B-+)
- R80 pad 1: Net-(U16B-+) -> Net-(U20B-+)
- R83 pad 2: Net-(U16B--) -> Net-(U20B--)
- U16 pad 1: Net-(SW10-A) -> Net-(U16A--)
- U16 pad 10: Net-(U16A-+) -> Net-(U16C-+)
- U16 pad 14: Net-(R132-Pad1) -> Net-(U16D--)
- U16 pad 2: Net-(SW10-B) -> Net-(U16A--)
- U16 pad 7: Net-(R83-Pad1) -> Net-(U16B--)
- U16 pad 8: Net-(SW12-A) -> Net-(U16C--)
- U16 pad 9: Net-(SW12-B) -> Net-(U16C--)
- U18 pad 10: Net-(U18C-+) -> Net-(U18B-+)
- U18 pad 12: Net-(U18D-+) -> Net-(U18A-+)
- U19 pad 10: Net-(U19C-+) -> Net-(U19B-+)
- U19 pad 12: Net-(U19C-+) -> Net-(U19A-+)
- U19 pad 5: Net-(U19A-+) -> Net-(U19B-+)
- U20 pad 1: Net-(U20A--) -> Net-(SW10-A)
- U20 pad 10: Net-(U20C-+) -> Net-(U20A-+)
- U20 pad 12: Net-(U20C-+) -> Net-(U20D-+)
- U20 pad 14: Net-(U20D--) -> Net-(R132-Pad1)
- U20 pad 2: Net-(U20A--) -> Net-(SW10-B)
- U20 pad 5: Net-(U20A-+) -> Net-(U20B-+)
- U20 pad 7: Net-(U20B--) -> Net-(R83-Pad1)
- U20 pad 8: Net-(U20C--) -> Net-(SW12-A)
- U20 pad 9: Net-(U20C--) -> Net-(SW12-B)
- U21 pad 3: Net-(U16A-+) -> Net-(U20A-+)
- Z180 pad 2: Net-(U16A-+) -> Net-(U20A-+)
- Z187 pad 1: Net-(U17B--) -> Net-(U16D--)
- Z188 pad 1: Net-(U18B--) -> Net-(U16C--)
- Z214 pad 1: Net-(U17D--) -> Net-(U17B--)
- Z215 pad 1: Net-(U18D--) -> Net-(U17A--)
- Z221 pad 2: Net-(U19A-+) -> Net-(U19B-+)
- Z222 pad 2: Net-(U19C-+) -> Net-(U19A-+)
- Z223 pad 2: Net-(U20A-+) -> Net-(U18B-+)
- Z224 pad 2: Net-(U20C-+) -> Net-(U18A-+)
- Z228 pad 1: Net-(U19A--) -> Net-(U19C--)
- Z229 pad 1: Net-(U19C--) -> Net-(U19D--)
- Z230 pad 1: Net-(U19D--) -> Net-(U19A--)
- Z231 pad 1: Net-(U20A--) -> Net-(U18C--)
- Z232 pad 1: Net-(U20B--) -> Net-(U18B--)
- Z233 pad 1: Net-(U20C--) -> Net-(U18D--)
- Z234 pad 1: Net-(U20D--) -> Net-(U18A--)
- Z238 pad 1: Net-(U19A--) -> Net-(U19C--)
- Z239 pad 1: Net-(U19C--) -> Net-(U19D--)
- Z241 pad 1: Net-(U20A--) -> Net-(U18C--)
- Z243 pad 1: Net-(U20C--) -> Net-(U18D--)
Routing:
- net Net-(U19A-+): track 0.00 -> 126.7 mm
- net Net-(U19B-+): track 0.00 -> 108.8 mm
- net Net-(R108-Pad1): track 0.00 -> 47.1 mm
- net Net-(R107-Pad1): track 0.00 -> 28.2 mm
- net Net-(U16D--): track 0.00 -> 23.7 mm, vias 0 -> 1
- net Net-(U17A--): track 0.00 -> 23.5 mm, vias 0 -> 1
- net Net-(U18B-+): track 0.00 -> 21.9 mm
- net Net-(U18A-+): track 0.00 -> 21.9 mm
- net Net-(U17B--): track 0.00 -> 21.0 mm, vias 0 -> 1
- net Net-(U16C--): track 0.00 -> 20.9 mm, vias 0 -> 1
- net Net-(U16B--): track 0.00 -> 19.2 mm
- net Net-(U17C--): track 0.00 -> 19.2 mm
- net Net-(U16A--): track 0.00 -> 19.1 mm
- net Net-(U17D--): track 0.00 -> 18.9 mm
- net Net-(U15D--): track 5.31 -> 23.5 mm, vias 0 -> 1
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Other:
- board text added: "U14"
