File: KiCad/Output.kicad_pcb (KiCad board)
At the start: 4 copper layers, 150 x 119.5 mm, 370 parts, among them J22 EMK_In, J24 Mic_Effekt_In, J25 Mic_Effekt_In, J26 Phono/Line_In, J27 Mic_Effekt_In, J28 Pegel_Out, J29 Pegel_Out, J37 AUX_Send_3, J38 AUX_Send_1, J39 AUX_Send_2, J40 Bass_Out, J41 Kick_Out, J42 Mid_Out, J43 High_Out, J44 Line_Out_L, J45 Line_Out_R, SW10 SW_SPDT, SW11 SW_SPDT, SW12 SW_SPDT, SW3 SW_SPDT, SW4 SW_SPDT, SW5 SW_SPDT, SW6 SW_SPDT, SW7 SW_SPDT, SW8 SW_SPDT, U10 TL074, U11 TL074, U12 TL074, U13 TL074, U14 TL074, U15 TL074, U16 TL074, U17 TL074, U18 TL074, U19 TL074, U20 TL074, U21 TL074, U22 TL074, U8 TL074, U9 TL074

Commit message: PCB Update
Parts:
- C104, C105, C92, C93, C96, C97, R145, R146, R147, R148, R149, Z211, Z220, Z225, Z226, Z227, Z230, Z232, Z234, Z235, Z236, Z237, Z240, Z242, Z244, Z245, Z246, Z247, Z250, Z252, Z254, Z255, Z256: moved to B.Cu
- Z117, Z118, Z119, Z121, Z175, Z176, Z177, Z205, Z206, Z207, Z208, Z209, Z210: moved to F.Cu
- moved C97 339.4 mm to (207.0, 49.5), turned to 180 degrees
- moved C96 331.2 mm to (199.4, 49.5), turned to 180 degrees
- moved R147 322.8 mm to (191.8, 44.5), turned to 180 degrees
- moved R146 317.9 mm to (191.8, 54.6), turned to 180 degrees
- moved Z237 314.0 mm to (199.4, 57.1), turned to 180 degrees
- moved Z230 311.2 mm to (199.4, 44.5)
- moved C93 307.4 mm to (176.5, 77.5), turned to 180 degrees
- moved Z240 305.5 mm to (199.4, 41.9), turned to 180 degrees
- moved Z227 305.0 mm to (199.4, 54.6)
- moved Z247 300.4 mm to (191.8, 57.1)
- moved C92 299.2 mm to (168.9, 77.5), turned to 180 degrees
- moved Z250 291.9 mm to (191.8, 41.9)
- moved Z236 288.0 mm to (168.9, 49.5), turned to 180 degrees
- moved R149 286.3 mm to (161.3, 72.4), turned to 180 degrees
- moved Z246 282.2 mm to (168.9, 47.0), turned to 180 degrees
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Connections:
- R121 pad 1: Net-(U21B--) -> Net-(U22B--)
- R122 pad 1: Net-(U21B-+) -> Net-(U22B-+)
- R125 pad 1: Net-(U21B-+) -> Net-(U22B-+)
- R131 pad 2: Net-(U21B--) -> Net-(U22B--)
- U21 pad 1: Net-(SW11-A) -> Net-(U21A--)
- U21 pad 12: Net-(U21D-+) -> Net-(U21A-+)
- U21 pad 2: Net-(SW11-B) -> Net-(U21A--)
- U21 pad 3: Net-(U20A-+) -> Net-(U21A-+)
- U21 pad 5: Net-(U21B-+) -> GND_O
- U21 pad 7: Net-(R131-Pad1) -> Net-(U21B--)
- U22 pad 1: Net-(U22A--) -> Net-(SW11-A)
- U22 pad 2: Net-(U22A--) -> Net-(SW11-B)
- U22 pad 3: Net-(U21D-+) -> Net-(U20A-+)
- U22 pad 5: GND_O -> Net-(U22B-+)
- U22 pad 7: Net-(U22B--) -> Net-(R131-Pad1)
- Z226 pad 2: Net-(U21D-+) -> Net-(U21A-+)
- Z235 pad 1: Net-(U21D--) -> Net-(U21A--)
- Z236 pad 1: Net-(U22A--) -> Net-(U21D--)
- Z245 pad 1: Net-(U21D--) -> Net-(U21A--)
- Z246 pad 1: Net-(U22A--) -> Net-(U21D--)
- Z257 pad 2: Net-(U21D-+) -> Net-(U21A-+)
- Z259 pad 1: Net-(U21D-+) -> Net-(U21A-+)
Routing:
- net Net-(U21C--): track 0.00 -> 110.5 mm, vias 0 -> 2
- net Net-(U18C--): track 2.54 -> 70.6 mm
- net Net-(U21A-+): track 0.00 -> 55.0 mm
- net Net-(U21D--): track 0.00 -> 49.1 mm
- net Net-(U21A--): track 0.00 -> 46.7 mm
- net Net-(U19D--): track 2.54 -> 41.8 mm
- net Net-(U19C--): track 2.54 -> 39.7 mm
- net Net-(U18D--): track 2.54 -> 26.3 mm
- net Net-(Z232-Pad2): track 0.00 -> 18.6 mm
- net Net-(Z227-Pad2): track 0.00 -> 18.6 mm
- net Net-(Z230-Pad2): track 0.00 -> 18.6 mm
- net Net-(Z234-Pad2): track 0.00 -> 16.1 mm
- net Net-(Z220-Pad1): track 0.00 -> 11.7 mm
- net +15V_O: track 27.7 -> 36.0 mm
- net -15V_O: track 27.7 -> 36.0 mm
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Other:
- board size 150 x 119.5 mm -> 150 x 120.7 mm

Commit message: PCB Update
Parts:
- C108, C109, C35, C37, R100, R69, R70, R76, R77, R78, R79, R80, R83, R85, R99, Z158, Z163, Z166, Z169, Z175, Z176, Z177, Z178, Z179, Z180: moved to B.Cu
- RV16: footprint Connector_PinSocket_2.54mm_LongPads:PinSocket_1x06_P2.54mm_Vertical_LongPads -> Connector_PinSocket_2.54mm_LongPads:PinSocket_2x03_P2.54mm_Vertical_LongPads
- moved R79 130.7 mm to (157.5, 80.0)
- moved R85 123.2 mm to (149.9, 80.0)
- moved R99 123.1 mm to (149.9, 85.1), turned to 180 degrees
- moved Z169 121.2 mm to (157.5, 85.1)
- moved R83 120.4 mm to (146.1, 67.3), turned to 180 degrees
- moved R100 119.8 mm to (149.9, 82.5)
- moved R80 115.7 mm to (142.2, 72.4), turned to 180 degrees
- moved R77 115.4 mm to (142.2, 69.8), turned to 180 degrees
- moved R78 115.4 mm to (142.2, 74.9), turned to 180 degrees
- moved Z178 112.7 mm to (152.0, 49.5), turned to 180 degrees
- moved Z179 112.7 mm to (152.0, 52.5), turned to 180 degrees
- moved Z180 112.7 mm to (152.0, 55.4), turned to 180 degrees
- moved J37 109.8 mm to (130.8, 47.0), turned to 180 degrees
- moved R76 109.0 mm to (134.6, 85.1), turned to 180 degrees
- moved C35 108.6 mm to (157.5, 82.5)
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Connections:
- R121 pad 1: Net-(U22B--) -> Net-(U20B--)
- R122 pad 1: Net-(U22B-+) -> Net-(U20B-+)
- R125 pad 1: Net-(U22B-+) -> Net-(U20B-+)
- R131 pad 2: Net-(U22B--) -> Net-(U20B--)
- R69 pad 1: Net-(U22D--) -> Net-(U22B--)
- R70 pad 1: Net-(U22D--) -> Net-(U22B--)
- R76 pad 2: Net-(U22D--) -> Net-(U22B--)
- R77 pad 1: Net-(U20B--) -> Net-(U22D--)
- R78 pad 1: Net-(U20B-+) -> Net-(U22D-+)
- R80 pad 1: Net-(U20B-+) -> Net-(U22D-+)
- R83 pad 2: Net-(U20B--) -> Net-(U22D--)
- U20 pad 1: Net-(SW10-A) -> Net-(SW11-A)
- U20 pad 2: Net-(SW10-B) -> Net-(SW11-B)
- U20 pad 7: Net-(R83-Pad1) -> Net-(R131-Pad1)
- U22 pad 1: Net-(SW11-A) -> Net-(SW10-A)
- U22 pad 14: Net-(R76-Pad1) -> Net-(R83-Pad1)
- U22 pad 2: Net-(SW11-B) -> Net-(SW10-B)
- U22 pad 7: Net-(R131-Pad1) -> Net-(R76-Pad1)
- Z158 pad 1: Net-(U22D-+) -> Net-(U22B-+)
Routing:
- net Net-(U19C--): track 39.7 -> 127.9 mm, vias 0 -> 1
- net Net-(U19D--): track 41.8 -> 116.0 mm, vias 0 -> 1
- net Net-(R69-Pad2): track 0.00 -> 39.8 mm, vias 0 -> 2
- net Net-(U21C--): track 110.5 -> 71.4 mm, vias 2 -> 0
- net Net-(U18D--): track 26.3 -> 63.6 mm, vias 0 -> 1
- net Net-(R83-Pad1): track 0.00 -> 34.6 mm, vias 0 -> 1
- net Net-(R79-Pad2): track 0.00 -> 25.9 mm, vias 0 -> 1
- net Net-(U18C--): track 70.6 -> 94.0 mm, vias 0 -> 1
- net Net-(R99-Pad1): track 0.00 -> 21.8 mm
- net Net-(Z163-Pad2): track 0.00 -> 21.6 mm
- net Net-(U21D--): track 49.1 -> 65.2 mm, vias 0 -> 1
- net Net-(U21A-+): track 55.0 -> 69.7 mm, vias 0 -> 1
- net Net-(SW10-B): track 0.00 -> 14.2 mm
- net Net-(U20A-+): track 0.00 -> 12.0 mm, vias 0 -> 1
- net Net-(U22B--): track 0.00 -> 11.0 mm
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- added copper zone on B.Cu, net Net-(R57-Pad1)
- added copper zone on B.Cu, net Net-(R79-Pad2)
- added copper zone on B.Cu, net Net-(U21C--)
Other:
- board size 150 x 120.7 mm -> 150 x 122 mm

Commit message: PCB Update
Parts:
- C100, C101, R121, R122, R123, R124, R125, R126, R131, R132, Z117, Z118, Z119, Z121, Z205, Z206, Z207, Z208, Z209, Z210: moved to B.Cu
- moved J22 166.1 mm to (210.8, 133.3)
- moved R131 115.7 mm to (138.4, 39.4)
- moved R122 113.4 mm to (142.2, 44.5)
- moved R121 113.3 mm to (142.2, 41.9)
- moved R124 112.5 mm to (142.2, 54.6)
- moved R123 111.6 mm to (142.2, 57.1)
- moved R132 110.2 mm to (138.4, 59.7)
- moved SW11 110.0 mm to (149.9, 41.9)
- moved RV21 108.8 mm to (153.7, 41.9)
- moved R125 107.6 mm to (134.6, 47.0), turned to 180 degrees
- moved R126 107.0 mm to (134.6, 52.1), turned to 180 degrees
- moved C101 101.8 mm to (149.9, 49.5), turned to 180 degrees
- moved SW12 98.9 mm to (149.9, 57.1), turned to 180 degrees
- moved RV22 98.9 mm to (153.7, 57.1), turned to 180 degrees
- moved Z206 87.9 mm to (123.2, 49.5)
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Connections:
- R121 pad 1: Net-(U20B--) -> Net-(U20A--)
- R122 pad 1: Net-(U20B-+) -> Net-(U20A-+)
- R123 pad 1: Net-(U20D--) -> Net-(U20B--)
- R124 pad 1: Net-(U20D-+) -> Net-(U20B-+)
- R125 pad 1: Net-(U20B-+) -> Net-(U20A-+)
- R126 pad 1: Net-(U20D-+) -> Net-(U20B-+)
- R131 pad 2: Net-(U20B--) -> Net-(U20A--)
- R132 pad 2: Net-(U20D--) -> Net-(U20B--)
- U20 pad 1: Net-(SW11-A) -> Net-(R131-Pad1)
- U20 pad 10: Net-(U20A-+) -> Net-(U20C-+)
- U20 pad 12: Net-(U20D-+) -> Net-(U20C-+)
- U20 pad 13: Net-(U20D--) -> Net-(SW11-B)
- U20 pad 14: Net-(R132-Pad1) -> Net-(SW11-A)
- U20 pad 2: Net-(SW11-B) -> Net-(U20A--)
- U20 pad 7: Net-(R131-Pad1) -> Net-(R132-Pad1)
- U22 pad 3: Net-(U20A-+) -> Net-(U20C-+)
- Z180 pad 2: Net-(U20A-+) -> Net-(U20C-+)
Routing:
- net -15V_O: track 38.8 -> 82.9 mm
- net Net-(R131-Pad1): track 0.00 -> 40.3 mm
- net +15V_O: track 38.8 -> 79.0 mm
- net Net-(U20C-+): track 0.00 -> 30.7 mm, vias 0 -> 1
- net Net-(R132-Pad1): track 0.00 -> 25.1 mm
- net Net-(U10A-+): track 91.9 -> 109.6 mm
- net Net-(R83-Pad1): track 34.6 -> 50.1 mm, vias 1 -> 0
- net Net-(Z220-Pad1): track 18.8 -> 5.08 mm
- net Net-(SW12-B): track 0.00 -> 13.0 mm
- net Net-(SW11-B): track 0.00 -> 13.0 mm
- net Net-(U19A-+): track 126.7 -> 114.7 mm
- net Net-(U19B-+): track 108.8 -> 96.9 mm
- net Net-(SW12-A): track 0.00 -> 10.4 mm
- net Net-(SW11-A): track 0.00 -> 10.4 mm
- net Net-(R63-Pad1): track 46.9 -> 57.2 mm
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- added copper zone on In2.Cu, net +15V_O
- added copper zone on In2.Cu, net -15V_O
- added copper zone on F.Cu, net Net-(R79-Pad2)
- removed copper zone on B.Cu, net Net-(R79-Pad2)
