File: KiCad/Output.kicad_sch (KiCad schematic)
At the start: 633 parts, among them J1 R_Phono_In, J10 VCC_IN, J11 VCC_OUT, J12 EMK_In, J13 EMK_Out, J14 EMK_Out, J15 Mic_Effekt_Out, J16 Mic_Effekt_Out, J17 Mic_Effekt_Out, J18 Mic_Effekt_Out, J19 Phono/Line_Out, J2 L_Phono_In, J20 Mic_Effekt_Out, J21 EMK_Out, J22 EMK_In, J23 EMK_In, J24 Mic_Effekt_In, J25 Mic_Effekt_In, J26 Phono/Line_In, J27 Mic_Effekt_In, J28 Pegel_Out, J29 Pegel_Out, J3 R_Line_In, J30 Pegel_In, J31 Pegel_In, J32 Pegel_In, J33 Pegel_In, J34 LED_Out, J35 LED_In, J36 VU_Meter_Out, J37 AUX_Send_3, J38 AUX_Send_1, J39 AUX_Send_2, J4 L_Line_In, J40 Bass_Out, J41 Kick_Out, J42 Mid_Out, J43 High_Out, J44 Line_Out_L, J45 Line_Out_R, J5 Mic_In, J6 Effekt_In, J7 AUX_RET_1, J8 AUX_RET_2, J9 AUX_RET_3, SW1 SW_DPST, SW10 SW_SPDT, SW11 SW_SPDT, SW12 SW_SPDT, SW2 SW_SPDT, SW3 SW_SPDT, SW4 SW_SPDT, SW5 SW_SPDT, SW6 SW_SPDT, SW7 SW_SPDT, SW8 SW_SPDT, SW9 SW_Rotary_1x4, U1 TL074, U10 TL074, U11 TL074, U12 TL074, U13 TL074, U14 TL074, U15 TL074, U16 TL074, U17 TL074, U18 TL074, U19 TL074, U2 TL074, U20 TL074, U21 TL074, U22 TL074, U23 TL074, U24 TL074, U25 INA128U, U3 TL074, U4 TL074, U5 TL074, U6 REC10K-2409, U7 REC10K-2415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

Commit message: PCB Update
Parts:
- removed C114, C115: 100n, Capacitor_SMD:C_0805_2012Metric_Pad1.18x1.45mm_HandSolder, symbol Device:C_Small
- removed J21: EMK_Out, Connector_PinSocket_2.54mm_LongPads:PinSocket_1x05_P2.54mm_Vertical_LongPads, symbol Connector:Conn_01x05_Socket
- removed J23: EMK_In, Connector_PinHeader_2.54mm_LongPads:PinHeader_1x05_P2.54mm_Vertical_LongPads, symbol Connector:Conn_01x05_Pin
- removed L1: 470uF, 1.6A, WE-SL575:WE-SL575, symbol Device:L_Coupled
- added J21: Conn_01x05_bridged, Connector_Bridged_2.54mm_LongPads:Bridge_2x05_P2.54mm_Vertical_LongPads, symbol conn_01x05_bridged:Conn_01x05_bridged
- added L1: ~, WE-SL575:WE-SL575, symbol Common_Mode_Choke:Common_Mode_Choke
- C1, C12, C13, C14, C15, C16, C17, C21, C22, C27, C28, C29, C3, C30, C31, C32, C33, C34, C7, C8, J1, J12, J15, J16, J17, J18, J19, J2, J20, J3, J4, J5, J6, J7, J8, J9, R1, R10, R11, R12, R13, R14, R15, R16, R17, R18, R19, R2, R20, R21, R22, R23, R24, R28, R29, R3, R30, R31, R32, R4, R5, R6, R7, R8, R9, RV1, RV2, RV3, RV4, RV5, RV6, SW2, U1, U2, U25, U3, U4, U5, Z1, Z10, Z100, Z11, Z12, Z13, Z14, Z15, Z16, Z17, Z18, Z19, Z2, Z20, Z21, Z22, Z23, Z24, Z25, Z26, Z27, Z28, Z29, Z3, Z30, Z31, Z32, Z33, Z34, Z35, Z36, Z37, Z38, Z39, Z4, Z40, Z41, Z42, Z43, Z44, Z45, Z46, Z47, Z48, Z49, Z5, Z50, Z51, Z52, Z53, Z54, Z55, Z56, Z57, Z58, Z59, Z6, Z60, Z61, Z62, Z63, Z64, Z65, Z66, Z67, Z68, Z69, Z7, Z70, Z71, Z72, Z73, Z74, Z75, Z76, Z77, Z78, Z79, Z8, Z80, Z81, Z82, Z83, Z84, Z85, Z86, Z87, Z88, Z89, Z9, Z90, Z91, Z92, Z93, Z94, Z95, Z96, Z97, Z98, Z99: now not fitted; now left out of the parts list
- C100, C101, C102, C103, C104, C105, C106, C107, C108, C109, C110, C111, C35, C37, C38, C39, C40, C41, C42, C43, C44, C45, C48, C49, C50, C51, C52, C53, C54, C55, C58, C59, C60, C61, C62, C63, C64, C65, C66, C67, C68, C69, C70, C71, C72, C73, C74, C75, C76, C77, C78, C79, C80, C81, C82, C83, C84, C85, C86, C87, C88, C89, C90, C91, C92, C93, C94, C95, C96, C97, C98, C99, J22, J24, J25, J26, J27, J28, J29, J37, J38, J39, J40, J41, J42, J43, J44, J45, R100, R101, R102, R103, R104, R105, R106, R107, R108, R109, R110, R111, R112, R113, R114, R115, R116, R117, R118, R119, R120, R121, R122, R123, R124, R125, R126, R127, R128, R129, R130, R131, R132, R133, R134, R135, R136, R137, R138, R139, R140, R141, R142, R143, R144, R145, R146, R147, R148, R149, R33, R34, R35, R36, R37, R38, R39, R40, R41, R42, R43, R44, R45, R46, R47, R48, R49, R50, R51, R52, R53, R54, R55, R56, R57, R58, R61, R62, R63, R64, R65, R66, R69, R70, R73, R74, R76, R77, R78, R79, R80, R83, R85, R87, R88, R89, R90, R91, R92, R93, R94, R95, R96, R97, R98, R99, RV10, RV11, RV12, RV13, RV14, RV15, RV16, RV17, RV18, RV19, RV20, RV21, RV22, RV7, RV8, RV9, SW10, SW11, SW12, SW3, SW4, SW5, SW6, SW7, SW8, U10, U11, U12, U13, U14, U15, U16, U17, U18, U19, U20, U21, U22, U8, U9, Z101, Z102, Z103, Z104, Z105, Z106, Z107, Z108, Z109, Z110, Z111, Z112, Z113, Z114, Z115, Z116, Z117, Z118, Z119, Z120, Z121, Z138, Z139, Z140, Z141, Z142, Z143, Z144, Z145, Z146, Z147, Z148, Z149, Z150, Z151, Z152, Z153, Z154, Z155, Z156, Z157, Z158, Z159, Z160, Z161, Z162, Z163, Z164, Z165, Z166, Z169, Z175, Z176, Z177, Z178, Z179, Z180, Z181, Z182, Z183, Z184, Z185, Z186, Z187, Z188, Z189, Z190, Z191, Z192, Z193, Z194, Z195, Z196, Z197, Z198, Z199, Z200, Z201, Z202, Z203, Z204, Z205, Z206, Z207, Z208, Z209, Z210, Z211, Z212, Z213, Z214, Z215, Z216, Z217, Z218, Z219, Z220, Z221, Z222, Z223, Z224, Z225, Z226, Z227, Z228, Z229, Z230, Z231, Z232, Z233, Z234, Z235, Z236, Z237, Z238, Z239, Z240, Z241, Z242, Z243, Z244, Z245, Z246, Z247, Z248, Z249, Z250, Z251, Z252, Z253, Z254, Z255, Z256: now fitted; now in the parts list
- C112, C113: value 100n -> 10n; now not fitted; now left out of the parts list
- C2, C5: footprint Capacitor_SMD:C_0805_2012Metric_Pad1.18x1.45mm_HandSolder -> Capacitor_SMD:C_1210_3225Metric_Pad1.33x2.70mm_HandSolder
- L2, L3, L4, L5: footprint Connector_PinSocket_2.54mm_LongPads:PinSocket_1x02_P2.54mm_Vertical_LongPads -> Inductor_SMD:L_1206_3216Metric
- renumbered U24 to U23, U23 to U24
Connections:
- net +15V: now also J22.5 (Pin_5); no longer C46.2, C56.2, J13.3 (Pin_3), J14.3 (Pin_3), J22.3 (Pin_3), R26.1, R72.1, U23.4 (V+), U24.4 (V+)
- net +9V: now also J22.2 (Pin_2); no longer J13.1 (Pin_1), J14.1 (Pin_1), J22.1 (Pin_1), J36.3 (Pin_3), R25.1
- net -15V: now also J22.3 (Pin_3); no longer C47.2, C57.2, J13.4 (Pin_4), J14.4 (Pin_4), J22.4 (Pin_4), R27.1, U23.11 (V-), U24.11 (V-)
- net 9V_GND: now also J22.1 (Pin_1); no longer C10.2, C18.2, C24.1, J13.2 (Pin_2), J14.2 (Pin_2), J22.2 (Pin_2), J36.4 (Pin_4), L3.2
- net GND: now also J22.4 (Pin_4); no longer C112.1, C112.2, C113.1, C113.2, C19.2, C20.1, C36.2, C46.1, C47.1, C56.1, C57.1, D3.2 (A), J13.5 (Pin_5), J14.5 (Pin_5), J22.5 (Pin_5), J36.2 (Pin_2), R75.1, R86.1, U23.3 (+), U23.5 (+), U7.5 (COM), Z122.2, Z123.2, Z124.2, Z125.2, Z126.2, Z127.2, Z128.2, Z129.2, Z134.2, Z135.2, Z136.2, Z137.2, Z170.2, Z171.2, Z174.2
- net Pegel_Aux_Return: now also SW9.2, U24.1, U24.2 (-); no longer SW9.3, U24.8, U24.9 (-)
- net Pegel_Mic_Effekt: now also SW9.3; no longer SW9.2
- net Pegel_Post: now also SW9.1, U24.6 (-), U24.7; no longer SW9.4, U24.13 (-), U24.14
- net Pegel_Pre: now also SW9.4; no longer SW9.1
- net at Z133.2, Z137.1: now also U24.5 (+); no longer U24.12 (+)
- net at D1.1 (K), R59.2, R60.1: now also U23.13 (-); no longer U23.2 (-)
- net at C2.1, SW1.4: now also L1.1
- net at C11.1, C4.2, C5.1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: now also C113.2, L1.2
- net at C2.2, SW1.2: now also L1.4
- net at C10.1, C12.1, C5.2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: now also C112.1, L1.3
- net at Z132.2, Z136.1: now also U24.3 (+); no longer U24.10 (+)
- net at D1.2 (A), D2.1 (K): now also U23.14; no longer U23.1
- net at R67.2, R68.2, R71.1: now also U23.9 (-); no longer U23.6 (-)
- net at R71.2, U24.10 (+), U24.12 (+): now also U23.8; no longer U23.7
- net FILT_GND renamed GND_15V_FILT
- net GND_15V_FILT: no longer C23.1, C24.2
- new net +15V_M: C46.2, C56.2, J21.6 (Pin_5), R72.1, U23.4 (V+), U24.4 (V+)
- new net +15V_P: J13.5 (Pin_5), J14.5 (Pin_5), J21.5 (Pin_5), R26.1
- new net +9V_M: J21.9 (Pin_2), J36.4 (Pin_4)
- new net +9V_P: J13.2 (Pin_2), J14.2 (Pin_2), J21.2 (Pin_2), R25.1
- new net -15V_M: C47.2, C57.2, J21.8 (Pin_3), U23.11 (V-), U24.11 (V-)
- new net -15V_P: J13.3 (Pin_3), J14.3 (Pin_3), J21.3 (Pin_3), R27.1
- new net 9V_GND_M: J21.10 (Pin_1), J36.3 (Pin_3)
- new net 9V_GND_P: C10.2, C18.2, C24.1, J13.1 (Pin_1), J14.1 (Pin_1), J21.1 (Pin_1), L3.2
- new net GND_9V_FILT: C112.2, C113.1, C23.1, C24.2
- new net GND_M: C36.2, C46.1, C47.1, C56.1, C57.1, D3.2 (A), J21.7 (Pin_4), J36.2 (Pin_2), R75.1, R86.1, U23.10 (+), U23.12 (+), Z122.2, Z123.2, Z124.2, Z125.2, Z126.2, Z127.2, Z128.2, Z129.2, Z134.2, Z135.2, Z136.2, Z137.2, Z170.2, Z171.2, Z174.2
- new net GND_P: C19.2, C20.1, J13.4 (Pin_4), J14.4 (Pin_4), J21.4 (Pin_4), U7.5 (COM)
Other:
- moved on the sheet: C2, C24, C25, C26, C4, C46, C5, C56, C6, J10, J11, J36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

Commit message: PCB Update
Parts:
- added Z257, Z258, Z259: ~, Resistor_SMD:R_0805_2012Metric_Pad1.20x1.40mm_HandSolder, symbol Device:R
Connections:
- net GND: now also Z258.2, Z259.2
- net at U21.12 (+), U22.3 (+), Z226.2: now also Z257.2, Z259.1; no longer J29.1 (Pin_1)
- new net: J29.1 (Pin_1), Z257.1, Z258.1
Other:
- moved on the sheet: Z235, Z236, Z245, Z246, Z255, Z256

Commit message: PCB Update
Parts:
- removed SW10, SW11, SW12, SW3, SW4, SW5, SW6, SW7, SW8: SW_SPDT, Connector_PinHeader_2.54mm_LongPads:PinHeader_1x03_P2.54mm_Vertical_LongPads, symbol Switch:SW_SPDT
- added SW10, SW11, SW12, SW3, SW4, SW5, SW6, SW7, SW8: SW_SPDT, Connector_PinHeader_2.54mm_LongPads:PinHeader_1x02_P2.54mm_Vertical_LongPads, symbol sw_spdt_2:SW_SPDT
- renumbered U9 to U8, U8 to U9
Connections:
- net at R35.1, RV7.1, U10.1: now also SW3.1 (A)
- net at R36.1, RV7.2, RV7.3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: now also SW3.2 (B)
- net at R37.1, RV8.1, U11.7: now also SW4.1 (A)
- net at R38.1, RV8.2, RV8.3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: now also SW4.2 (B)
- net at R40.2, R49.2: now also U8.12 (+); no longer U8.5 (+)
- net at R39.2, R55.1: now also U8.13 (-); no longer U8.6 (-)
- net at R55.2, Z140.1: now also U8.14; no longer U8.7
- net at R123.2, RV22.1, U14.8: now also SW12.1 (A)
- net at R124.2, RV22.2, RV22.3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: now also SW12.2 (B)
- net at U10.3 (+), U11.5 (+), U12.10 (+)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: now also U8.5 (+); no longer U8.3 (+)
- net at R34.1, R45.2, U13.8: now also SW8.1 (A)
- net at R34.2, R46.2, U13.9 (-): now also SW8.2 (B)
- net at R41.2, R56.1: now also U8.9 (-); no longer U8.6 (-)
- net at R56.2, Z141.1: now also U8.8; no longer U8.7
- net at R41.1, RV10.1: now also U8.7, SW6.1 (A); no longer U8.1
- net at R42.1, RV10.2, RV10.3: now also U8.6 (-), SW6.2 (B); no longer U8.2 (-)
- net at R42.2, R50.2: now also U8.10 (+); no longer U8.5 (+)
- net at C42.1, RV17.1, RV17.2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: now also U9.3 (+); no longer U9.12 (+)
- net at R33.1, R43.2, U12.8: now also SW7.1 (A)
- net at R33.2, R44.2, U12.9 (-): now also SW7.2 (B)
- net at RV12.2: now also U9.5 (+); no longer U9.10 (+)
- net at R101.2, RV12.3, Z181.1: now also U9.1; no longer U9.14
- net at R101.1, R91.2: now also U9.2 (-); no longer U9.13 (-)
- net at R122.2, RV21.2, RV21.3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: now also SW11.2 (B)
- net at R39.1, RV9.1, U8.1: now also SW5.1 (A)
- net at R40.1, RV9.2, RV9.3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: now also SW5.2 (B)
- net at R121.2, RV21.1, U21.1: now also SW11.1 (A)
- net at R77.2, RV11.1, U14.1: now also SW10.1 (A)
- net at R78.2, RV11.2, RV11.3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: now also SW10.2 (B)
- new net: C38.2, U9.6 (-), U9.7
- no-connect marks 12 -> 3

Commit message: PCB Update
Parts:
- removed J13, J14: EMK_Out, Connector_PinSocket_2.54mm_LongPads:PinSocket_1x05_P2.54mm_Vertical_LongPads, symbol Connector:Conn_01x05_Socket
- added C114, C116, C117, C118: 100n, Capacitor_SMD:C_0805_2012Metric_Pad1.18x1.45mm_HandSolder, symbol Device:C_Small
- added C115: 10n, Capacitor_SMD:C_1210_3225Metric_Pad1.33x2.70mm_HandSolder, symbol Device:C_Small
- added H1, H2, H3, H4, H6, H7, H8: MountingHole, MountingHole:MountingHole_3.2mm_M3_Pad, symbol Mechanical:MountingHole
- added H5: MountingHole_Pad, MountingHole:MountingHole_3.2mm_M3_Pad, symbol Mechanical:MountingHole_Pad
- renumbered U9 to U10, U9 to U11, U10 to U9, U11 to U9
Connections:
- net GND_M: now also C115.2
- net at C43.1, RV18.1, RV18.2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: now also U11.5 (+); no longer U11.12 (+)
- net at R102.1, R93.2: now also U11.6 (-); no longer U11.13 (-)
- net at R102.2, RV13.3, Z182.1: now also U11.7; no longer U11.14
- net at R35.2, R53.1: now also U9.13 (-); no longer U9.6 (-)
- net at R53.2, Z138.1: now also U9.14; no longer U9.7
- net at R36.2, R47.2: now also U9.12 (+); no longer U9.5 (+)
- net +15V renamed +15V_O
- net +15V_O: no longer C13.2, C16.2, C28.2, C31.2, C33.2, C7.2, J12.5 (Pin_5), U1.4 (V+), U2.4 (V+), U25.7 (V+), U3.4 (V+), U4.4 (V+), U5.4 (V+)
- net +9V renamed +9V_I
- net +9V_I: no longer J22.2 (Pin_2)
- net -15V renamed -15V_O
- net -15V_O: no longer C14.2, C17.2, C29.2, C32.2, C34.2, C8.2, J12.3 (Pin_3), U1.11 (V-), U2.11 (V-), U25.4 (V-), U3.11 (V-), U4.11 (V-), U5.11 (V-)
- net 9V_GND renamed 9V_GND_I
- net 9V_GND_I: no longer J22.1 (Pin_1)
- net GND renamed GND_O
- net GND_O: no longer C13.1, C14.1, C16.1, C17.1, C28.1, C29.1, C3.2, C30.2, C31.1, C32.1, C33.1, C34.1, C7.1, C8.1, J1.2 (Pin_2), J12.4 (Pin_4), J2.2 (Pin_2), J3.2 (Pin_2), J4.2 (Pin_2), J5.1 (Pin_1), J6.2 (Pin_2), J7.2 (Pin_2), J8.2 (Pin_2), J9.2 (Pin_2), R18.1, R24.1, R31.1, R4.1, U25.5 (REF), Z1.2, Z10.2, Z100.2, Z2.2, Z21.2, Z22.2, Z23.2, Z24.2, Z25.2, Z26.2, Z27.2, Z28.2, Z29.2, Z3.2, Z30.2, Z38.2, Z39.2, Z4.2, Z40.2, Z41.2, Z42.2, Z43.2, Z44.2, Z5.2, Z52.2, Z53.2, Z54.2, Z57.2, Z58.2, Z6.2, Z60.2, Z66.2, Z67.2, Z7.2, Z70.2, Z72.2, Z73.2, Z77.2, Z8.2, Z80.2, Z81.2, Z82.2, Z83.2, Z84.2, Z9.2, Z90.2, Z91.2, Z92.2, Z93.2, Z94.2, Z95.2, Z96.2, Z97.2, Z98.2, Z99.2
- new net: C115.1, H5.1
- new net +15V_I: C13.2, C16.2, C28.2, C31.2, C33.2, C7.2, J12.5 (Pin_5), U1.4 (V+), U2.4 (V+), U25.7 (V+), U3.4 (V+), U4.4 (V+), U5.4 (V+)
- new net +9V_O: J22.2 (Pin_2)
- new net -15V_I: C14.2, C17.2, C29.2, C32.2, C34.2, C8.2, J12.3 (Pin_3), U1.11 (V-), U2.11 (V-), U25.4 (V-), U3.11 (V-), U4.11 (V-), U5.11 (V-)
- new net 9V_GND_O: J22.1 (Pin_1)
- new net GND_I: C114.1, C114.2, C116.1, C116.2, C117.1, C117.2, C118.1, C118.2, C13.1, C14.1, C16.1, C17.1, C28.1, C29.1, C3.2, C30.2, C31.1, C32.1, C33.1, C34.1, C7.1, C8.1, J1.2 (Pin_2), J12.4 (Pin_4), J2.2 (Pin_2), J3.2 (Pin_2), J4.2 (Pin_2), J5.1 (Pin_1), J6.2 (Pin_2), J7.2 (Pin_2), J8.2 (Pin_2), J9.2 (Pin_2), R18.1, R24.1, R31.1, R4.1, U25.5 (REF), Z1.2, Z10.2, Z100.2, Z2.2, Z21.2, Z22.2, Z23.2, Z24.2, Z25.2, Z26.2, Z27.2, Z28.2, Z29.2, Z3.2, Z30.2, Z38.2, Z39.2, Z4.2, Z40.2, Z41.2, Z42.2, Z43.2, Z44.2, Z5.2, Z52.2, Z53.2, Z54.2, Z57.2, Z58.2, Z6.2, Z60.2, Z66.2, Z67.2, Z7.2, Z70.2, Z72.2, Z73.2, Z77.2, Z8.2, Z80.2, Z81.2, Z82.2, Z83.2, Z84.2, Z9.2, Z90.2, Z91.2, Z92.2, Z93.2, Z94.2, Z95.2, Z96.2, Z97.2, Z98.2, Z99.2
Other:
- moved on the sheet: C10, C11, C112, C113, C12, C18, C19, C2, C20, C23, C24, C25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

Commit message: PCB Update
Parts:
- renumbered U13 to U10, U12 to U10, U10 to U11, U22 to U11, U10 to U12, U10 to U13, U11 to U13, U11 to U22
Connections:
- net GND_O: now also U11.10 (+), U11.12 (+); no longer U11.10 (+), U11.12 (+)
- net at R64.2, R65.2, R66.2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: now also U11.6 (-); no longer U11.13 (-)
- net at RV14.2: now also U13.10 (+); no longer U13.12 (+)
- net at R58.1, Z143.1: now also U10.8; no longer U10.14
- net at C43.1, RV18.1, RV18.2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: now also U22.12 (+); no longer U22.5 (+)
- net at R102.1, R93.2: now also U22.13 (-); no longer U22.6 (-)
- net at R102.2, RV13.3, Z182.1: now also U22.14; no longer U22.7
- net at R61.2, R62.2, R63.2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: now also U11.2 (-); no longer U11.9 (-)
- net at R73.2, Z159.1: now also U11.1; no longer U11.8
- net at U8.3 (+), U8.5 (+), U9.3 (+)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: now also U10.3 (+); no longer U10.10 (+)
- net at Z112.2, Z116.1: now also U10.5 (+); no longer U10.10 (+)
- net at R34.1, R45.2, SW8.1 (A): now also U10.7; no longer U10.8
- net at R34.2, R46.2, SW8.2 (B): now also U10.6 (-); no longer U10.9 (-)
- net at C42.1, RV17.1, RV17.2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: now also U12.12 (+); no longer U12.3 (+)
- net at R33.1, R43.2, SW7.1 (A): now also U10.1; no longer U10.8
- net at R33.2, R44.2, SW7.2 (B): now also U10.2 (-); no longer U10.9 (-)
- net at C44.1, RV19.1, RV19.2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: now also U13.12 (+); no longer U13.3 (+)
- net at RV12.2: now also U12.10 (+); no longer U12.5 (+)
- net at R101.2, RV12.3, Z181.1: now also U12.14; no longer U12.1
- net at R103.1, R95.2: now also U13.13 (-); no longer U13.2 (-)
- net at R101.1, R91.2: now also U12.13 (-); no longer U12.2 (-)
- net at R74.2, Z160.1: now also U11.7; no longer U11.14
- net at R46.1, R52.1: now also U10.10 (+); no longer U10.12 (+)
- net at Z156.1: now also U11.3 (+); no longer U11.10 (+)
- net at R45.1, R58.2: now also U10.9 (-); no longer U10.13 (-)
- net at R103.2, RV14.3, Z183.1: now also U13.14; no longer U13.1
- net at Z157.1: now also U11.5 (+); no longer U11.12 (+)
- new net: C40.2, U13.8, U13.9 (-)
- new net: U11.13 (-), U11.14
- new net: C38.2, U12.8, U12.9 (-)
- new net: U11.8, U11.9 (-)
Other:
- moved on the sheet: U11C, U11D, U22B

Commit message: PCB Update
Parts:
- renumbered U22 to U12, U12 to U22
Connections:
- net at C45.1, RV20.1, RV20.2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: now also U22.10 (+); no longer U22.3 (+)
- net at C43.1, RV18.1, RV18.2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: now also U12.5 (+); no longer U12.12 (+)
- net at R102.1, R93.2: now also U12.6 (-); no longer U12.13 (-)
- net at R102.2, RV13.3, Z182.1: now also U12.7; no longer U12.14
- net at RV15.2: now also U22.12 (+); no longer U22.5 (+)
- net at R104.2, RV15.3, Z184.1: now also U22.8; no longer U22.1
- net at R104.1, R97.2: now also U22.9 (-); no longer U22.2 (-)
- net at RV13.2: now also U12.3 (+); no longer U12.10 (+)
- new net: C41.2, U22.13 (-), U22.14
- new net: C39.2, U12.1, U12.2 (-)
Changed lines of the file:
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@@
 		(at 613.41 140.97 0)
 		(mirror x)
-		(unit 4)
+		(unit 2)
 		(exclude_from_sim no)
 		(in_bom yes)
 		(on_board yes)
 		(dnp no)
-		(property "Reference" "U22"
+		(property "Reference" "U12"
 			(at 613.41 135.382 0)
 			(effects
@@
 			(project "DiKo_PreAmp"
 				(path "/81a92cd6-862a-4567-ad33-f8a3bc120591"
-					(reference "U22")
-					(unit 4)
+					(reference "U12")
+					(unit 2)
 				)
 			)
@@
 		(lib_id "Amplifier_Operational:TL074")
 		(at 561.34 170.18 0)
-		(unit 3)
+		(unit 1)
 		(exclude_from_sim no)
 		(in_bom yes)
@@
 		(dnp no)
 		(fields_autoplaced yes)
-		(property "Reference" "U22"
+		(property "Reference" "U12"
 			(at 561.34 160.02 0)
 			(effects
@@
 			(project "DiKo_PreAmp"
 				(path "/81a92cd6-862a-4567-ad33-f8a3bc120591"
-					(reference "U22")
-					(unit 3)
+					(reference "U12")
+					(unit 1)
 				)
 			)
@@
 		(at 613.41 274.32 0)
 		(mirror x)
-		(unit 1)
+		(unit 3)
 		(exclude_from_sim no)
 		(in_bom yes)
 		(on_board yes)
 		(dnp no)
-		(property "Reference" "U12"
+		(property "Reference" "U22"
 			(at 613.41 268.732 0)
 			(effects
@@
 			(project "DiKo_PreAmp"
 				(path "/81a92cd6-862a-4567-ad33-f8a3bc120591"
-					(reference "U12")
-					(unit 1)
+					(reference "U22")
+					(unit 3)
 				)
 			)
@@
 		(lib_id "Amplifier_Operational:TL074")
 		(at 561.34 303.53 0)
-		(unit 2)
+		(unit 4)
 		(exclude_from_sim no)
 		(in_bom yes)
@@
 		(dnp no)
 		(fields_autoplaced yes)
-		(property "Reference" "U12"
+		(property "Reference" "U22"
 			(at 561.34 293.37 0)
 			(effects
@@
 			(project "DiKo_PreAmp"
 				(path "/81a92cd6-862a-4567-ad33-f8a3bc120591"
-					(reference "U12")
-					(unit 2)
+					(reference "U22")
+					(unit 4)
 				)
 			)

Commit message: PCB Update
Parts:
- RV17, RV20: footprint Connector_PinSocket_2.54mm_LongPads:PinSocket_1x06_P2.54mm_Vertical_LongPads -> Connector_PinSocket_2.54mm_LongPads:PinSocket_2x03_P2.54mm_Vertical_LongPads
- RV18, RV19: footprint Connector_PinSocket_2.54mm_LongPads:PinSocket_1x06_P2.54mm_Vertical_LongPads -> Connector_PinSocket_2.54mm_LongPads:PinSocket_2x03_P2.54mm_Vertical_LongPads_Mirrored
- renumbered U22 to U13, U13 to U22
Connections:
- net at R93.1, RV13.1: now also Z152.2; no longer Z153.2
- net at C37.1, R85.1: now also U22.10 (+); no longer U22.5 (+)
- net at RV14.2: now also U13.3 (+); no longer U13.10 (+)
- net at R76.1, Z163.1: now also U22.14; no longer U22.1
- net at R69.1, R70.1, R76.2: now also U22.13 (-); no longer U22.2 (-)
- net at Z158.1: now also U22.12 (+); no longer U22.3 (+)
- net at C43.1, RV18.1, RV18.2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: now also U12.12 (+); no longer U12.5 (+)
- net at R102.1, R93.2: now also U12.13 (-); no longer U12.6 (-)
- net at R102.2, RV13.3, Z182.1: now also U12.14; no longer U12.7
- net at RV15.2: now also U13.5 (+); no longer U13.12 (+)
- net at R99.1, RV16.3, Z178.1: now also U22.8; no longer U22.7
- net at C42.1, RV17.1, RV17.2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: now also U12.10 (+); no longer U12.12 (+)
- net at R91.1, RV12.1: now also Z153.2; no longer Z152.2
- net at RV12.2: now also U12.5 (+); no longer U12.10 (+)
- net at R101.2, RV12.3, Z181.1: now also U12.8; no longer U12.14
- net at R100.1, R99.2: now also U22.9 (-); no longer U22.6 (-)
- net at C48.1: now also Z199.2; no longer Z197.2
- net at R101.1, R91.2: now also U12.9 (-); no longer U12.13 (-)
- net at C49.1: now also Z197.2; no longer Z199.2
- new net: C40.2, U13.1, U13.2 (-)
- new net: C41.2, U13.6 (-), U13.7
- new net: C38.2, U12.6 (-), U12.7
Other:
- moved on the sheet: C38, C39, C42, C43, R101, R102, R87, R88, R91, R92, R93, R94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

Commit message: PCB Update
Parts:
- removed Z185, Z193, Z198: ~, Resistor_SMD:R_0805_2012Metric_Pad1.20x1.40mm_HandSolder, symbol Device:R_Small
- added Z185, Z193, Z198: ~, Resistor_SMD:R_0805_2012Metric_Pad1.20x1.40mm_HandSolder, symbol Device:R
- renumbered U16 to U14, U15 to U14, U16 to U15, U14 to U16
Connections:
- net GND_O: now also Z193.2
- net at C59.2, R118.2: now also U14.5 (+); no longer U14.3 (+)
- net at C82.2, R141.2: now also U14.12 (+); no longer U14.5 (+)
- net at C63.2, R114.2: now also U15.5 (+); no longer U15.10 (+)
- net at C53.2, R128.1: now also U15.6 (-), U15.7; no longer U15.8, U15.9 (-)
- net at C52.2, R127.1: now also U15.1, U15.2 (-); no longer U15.8, U15.9 (-)
- net at C75.2, Z213.1: now also U15.8, U15.9 (-); no longer U15.13 (-), U15.14
- net at C83.2, R142.2: now also U14.10 (+); no longer U14.5 (+)
- net at R134.2, Z186.1: now also U14.8, U14.9 (-); no longer U14.6 (-), U14.7
- net at C62.2, R113.2: now also U15.3 (+); no longer U15.10 (+)
- net at C87.2, R138.2: now also U15.10 (+); no longer U15.12 (+)
- net at R105.1: now also Z198.2
- net at C71.1, R110.2: now also U14.6 (-), U14.7; no longer U14.1, U14.2 (-)
- new net: R133.2, U14.13 (-), U14.14, Z185.1
- new net: Z185.2, Z193.1, Z198.1
Other:
- moved on the sheet: R105
