File: KiCad/Output.kicad_sch (KiCad schematic)
At the start: 644 parts, among them J1 R_Phono_In, J10 VCC_IN, J11 VCC_OUT, J12 EMK_In, J15 Mic_Effekt_Out, J16 Mic_Effekt_Out, J17 Mic_Effekt_Out, J18 Mic_Effekt_Out, J19 Phono/Line_Out, J2 L_Phono_In, J20 Mic_Effekt_Out, J21 Conn_01x05_bridged, J22 EMK_In, J24 Mic_Effekt_In, J25 Mic_Effekt_In, J26 Phono/Line_In, J27 Mic_Effekt_In, J28 Pegel_Out, J29 Pegel_Out, J3 R_Line_In, J30 Pegel_In, J31 Pegel_In, J32 Pegel_In, J33 Pegel_In, J34 LED_Out, J35 LED_In, J36 VU_Meter_Out, J37 AUX_Send_3, J38 AUX_Send_1, J39 AUX_Send_2, J4 L_Line_In, J40 Bass_Out, J41 Kick_Out, J42 Mid_Out, J43 High_Out, J44 Line_Out_L, J45 Line_Out_R, J5 Mic_In, J6 Effekt_In, J7 AUX_RET_1, J8 AUX_RET_2, J9 AUX_RET_3, SW1 SW_DPST, SW10 SW_SPDT, SW11 SW_SPDT, SW12 SW_SPDT, SW2 SW_SPDT, SW3 SW_SPDT, SW4 SW_SPDT, SW5 SW_SPDT, SW6 SW_SPDT, SW7 SW_SPDT, SW8 SW_SPDT, SW9 SW_Rotary_1x4, U1 TL074, U10 TL074, U11 TL074, U12 TL074, U13 TL074, U14 TL074, U15 TL074, U16 TL074, U17 TL074, U18 TL074, U19 TL074, U2 TL074, U20 TL074, U21 TL074, U22 TL074, U23 TL074, U24 TL074, U25 INA128U, U3 TL074, U4 TL074, U5 TL074, U6 REC10K-2409, U7 REC10K-2415, U8 TL074, U9 TL074

Commit message: PCB Update
Parts:
- renumbered U17 to U16, U18 to U16, U18 to U17, U20 to U18, U16 to U20
Connections:
- net at U18.5 (+), Z223.2: now also U18.10 (+); no longer U18.3 (+)
- net at Z228.1, Z238.1: now also U19.8, U19.9 (-); no longer U19.1, U19.2 (-)
- net at C61.2, R120.2: now also U16.5 (+); no longer U16.3 (+)
- net at C88.2, R139.2: now also U17.5 (+); no longer U17.12 (+)
- net at U19.5 (+), Z221.2: now also U19.10 (+); no longer U19.3 (+)
- net at C89.2, R140.2: now also U17.3 (+); no longer U17.12 (+)
- net at Z231.1, Z241.1: now also U18.8, U18.9 (-); no longer U18.1, U18.2 (-)
- net at Z229.1, Z239.1: now also U19.13 (-), U19.14; no longer U19.8, U19.9 (-)
- net at C84.2, R143.2: now also U16.12 (+); no longer U16.5 (+)
- net at C65.2, R116.2: now also U17.12 (+); no longer U17.10 (+)
- net at C76.2, Z214.1: now also U17.6 (-), U17.7; no longer U17.13 (-), U17.14
- net at R136.2, Z188.1: now also U16.8, U16.9 (-); no longer U16.6 (-), U16.7
- net at C77.2, Z215.1: now also U17.1, U17.2 (-); no longer U17.13 (-), U17.14
- net at Z233.1, Z243.1: now also U18.13 (-), U18.14; no longer U18.8, U18.9 (-)
- net at C73.1, R112.2: now also U16.6 (-), U16.7; no longer U16.1, U16.2 (-)
- net at C55.2, R130.1: now also U17.13 (-), U17.14; no longer U17.8, U17.9 (-)
- net at C85.2, R144.2: now also U16.10 (+); no longer U16.5 (+)
- net at R135.2, Z187.1: now also U16.13 (-), U16.14; no longer U16.6 (-), U16.7
- new net: U19.1, U19.2 (-), Z230.1
- new net: U18.1, U18.2 (-), Z234.1
- new net: U18.12 (+), U18.3 (+), Z224.2
- new net: U19.12 (+), U19.3 (+), Z222.2
Changed lines of the file:
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@@
 		(on_board yes)
 		(dnp no)
-		(property "Reference" "U17"
+		(property "Reference" "U16"
 			(at 679.958 186.182 0)
 			(effects
@@
 			(project "DiKo_PreAmp"
 				(path "/81a92cd6-862a-4567-ad33-f8a3bc120591"
-					(reference "U17")
+					(reference "U16")
 					(unit 1)
 				)
@@
 		(lib_id "Amplifier_Operational:TL074")
 		(at 764.54 57.15 0)
-		(unit 1)
+		(unit 3)
 		(exclude_from_sim no)
 		(in_bom yes)
@@
 				(path "/81a92cd6-862a-4567-ad33-f8a3bc120591"
 					(reference "U19")
-					(unit 1)
+					(unit 3)
 				)
 			)
@@
 		(lib_id "Amplifier_Operational:TL074")
 		(at 764.54 191.77 0)
-		(unit 1)
+		(unit 3)
 		(exclude_from_sim no)
 		(in_bom yes)
@@
 		(dnp no)
 		(fields_autoplaced yes)
-		(property "Reference" "U20"
+		(property "Reference" "U18"
 			(at 764.54 181.61 0)
 			(effects
@@
 			(project ""
 				(path "/81a92cd6-862a-4567-ad33-f8a3bc120591"
-					(reference "U20")
-					(unit 1)
+					(reference "U18")
+					(unit 3)
 				)
 			)
@@
 		(lib_id "Amplifier_Operational:TL074")
 		(at 764.54 294.64 0)
-		(unit 4)
+		(unit 1)
 		(exclude_from_sim no)
 		(in_bom yes)
@@
 		(dnp no)
 		(fields_autoplaced yes)
-		(property "Reference" "U20"
+		(property "Reference" "U18"
 			(at 764.54 284.48 0)
 			(effects
@@
 			(project ""
 				(path "/81a92cd6-862a-4567-ad33-f8a3bc120591"
-					(reference "U20")
-					(unit 4)
+					(reference "U18")
+					(unit 1)
 				)
 			)
@@
 		(at 725.17 226.06 0)
 		(mirror x)
-		(unit 4)
+		(unit 2)
 		(exclude_from_sim no)
 		(in_bom yes)
@@
 				(path "/81a92cd6-862a-4567-ad33-f8a3bc120591"
 					(reference "U17")
-					(unit 4)
+					(unit 2)
 				)
 			)
@@
 		(dnp no)
 		(fields_autoplaced yes)
-		(property "Reference" "U16"
+		(property "Reference" "U20"
 			(at 640.08 389.89 0)
 			(effects
@@
 			(project "DiKo_PreAmp"
 				(path "/81a92cd6-862a-4567-ad33-f8a3bc120591"
-					(reference "U16")
+					(reference "U20")
 					(unit 3)
 				)
@@
 		(on_board yes)
 		(dnp no)
-		(property "Reference" "U16"
+		(property "Reference" "U20"
 			(at 568.96 418.338 0)
 			(effects
@@
 			(project "DiKo_PreAmp"
 				(path "/81a92cd6-862a-4567-ad33-f8a3bc120591"
-					(reference "U16")
+					(reference "U20")
 					(unit 2)
 				)
@@
 		(on_board yes)
 		(dnp no)
-		(property "Reference" "U16"
+		(property "Reference" "U20"
 			(at 695.96 418.338 0)
 			(effects
@@
 			(project "DiKo_PreAmp"
 				(path "/81a92cd6-862a-4567-ad33-f8a3bc120591"
-					(reference "U16")
+					(reference "U20")
 					(unit 4)
 				)
@@
 		(at 725.17 191.77 0)
 		(mirror x)
-		(unit 2)
+		(unit 4)
 		(exclude_from_sim no)
 		(in_bom yes)
 		(on_board yes)
 		(dnp no)
-		(property "Reference" "U17"
+		(property "Reference" "U16"
 			(at 725.17 185.928 0)
 			(effects
@@
 			(project "DiKo_PreAmp"
 				(path "/81a92cd6-862a-4567-ad33-f8a3bc120591"
-					(reference "U17")
-					(unit 2)
+					(reference "U16")
+					(unit 4)
 				)
 			)
@@
 		(at 725.17 257.81 0)
 		(mirror x)
-		(unit 2)
+		(unit 3)
 		(exclude_from_sim no)
 		(in_bom yes)
 		(on_board yes)
 		(dnp no)
-		(property "Reference" "U18"
+		(property "Reference" "U16"
 			(at 725.17 251.968 0)
 			(effects
@@
 			(project "DiKo_PreAmp"
 				(path "/81a92cd6-862a-4567-ad33-f8a3bc120591"
-					(reference "U18")
-					(unit 2)
+					(reference "U16")
+					(unit 3)
 				)
 			)
@@
 		(lib_id "Amplifier_Operational:TL074")
 		(at 764.54 124.46 0)
-		(unit 3)
+		(unit 4)
 		(exclude_from_sim no)
 		(in_bom yes)
@@
 				(path "/81a92cd6-862a-4567-ad33-f8a3bc120591"
 					(reference "U19")
-					(unit 3)
+					(unit 4)
 				)
 			)
@@
 		(lib_id "Amplifier_Operational:TL074")
 		(at 764.54 161.29 0)
-		(unit 4)
+		(unit 1)
 		(exclude_from_sim no)
 		(in_bom yes)
@@
 				(path "/81a92cd6-862a-4567-ad33-f8a3bc120591"
 					(reference "U19")
-					(unit 4)
+					(unit 1)
 				)
 			)
@@
 		(at 725.17 292.1 0)
 		(mirror x)
-		(unit 4)
+		(unit 1)
 		(exclude_from_sim no)
 		(in_bom yes)
 		(on_board yes)
 		(dnp no)
-		(property "Reference" "U18"
+		(property "Reference" "U17"
 			(at 725.17 286.258 0)
 			(effects
@@
 			(project "DiKo_PreAmp"
 				(path "/81a92cd6-862a-4567-ad33-f8a3bc120591"
-					(reference "U18")
-					(unit 4)
+					(reference "U17")
+					(unit 1)
 				)
 			)
@@
 		(dnp no)
 		(fields_autoplaced yes)
-		(property "Reference" "U16"
+		(property "Reference" "U20"
 			(at 513.08 389.89 0)
 			(effects
@@
 			(project "DiKo_PreAmp"
 				(path "/81a92cd6-862a-4567-ad33-f8a3bc120591"
-					(reference "U16")
+					(reference "U20")
 					(unit 1)
 				)
@@
 		(at 679.45 257.81 0)
 		(mirror x)
-		(unit 1)
+		(unit 2)
 		(exclude_from_sim no)
 		(in_bom yes)
 		(on_board yes)
 		(dnp no)
-		(property "Reference" "U18"
+		(property "Reference" "U16"
 			(at 679.958 252.222 0)
 			(effects
@@
 			(project "DiKo_PreAmp"
 				(path "/81a92cd6-862a-4567-ad33-f8a3bc120591"
-					(reference "U18")
-					(unit 1)
+					(reference "U16")
+					(unit 2)
 				)
 			)
@@
 		(dnp no)
 		(fields_autoplaced yes)
-		(property "Reference" "U20"
+		(property "Reference" "U18"
 			(at 764.54 218.44 0)
 			(effects
@@
 			(project ""
 				(path "/81a92cd6-862a-4567-ad33-f8a3bc120591"
-					(reference "U20")
+					(reference "U18")
 					(unit 2)
 				)
@@
 		(lib_id "Amplifier_Operational:TL074")
 		(at 764.54 257.81 0)
-		(unit 3)
+		(unit 4)
 		(exclude_from_sim no)
 		(in_bom yes)
@@
 		(dnp no)
 		(fields_autoplaced yes)
-		(property "Reference" "U20"
+		(property "Reference" "U18"
 			(at 764.54 247.65 0)
 			(effects
@@
 			(project ""
 				(path "/81a92cd6-862a-4567-ad33-f8a3bc120591"
-					(reference "U20")
-					(unit 3)
+					(reference "U18")
+					(unit 4)
 				)
 			)
@@
 		(at 679.45 292.1 0)
 		(mirror x)
-		(unit 3)
+		(unit 4)
 		(exclude_from_sim no)
 		(in_bom yes)
 		(on_board yes)
 		(dnp no)
-		(property "Reference" "U18"
+		(property "Reference" "U17"
 			(at 679.45 286.258 0)
 			(effects
@@
 			(project "DiKo_PreAmp"
 				(path "/81a92cd6-862a-4567-ad33-f8a3bc120591"
-					(reference "U18")
-					(unit 3)
+					(reference "U17")
+					(unit 4)
 				)
 			)

Commit message: PCB Update
Parts:
- renumbered U22 to U21, U21 to U22
Connections:
- net at Z226.2, Z257.2, Z259.1: now also U21.12 (+), U21.3 (+); no longer U21.12 (+), U21.3 (+)
- net at Z236.1, Z246.1: now also U21.13 (-), U21.14; no longer U21.1, U21.2 (-)
- net at Z235.1, Z245.1: now also U21.1, U21.2 (-); no longer U21.13 (-), U21.14
Changed lines of the file:
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@@
 		(lib_id "Amplifier_Operational:TL074")
 		(at 764.54 397.51 0)
-		(unit 1)
+		(unit 4)
 		(exclude_from_sim no)
 		(in_bom yes)
@@
 		(dnp no)
 		(fields_autoplaced yes)
-		(property "Reference" "U22"
+		(property "Reference" "U21"
 			(at 764.54 387.35 0)
 			(effects
@@
 			(project ""
 				(path "/81a92cd6-862a-4567-ad33-f8a3bc120591"
-					(reference "U22")
-					(unit 1)
+					(reference "U21")
+					(unit 4)
 				)
 			)
@@
 		(dnp no)
 		(fields_autoplaced yes)
-		(property "Reference" "U22"
+		(property "Reference" "U21"
 			(at 793.75 328.93 0)
 			(effects
@@
 			(project "DiKo_PreAmp"
 				(path "/81a92cd6-862a-4567-ad33-f8a3bc120591"
-					(reference "U22")
+					(reference "U21")
 					(unit 2)
 				)
@@
 		(on_board yes)
 		(dnp no)
-		(property "Reference" "U21"
+		(property "Reference" "U22"
 			(at 695.96 363.728 0)
 			(effects
@@
 			(project ""
 				(path "/81a92cd6-862a-4567-ad33-f8a3bc120591"
-					(reference "U21")
+					(reference "U22")
 					(unit 2)
 				)
@@
 		(lib_id "Amplifier_Operational:TL074")
 		(at 764.54 369.57 0)
-		(unit 4)
+		(unit 1)
 		(exclude_from_sim no)
 		(in_bom yes)
@@
 				(path "/81a92cd6-862a-4567-ad33-f8a3bc120591"
 					(reference "U21")
-					(unit 4)
+					(unit 1)
 				)
 			)
@@
 		(dnp no)
 		(fields_autoplaced yes)
-		(property "Reference" "U21"
+		(property "Reference" "U22"
 			(at 640.08 335.28 0)
 			(effects
@@
 			(project ""
 				(path "/81a92cd6-862a-4567-ad33-f8a3bc120591"
-					(reference "U21")
+					(reference "U22")
 					(unit 1)
 				)

Commit message: PCB Update
Parts:
- RV16: footprint Connector_PinSocket_2.54mm_LongPads:PinSocket_1x06_P2.54mm_Vertical_LongPads -> Connector_PinSocket_2.54mm_LongPads:PinSocket_2x03_P2.54mm_Vertical_LongPads
- renumbered U22 to U20, U20 to U22
Connections:
- net at R83.1, Z175.1, Z176.1: now also U22.14; no longer U22.7
- net at Z158.1: now also U22.5 (+); no longer U22.12 (+)
- net at R69.1, R70.1, R76.2: now also U22.6 (-); no longer U22.13 (-)
- net at R76.1, Z163.1: now also U22.7; no longer U22.14
- net at R78.1, R80.1: now also U22.12 (+); no longer U22.5 (+)
- net at R77.1, R83.2: now also U22.13 (-); no longer U22.6 (-)
Changed lines of the file:
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@@
 		(at 514.35 354.33 0)
 		(mirror x)
-		(unit 4)
+		(unit 2)
 		(exclude_from_sim no)
 		(in_bom yes)
@@
 				(path "/81a92cd6-862a-4567-ad33-f8a3bc120591"
 					(reference "U22")
-					(unit 4)
+					(unit 2)
 				)
 			)
@@
 		(at 568.96 424.18 0)
 		(mirror x)
-		(unit 2)
+		(unit 4)
 		(exclude_from_sim no)
 		(in_bom yes)
 		(on_board yes)
 		(dnp no)
-		(property "Reference" "U20"
+		(property "Reference" "U22"
 			(at 568.96 418.338 0)
 			(effects
@@
 			(project "DiKo_PreAmp"
 				(path "/81a92cd6-862a-4567-ad33-f8a3bc120591"
-					(reference "U20")
-					(unit 2)
+					(reference "U22")
+					(unit 4)
 				)
 			)
@@
 		(on_board yes)
 		(dnp no)
-		(property "Reference" "U22"
+		(property "Reference" "U20"
 			(at 695.96 363.728 0)
 			(effects
@@
 			(project ""
 				(path "/81a92cd6-862a-4567-ad33-f8a3bc120591"
-					(reference "U22")
+					(reference "U20")
 					(unit 2)
 				)
@@
 			)
 		)
-		(property "Footprint" "Connector_PinSocket_2.54mm_LongPads:PinSocket_1x06_P2.54mm_Vertical_LongPads"
+		(property "Footprint" "Connector_PinSocket_2.54mm_LongPads:PinSocket_2x03_P2.54mm_Vertical_LongPads"
 			(at 568.96 360.045 0)
 			(effects
@@
 		(dnp no)
 		(fields_autoplaced yes)
-		(property "Reference" "U20"
+		(property "Reference" "U22"
 			(at 513.08 389.89 0)
 			(effects
@@
 			(project "DiKo_PreAmp"
 				(path "/81a92cd6-862a-4567-ad33-f8a3bc120591"
-					(reference "U20")
+					(reference "U22")
 					(unit 1)
 				)
@@
 		(dnp no)
 		(fields_autoplaced yes)
-		(property "Reference" "U22"
+		(property "Reference" "U20"
 			(at 640.08 335.28 0)
 			(effects
@@
 			(project ""
 				(path "/81a92cd6-862a-4567-ad33-f8a3bc120591"
-					(reference "U22")
+					(reference "U20")
 					(unit 1)
 				)

Commit message: PCB Update
Connections:
- net at R124.1, R126.1: now also U20.5 (+); no longer U20.12 (+)
- net at R122.1, R125.1: now also U20.3 (+); no longer U20.5 (+)
- net at R131.1, Z205.1, Z207.1: now also U20.1; no longer U20.7
- net at R121.1, R131.2: now also U20.2 (-); no longer U20.6 (-)
- net at R123.1, R132.2: now also U20.6 (-); no longer U20.13 (-)
- net at R132.1, Z206.1, Z208.1: now also U20.7; no longer U20.14
- net at U20.10 (+), U22.3 (+), Z180.2: now also U20.12 (+); no longer U20.3 (+)
- net at R122.2, RV21.2, RV21.3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: now also U20.13 (-); no longer U20.2 (-)
- net at R121.2, RV21.1, SW11.1 (A): now also U20.14; no longer U20.1
Changed lines of the file:
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@@
 		(at 695.96 424.18 0)
 		(mirror x)
-		(unit 4)
+		(unit 2)
 		(exclude_from_sim no)
 		(in_bom yes)
@@
 				(path "/81a92cd6-862a-4567-ad33-f8a3bc120591"
 					(reference "U20")
-					(unit 4)
+					(unit 2)
 				)
 			)
@@
 		(at 695.96 369.57 0)
 		(mirror x)
-		(unit 2)
+		(unit 1)
 		(exclude_from_sim no)
 		(in_bom yes)
@@
 				(path "/81a92cd6-862a-4567-ad33-f8a3bc120591"
 					(reference "U20")
-					(unit 2)
+					(unit 1)
 				)
 			)
@@
 		(lib_id "Amplifier_Operational:TL074")
 		(at 640.08 345.44 0)
-		(unit 1)
+		(unit 4)
 		(exclude_from_sim no)
 		(in_bom yes)
@@
 				(path "/81a92cd6-862a-4567-ad33-f8a3bc120591"
 					(reference "U20")
-					(unit 1)
+					(unit 4)
 				)
 			)

Commit message: PCB Update
Parts:
- added C119: 10n, Capacitor_SMD:C_1210_3225Metric_Pad1.33x2.70mm_HandSolder, symbol Device:C_Small
- added C120, C121, C122: 100n, Capacitor_SMD:C_0805_2012Metric_Pad1.18x1.45mm_HandSolder, symbol Device:C_Small
- added H10, H11, H12: MountingHole, MountingHole:MountingHole_3.2mm_M3_Pad, symbol Mechanical:MountingHole
- added H9: MountingHole_Pad, MountingHole:MountingHole_3.2mm_M3_Pad, symbol Mechanical:MountingHole_Pad
Connections:
- net GND_O: now also C119.2, C120.1, C120.2, C121.1, C121.2, C122.1, C122.2
- new net: C119.1, H9.1
Other:
- moved on the sheet: J22

Commit message: PCB Update
Parts:
- removed C120, C121, C122: 100n, Capacitor_SMD:C_0805_2012Metric_Pad1.18x1.45mm_HandSolder, symbol Device:C_Small

Commit message: PCB Final Update
Parts:
- removed J22: EMK_In, Connector_PinHeader_2.54mm_LongPads:PinHeader_1x05_P2.54mm_Vertical_LongPads, symbol Connector:Conn_01x05_Pin
- added J22: Conn_02x07_Odd_Even, Connector_PinHeader_2.54mm:PinHeader_2x07_P2.54mm_Vertical, symbol Connector_Generic:Conn_02x07_Odd_Even
Connections:
- net +15V_O: now also J22.13 (Pin_13), J22.14 (Pin_14)
- net +9V_O: now also J22.5 (Pin_5), J22.6 (Pin_6)
- net -15V_O: now also J22.7 (Pin_7), J22.8 (Pin_8)
- net 9V_GND_O: now also J22.1 (Pin_1), J22.2 (Pin_2), J22.3 (Pin_3), J22.4 (Pin_4)
- net GND_O: now also J22.10 (Pin_10), J22.11 (Pin_11), J22.12 (Pin_12), J22.9 (Pin_9)
