File: KiCad/KS_BP.kicad_sch (KiCad schematic)
At the start: 172 parts, among them J1 Bass_Out, J2 Bass_Out, J3 Bass_Out, J31 Conn_02x07_Odd_Even, J32 Conn_02x07_Odd_Even, J33 Conn_02x07_Odd_Even, J34 Conn_02x07_Odd_Even, J4 Bass_Out, J5 Bass_Out, J6 Bass_Out, J7 Bass_Out, J8 Bass_Out, SW1 SW_SPDT, SW2 SW_SPDT, SW3 SW_SPDT, SW4 SW_SPDT, U1 TL074, U10 TL074, U11 TL074, U12 TL074, U2 TL074, U3 TL074, U4 TL074, U5 TL074, U6 TL074, U7 TL074, U8 TL074, U9 TL074

Commit message: Upadte
Parts:
- removed C12, C21, C22, C29, C30, C9: 10n, Capacitor_SMD:C_0805_2012Metric_Pad1.18x1.45mm_HandSolder, symbol Device:C_Small
- removed C15, C16, C23, C24, C31, C32: 220n, Capacitor_SMD:C_0805_2012Metric_Pad1.18x1.45mm_HandSolder, symbol Device:C_Small
- removed C17, C18, C25, C26, C33, C34: 150n, Capacitor_SMD:C_0805_2012Metric_Pad1.18x1.45mm_HandSolder, symbol Device:C_Small
- removed C19, C27, C35: 1u, Capacitor_SMD:C_0805_2012Metric_Pad1.18x1.45mm_HandSolder, symbol Device:C_Small
- removed C20, C28, C36: 100n, Capacitor_SMD:C_0805_2012Metric_Pad1.18x1.45mm_HandSolder, symbol Device:C_Small
- removed J2, J3, J4, J6, J7, J8: Bass_Out, Connector_PinSocket_2.54mm_LongPads:PinSocket_1x02_P2.54mm_Vertical_LongPads, symbol Connector:Conn_01x02_Socket
- removed J32, J33, J34: Conn_02x07_Odd_Even, Connector_PinHeader_2.54mm:PinHeader_2x07_P2.54mm_Vertical, symbol Connector_Generic:Conn_02x07_Odd_Even
- removed R12, R30, R42: 680k, Resistor_SMD:R_0805_2012Metric_Pad1.20x1.40mm_HandSolder, symbol Device:R
- removed R15, R164, R165, R166, R26, R3, R37, R38, R9: 1k, Resistor_SMD:R_0805_2012Metric_Pad1.20x1.40mm_HandSolder, symbol Device:R
- removed R16, R27, R28, R39, R4, R40, Z10, Z45, Z60, Z68, Z71, Z74: 100k, Resistor_SMD:R_0805_2012Metric_Pad1.20x1.40mm_HandSolder, symbol Device:R
- removed R21, R32, R44: 75k, Resistor_SMD:R_0805_2012Metric_Pad1.20x1.40mm_HandSolder, symbol Device:R
- removed R22, R23, R33, R34, R45, R46: 15k, Resistor_SMD:R_0805_2012Metric_Pad1.20x1.40mm_HandSolder, symbol Device:R
- removed R24, R25, R35, R36, R47, R48: 7k5, Resistor_SMD:R_0805_2012Metric_Pad1.20x1.40mm_HandSolder, symbol Device:R
- removed R29, R41, R7: 560k, Resistor_SMD:R_0805_2012Metric_Pad1.20x1.40mm_HandSolder, symbol Device:R
- removed R31, R43, R8: 10k, Resistor_SMD:R_0805_2012Metric_Pad1.20x1.40mm_HandSolder, symbol Device:R
- removed SW2, SW3, SW4: SW_SPDT, Connector_PinHeader_2.54mm_LongPads:PinHeader_1x02_P2.54mm_Vertical_LongPads, symbol sw_spdt_2:SW_SPDT
- removed U10, U11, U12, U4, U5, U7, U8, U9: TL074, Package_DIP:DIP-14_W7.62mm_Socket_LongPads, symbol Amplifier_Operational:TL074
- removed unit 1 of U3
- removed unit 4 of U3
- removed unit 3 of U6
- removed Z11, Z12, Z24, Z26, Z27, Z30, Z31, Z38, Z40, Z41, Z43, Z49, Z5, Z51, Z52, Z54, Z55, Z57, Z6: 0R, Resistor_SMD:R_0805_2012Metric_Pad1.20x1.40mm_HandSolder, symbol Device:R
- removed Z14, Z15, Z16, Z50, Z58, Z70, Z73, Z76, Z9: (no value), Resistor_SMD:R_0805_2012Metric_Pad1.20x1.40mm_HandSolder, symbol Device:R
- removed Z2, Z44, Z59, Z69, Z72, Z75: 1u, Resistor_SMD:R_0805_2012Metric_Pad1.20x1.40mm_HandSolder, symbol Device:R
- removed Z35, Z37, Z39, Z42, Z53, Z56: 820k, Resistor_SMD:R_0805_2012Metric_Pad1.20x1.40mm_HandSolder, symbol Device:R
- added C209, C210, C301, C302, C401, C402, C501, C706, C709, C713, C718: 10n, symbol Device:C_Small
- added C211, C212, C303, C304, C403, C404: 220n, symbol Device:C_Small
- added C213, C214, C305, C306, C405, C406: 150n, symbol Device:C_Small
- added C215, C307, C407: 1u, symbol Device:C_Small
- added C216, C308, C408, C704, C707, C715: 100n, symbol Device:C_Small
- added C502: 2n2, symbol Device:C_Small
- added C503: 47u, symbol Device:C_Small
- added C601: 4u7, symbol Device:C_Small
- added C701, C702: 10u, symbol Device:C_Small
- added C703, C711, C712, C719: 470p, symbol Device:C_Small
- added C705, C708, C716: 10u, symbol Device:C_Polarized_Small
- added C710, C714, C717: 1n, symbol Device:C_Small
- added D601, D602, D604: D, symbol Device:D
- added D603: LED, symbol Device:LED
- added J107, J108, J109, J110, J111, J112: Conn_02x07_Odd_Even, symbol Connector_Generic:Conn_02x07_Odd_Even
- added J204, J301, J401: Bass_IN, symbol Connector:Conn_01x02_Socket
- added J205, J302, J402: Bass_Out, symbol Connector:Conn_01x02_Socket
- added J501, J502, J503, J504, J601, J602, J603, J604: L_Phono_In, symbol Connector:Conn_01x02_Pin
- added J505, J506: Phono/Line_Out, symbol Connector:Conn_01x02_Socket
- added J605: VU_Meter_Out, symbol Connector:Conn_01x04_Socket
- added J606: LED_In, symbol Connector:Conn_01x02_Pin
- added J607: LED_Out, symbol Connector:Conn_01x02_Socket
- added J701: VCC_IN, symbol Connector:Conn_01x02_Pin
- added J702: VCC_OUT, symbol Connector:Conn_01x02_Pin
- added L701: (no value), WE-SL575:WE-SL575, symbol Common_Mode_Choke:Common_Mode_Choke
- added L702, L703, L704, L705: Dämpfungsperle, 220 Ohm @ 100MHz, 0.5A, symbol Device:L_Ferrite
- added R214, R218, R301, R305, R401, R405, Z253, Z272, Z305, Z324, Z405, Z424, Z534, Z540: 100k, symbol Device:R
- added R215, R216, R217, R302, R303, R304, R402, R403, R404, R508, R609, R610: 1k, symbol Device:R
- added R219, R306, R406: 560k, symbol Device:R
- added R220, R307, R407: 680k, symbol Device:R
- added R221, R308, R408, R501, R502, R503, R504, R505, R601, R602, R603, R604, R607, R612: 10k, symbol Device:R
- added R222, R309, R409: 75k, symbol Device:R
- added R223, R224, R310, R311, R410, R411, R611, R614: 15k, symbol Device:R
- added R225, R226, R312, R313, R412, R413: 7k5, symbol Device:R
- added R506: 390k, symbol Device:R
- added R507, R605, R606: 33k, symbol Device:R
- added R608: 16k5, symbol Device:R
- added R613: 2k2, symbol Device:R
- added R615: 500R, symbol Device:R
- added SW202, SW301, SW401: SW_SPDT, symbol sw_spdt_2:SW_SPDT
- added SW501: SW_SPDT, symbol Switch:SW_SPDT
- added SW701: SW_DPST, symbol Switch:SW_DPST
- added U103, U107, U108, U109, U110, U111, U112, U113, U114, U203, U204, U205, U206, U301, U302, U303, U401, U402, U403, U501, U502, U503, U504, U601, U602, U603, U604: TL074, symbol OPV_De:TL074
- added unit 5 of U104
- added unit 5 of U105
- added unit 5 of U106
- added U701: REC10K-2415, REC10K-2415DAW_H2:CONV_REC10K-2415DAW_H2, symbol REC10K-2415DAW_H2:REC10K-2415DAW_H2
- added U702: REC10K-2409, REC10K-2409SAW_H2:CONV_REC10K-2409SAW_H2, symbol REC10K-2409SAW_H2:REC10K-2409SAW_H2
- added Z226, Z227, Z234, Z235, Z240, Z241, Z243, Z250, Z251, Z255, Z256, Z258, Z259, Z261, Z262, Z264, Z265, Z267, Z268, Z302, Z303, Z307, Z308, Z310, Z311, Z313, Z314, Z316, Z317, Z319, Z320, Z402, Z403, Z407, Z408, Z410, Z411, Z413, Z414, Z416, Z417, Z419, Z420, Z626, Z627, Z628, Z629, Z632, Z701, Z702, Z703: 0R, symbol Device:R
- added Z230, Z236, Z242, Z252, Z254, Z257, Z260, Z266, Z271, Z304, Z306, Z309, Z312, Z318, Z323, Z404, Z406, Z409, Z412, Z418, Z423, Z502, Z503, Z504, Z506, Z508, Z509, Z510, Z512, Z514, Z515, Z516, Z518, Z520, Z521, Z522, Z524, Z525, Z526, Z527, Z528, Z529, Z530, Z531, Z532, Z535, Z536, Z537, Z538, Z541, Z542, Z543, Z544, Z602, Z603, Z604, Z606, Z608, Z609, Z610, Z612, Z614, Z615, Z616, Z618, Z620, Z621, Z622, Z624, Z625, Z630, Z631: (no value), symbol Device:R
- added Z249, Z269, Z301, Z321, Z401, Z421: 1u, symbol Device:R
- added Z263, Z270, Z315, Z322, Z415, Z422, Z505, Z511, Z517, Z523, Z605, Z611, Z617, Z623: 820k, symbol Device:R
- added Z501, Z507, Z513, Z519, Z601, Z607, Z613, Z619: 4u7, symbol Device:R
- added Z533, Z539: 100R, symbol Device:R
- C109: renamed from C5; footprint Capacitor_SMD:C_0805_2012Metric_Pad1.18x1.45mm_HandSolder -> (none)
- C110: renamed from C6; footprint Capacitor_SMD:C_0805_2012Metric_Pad1.18x1.45mm_HandSolder -> (none)
- C111: renamed from C8; footprint Capacitor_SMD:C_0805_2012Metric_Pad1.18x1.45mm_HandSolder -> (none)
- C112: renamed from C7; footprint Capacitor_SMD:C_0805_2012Metric_Pad1.18x1.45mm_HandSolder -> (none)
- C113: renamed from C10; footprint Capacitor_SMD:C_0805_2012Metric_Pad1.18x1.45mm_HandSolder -> (none)
- C114: renamed from C13; footprint Capacitor_SMD:C_0805_2012Metric_Pad1.18x1.45mm_HandSolder -> (none)
- C115: renamed from C11; footprint Capacitor_SMD:C_0805_2012Metric_Pad1.18x1.45mm_HandSolder -> (none)
- C116: renamed from C14; footprint Capacitor_SMD:C_0805_2012Metric_Pad1.18x1.45mm_HandSolder -> (none)
- J104: renamed from J5; value Bass_Out -> Bass_IN; footprint Connector_PinSocket_2.54mm_LongPads:PinSocket_1x02_P2.54mm_Vertical_LongPads -> (none); Gegenstück Mouser Teilenr. 61301611821 -> (none); Mouser-Teilenr. 710-61301611121 -> (none)
- J105: renamed from J1; footprint Connector_PinSocket_2.54mm_LongPads:PinSocket_1x02_P2.54mm_Vertical_LongPads -> (none); Gegenstück Mouser Teilenr. 61301611821 -> (none); Mouser-Teilenr. 710-61301611121 -> (none)
- J106: renamed from J31; footprint Connector_PinHeader_2.54mm:PinHeader_2x07_P2.54mm_Vertical -> (none); Gegenstück Mouser Teilenr. 164-9007-E -> (none); Mouser-Teilenr. 649-67996-414HLF -> (none)
- R114: renamed from R2; footprint Resistor_SMD:R_0805_2012Metric_Pad1.20x1.40mm_HandSolder -> (none)
- R115: renamed from R1; footprint Resistor_SMD:R_0805_2012Metric_Pad1.20x1.40mm_HandSolder -> (none)
- R116: renamed from R163; footprint Resistor_SMD:R_0805_2012Metric_Pad1.20x1.40mm_HandSolder -> (none)
- R117: renamed from R13; footprint Resistor_SMD:R_0805_2012Metric_Pad1.20x1.40mm_HandSolder -> (none)
- R118: renamed from R14; footprint Resistor_SMD:R_0805_2012Metric_Pad1.20x1.40mm_HandSolder -> (none)
- R119: renamed from R5; footprint Resistor_SMD:R_0805_2012Metric_Pad1.20x1.40mm_HandSolder -> (none)
- R120: renamed from R10; footprint Resistor_SMD:R_0805_2012Metric_Pad1.20x1.40mm_HandSolder -> (none)
- R121: renamed from R6; footprint Resistor_SMD:R_0805_2012Metric_Pad1.20x1.40mm_HandSolder -> (none)
- R122: renamed from R11; footprint Resistor_SMD:R_0805_2012Metric_Pad1.20x1.40mm_HandSolder -> (none)
- R123: renamed from R17; footprint Resistor_SMD:R_0805_2012Metric_Pad1.20x1.40mm_HandSolder -> (none)
- R124: renamed from R18; footprint Resistor_SMD:R_0805_2012Metric_Pad1.20x1.40mm_HandSolder -> (none)
- R125: renamed from R20; footprint Resistor_SMD:R_0805_2012Metric_Pad1.20x1.40mm_HandSolder -> (none)
- R126: renamed from R19; footprint Resistor_SMD:R_0805_2012Metric_Pad1.20x1.40mm_HandSolder -> (none)
- SW102: renamed from SW1; footprint Connector_PinHeader_2.54mm_LongPads:PinHeader_1x02_P2.54mm_Vertical_LongPads -> (none)
- U104: renamed from U1; footprint Package_DIP:DIP-14_W7.62mm_Socket_LongPads -> (none); symbol Amplifier_Operational:TL074 -> OPV_De:TL074
- U104: renamed from U3; footprint Package_DIP:DIP-14_W7.62mm_Socket_LongPads -> (none); symbol Amplifier_Operational:TL074 -> OPV_De:TL074
- U105: renamed from U2; footprint Package_DIP:DIP-14_W7.62mm_Socket_LongPads -> (none); symbol Amplifier_Operational:TL074 -> OPV_De:TL074
- U106: renamed from U6; footprint Package_DIP:DIP-14_W7.62mm_Socket_LongPads -> (none); symbol Amplifier_Operational:TL074 -> OPV_De:TL074
- Z225: renamed from Z66; footprint Resistor_SMD:R_0805_2012Metric_Pad1.20x1.40mm_HandSolder -> (none)
- Z228: renamed from Z65; footprint Resistor_SMD:R_0805_2012Metric_Pad1.20x1.40mm_HandSolder -> (none)
- Z229: renamed from Z67; footprint Resistor_SMD:R_0805_2012Metric_Pad1.20x1.40mm_HandSolder -> (none)
- Z231: renamed from Z4; footprint Resistor_SMD:R_0805_2012Metric_Pad1.20x1.40mm_HandSolder -> (none)
- Z232: renamed from Z3; footprint Resistor_SMD:R_0805_2012Metric_Pad1.20x1.40mm_HandSolder -> (none)
- Z233: renamed from Z13; footprint Resistor_SMD:R_0805_2012Metric_Pad1.20x1.40mm_HandSolder -> (none)
- Z237: renamed from Z29; footprint Resistor_SMD:R_0805_2012Metric_Pad1.20x1.40mm_HandSolder -> (none)
- Z238: renamed from Z28; footprint Resistor_SMD:R_0805_2012Metric_Pad1.20x1.40mm_HandSolder -> (none)
- Z239: renamed from Z36; footprint Resistor_SMD:R_0805_2012Metric_Pad1.20x1.40mm_HandSolder -> (none)
- Z244: renamed from Z25; footprint Resistor_SMD:R_0805_2012Metric_Pad1.20x1.40mm_HandSolder -> (none)
- Z245: renamed from Z1; footprint Resistor_SMD:R_0805_2012Metric_Pad1.20x1.40mm_HandSolder -> (none)
- Z246: renamed from Z34; footprint Resistor_SMD:R_0805_2012Metric_Pad1.20x1.40mm_HandSolder -> (none)
- Z247: renamed from Z7; footprint Resistor_SMD:R_0805_2012Metric_Pad1.20x1.40mm_HandSolder -> (none)
- Z248: renamed from Z8; footprint Resistor_SMD:R_0805_2012Metric_Pad1.20x1.40mm_HandSolder -> (none)
Connections:
- net +15V_O: no longer J106.13 (Pin_13), J106.14 (Pin_14)
- net +9V_O: no longer J106.5 (Pin_5), J106.6 (Pin_6)
- net -15V_O: no longer J106.7 (Pin_7), J106.8 (Pin_8)
- net 9V_GND_O: no longer J106.1 (Pin_1), J106.2 (Pin_2), J106.3 (Pin_3), J106.4 (Pin_4)
- net at Z244.1, Z246.1: now also Z243.2
- net at R119.2, U105.1, U105.2 (-): now also Z235.1; no longer C112.1
- net at R114.2, U104.14: now also Z231.2; no longer Z232.1
- net at C115.2, U106.13 (-), U106.14: now also Z243.1
- net at C113.2, U106.1, U106.2 (-): now also Z241.1; no longer R126.1
- net at C109.1: now also Z232.1; no longer Z231.2
- net at R121.2, U105.13 (-), U105.14: now also Z237.2; no longer Z238.1
- net at R123.1: now also Z238.1; no longer Z237.2
- net at J104.1 (Pin_1), Z225.2: now also Z228.1; no longer Z229.1
- net GND_O renamed GND1
- net GND1: now also C214.1, C216.1, C306.1, C308.1, C406.1, C408.1, J107.10 (Pin_10), J107.11 (Pin_11), J107.12 (Pin_12), J107.9 (Pin_9), J108.10 (Pin_10), J108.11 (Pin_11)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
- new net: Z255.1, Z256.2, Z257.1
- new net: R214.2, U204.14, Z255.2
- new net: C401.2, C402.1, R406.1
- new net: C402.2, R407.2, U402.3 (+)
- new net: R302.1, R303.2, SW301.1 (A), U301.1
- new net: R301.1, R302.2, U301.13 (-)
- new net: R501.2, R502.2, R503.2, R504.2, R505.1, U502.13 (-)
- new net: R505.2, U502.14, Z525.2
- new net: Z319.2, Z320.1, Z322.1
- new net: L702.1, U701.6 (+VOUT)
- new net: C703.2, C704.1, L702.2, Z701.1
- new net: Z602.2, Z603.1, Z606.1
- new net: J205.1 (Pin_1), Z269.2, Z272.1
- new net: U204.3 (+), Z251.1
- new net: Z250.1, Z251.2, Z254.1
- new net: Z608.2, Z609.1, Z612.1
- new net: R602.1, Z609.2
- new net: SW501.2 (B), Z526.1
- new net: Z526.2, Z527.1, Z528.1
- new net: U301.10 (+), Z301.1, Z305.1
- new net: C307.1, R312.1, R313.2
- new net: C308.2, R312.2, U303.12 (+)
- new net: R216.1, R217.1, SW202.2 (B), U204.2 (-)
- new net: R217.2, R218.2, U204.12 (+)
- new net: J607.2 (Pin_2), Z632.1
- new net: C701.1, C703.1, C706.1, L701.2, U701.1 (+VIN), U702.1 (+VIN)
- new net: C301.2, C302.1, R306.1
- new net: C302.2, R307.2, U302.3 (+)
- new net: R601.2, R602.2, R603.2, R604.2, R607.1, U601.13 (-)
- new net: Z310.1, Z311.2, Z312.1
- new net: J701.1 (Pin_1), J702.1 (Pin_1), SW701.3
- new net: J701.2 (Pin_2), J702.2 (Pin_2), SW701.1
- new net: R502.1, Z509.2
- new net: Z267.2, Z268.1, Z270.1
- new net: C209.1, Z256.1
- new net: C209.2, C210.1, R219.1
- new net: R413.1, Z416.2
- new net: C407.1, R412.1, R413.2
- new net: R605.2, R611.1, U601.8, Z626.2
- new net: C601.1, J605.1 (Pin_1), R611.2, R612.2
- new net: R604.1, Z621.2
- new net: J603.1 (Pin_1), Z613.1, Z616.1
- new net: U603.5 (+), Z613.2, Z617.1
- new net: C701.2, C709.1, C711.1, C718.1, C719.1, L701.3, U701.2 (-VIN), U702.2 (-VIN)
- new net: U502.12 (+), Z530.1
- new net: C403.1, C404.2, R408.1
- new net: C403.2, R409.2, U402.12 (+)
- new net: D601.2 (A), R608.1, R609.2
- new net: R605.1, R606.2, R608.2, U601.9 (-)
- new net: R313.1, Z316.2
- new net: C408.2, R412.2, U403.12 (+)
- new net: C407.2, U403.13 (-), U403.14, Z419.1
- new net: U602.5 (+), Z607.2, Z611.1
- new net: U602.6 (-), U602.7, Z608.1
- new net: Z402.1, Z403.2, Z406.1
- new net: U401.8, U401.9 (-), Z402.2
- new net: R303.1, R304.1, SW301.2 (B), U301.2 (-)
- new net: U301.3 (+), Z303.1
- new net: U502.10 (+), Z538.1
- new net: Z537.1, Z538.2, Z540.1
- new net: SW501.1 (A), Z531.2
- new net: SW501.3 (C), Z537.2
- new net: R503.1, Z515.2
- new net: R402.1, R403.2, SW401.1 (A), U401.1
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Other:
- note added: "Mitschrifft: T Stücke sollten mit kleinerem Gehäuse gebaut werden dammit lötzinn reicht zum überbrücken. Rückgekoppelte opvs mit kapazität bandbreite begrenzen schwingung vermeiden. achtung invertierender verstärker muss zweifach angewendet werden damit phasen passen! Pegelanzeige braucht einstell Poti (Schraubendreher Poti) Die kapazitäten gegen masse vor den dc/dc wandlern können auch frei geha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"
- note removed: "BP4 Sub 30Hz/-3dB 150Hz/-6dB"
- title: Vorverstärker 1 -> Vorverstärker
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
Commit message: update
Parts:
- removed C209, C210, C713, C718: 10n, symbol Device:C_Small
- removed C211, C212: 220n, symbol Device:C_Small
- removed C213, C214: 150n, symbol Device:C_Small
- removed C215: 1u, symbol Device:C_Small
- removed C216, C715: 100n, symbol Device:C_Small
- removed C601: 4u7, symbol Device:C_Small
- removed C712, C719: 470p, symbol Device:C_Small
- removed C714, C717: 1n, symbol Device:C_Small
- removed C716: 10u, symbol Device:C_Polarized_Small
- removed D601, D602, D604: D, symbol Device:D
- removed D603: LED, symbol Device:LED
- removed J107, J108, J109, J110, J111, J112: Conn_02x07_Odd_Even, symbol Connector_Generic:Conn_02x07_Odd_Even
- removed J204: Bass_IN, symbol Connector:Conn_01x02_Socket
- removed J205: Bass_Out, symbol Connector:Conn_01x02_Socket
- removed J501, J502, J601, J602, J603, J604: L_Phono_In, symbol Connector:Conn_01x02_Pin
- removed J605: VU_Meter_Out, symbol Connector:Conn_01x04_Socket
- removed J606: LED_In, symbol Connector:Conn_01x02_Pin
- removed J607: LED_Out, symbol Connector:Conn_01x02_Socket
- removed L704, L705: Dämpfungsperle, 220 Ohm @ 100MHz, 0.5A, symbol Device:L_Ferrite
- removed R214, R218, Z253, Z272: 100k, symbol Device:R
- removed R215, R216, R217, R609, R610: 1k, symbol Device:R
- removed R219: 560k, symbol Device:R
- removed R220: 680k, symbol Device:R
- removed R221, R501, R502, R601, R602, R603, R604, R607, R612: 10k, symbol Device:R
- removed R222: 75k, symbol Device:R
- removed R223, R224, R611, R614: 15k, symbol Device:R
- removed R225, R226: 7k5, symbol Device:R
- removed R605, R606: 33k, symbol Device:R
- removed R608: 16k5, symbol Device:R
- removed R613: 2k2, symbol Device:R
- removed R615: 500R, symbol Device:R
- removed SW202: SW_SPDT, symbol sw_spdt_2:SW_SPDT
- removed unit 5 of U103
- removed unit 5 of U104
- removed unit 5 of U105
- removed unit 5 of U106
- removed U107, U108, U109, U110, U111, U112, U113, U114, U203, U204, U205, U206, U303, U403, U601, U602, U603, U604: TL074, symbol OPV_De:TL074
- removed unit 2 of U501
- removed unit 2 of U502
- removed U702: REC10K-2409, REC10K-2409SAW_H2:CONV_REC10K-2409SAW_H2, symbol REC10K-2409SAW_H2:REC10K-2409SAW_H2
- removed Z249, Z269: 1u, symbol Device:R
- removed Z250, Z251, Z255, Z256, Z258, Z259, Z261, Z262, Z264, Z265, Z267, Z268, Z626, Z627, Z628, Z629, Z632, Z703: 0R, symbol Device:R
- removed Z252, Z254, Z257, Z260, Z266, Z271, Z502, Z503, Z504, Z506, Z508, Z509, Z510, Z512, Z527, Z528, Z602, Z603, Z604, Z606, Z608, Z609, Z610, Z612, Z614, Z615, Z616, Z618, Z620, Z621, Z622, Z624, Z625, Z630, Z631: (no value), symbol Device:R
- removed Z263, Z270, Z505, Z511, Z605, Z611, Z617, Z623: 820k, symbol Device:R
- removed Z501, Z507, Z601, Z607, Z613, Z619: 4u7, symbol Device:R
- added C201, C202: 10n, symbol Device:C_Small
- added C203, C204: 220n, symbol Device:C_Small
- added C205, C206: 150n, symbol Device:C_Small
- added C207: 1u, symbol Device:C_Small
- added C208: 100n, symbol Device:C_Small
- added C605: 1n, symbol Device:C_Small
- added J201: Bass_IN, symbol Connector:Conn_01x02_Socket
- added J202: Bass_Out, symbol Connector:Conn_01x02_Socket
- added J203, J303, J403, J507, J603: Conn_02x07_Odd_Even, symbol Connector_Generic:Conn_02x07_Odd_Even
- added J505: L_Phono_In, symbol Connector:Conn_01x02_Pin
- added J506: Phono/Line_Out, symbol Connector:Conn_01x02_Socket
- added R201, R205, Z205, Z224, Z523: 100k, symbol Device:R
- added R202, R203, R204: 1k, symbol Device:R
- added R206: 560k, symbol Device:R
- added R207: 680k, symbol Device:R
- added R208: 10k, symbol Device:R
- added R209: 75k, symbol Device:R
- added R210, R211: 15k, symbol Device:R
- added R212, R213: 7k5, symbol Device:R
- added SW201: SW_SPDT, symbol sw_spdt_2:SW_SPDT
- added unit 5 of U101
- added unit 5 of U102
- added U201, U202: TL074, symbol OPV_De:TL074
- added unit 2 of U301
- added unit 5 of U301
- added unit 2 of U302
- added unit 5 of U302
- added unit 5 of U401
- added unit 2 of U401
- added unit 2 of U402
- added unit 5 of U402
- added unit 5 of U501
- added unit 4 of U502
- added unit 1 of U502
- added unit 5 of U502
- added Z201, Z221: 1u, symbol Device:R
- added Z202, Z203, Z207, Z208, Z210, Z211, Z213, Z214, Z216, Z217, Z219, Z220: 0R, symbol Device:R
- added Z204, Z206, Z209, Z212, Z218, Z223, Z518, Z519, Z522, Z537, Z539, Z540, Z541, Z542: (no value), symbol Device:R
- added Z215, Z222, Z538: 820k, symbol Device:R
- added Z535: 4u7, symbol Device:R
- added Z536: 100R, symbol Device:R
- SW601: renamed from SW701; symbol Switch:SW_DPST -> sw_dpst_2:SW_DPST
- renumbered C109 to C101, C110 to C102, C111 to C103, C112 to C104, C113 to C105, C114 to C106, C115 to C107, C116 to C108, C701 to C601, C702 to C602, C703 to C603, C706 to C604, C704 to C606, C705 to C607, C707 to C608, C708 to C609, C709 to C610, C710 to C611, C711 to C612, J104 to J101, J105 to J102, J106 to J103, J503 to J501, J504 to J502, J505 to J503, J506 to J504, J701 to J601, J702 to J602, L701 to L601, L702 to L602, L703 to L603, R114 to R101, R115 to R102, R116 to R103, R117 to R104, R118 to R105, R119 to R106, R120 to R107, R121 to R108, R122 to R109, R123 to R110, R124 to R111, R125 to R112, R126 to R113, R503 to R501, R504 to R502, R505 to R503, R506 to R504, R507 to R505, R508 to R506, SW102 to SW101, U104 to U101, U103 to U101, U105 to U101, U104 to U102, U106 to U102, U105 to U102, U504 to U501, U502 to U501, U503 to U501, U501 to U502, U701 to U601, Z225 to Z101, Z226 to Z102, Z227 to Z103, Z228 to Z104, Z229 to Z105, Z230 to Z106, Z231 to Z107, Z232 to Z108, Z233 to Z109, Z234 to Z110, Z235 to Z111, Z236 to Z112, Z237 to Z113, Z238 to Z114, Z239 to Z115, Z240 to Z116, Z241 to Z117, Z242 to Z118, Z243 to Z119, Z244 to Z120, Z245 to Z121, Z246 to Z122, Z247 to Z123, Z248 to Z124, Z513 to Z501, Z514 to Z502, Z515 to Z503, Z516 to Z504, Z517 to Z505, Z518 to Z506, Z519 to Z507, Z520 to Z508, Z521 to Z509, Z522 to Z510, Z523 to Z511, Z524 to Z512, Z525 to Z513, Z529 to Z514, Z530 to Z515, Z531 to Z516, Z532 to Z517, Z533 to Z520, Z534 to Z521, Z535 to Z524, Z536 to Z525, Z537 to Z527, Z538 to Z528, Z539 to Z529, Z540 to Z530, Z541 to Z531, Z542 to Z532, Z543 to Z533, Z544 to Z534, Z701 to Z601, Z702 to Z602
Connections:
- net +15V_P is gone; now on net +15V: C607.1, Z601.2
- net +9V1 is gone; now on net GND: J103.5 (Pin_5), J103.6 (Pin_6)
- net -15V1 is gone; now on net GND: J103.7 (Pin_7), J103.8 (Pin_8)
- net 9VGND1 is gone; now on net -15V: J103.1 (Pin_1), J103.2 (Pin_2), J103.3 (Pin_3), J103.4 (Pin_4)
- net GND_I is gone; now on net GND: J501.2 (Pin_2), J502.2 (Pin_2), J503.2 (Pin_2), J504.2 (Pin_2), R506.1, Z504.2, Z505.2, Z506.2, Z510.2, Z511.2, Z512.2, Z515.2, Z521.2, Z524.2, Z525.2, Z530.2, Z532.2, Z533.2, Z534.2
- net GND_P is gone; now on net GND: C606.2, C607.2, C608.1, C609.1, U601.5 (COM)
- net at C402.2, R407.2: now also U401.12 (+); no longer U402.3 (+)
- net at R106.2, Z111.1: now also U101.13 (-), U101.14; no longer U101.1, U101.2 (-)
- net at C107.2, Z119.1: now also U102.8, U102.9 (-); no longer U102.13 (-), U102.14
- net at R302.1, R303.2, SW301.1 (A): now also U301.7; no longer U301.1
- net at R301.1, R302.2: now also U301.9 (-); no longer U301.13 (-)
- net at R501.2, R502.2, R503.1: now also U501.9 (-); no longer U501.13 (-)
- net at R503.2, Z513.2: now also U501.8; no longer U501.14
- net at Z121.1, Z123.1: now also U102.13 (-), U102.14; no longer U102.8, U102.9 (-)
- net at C603.2, C606.1, L602.2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: now also C605.1
- net at R103.1, R104.1, SW101.2 (B): now also U101.6 (-); no longer U101.2 (-)
- net at R102.1, R103.2, SW101.1 (A): now also U101.7; no longer U101.1
- net at Z526.1: now also U502.2 (-), Z522.2; no longer SW501.2 (B)
- net GND: now reaches Z526.2
- net GND: now also C106.1, C108.1, C306.1, C308.1, C406.1, C408.1, J101.2 (Pin_2), J102.2 (Pin_2), J103.10 (Pin_10), J103.9 (Pin_9), J301.2 (Pin_2), J302.2 (Pin_2), J401.2 (Pin_2), J402.2 (Pin_2), R105.1, R107.1, R109.1, R305.1, R307.1, R309.1, R405.1, R407.1, R409.1, Z104.2, Z105.2, Z106.2, Z109.2, Z112.2, Z115.2, Z118.2, Z122.2, Z123.2, Z124.2, Z304.2, Z305.2, Z306.2, Z309.2, Z312.2, Z315.2, Z318.2, Z322.2, Z323.2, Z324.2, Z404.2, Z405.2, Z406.2, Z409.2, Z412.2, Z415.2, Z418.2, Z422.2, Z423.2, Z424.2, C206.1, C208.1, J201.2 (Pin_2), J202.2 (Pin_2), J203.10 (Pin_10), J203.5 (Pin_5), J203.6 (Pin_6), J203.7 (Pin_7), J203.8 (Pin_8), J203.9 (Pin_9), J303.10 (Pin_10), J303.5 (Pin_5), J303.6 (Pin_6), J303.7 (Pin_7), J303.8 (Pin_8), J303.9 (Pin_9), J403.10 (Pin_10), J403.5 (Pin_5), J403.6 (Pin_6), J403.7 (Pin_7), J403.8 (Pin_8), J403.9 (Pin_9), J505.2 (Pin_2), J506.2 (Pin_2), J507.10 (Pin_10), J507.5 (Pin_5), J507.6 (Pin_6), J507.7 (Pin_7), J507.8 (Pin_8), J507.9 (Pin_9), J603.10 (Pin_10), J603.5 (Pin_5), J603.6 (Pin_6), J603.7 (Pin_7), J603.8 (Pin_8), J603.9 (Pin_9), R205.1, R207.1, R209.1, Z204.2, Z205.2, Z206.2, Z209.2, Z212.2, Z215.2, Z218.2, Z222.2, Z223.2, Z224.2, Z523.2, Z537.2, Z538.2, Z540.2, Z541.2, Z542.2
- net at Z301.1, Z305.1: now also U301.3 (+); no longer U301.10 (+)
- net at C308.2, R312.2: now also U302.10 (+)
- net at C603.1, C604.1, U601.1 (+VIN): now also C601.2, L601.3; no longer C601.1, L601.2
- net at C302.2, R307.2: now also U301.12 (+); no longer U302.3 (+)
- net at R104.2, R105.2: now also U101.10 (+); no longer U101.12 (+)
- net at R101.1, R102.2: now also U101.9 (-); no longer U101.13 (-)
- net at R101.2, Z107.2: now also U101.8; no longer U101.14
- net at C103.2, R109.2: now also U102.3 (+); no longer U102.12 (+)
- net at C610.1, C612.1, U601.2 (-VIN): now also C601.1, L601.2; no longer C601.2, L601.3
- net at Z515.1: now also U501.10 (+); no longer U501.12 (+)
- net at Z120.2: now also U102.12 (+); no longer U102.10 (+)
- net at C403.2, R409.2: now also U402.3 (+); no longer U402.12 (+)
- net at C408.2, R412.2: now also U402.10 (+)
- net at C407.2, Z419.1: now also U402.8, U402.9 (-)
- net at R303.1, R304.1, SW301.2 (B): now also U301.6 (-); no longer U301.2 (-)
- net at Z303.1: now also U301.5 (+); no longer U301.3 (+)
- net at SW501.1 (A): now also Z527.2; no longer Z516.2
- net at SW501.3 (C): now also Z516.2; no longer Z527.2
- net at R402.1, R403.2, SW401.1 (A): now also U401.7; no longer U401.1
- net at R403.1, R404.1, SW401.2 (B): now also U401.6 (-); no longer U401.2 (-)
- net at C502.1, C503.2, R505.2: now also U502.6 (-); no longer U502.9 (-)
- net at C307.2, Z319.1: now also U302.8, U302.9 (-)
- net at C305.2, Z317.1: now also U302.6 (-), U302.7
- net at C102.2, R107.2: now also U101.12 (+); no longer U101.3 (+)
- net at C108.2, R112.2: now also U102.10 (+); no longer U102.12 (+)
- net at C405.2, Z417.1: now also U402.6 (-), U402.7
- net at C406.2, R411.2: now also U402.5 (+)
- net at C501.2, R504.1, Z520.1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: now also U502.7; no longer U502.8
- net at R301.2, Z307.2: now also U301.8; no longer U301.14
- net at R304.2, R305.2: now also U301.10 (+); no longer U301.12 (+)
- net at C105.2, Z117.1: now also U102.6 (-), U102.7; no longer U102.1, U102.2 (-)
- net at R306.2, Z311.1: now also U301.13 (-), U301.14; no longer U302.1, U302.2 (-)
- net at Z320.2: now also U302.12 (+); no longer U302.10 (+)
- net at Z501.2, Z505.1: now also U501.3 (+); no longer U501.5 (+)
- net at R406.2, Z411.1: now also U401.13 (-), U401.14; no longer U402.1, U402.2 (-)
- net at Z401.1, Z405.1: now also U401.3 (+); no longer U401.10 (+)
- net at Z403.1: now also U401.5 (+); no longer U401.3 (+)
- net at Z321.1, Z323.1: now also U302.13 (-), U302.14; no longer U302.8, U302.9 (-)
- net at Z421.1, Z423.1: now also U402.13 (-), U402.14; no longer U402.8, U402.9 (-)
- net at C303.2, R309.2: now also U302.3 (+); no longer U302.12 (+)
- net at C306.2, R311.2: now also U302.5 (+)
- net at C106.2, R111.2: now also U102.5 (+); no longer U102.3 (+)
- net at R404.2, R405.2: now also U401.10 (+); no longer U401.12 (+)
- net at R308.2, Z313.2: now also U302.1, U302.2 (-); no longer U302.13 (-), U302.14
- net at Z420.2: now also U402.12 (+); no longer U402.10 (+)
- net at R408.2, Z413.2: now also U402.1, U402.2 (-); no longer U402.13 (-), U402.14
- net at Z101.1, Z105.1: now also U101.3 (+); no longer U101.10 (+)
- net at R401.1, R402.2: now also U401.9 (-); no longer U401.13 (-)
- net at R401.2, Z407.2: now also U401.8; no longer U401.14
- net at Z517.1: now also U502.3 (+); no longer U502.10 (+)
- net at R108.2, Z113.2: now also U102.1, U102.2 (-); no longer U102.13 (-), U102.14
- net at Z103.1: now also U101.5 (+); no longer U101.3 (+)
- net at U501.14, Z514.1: now also SW501.2 (B)
- net +15V1 renamed +15V
- net +15V: now also J103.11 (Pin_11), J103.12 (Pin_12), J203.11 (Pin_11), J203.12 (Pin_12), J203.13 (Pin_13), J203.14 (Pin_14), J303.11 (Pin_11), J303.12 (Pin_12), J303.13 (Pin_13), J303.14 (Pin_14), J403.11 (Pin_11), J403.12 (Pin_12), J403.13 (Pin_13), J403.14 (Pin_14), J507.11 (Pin_11), J507.12 (Pin_12), J507.13 (Pin_13), J507.14 (Pin_14), J603.11 (Pin_11), J603.12 (Pin_12), J603.13 (Pin_13), J603.14 (Pin_14), U101.4 (V+), U102.4 (V+), U201.4 (V+), U202.4 (V+), U301.4 (V+), U302.4 (V+), U401.4 (V+), U402.4 (V+), U501.4 (V+), U502.4 (V+)
- net -15V_P renamed -15V
- net -15V: now also J203.1 (Pin_1), J203.2 (Pin_2), J203.3 (Pin_3), J203.4 (Pin_4), J303.1 (Pin_1), J303.2 (Pin_2), J303.3 (Pin_3), J303.4 (Pin_4), J403.1 (Pin_1), J403.2 (Pin_2), J403.3 (Pin_3), J403.4 (Pin_4), J507.1 (Pin_1), J507.2 (Pin_2), J507.3 (Pin_3), J507.4 (Pin_4), J603.1 (Pin_1), J603.2 (Pin_2), J603.3 (Pin_3), J603.4 (Pin_4), U101.11 (V-), U102.11 (V-), U201.11 (V-), U202.11 (V-), U301.11 (V-), U302.11 (V-), U401.11 (V-), U402.11 (V-), U501.11 (V-), U502.11 (V-)
- removed net GND1: C106.1, C108.1, C306.1, C308.1, C406.1, C408.1, J101.2 (Pin_2), J102.2 (Pin_2), J103.10 (Pin_10), J103.11 (Pin_11), J103.12 (Pin_12), J103.9 (Pin_9), J301.2 (Pin_2), J302.2 (Pin_2), J401.2 (Pin_2), J402.2 (Pin_2), R105.1, R107.1, R109.1, R305.1, R307.1, R309.1, R405.1, R407.1, R409.1, Z104.2, Z105.2, Z106.2, Z109.2, Z112.2, Z115.2, Z118.2, Z122.2, Z123.2, Z124.2, Z304.2, Z305.2, Z306.2, Z309.2, Z312.2, Z315.2, Z318.2, Z322.2, Z323.2, Z324.2, Z404.2, Z405.2, Z406.2, Z409.2, Z412.2, Z415.2, Z418.2, Z422.2, Z423.2, Z424.2
- net GND_15V_FILT renamed GND_FILT
- net GND_FILT: now also C605.2
- new net: Z210.1, Z211.2, Z212.1
- new net: C204.1, Z210.2
- new net: U201.5 (+), Z203.1
- new net: R203.1, R204.1, SW201.2 (B), U201.6 (-)
- new net: R202.1, R203.2, SW201.1 (A), U201.7
- new net: U301.1, U301.2 (-), Z302.2
- new net: U201.3 (+), Z201.1, Z205.1
- new net: U502.14, Z536.1, Z539.1, Z540.1
- new net: J506.1 (Pin_1), Z536.2, Z541.1
- new net: C205.2, U202.6 (-), U202.7, Z217.1
- new net: Z216.1, Z217.2, Z218.1
- new net: Z219.2, Z220.1, Z222.1
- new net: U202.12 (+), Z220.2
- new net: U202.13 (-), U202.14, Z221.1, Z223.1
- new net: U502.12 (+), Z535.2, Z538.1
- new net: Z202.1, Z203.2, Z206.1
- new net: U201.1, U201.2 (-), Z202.2
- new net: R213.1, Z216.2
- new net: Z518.1, Z519.2, Z523.1
- new net: U502.1, Z518.2, Z522.1
- new net: C203.1, C204.2, R208.1
- new net: Z207.1, Z208.2, Z209.1
- new net: U501.1, U501.2 (-), Z502.1
- new net: U502.13 (-), Z539.2, Z542.1
- new net: C201.2, C202.1, R206.1
- new net: R206.2, U201.13 (-), U201.14, Z211.1
- new net: Z213.1, Z214.2, Z215.1
- new net: R208.2, U202.1, U202.2 (-), Z213.2
- new net: R204.2, R205.2, U201.10 (+)
- new net: R201.2, U201.8, Z207.2
- new net: R201.1, R202.2, U201.9 (-)
- new net: J505.1 (Pin_1), Z535.1, Z537.1
- new net: C203.2, R209.2, U202.3 (+)
- new net: C202.2, R207.2, U201.12 (+)
- new net: C206.2, R211.2, U202.5 (+)
- new net: C208.2, R212.2, U202.10 (+)
- new net: J202.1 (Pin_1), Z221.2, Z224.1
- new net: U101.1, U101.2 (-), Z102.2
- new net: R210.1, Z214.1
- new net: C205.1, R210.2, R211.1
- new net: J201.1 (Pin_1), Z201.2, Z204.1
- new net: U502.5 (+), Z519.1
- new net: C207.1, R212.1, R213.2
- new net: U401.1, U401.2 (-), Z402.2
- new net: C201.1, Z208.1
- new net: C207.2, U202.8, U202.9 (-), Z219.1
- no-connect marks 3 -> 1
Other:
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
Commit message: update
Parts:
- removed Z104: (no value), symbol Device:R
- added C109, C110, C111, C112: 100n, symbol Device:C_Small
- added D601, D602: BZV55B12, Diode_SMD:D_MiniMELF, symbol Diode:BZV55B12
- added Z125: 100k, symbol Device:R
Connections:
- net GND: now also D601.2 (A)
- net at Z101.1, Z105.1: now also Z125.1; no longer U101.3 (+)
- new net: D602.2 (A), U101.3 (+), Z125.2
- new net: D601.1 (K), D602.1 (K)
Other:
- moved on the sheet: J101, Z101, Z105

Commit message: Update
Parts:
- removed C501: 10n, symbol Device:C_Small
- removed C502: 2n2, symbol Device:C_Small
- removed C503: 47u, symbol Device:C_Small
- removed D601, D602: BZV55B12, Diode_SMD:D_MiniMELF, symbol Diode:BZV55B12
- removed J101, J201, J301, J401: Bass_IN, symbol Connector:Conn_01x02_Socket
- removed J501, J502, J505: L_Phono_In, symbol Connector:Conn_01x02_Pin
- removed J503, J504: Phono/Line_Out, symbol Connector:Conn_01x02_Socket
- removed R501, R502, R503: 10k, symbol Device:R
- removed R504: 390k, symbol Device:R
- removed R505: 33k, symbol Device:R
- removed R506: 1k, symbol Device:R
- removed SW501: SW_SPDT, symbol Switch:SW_SPDT
- removed unit 2 of U501
- removed unit 3 of U501
- removed unit 1 of U501
- removed unit 4 of U501
- removed unit 4 of U502
- removed unit 1 of U502
- removed unit 2 of U502
- removed unit 3 of U502
- removed Z101: 1u, symbol Device:R
- removed Z105, Z125, Z523, Z530: 100k, symbol Device:R
- removed Z501: 4u7, symbol Device:R
- removed Z502, Z503, Z514, Z515, Z516, Z517, Z518, Z519, Z524, Z525, Z528, Z531, Z532, Z533, Z534, Z539, Z540, Z541, Z542: (no value), symbol Device:R
- removed Z520, Z529, Z536: 100R, symbol Device:R
- added C504, C507, C508, C510: 10n, symbol Device:C_Small
- added C505, C511: 2n2, symbol Device:C_Small
- added C506, C509: 47u, symbol Device:C_Small
- added D609, D610, D611, D612, D613, D614, D615, D616, D617, D618, D619, D620, D621, D622, D623, D624, D625, D626, D627, D628, D629, D630, D631, D632: BZV55B12, Diode_SMD:D_MiniMELF, symbol Diode:BZV55B12
- added J107, J108, J109, J110, J111, J112, J113, J114, J115, J116, J117, J118: Bass_IN, symbol Connector:Conn_01x02_Socket
- added J404: Bass_Out, symbol Connector:Conn_01x02_Socket
- added J505: Phono/Line_Out, symbol Connector:Conn_01x02_Socket
- added R507, R508, R509, R510, R511, R512, R513, R514, R515, R516, R517, R518, R519, R520: 10k, symbol Device:R
- added R521, R525, R526, R527: 390k, symbol Device:R
- added R522, R524, R528, R529: 33k, symbol Device:R
- added R523, R530: 1k, symbol Device:R
- added SW503, SW504: SW_SPDT, symbol Switch:SW_SPDT
- added U503, U504, U505, U506, U507, U508, U509, U510: TL074, symbol OPV_De:TL074
- added Z134, Z135, Z140, Z141, Z146, Z147, Z152, Z153, Z154, Z155, Z156, Z157, Z226, Z426: 1u, symbol Device:R
- added Z136, Z137, Z138, Z139, Z142, Z143, Z144, Z145, Z148, Z149, Z150, Z151, Z158, Z159, Z160, Z161, Z162, Z163, Z164, Z165, Z166, Z167, Z168, Z169, Z227, Z427: 100k, symbol Device:R
- added Z225, Z228, Z229, Z230, Z231, Z425, Z543, Z544, Z545, Z546, Z547, Z548, Z549, Z550, Z551, Z552, Z553, Z554, Z555, Z556, Z557, Z558, Z559, Z560, Z561, Z563, Z564, Z565, Z566, Z567, Z568, Z569, Z570, Z571, Z572, Z573, Z581, Z582: (no value), symbol Device:R
- Z505, Z511, Z538: value 820k -> (none)
- Z507, Z535: value 4u7 -> (none)
- Z521: value 100k -> 100R
- Z522: value (none) -> 100R
Connections:
- net GND: now also Z507.2, Z508.2, Z527.2, C507.1, C508.1, D610.2 (A), D612.2 (A), D614.2 (A), D616.2 (A), D618.2 (A), D620.2 (A), D622.2 (A), D624.2 (A), D626.2 (A), D628.2 (A), D630.2 (A), D632.2 (A), J107.2 (Pin_2), J108.2 (Pin_2), J109.2 (Pin_2), J110.2 (Pin_2), J111.2 (Pin_2), J112.2 (Pin_2), J113.2 (Pin_2), J114.2 (Pin_2), J115.2 (Pin_2), J116.2 (Pin_2), J117.2 (Pin_2), J118.2 (Pin_2), J404.2 (Pin_2), J505.2 (Pin_2), R523.1, R525.2, R526.2, R530.1, Z136.2, Z137.2, Z142.2, Z143.2, Z148.2, Z149.2, Z158.2, Z159.2, Z160.2, Z161.2, Z162.2, Z163.2, Z225.2, Z227.2, Z425.2, Z427.2, Z545.2, Z548.2, Z549.2, Z554.2, Z555.2, Z563.2, Z564.2, Z565.2, Z566.2, Z567.2, Z573.2, Z581.2, Z582.2; no longer Z504.2, Z505.2, Z506.2, Z510.2, Z511.2, Z512.2, Z521.2, Z538.2
- net at Z513.2: now also R519.1
- net at Z526.1: now also Z521.1, C504.2, R521.1, U509.7; no longer Z522.2
- net at J506.1 (Pin_1): now also Z522.2, Z582.1
- net at Z535.2: now also U503.12 (+), Z544.2; no longer Z538.1
- net at Z522.1: now also Z527.1, C510.2, R527.1, U510.7
- net at Z506.1: now also U508.1, U508.2 (-)
- net at Z537.1: now also Z510.2, Z511.1; no longer Z535.1
- net at Z301.2, Z304.1: now also Z230.2
- net at Z507.1: now also Z504.2, Z505.1; no longer Z510.1
- net at Z509.2: now also R518.1
- net at Z508.1: now also Z506.2, Z509.1
- net at U101.3 (+): now also Z226.1, Z227.1
- net at Z201.2, Z204.1: now also Z229.2
- net at Z401.2, Z404.1: now also Z231.2
- net at Z504.1: now also U503.1, U503.2 (-)
- net at Z513.1: now also Z512.2, Z567.1
- new net: SW503.1 (A), Z425.1, Z426.1
- new net: D629.1 (K), D630.1 (K)
- new net: D629.2 (A), U508.3 (+), Z168.2
- new net: D617.1 (K), D618.1 (K)
- new net: U508.10 (+), Z573.1
- new net: R520.2, U508.8, Z572.2
- new net: R514.2, R515.2, R516.2, R517.2, R518.2, R519.2, R520.1, U508.9 (-)
- new net: C507.2, R525.1, U509.5 (+)
- new net: Z228.1, Z229.1, Z230.1, Z231.1
- new net: C505.1, R522.2, R524.1
- new net: C504.1, C505.2, R521.2, R522.1
- new net: C506.1, R523.2
- new net: C506.2, R524.2, U509.6 (-)
- new net: D625.1 (K), D626.1 (K)
- new net: Z559.2, Z564.1, Z569.1
- new net: Z135.1, Z137.1, Z139.1
- new net: U508.13 (-), Z572.1
- new net: Z552.2, Z554.1, Z556.1
- new net: R512.1, Z556.2
- new net: Z154.1, Z160.1, Z166.1
- new net: D625.2 (A), U507.3 (+), Z166.2
- new net: R509.1, Z511.2
- new net: R507.1, R508.2, R509.2, R510.2, R511.2, R512.2, R513.2, U503.9 (-)
- new net: D619.2 (A), U505.5 (+), Z151.2
- new net: U505.6 (-), U505.7, Z553.1
- new net: R510.1, Z550.2
- new net: Z155.1, Z161.1, Z167.1
- new net: D627.2 (A), U507.5 (+), Z167.2
- new net: R514.1, Z568.2
- new net: J118.1 (Pin_1), Z157.2
- new net: Z140.1, Z142.1, Z144.1
- new net: Z225.1, Z226.2, Z228.2
- new net: D611.2 (A), U503.5 (+), Z139.2
- new net: R513.1, Z557.2
- new net: J112.1 (Pin_1), Z147.2
- new net: SW504.1 (A), Z535.1
- new net: SW503.2 (B), SW504.2 (B), U503.14
- new net: SW504.3 (C), Z544.1
- new net: Z157.1, Z163.1, Z169.1
- new net: U508.12 (+), Z543.2
- new net: U508.14, Z543.1
- new net: Z134.1, Z136.1, Z138.1
- new net: D609.2 (A), U503.3 (+), Z138.2
- new net: J108.1 (Pin_1), Z135.2
- new net: Z553.2, Z555.1, Z557.1
- new net: D631.1 (K), D632.1 (K)
- new net: Z156.1, Z162.1, Z168.1
- new net: R515.1, Z569.2
- new net: U505.1, U505.2 (-), Z552.1
- new net: J505.1 (Pin_1), Z521.2, Z581.1
- new net: D617.2 (A), U505.3 (+), Z150.2
- new net: Z547.2, Z549.1, Z551.1
- new net: Z146.1, Z148.1, Z150.1
- new net: Z152.1, Z158.1, Z164.1
- new net: J113.1 (Pin_1), Z152.2
- new net: D615.1 (K), D616.1 (K)
- new net: D615.2 (A), U504.5 (+), Z145.2
- new net: Z147.1, Z149.1, Z151.1
- new net: U507.6 (-), U507.7, Z561.1
- new net: R508.1, Z505.2
- new net: D631.2 (A), U508.5 (+), Z169.2
- new net: U508.6 (-), U508.7, Z512.1
- new net: D613.2 (A), U504.3 (+), Z144.2
- new net: U506.6 (-), U506.7, Z559.1
- new net: D613.1 (K), D614.1 (K)
- new net: U504.1, U504.2 (-), Z546.1
- new net: Z546.2, Z548.1, Z550.1
- new net: J107.1 (Pin_1), Z134.2
- new net: D611.1 (K), D612.1 (K)
- new net: J109.1 (Pin_1), Z140.2
- new net: C510.1, C511.2, R527.2, R528.1
- new net: C511.1, R528.2, R529.1
- new net: Z558.2, Z563.1, Z568.1
- new net: U503.13 (-), Z538.1
- new net: U506.1, U506.2 (-), Z558.1
- new net: J404.1 (Pin_1), Z426.2, Z427.1
- new net: C509.2, R529.2, U510.6 (-)
- new net: D621.1 (K), D622.1 (K)
- new net: D621.2 (A), U506.3 (+), Z164.2
- new net: U507.1, U507.2 (-), Z560.1
- new net: Z560.2, Z565.1, Z570.1
- new net: U503.10 (+), Z545.1
- new net: R507.2, U503.8, Z538.2
- new net: D619.1 (K), D620.1 (K)
- new net: C508.2, R526.1, U510.5 (+)
- new net: J111.1 (Pin_1), Z146.2
- new net: U504.6 (-), U504.7, Z547.1
- new net: J117.1 (Pin_1), Z156.2
- new net: D623.1 (K), D624.1 (K)
- new net: U503.6 (-), U503.7, Z510.1
- new net: D627.1 (K), D628.1 (K)
- new net: J116.1 (Pin_1), Z155.2
- new net: J115.1 (Pin_1), Z154.2
- new net: D623.2 (A), U506.5 (+), Z165.2
- new net: Z141.1, Z143.1, Z145.1
- new net: Z153.1, Z159.1, Z165.1
- new net: R517.1, Z571.2
- new net: J114.1 (Pin_1), Z153.2
- new net: D609.1 (K), D610.1 (K)
- new net: J110.1 (Pin_1), Z141.2
- new net: R516.1, Z570.2
- new net: Z561.2, Z566.1, Z571.1
- new net: C509.1, R530.2
- new net: R511.1, Z551.2
- no-connect marks 1 -> 2
Other:
- moved on the sheet: C101, C102, C103, C104, C105, C106, C107, C108, C109, C110, C111, C112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
