File: KiCad/Pre_Amp.kicad_sch (KiCad schematic)
At the start: 365 parts, among them J102 Bass_Out, J103 Conn_02x07_Odd_Even, J104 Bass_IN, J105 Bass_IN, J106 Bass_IN, J107 Bass_IN, J108 Bass_IN, J109 Bass_IN, J110 Bass_IN, J111 Bass_IN, J112 Bass_IN, J202 Bass_Out, J203 Conn_02x07_Odd_Even, J302 Bass_Out, J303 Conn_02x07_Odd_Even, J402 Bass_Out, J403 Conn_02x07_Odd_Even, J404 Bass_Out, J503 Phono/Line_Out, J504 Phono/Line_Out, J507 Conn_02x07_Odd_Even, J601 VCC_IN, J602 VCC_OUT, J603 Conn_02x07_Odd_Even, SW101 SW_SPDT, SW201 SW_SPDT, SW301 SW_SPDT, SW401 SW_SPDT, SW501 SW_SPDT, SW502 SW_SPDT, SW601 SW_DPST, U101 TL074, U102 TL074, U201 TL074, U202 TL074, U301 TL074, U302 TL074, U401 TL074, U402 TL074, U501 TL074, U502 TL074, U503 TL074, U504 TL074, U505 TL074, U601 REC10K-2415

Commit message: Update
Parts:
- removed D603, D604, D605, D606, D607, D608, D609, D610, D611, D612, D613, D614, D615, D616, D617, D618, D619, D620: BZV55B12, Diode_SMD:D_MiniMELF, symbol Diode:BZV55B12
- removed J103, J203, J303, J403, J507: Conn_02x07_Odd_Even, symbol Connector_Generic:Conn_02x07_Odd_Even
- removed J105, J106, J107, J108, J109, J110, J111, J112: Bass_IN, symbol Connector:Conn_01x02_Socket
- removed J404: Bass_Out, symbol Connector:Conn_01x02_Socket
- removed J503, J504: Phono/Line_Out, symbol Connector:Conn_01x02_Socket
- removed R501, R502, R503, R507, R508, R509, R510, R511, R512, R513: 10k, symbol Device:R
- removed R504: 390k, symbol Device:R
- removed R505: 33k, symbol Device:R
- removed R506: 1k, symbol Device:R
- removed SW501, SW502: SW_SPDT, symbol Switch:SW_SPDT
- removed unit 2 of U501
- removed unit 3 of U501
- removed unit 1 of U501
- removed unit 4 of U501
- removed unit 4 of U502
- removed unit 1 of U502
- removed unit 2 of U502
- removed unit 3 of U502
- removed U503, U504, U505: TL074, symbol OPV_De:TL074
- removed Z143, Z144, Z145, Z148, Z149, Z150, Z151, Z427, Z521, Z523, Z530: 100k, symbol Device:R
- removed Z146, Z147, Z426: 1u, symbol Device:R
- removed Z425, Z502, Z503, Z504, Z505, Z506, Z507, Z508, Z509, Z510, Z511, Z512, Z513, Z514, Z515, Z516, Z517, Z518, Z519, Z522, Z524, Z525, Z526, Z527, Z528, Z531, Z532, Z533, Z534, Z535, Z537, Z538, Z539, Z540, Z541, Z542, Z543, Z545, Z546, Z547, Z548, Z549, Z550, Z551, Z552, Z553, Z554, Z555, Z556, Z557: (no value), symbol Device:R
- removed Z520, Z529, Z536: 100R, symbol Device:R
- added C101, C102, C104, C107: 10n, symbol Device:C_Small
- added C103: 2n2, symbol Device:C_Small
- added C105: 47u, symbol Device:C_Small
- added C108, C113, C201, C202, C203, C204, C301, C302, C303, C304, C401, C402, C403, C404, C504: 100n, symbol Device:C_Small
- added C210: 150n, symbol Device:C_Small
- added D101, D102, D103, D104, D105, D106, D107, D108: D, symbol Device:D
- added J101, J102, J103: Bass_IN, symbol Connector:Conn_01x02_Socket
- added R101, R102, R106, R110, R111: 10k, symbol Device:R
- added R103, R104, R107, R112, R114: 390k, symbol Device:R
- added R105, R108: 33k, symbol Device:R
- added R109: 1k, symbol Device:R
- added R213: 7k5, symbol Device:R
- added SW101: SW_SPDT, symbol Switch:SW_SPDT
- added unit 4 of U101
- added unit 3 of U101
- added unit 1 of U101
- added unit 2 of U101
- added unit 3 of U102
- added unit 4 of U102
- added unit 1 of U102
- added U103: TL074, symbol OPV_De:TL074
- added unit 2 of U202
- added Z101, Z102, Z103, Z105, Z106, Z111, Z114, Z115, Z119, Z120, Z122, Z123, Z124, Z125, Z218: (no value), symbol Device:R
- added Z107, Z108, Z109, Z110, Z216, Z217: 0R, symbol Device:R
- added Z112, Z113: 820k, symbol Device:R
- added Z221: 1u, symbol Device:R
- C106: value 150n -> 10n
- C501: value 10n -> 100n
- C502: value 2n2 -> 100n
- C503: value 47u -> 100n
- R113: value 7k5 -> 10k
- Z104, Z121, Z128, Z131: value 1u -> (none)
- Z116, Z117: value 0R -> (none)
- Z126, Z127, Z129, Z130, Z132, Z133, Z136, Z139, Z142: value 100k -> (none)
- Z134, Z135: value 1u -> 0R
- Z137, Z138: value 100k -> 0R
- Z140, Z141: value 1u -> 820k
- renumbered C101 to C205, C102 to C206, C103 to C207, C104 to C208, C105 to C209, C107 to C211, C108 to C212, C201 to C305, C202 to C306, C203 to C307, C204 to C308, C205 to C309, C206 to C310, C207 to C311, C208 to C312, C301 to C405, C302 to C406, C303 to C407, C304 to C408, C305 to C409, C306 to C410, C307 to C411, C308 to C412, C401 to C505, C402 to C506, C403 to C507, C404 to C508, C405 to C509, C406 to C510, C407 to C511, C408 to C512, J102 to J201, J202 to J301, J302 to J401, J402 to J501, R101 to R201, R102 to R202, R103 to R203, R104 to R204, R105 to R205, R106 to R206, R107 to R207, R108 to R208, R109 to R209, R110 to R210, R111 to R211, R112 to R212, R201 to R301, R202 to R302, R203 to R303, R204 to R304, R205 to R305, R206 to R306, R207 to R307, R208 to R308, R209 to R309, R210 to R310, R211 to R311, R212 to R312, R213 to R313, R301 to R401, R302 to R402, R303 to R403, R304 to R404, R305 to R405, R306 to R406, R307 to R407, R308 to R408, R309 to R409, R310 to R410, R311 to R411, R312 to R412, R313 to R413, R401 to R501, R402 to R502, R403 to R503, R404 to R504, R405 to R505, R406 to R506, R407 to R507, R408 to R508, R409 to R509, R410 to R510, R411 to R511, R412 to R512, R413 to R513, SW101 to SW201, SW201 to SW301, SW301 to SW401, SW401 to SW501, U101 to U201, U102 to U202, U201 to U301, U202 to U302, U301 to U401, U302 to U402, U401 to U501, U402 to U502, Z226 to Z201, Z102 to Z202, Z103 to Z203, Z225 to Z204, Z227 to Z205, Z106 to Z206, Z107 to Z207, Z108 to Z208, Z109 to Z209, Z110 to Z210, Z111 to Z211, Z112 to Z212, Z113 to Z213, Z114 to Z214, Z115 to Z215, Z119 to Z219, Z120 to Z220, Z122 to Z222, Z123 to Z223, Z124 to Z224, Z201 to Z301, Z202 to Z302, Z203 to Z303, Z204 to Z304, Z205 to Z305, Z206 to Z306, Z207 to Z307, Z208 to Z308, Z209 to Z309, Z210 to Z310, Z211 to Z311, Z212 to Z312, Z213 to Z313, Z214 to Z314, Z215 to Z315, Z216 to Z316, Z217 to Z317, Z218 to Z318, Z219 to Z319, Z220 to Z320, Z221 to Z321, Z222 to Z322, Z223 to Z323, Z224 to Z324, Z301 to Z401, Z302 to Z402, Z303 to Z403, Z304 to Z404, Z305 to Z405, Z306 to Z406, Z307 to Z407, Z308 to Z408, Z309 to Z409, Z310 to Z410, Z311 to Z411, Z312 to Z412, Z313 to Z413, Z314 to Z414, Z315 to Z415, Z316 to Z416, Z317 to Z417, Z318 to Z418, Z319 to Z419, Z320 to Z420, Z321 to Z421, Z322 to Z422, Z323 to Z423, Z324 to Z424, Z401 to Z501, Z402 to Z502, Z403 to Z503, Z404 to Z504, Z405 to Z505, Z406 to Z506, Z407 to Z507, Z408 to Z508, Z409 to Z509, Z410 to Z510, Z411 to Z511, Z412 to Z512, Z413 to Z513, Z414 to Z514, Z415 to Z515, Z416 to Z516, Z417 to Z517, Z418 to Z518, Z419 to Z519, Z420 to Z520, Z421 to Z521, Z422 to Z522, Z423 to Z523, Z424 to Z524
Connections:
- net +15V: now also C110.2, C112.2, C501.2, C503.2, C108.2, C201.2, C203.2, C301.2, C303.2, C401.2, C403.2, U103.4 (V+)
- net -15V: now also C109.2, C111.2, C502.2, C113.2, C202.2, C204.2, C302.2, C304.2, C402.2, C404.2, C504.2, U103.11 (V-)
- net GND: now also C109.1, C110.1, C111.1, C112.1, C501.1, C502.1, C503.1, Z121.2, Z127.2, Z139.2, Z140.2, Z141.2, C101.1, C104.1, C107.1, C108.1, C113.1, C201.1, C202.1, C203.1, C204.1, C210.1, C301.1, C302.1, C303.1, C304.1, C401.1, C402.1, C403.1, C404.1, C504.1, D101.1 (K), D102.2 (A), D103.1 (K), D104.2 (A), D105.1 (K), D106.2 (A), D107.1 (K), D108.2 (A), J101.2 (Pin_2), J102.2 (Pin_2), J103.2 (Pin_2), R103.2, R107.2, R109.1, R112.2, R114.2, Z111.2, Z112.2, Z113.2, Z120.2, Z218.2; no longer Z118.2, Z126.2, Z129.2, Z132.2, Z137.2, Z142.2
- net at U202.13 (-), U202.14, Z223.1: now also Z221.1; no longer Z121.1
- net at Z201.2, Z204.1, Z301.2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: now also SW101.2 (B)
- net at J201.1 (Pin_1), Z224.1: now also Z221.2; no longer Z121.2
- net at Z128.2: now also Z129.1, R114.1
- net at Z140.1: now also Z134.2, Z135.1; no longer Z142.1
- net at Z117.2, Z118.1: now also D103.2 (A); no longer Z116.1
- net at R113.1: now also Z132.2, Z136.1; no longer Z116.2
- net at C211.1, R212.1: now also R213.2; no longer R113.2
- net at Z133.2: now also R111.2, U103.1
- net at Z130.2: now also Z131.1, D107.2 (A)
- net at Z131.2: now also D108.1 (K), U102.12 (+)
- net at Z138.2: now also U103.12 (+)
- net at Z135.2: now also U103.10 (+)
- net at Z141.1: now also Z137.2, Z138.1
- net at Z104.2: now also D102.1 (K), U101.3 (+); no longer J104.1 (Pin_1)
- new net: C107.2, Z129.2, Z130.1
- new net: C101.2, Z102.2, Z103.1
- new net: R213.1, Z216.2
- new net: D104.1 (K), U102.3 (+), Z118.2
- new net: D106.1 (K), U102.10 (+), Z125.2
- new net: U102.5 (+), Z121.1
- new net: R101.2, R102.1, R106.2, U102.6 (-)
- new net: R102.2, U102.7, Z106.2
- new net: R110.2, R111.1, R113.2, U103.2 (-)
- new net: C103.1, R105.2, R108.1
- new net: C102.1, C103.2, R104.2, R105.1
- new net: C105.1, R109.2
- new net: C105.2, R108.2, U101.9 (-)
- new net: R106.1, Z119.2, Z120.1
- new net: U103.8, U103.9 (-), Z137.1
- new net: Z109.2, Z110.1, Z113.1
- new net: U101.12 (+), Z110.2
- new net: U101.6 (-), Z106.1
- new net: R110.1, Z126.2, Z127.1
- new net: D101.2 (A), Z103.2, Z104.1
- new net: SW101.3 (C), U101.13 (-), U101.14
- new net: R101.1, Z105.2, Z111.1
- new net: J102.1 (Pin_1), Z115.1
- new net: R107.1, Z115.2, Z116.1
- new net: U102.8, U102.9 (-), Z126.1
- new net: R112.1, Z122.2, Z123.1
- new net: C106.2, Z123.2, Z124.1
- new net: C102.2, R104.1, U101.8, Z109.1
- new net: U103.5 (+), Z142.2
- new net: U103.6 (-), Z133.1
- new net: U103.7, Z134.1, Z142.1
- new net: U103.3 (+), Z139.1
- new net: J101.1 (Pin_1), Z101.1
- new net: R103.1, Z101.2, Z102.1
- new net: U101.7, Z107.1, Z114.1
- new net: Z107.2, Z108.1, Z112.1
- new net: C209.2, U202.6 (-), U202.7, Z217.1
- new net: U101.10 (+), Z108.2
- new net: Z216.1, Z217.2, Z218.1
- new net: U102.1, U102.2 (-), Z119.1
- new net: U101.1, U101.2 (-), Z105.1
- new net: D105.2 (A), Z124.2, Z125.1
- new net: C104.2, Z116.2, Z117.1
- new net: C210.2, R211.2, U202.5 (+)
- new net: U102.13 (-), U102.14, Z132.1
- new net: J104.1 (Pin_1), Z128.1
- new net: SW101.1 (A), U103.13 (-), U103.14
- new net: U101.5 (+), Z114.2
- new net: J103.1 (Pin_1), Z122.1
Other:
- moved on the sheet: C205, C206, C207, C208, C209, C211, C212, C305, C306, C307, C308, C309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

Commit message: Update
Parts:
- removed C201, C202, C203, C204, C212, C301, C302, C303, C304, C312, C401, C402, C403, C404, C412, C501, C502, C503, C504, C512: 100n, symbol Device:C_Small
- removed C205, C206, C305, C306, C405, C406, C505, C506: 10n, symbol Device:C_Small
- removed C207, C208, C307, C308, C407, C408, C507, C508: 220n, symbol Device:C_Small
- removed C209, C210, C309, C310, C409, C410, C509, C510: 150n, symbol Device:C_Small
- removed C211, C311, C411, C511: 1u, symbol Device:C_Small
- removed J201, J301, J401, J501: Bass_Out, symbol Connector:Conn_01x02_Socket
- removed R201, R205, R301, R305, R401, R405, R501, R505, Z305, Z324, Z405, Z424, Z505, Z524: 100k, symbol Device:R
- removed R202, R203, R204, R302, R303, R304, R402, R403, R404, R502, R503, R504: 1k, symbol Device:R
- removed R206, R306, R406, R506: 560k, symbol Device:R
- removed R207, R307, R407, R507: 680k, symbol Device:R
- removed R208, R308, R408, R508: 10k, symbol Device:R
- removed R209, R309, R409, R509: 75k, symbol Device:R
- removed R210, R211, R310, R311, R410, R411, R510, R511: 15k, symbol Device:R
- removed R212, R213, R312, R313, R412, R413, R512, R513: 7k5, symbol Device:R
- removed SW201, SW301, SW401, SW501: SW_SPDT, symbol sw_spdt_2:SW_SPDT
- removed U201, U202, U301, U302, U401, U402, U501, U502: TL074, symbol OPV_De:TL074
- removed Z301, Z321, Z401, Z421, Z501, Z521: 1u, symbol Device:R
- removed Z302, Z303, Z307, Z308, Z310, Z311, Z313, Z314, Z316, Z317, Z319, Z320, Z402, Z403, Z407, Z408, Z410, Z411, Z413, Z414, Z416, Z417, Z419, Z420, Z502, Z503, Z507, Z508, Z510, Z511, Z513, Z514, Z516, Z517, Z519, Z520: 0R, symbol Device:R
- removed Z304, Z306, Z309, Z312, Z318, Z323, Z404, Z406, Z409, Z412, Z418, Z423, Z504, Z506, Z509, Z512, Z518, Z523: (no value), symbol Device:R
- removed Z315, Z322, Z415, Z422, Z515, Z522: 820k, symbol Device:R
- added C114, C115, C126, C127, C138, C139, C150, C151: 10n, symbol Device:C_Small
- added C116, C117, C118, C119, C125, C128, C129, C130, C131, C137, C140, C141, C142, C143, C149, C152, C153, C154, C155, C161: 100n, symbol Device:C_Small
- added C120, C121, C132, C133, C144, C145, C156, C157: 220n, symbol Device:C_Small
- added C122, C123, C134, C135, C146, C147, C158, C159: 150n, symbol Device:C_Small
- added C124, C136, C148, C160: 1u, symbol Device:C_Small
- added J105, J107, J109, J111: Stecker_In_Out_Switch, symbol Stecker_In_Out_Switch:Stecker_In_Out_Switch
- added J106, J108, J110, J112: Conn_02x07_Odd_Even, symbol Connector_Generic:Conn_02x07_Odd_Even
- added R115, R119, R128, R132, R141, R145, R154, R158, Z147, Z166, Z171, Z190, Z195, Z238: 100k, symbol Device:R
- added R116, R117, R118, R129, R130, R131, R142, R143, R144, R155, R156, R157: 1k, symbol Device:R
- added R120, R133, R146, R159: 560k, symbol Device:R
- added R121, R134, R147, R160: 680k, symbol Device:R
- added R122, R135, R148, R161: 10k, symbol Device:R
- added R123, R136, R149, R162: 75k, symbol Device:R
- added R124, R125, R137, R138, R150, R151, R163, R164: 15k, symbol Device:R
- added R126, R127, R139, R140, R152, R153, R165, R166: 7k5, symbol Device:R
- added U104, U105, U106, U107, U108, U109, U110, U111: TL074, symbol OPV_De:TL074
- added Z143, Z163, Z167, Z187, Z191, Z235: 1u, symbol Device:R
- added Z144, Z145, Z149, Z150, Z152, Z153, Z155, Z156, Z158, Z159, Z161, Z162, Z168, Z169, Z173, Z174, Z176, Z177, Z179, Z180, Z182, Z183, Z185, Z186, Z192, Z193, Z197, Z198, Z200, Z225, Z227, Z228, Z230, Z231, Z233, Z234: 0R, symbol Device:R
- added Z146, Z148, Z151, Z154, Z160, Z165, Z170, Z172, Z175, Z178, Z184, Z189, Z194, Z196, Z199, Z226, Z232, Z237: (no value), symbol Device:R
- added Z157, Z164, Z181, Z188, Z229, Z236: 820k, symbol Device:R
- Z201, Z221: value 1u -> 0R
- Z202, Z208, Z213, Z220: value 0R -> (none)
- Z204, Z206, Z209: value (none) -> 0R
- Z205: value 100k -> 820k
- Z211: value 0R -> 1u
- Z212: value (none) -> 820k
- Z214, Z219: value 0R -> 100k
- Z215: value 820k -> 1u
- Z222: value 820k -> 0R
- Z224: value 100k -> 0R
Connections:
- net +15V: now also C116.2, C118.2, C128.2, C130.2, C140.2, C142.2, C152.2, C154.2, J106.11 (Pin_11), J106.12 (Pin_12), J106.13 (Pin_13), J106.14 (Pin_14), J108.11 (Pin_11), J108.12 (Pin_12), J108.13 (Pin_13), J108.14 (Pin_14), J110.11 (Pin_11), J110.12 (Pin_12), J110.13 (Pin_13), J110.14 (Pin_14), J112.11 (Pin_11), J112.12 (Pin_12), J112.13 (Pin_13), J112.14 (Pin_14), U104.4 (V+), U105.4 (V+), U106.4 (V+), U107.4 (V+), U108.4 (V+), U109.4 (V+), U110.4 (V+), U111.4 (V+)
- net -15V: now also C117.2, C119.2, C129.2, C131.2, C141.2, C143.2, C153.2, C155.2, J106.1 (Pin_1), J106.2 (Pin_2), J106.3 (Pin_3), J106.4 (Pin_4), J108.1 (Pin_1), J108.2 (Pin_2), J108.3 (Pin_3), J108.4 (Pin_4), J110.1 (Pin_1), J110.2 (Pin_2), J110.3 (Pin_3), J110.4 (Pin_4), J112.1 (Pin_1), J112.2 (Pin_2), J112.3 (Pin_3), J112.4 (Pin_4), U104.11 (V-), U105.11 (V-), U106.11 (V-), U107.11 (V-), U108.11 (V-), U109.11 (V-), U110.11 (V-), U111.11 (V-)
- net GND: now also Z202.2, Z208.2, Z213.2, Z214.2, Z219.2, Z220.2, C116.1, C117.1, C118.1, C119.1, C123.1, C125.1, C128.1, C129.1, C130.1, C131.1, C135.1, C137.1, C140.1, C141.1, C142.1, C143.1, C147.1, C149.1, C152.1, C153.1, C154.1, C155.1, C159.1, C161.1, J105.3 (Pin_3), J105.4 (Pin_4), J105.5 (Pin_5), J105.6 (Pin_6), J105.7 (Pin_7), J105.8 (Pin_8), J106.10 (Pin_10), J106.5 (Pin_5), J106.6 (Pin_6), J106.7 (Pin_7), J106.8 (Pin_8), J106.9 (Pin_9), J107.3 (Pin_3), J107.4 (Pin_4), J107.5 (Pin_5), J107.6 (Pin_6), J107.7 (Pin_7), J107.8 (Pin_8), J108.10 (Pin_10), J108.5 (Pin_5), J108.6 (Pin_6), J108.7 (Pin_7), J108.8 (Pin_8), J108.9 (Pin_9), J109.3 (Pin_3), J109.4 (Pin_4), J109.5 (Pin_5), J109.6 (Pin_6), J109.7 (Pin_7), J109.8 (Pin_8), J110.10 (Pin_10), J110.5 (Pin_5), J110.6 (Pin_6), J110.7 (Pin_7), J110.8 (Pin_8), J110.9 (Pin_9), J111.3 (Pin_3), J111.4 (Pin_4), J111.5 (Pin_5), J111.6 (Pin_6), J111.7 (Pin_7), J111.8 (Pin_8), J112.10 (Pin_10), J112.5 (Pin_5), J112.6 (Pin_6), J112.7 (Pin_7), J112.8 (Pin_8), J112.9 (Pin_9), R119.1, R121.1, R123.1, R132.1, R134.1, R136.1, R145.1, R147.1, R149.1, R158.1, R160.1, R162.1, Z146.2, Z147.2, Z148.2, Z151.2, Z154.2, Z157.2, Z160.2, Z164.2, Z165.2, Z166.2, Z170.2, Z171.2, Z172.2, Z175.2, Z178.2, Z181.2, Z184.2, Z188.2, Z189.2, Z190.2, Z194.2, Z195.2, Z196.2, Z199.2, Z226.2, Z229.2, Z232.2, Z236.2, Z237.2, Z238.2; no longer Z204.2, Z206.2, Z209.2, Z215.2, Z222.2, Z224.2
- net at Z211.1: now also Z213.1, U108.13 (-), U108.14
- net at Z219.1: now also Z215.1, U110.3 (+)
- net at Z216.2: now also U110.1, U110.2 (-)
- net at Z221.1, Z223.1: now also Z222.2
- net at Z221.2: now also R154.2, U110.8; no longer Z224.1
- net at Z207.2: now also Z206.1, Z208.1
- net at U103.7, Z142.1: no longer Z134.1
- net at Z210.1, Z212.1: now also Z209.2; no longer Z211.2
- net at Z205.1: now also Z203.1, Z204.2; no longer Z201.1
- net at Z217.1: now also U110.5 (+)
- net at Z214.1: now also Z211.2, J109.10 (Pin_10), J109.9 (Pin_9)
- net at Z216.1, Z217.2: now also Z220.1; no longer Z218.1
- net at Z210.2: now also U108.12 (+)
- new net: Z149.1, Z150.2, Z151.1
- new net: U104.13 (-), U104.14, Z163.1, Z165.1
- new net: J105.10 (Pin_10), J105.9 (Pin_9), Z163.2, Z166.1
- new net: J105.1 (Pin_1), J105.2 (Pin_2), J107.1 (Pin_1), J107.2 (Pin_2), J109.1 (Pin_1), J109.2 (Pin_2), J111.1 (Pin_1), J111.2 (Pin_2), SW101.2 (B), Z143.2, Z146.1, Z167.2, Z170.1, Z191.2, Z194.1, Z215.2, Z218.1
- new net: C148.2, U109.1, U109.2 (-), Z209.1
- new net: C149.2, R152.2, U109.3 (+)
- new net: C135.2, R138.2, U107.12 (+)
- new net: C134.2, U107.13 (-), U107.14, Z183.1
- new net: C122.2, U105.13 (-), U105.14, Z159.1
- new net: Z158.1, Z159.2, Z160.1
- new net: C132.1, C133.2, R135.1
- new net: R135.2, U107.8, U107.9 (-), Z179.2
- new net: R154.1, R155.2, U110.9 (-)
- new net: Z192.1, Z193.2, Z196.1
- new net: C150.1, Z222.1
- new net: C150.2, C151.1, R159.1
- new net: C122.1, R124.2, R125.1
- new net: C123.2, R125.2, U105.12 (+)
- new net: U110.13 (-), U110.14, Z235.1, Z237.1
- new net: J111.10 (Pin_10), J111.9 (Pin_9), Z235.2, Z238.1
- new net: R118.2, R119.2, U104.10 (+)
- new net: R115.2, U104.8, Z149.2
- new net: R115.1, R116.2, U104.9 (-)
- new net: C125.2, R126.2, U105.3 (+)
- new net: C147.2, R151.2, U109.12 (+)
- new net: C158.2, U111.13 (-), U111.14, Z231.1
- new net: Z230.1, Z231.2, Z232.1
- new net: C160.2, U111.1, U111.2 (-), Z233.1
- new net: Z233.2, Z234.1, Z236.1
- new net: C136.2, U107.1, U107.2 (-), Z185.1
- new net: C137.2, R139.2, U107.3 (+)
- new net: C138.2, C139.1, R146.1
- new net: C139.2, R147.2, U109.5 (+)
- new net: R140.1, Z182.2
- new net: C136.1, R139.1, R140.2
- new net: C151.2, R160.2, U111.5 (+)
- new net: R144.2, R145.2, U108.10 (+)
- new net: U110.12 (+), Z234.2
- new net: C138.1, Z198.1
- new net: R141.1, R142.2, U108.9 (-)
- new net: R141.2, U108.8, Z197.2
- new net: C126.2, C127.1, R133.1
- new net: C127.2, R134.2, U107.5 (+)
- new net: R131.2, R132.2, U106.10 (+)
- new net: R124.1, Z156.1
- new net: Z155.1, Z156.2, Z157.1
- new net: Z152.1, Z153.2, Z154.1
- new net: C121.1, Z152.2
- new net: R122.2, U105.8, U105.9 (-), Z155.2
- new net: C158.1, R163.2, R164.1
- new net: C159.2, R164.2, U111.12 (+)
- new net: J111.13 (SW_Out), J111.14 (Pin_14), R155.1, R156.2, U110.7
- new net: J109.13 (SW_Out), J109.14 (Pin_14), R142.1, R143.2, U108.7
- new net: C120.2, R123.2, U105.10 (+)
- new net: Z224.1, Z225.2, Z226.1
- new net: J105.11 (SW_In), J105.12 (Pin_12), R117.1, R118.1, U104.6 (-)
- new net: U106.13 (-), U106.14, Z187.1, Z189.1
- new net: J107.10 (Pin_10), J107.9 (Pin_9), Z187.2, Z190.1
- new net: U104.12 (+), Z162.2
- new net: Z176.1, Z177.2, Z178.1
- new net: C114.1, Z150.1
- new net: C114.2, C115.1, R120.1
- new net: R159.2, U111.6 (-), U111.7, Z225.1
- new net: Z227.1, Z228.2, Z229.1
- new net: R161.2, U111.8, U111.9 (-), Z227.2
- new net: C161.2, R165.2, U111.3 (+)
- new net: U106.3 (+), Z167.1, Z171.1
- new net: J111.11 (SW_In), J111.12 (Pin_12), R156.1, R157.1, U110.6 (-)
- new net: U106.12 (+), Z186.2
- new net: C148.1, R152.1, R153.2
- new net: Z161.2, Z162.1, Z164.1
- new net: C144.1, C145.2, R148.1
- new net: R148.2, U109.8, U109.9 (-), Z203.2
- new net: R153.1, Z206.2
- new net: R166.1, Z230.2
- new net: C160.1, R165.1, R166.2
- new net: R157.2, R158.2, U110.10 (+)
- new net: R146.2, U109.6 (-), U109.7, Z201.1
- new net: C126.1, Z174.1
- new net: Z173.1, Z174.2, Z175.1
- new net: U108.1, U108.2 (-), Z192.2
- new net: C124.2, U105.1, U105.2 (-), Z161.1
- new net: C115.2, R121.2, U105.5 (+)
- new net: R120.2, U105.6 (-), U105.7, Z153.1
- new net: U108.3 (+), Z191.1, Z195.1
- new net: R128.2, U106.8, Z173.2
- new net: R128.1, R129.2, U106.9 (-)
- new net: J107.11 (SW_In), J107.12 (Pin_12), R130.1, R131.1, U106.6 (-)
- new net: J107.13 (SW_Out), J107.14 (Pin_14), R129.1, R130.2, U106.7
- new net: U106.5 (+), Z169.1
- new net: C120.1, C121.2, R122.1
- new net: C132.2, R136.2, U107.10 (+)
- new net: J105.13 (SW_Out), J105.14 (Pin_14), R116.1, R117.2, U104.7
- new net: Z182.1, Z183.2, Z184.1
- new net: Z168.1, Z169.2, Z172.1
- new net: Z197.1, Z198.2, Z199.1
- new net: C134.1, R137.2, R138.1
- new net: Z179.1, Z180.2, Z181.1
- new net: J109.11 (SW_In), J109.12 (Pin_12), R143.1, R144.1, U108.6 (-)
- new net: U104.5 (+), Z145.1
- new net: Z144.1, Z145.2, Z148.1
- new net: R163.1, Z228.1
- new net: C157.1, Z224.2
- new net: C156.1, C157.2, R161.1
- new net: C144.2, R149.2, U109.10 (+)
- new net: C156.2, R162.2, U111.10 (+)
- new net: R137.1, Z180.1
- new net: R127.1, Z158.2
- new net: R150.1, Z204.1
- new net: C146.1, R150.2, R151.1
- new net: R133.2, U107.6 (-), U107.7, Z177.1
- new net: Z185.2, Z186.1, Z188.1
- new net: C124.1, R126.1, R127.2
- new net: U108.5 (+), Z193.1
- new net: C146.2, U109.13 (-), U109.14, Z207.1
- new net: C133.1, Z176.2
- new net: Z200.1, Z201.2, Z202.1
- new net: C145.1, Z200.2
- new net: U106.1, U106.2 (-), Z168.2
- new net: U104.1, U104.2 (-), Z144.2
- new net: U104.3 (+), Z143.1, Z147.1
Other:
- moved on the sheet: U103B, Z142
