File: KiCad/SPICE/RIAA.kicad_sch (KiCad schematic)
At the start: 14 parts, among them U1 ${SIM.PARAMS}, U2 ${SIM.PARAMS}, U3 ${SIM.PARAMS}

Commit message: RIAA Spice
Parts:
- removed R5: 47k, Resistor_SMD:R_0805_2012Metric_Pad1.20x1.40mm_HandSolder, symbol Device:R
- removed R6: 1k, Resistor_SMD:R_0805_2012Metric_Pad1.20x1.40mm_HandSolder, symbol Device:R
- removed R7: 100k, Resistor_SMD:R_0805_2012Metric_Pad1.20x1.40mm_HandSolder, symbol Device:R
- removed R94: 2k, Resistor_SMD:R_0805_2012Metric_Pad1.20x1.40mm_HandSolder, symbol Device:R
- removed U1, U2: ${SIM.PARAMS}, symbol Simulation_SPICE:OPAMP
- removed V2: VSIN, symbol Simulation_SPICE:VSIN
- added C1: 10n, symbol Device:C
- added C2: 2n2, symbol Device:C
- added C3: 47u, symbol Device:C
- added C4: 2u2, symbol Device:C
- added R4: 100k, symbol Device:R
- R1: value 47k -> 390k; footprint Resistor_SMD:R_0805_2012Metric_Pad1.20x1.40mm_HandSolder -> (none); now in the parts list
- R2: value 1k -> 33k; footprint Resistor_SMD:R_0805_2012Metric_Pad1.20x1.40mm_HandSolder -> (none); now in the parts list
- R3: value 100k -> 1k; footprint Resistor_SMD:R_0805_2012Metric_Pad1.20x1.40mm_HandSolder -> (none); now in the parts list
Connections:
- net GND: now also R3.1, R4.1
- net out: now also C4.1, R4.2; no longer R3.1, U3.5
- net In: now reaches U3.1 (+)
- net In: now also V1.2
- net at R1.1: now also R2.2, C1.1, C2.2
- net at R1.2: now also U3.5, C1.2, C4.2; no longer R2.1
- new net: C3.1, R3.2
- new net: C2.1, C3.2, R2.1, U3.2 (-)
Other:
- moved on the sheet: V1
