File: KiCad/SPICE/Spannungsteiler.kicad_sch (KiCad schematic)
At the start: 6 parts, among them U1 ${SIM.PARAMS}

Commit message: VU Update
Parts:
- removed V3: VSIN, symbol Simulation_SPICE:VSIN
- added R3: 15k, symbol Device:R
- R1: value 1k -> 150k
Connections:
- net GND: now also R3.1
- net in: now also R1.2; no longer R1.1
- net at R2.1, U1.2 (-): no longer R1.2
- new net: R1.1, R3.2
Other:
- moved on the sheet: R1, R2, U1
