File: KiCad/SPICE/EQ.kicad_sch (KiCad schematic)
At the start: 14 parts, among them U4 ${SIM.PARAMS}, U5 ${SIM.PARAMS}

Commit message: Update
Parts:
- C33: value 1 n -> 1n5
Changed lines of the file:
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@@
 			)
 		)
-		(property "Sim.Params" "r=47k pos=1"
+		(property "Sim.Params" "r=50k pos=1"
 			(at 106.68 111.76 0)
 			(show_name yes)
@@
 			)
 		)
-		(property "Value" "1 n"
+		(property "Value" "1n5"
 			(at 179.07 106.6862 0)
 			(show_name no)
