File: KiCad/SPICE/Elektrometersubtrahierer.kicad_sch (KiCad schematic)
At the start: 14 parts, among them U1 ${SIM.PARAMS}, U2 ${SIM.PARAMS}, U3 ${SIM.PARAMS}

Commit message: Erste mal musik durch geschickt
Parts:
- R2, R6: value 1k -> 10k
- R3, R7: value 100k -> 10k
- R94: value 2k -> 1k
Changed lines of the file:
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@@
 			)
 		)
-		(property "Value" "1k"
+		(property "Value" "10k"
 			(at 149.86 100.33 90)
 			(show_name no)
@@
 			)
 		)
-		(property "Value" "100k"
+		(property "Value" "10k"
 			(at 158.75 113.0299 0)
 			(show_name no)
@@
 			)
 		)
-		(property "Value" "100k"
+		(property "Value" "10k"
 			(at 163.83 59.69 90)
 			(show_name no)
@@
 			)
 		)
-		(property "Value" "1k"
+		(property "Value" "10k"
 			(at 149.86 59.69 90)
 			(show_name no)
@@
 			)
 		)
-		(property "Value" "2k"
+		(property "Value" "1k"
 			(at 147.32 85.0899 0)
 			(show_name no)

Commit message: Update
Parts:
- added C1: 330p, symbol Device:C
- added R4: 2k2, symbol Device:R
- R1, R5: value 47k -> 15k
- R2, R6: value 10k -> 1k
- R3, R7: value 10k -> 47k
Connections:
- net at U2.1 (+), V2.1: now also C1.2, R4.2
- net at U1.1 (+), V1.2: now also C1.1, R4.1
Other:
- moved on the sheet: V1, V2
