File: KiCad/SPICE/Pegelanzeige.kicad_sch (KiCad schematic)
At the start: 23 parts, among them U4 ${SIM.PARAMS}, U5 ${SIM.PARAMS}, U6 ${SIM.PARAMS}, U7 ${SIM.PARAMS}

Commit message: VU Test
Parts:
- R3: value 10k -> 16k5
- R4, R5: value 20k -> 33k
- R8, R9: value 1k8 -> 2k2
Changed lines of the file:
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@@
 			)
 		)
-		(property "Value" "10k"
+		(property "Value" "16k5"
 			(at 151.13 77.47 90)
 			(show_name no)
@@
 			)
 		)
-		(property "Value" "20k"
+		(property "Value" "33k"
 			(at 151.13 63.5 90)
 			(show_name no)
@@
 			)
 		)
-		(property "Value" "1k8"
+		(property "Value" "2k2"
 			(at 251.46 80.0099 0)
 			(show_name no)
@@
 			)
 		)
-		(property "Value" "1k8"
+		(property "Value" "2k2"
 			(at 223.52 66.04 90)
 			(show_name no)
@@
 			)
 		)
-		(property "Value" "20k"
+		(property "Value" "33k"
 			(at 172.72 63.5 90)
 			(show_name no)

Commit message: VU Update
Parts:
- added R12: 33k, symbol Device:R
- added R13: 3k3, symbol Device:R
- R10: value 10k -> 1k
- R11: value 1k -> 100k
- R6: value 100R -> 2k2
- R7: value 3k3 -> 15k
Connections:
- net GND: now also R11.2, R13.2; no longer D4.1 (K)
- net LED: now also D3.1 (K), R10.1; no longer D4.2 (A)
- new net: R12.1, R13.1
Other:
- moved on the sheet: C1, D3, D4, R11, R8, R9

Commit message: VU Update
Parts:
- R10: value 1k -> 100R
- R11: value 100k -> 10k
Connections:
- net GND: now also D3.1 (K), D4.2 (A); no longer D3.2 (A), R11.2
- net at U5.5: now also R10.1; no longer R10.2
- net at D4.1 (K): now also R11.2
- removed net LED: D3.1 (K), R10.1, R11.1
- new net: D3.2 (A), R10.2

Commit message: Update
Parts:
- R6, R9: value 2k2 -> 10k
- R8: value 2k2 -> 15k
Changed lines of the file:
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@@
 			)
 		)
-		(property "Value" "2k2"
+		(property "Value" "10k"
 			(at 176.53 118.1099 0)
 			(show_name no)
@@
 			)
 		)
-		(property "Value" "2k2"
+		(property "Value" "10k"
 			(at 257.81 80.0099 0)
 			(show_name no)
@@
 			)
 		)
-		(property "Value" "2k2"
+		(property "Value" "15k"
 			(at 234.95 66.04 90)
 			(show_name no)
