File: KiCad/SPICE/Bandpass.kicad_sch (KiCad schematic)
At the start: 93 parts, among them U1 ${SIM.PARAMS}, U10 ${SIM.PARAMS}, U11 ${SIM.PARAMS}, U12 ${SIM.PARAMS}, U13 ${SIM.PARAMS}, U14 ${SIM.PARAMS}, U15 ${SIM.PARAMS}, U16 ${SIM.PARAMS}, U17 ${SIM.PARAMS}, U2 ${SIM.PARAMS}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

Commit message: Höhen Update
Parts:
- C25, C26, C27, C28: value 1n5 -> 3n
- R25, R27: value 15k -> 7k5
- R26, R28: value 30k -> 15k
Changed lines of the file:
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@@
 			)
 		)
-		(property "Value" "1n5"
+		(property "Value" "3n"
 			(at 57.15 309.88 90)
 			(show_name no)
@@
 			)
 		)
-		(property "Value" "1n5"
+		(property "Value" "3n"
 			(at 128.27 312.42 90)
 			(show_name no)
@@
 			)
 		)
-		(property "Value" "1n5"
+		(property "Value" "3n"
 			(at 115.57 312.42 90)
 			(show_name no)
@@
 			)
 		)
-		(property "Value" "15k"
+		(property "Value" "7k5"
 			(at 143.51 298.45 90)
 			(show_name no)
@@
 			)
 		)
-		(property "Value" "30k"
+		(property "Value" "15k"
 			(at 143.51 326.3899 0)
 			(show_name no)
@@
 			)
 		)
-		(property "Value" "15k"
+		(property "Value" "7k5"
 			(at 85.09 298.45 90)
 			(show_name no)
@@
 			)
 		)
-		(property "Value" "30k"
+		(property "Value" "15k"
 			(at 85.09 323.8499 0)
 			(show_name no)
@@
 			)
 		)
-		(property "Value" "1n5"
+		(property "Value" "3n"
 			(at 69.85 309.88 90)
 			(show_name no)

Commit message: Update
Parts:
- removed C10, C11, C12, C9: 100n, symbol Device:C
- removed C13, C15: 300n, symbol Device:C
- removed C14, C16: 150n, symbol Device:C
- removed C17, C18, C19, C20: 13n6, symbol Device:C
- removed C21, C23: 20n, symbol Device:C
- removed C22, C24: 10n, symbol Device:C
- removed C25, C26, C27, C28: 3n, symbol Device:C
- removed C29, C30: 2n2, symbol Device:C
- removed C31: 6n8, symbol Device:C
- removed C32: 1n, symbol Device:C
- removed R10, R12, R26, R28: 15k, symbol Device:R
- removed R11, R25, R27, R9: 7k5, symbol Device:R
- removed R117, R119, R130, R131, R17, R19: 10k, symbol Device:R
- removed R125: 1M, symbol Device:R
- removed R13, R14, R15, R16: 1k, symbol Device:R
- removed R18, R20: 20k, symbol Device:R
- removed R21, R22, R23, R24: 2k2, symbol Device:R
- removed R29, R30: 3k9, symbol Device:R
- removed R31, R32: 3k3, symbol Device:R
- removed U10, U11, U12, U13, U14, U15, U16, U17, U5, U6, U7, U8, U9: ${SIM.PARAMS}, symbol Simulation_SPICE:OPAMP
- removed V2, V5, V6: VSIN, symbol Simulation_SPICE:VSIN
Other:
- note removed: "f_g = 17kHz"
- note removed: "f_g = 4.9kHz"
- note removed: "f_g = 800Hz"
