File: KiCad/Designe_Blocks/Bandpass_Killswitch/Bandpass_Killswitch.kicad_sch (KiCad schematic)
At the start: 53 parts, among them J1 Stecker_In_Out_Switch, J2 Conn_02x07_Odd_Even, U1 TL074, U2 TL074

Commit message: Update
Parts:
- C1, C10, C11, C12, C2, C3, C4, C5, C6, C7, C8, C9: footprint Capacitor_SMD:C_0805_2012Metric -> (none)
- J1, J2: footprint PinHeader:PinHeader_2x07_P2.54mm_Vertical -> (none)
- R1, R10, R11, R12, R13, R2, R3, R4, R5, R6, R7, R8, R9, Z1, Z10, Z11, Z12, Z13, Z14, Z15, Z16, Z17, Z18, Z19, Z2, Z20, Z21, Z22, Z23, Z24, Z3, Z4, Z5, Z6, Z7, Z8, Z9: footprint Resistor_SMD:R_0805_2012Metric -> (none)
- U1, U2: footprint TL074CN:DIP794W53P254L1930H508Q14N -> (none)
Other:
- moved on the sheet: C1, C10, C11, C12, C2, C3, C4, C5, C6, C7, C8, C9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
