File: KiCad/Designe_Blocks/Input_Phono_Line/Input_Phono_Line.kicad_pcb (KiCad board)
At the start: 4 copper layers, 98 parts, among them J1 Stecker_In_Out_Switch, J2 Conn_02x07_Odd_Even, U1 TL074, U2 TL074, U3 TL074

Commit message: Update
Parts:
- added J3: Stecker_4In, PinHeader:PinHeader_2x07_P2.54mm_Vertical, F.Cu at (89.7, 56.1)
- C10, C11, C12, C13, C2, C3, C5, C8, C9, R1, R10, R11, R13, R14, R2, R4, R5, R6, R7, R9, Z1, Z10, Z11, Z12, Z13, Z14, Z15, Z16, Z17, Z18, Z19, Z24, Z25, Z26, Z27, Z28, Z29, Z30, Z31, Z36, Z37, Z38, Z39, Z40, Z41, Z42, Z43, Z44, Z45, Z46, Z47, Z48, Z49, Z54, Z55, Z56, Z57, Z6, Z7, Z8, Z9: moved to F.Cu
- J1: value Stecker_In_Out_Switch -> Stecker_1Out_Switch; footprint PinHeader:PinHeader_2x013_P2.54mm_Vertical (Kopie) -> PinHeader:PinHeader_2x07_P2.54mm_Vertical
- moved R2 195.0 mm to (44.9, 58.2), turned to 0 degrees
- moved R4 194.4 mm to (44.9, 61.1), turned to 0 degrees
- moved R5 194.4 mm to (44.9, 64.1), turned to 0 degrees
- moved R6 194.4 mm to (44.9, 67.0), turned to 0 degrees
- moved R7 194.4 mm to (44.9, 70.0), turned to 0 degrees
- moved R10 193.9 mm to (44.9, 75.9), turned to 0 degrees
- moved R11 193.9 mm to (44.9, 78.8), turned to 0 degrees
- moved R9 193.9 mm to (44.9, 72.9), turned to 0 degrees
- moved Z10 187.8 mm to (49.3, 75.9), turned to 0 degrees
- moved Z11 187.8 mm to (49.3, 78.8), turned to 0 degrees
- moved R13 186.4 mm to (49.3, 55.2), turned to 0 degrees
- moved R14 186.4 mm to (49.3, 58.2), turned to 0 degrees
- moved Z1 185.8 mm to (49.3, 61.1), turned to 0 degrees
- moved Z7 183.7 mm to (49.3, 67.0), turned to 0 degrees
- moved Z8 183.7 mm to (49.3, 70.0), turned to 0 degrees
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Connections:
- C5 pad 2: Net-(U2A--) -> Net-(U3A--)
- J1 pad 1: Net-(J1A-Phono_L) -> Net-(J1B-Out-Pad1)
- J1 pad 10: GND -> Net-(J1A-SW_2)
- J1 pad 11: GND -> Net-(J1A-SW_3)
- J1 pad 12: GND -> Net-(J1A-SW_3)
- J1 pad 13: GND -> Net-(J1A-SW_Out-Pad13)
- J1 pad 14: GND -> Net-(J1A-SW_Out-Pad13)
- J1 pad 2: Net-(J1A-Phono_L) -> Net-(J1B-Out-Pad1)
- J1 pad 3: Net-(J1B-Phono_R-Pad3) -> GND
- J1 pad 4: Net-(J1B-Phono_R-Pad3) -> GND
- J1 pad 9: GND -> Net-(J1A-SW_2)
- R10 pad 2: Net-(U3C--) -> Net-(U2C--)
- R11 pad 1: Net-(U3C--) -> Net-(U2C--)
- R14 pad 2: Net-(U3C--) -> Net-(U2C--)
- R7 pad 2: Net-(U2A--) -> Net-(U3A--)
- U1 pad 12: Net-(D4-K) -> GND
- U1 pad 5: GND -> Net-(D4-K)
- U2 pad 1: Net-(C2-Pad2) -> Net-(U2-Pad1)
- U2 pad 12: Net-(U2D-+) -> GND
- U2 pad 14: Net-(J1E-SW_3) -> Net-(U2-Pad14)
- U2 pad 3: Net-(U2A-+) -> Net-(D6-K)
- U2 pad 5: Net-(U2B-+) -> Net-(D8-K)
- U2 pad 7: Net-(U2B--) -> Net-(U2-Pad7)
- U2 pad 8: Net-(J1E-SW_2) -> Net-(R11-Pad2)
- U3 pad 1: Net-(U3-Pad1) -> Net-(C2-Pad2)
- U3 pad 12: GND -> Net-(U3D-+)
- U3 pad 14: Net-(U3-Pad14) -> Net-(U3D--)
- U3 pad 3: Net-(D6-K) -> Net-(U3A-+)
- U3 pad 5: Net-(D8-K) -> Net-(U3B-+)
- U3 pad 7: Net-(U3-Pad7) -> Net-(J1A-SW_3)
- U3 pad 8: Net-(R11-Pad2) -> Net-(J1A-SW_2)
- Z1 pad 1: Net-(U1-Pad7) -> Net-(U1-Pad14)
- Z1 pad 2: Net-(U1B--) -> Net-(U1D--)
- Z11 pad 2: Net-(U2B-+) -> Net-(U3D-+)
- Z18 pad 2: Net-(U2C-+) -> Net-(U3C-+)
- Z19 pad 1: Net-(U2B--) -> Net-(U3D--)
- Z2 pad 1: Net-(J1A-Phono_L) -> Net-(J3A-Phono_L)
- Z20 pad 1: Net-(J1B-Phono_R-Pad3) -> Net-(J3B-Phono_R-Pad3)
- Z24 pad 1: Net-(U1-Pad14) -> Net-(U1-Pad7)
- Z27 pad 1: Net-(U1-Pad14) -> Net-(U1-Pad7)
- Z27 pad 2: Net-(U1D--) -> Net-(U1B--)
- Z28 pad 1: Net-(U2C--) -> Net-(U3C--)
- Z28 pad 2: Net-(J1E-SW_2) -> Net-(J1A-SW_2)
- Z29 pad 1: Net-(U1D--) -> Net-(U1B--)
- Z30 pad 1: Net-(J1E-SW_2) -> Net-(J1A-SW_2)
- Z31 pad 1: Net-(U3-Pad14) -> Net-(U2-Pad14)
- Z31 pad 2: Net-(U3D--) -> Net-(U2D--)
- Z32 pad 1: Net-(J1C-Line_L-Pad17) -> Net-(J3C-Line_L-Pad11)
- Z36 pad 1: Net-(U3-Pad1) -> Net-(U2-Pad1)
- Z37 pad 1: Net-(U3D--) -> Net-(U2D--)
- Z38 pad 1: Net-(U3-Pad14) -> Net-(U2-Pad14)
- Z39 pad 2: Net-(U2D-+) -> Net-(U3B-+)
- Z40 pad 2: Net-(J1E-SW_Out-Pad25) -> Net-(J1A-SW_Out-Pad13)
- Z41 pad 1: Net-(J1F-Out) -> Net-(J1B-Out-Pad1)
- Z43 pad 1: Net-(U3-Pad1) -> Net-(U2-Pad1)
- Z43 pad 2: Net-(U3A--) -> Net-(U2A--)
- Z45 pad 1: Net-(J1E-SW_Out-Pad25) -> Net-(J1A-SW_Out-Pad13)
- Z46 pad 1: Net-(J1E-SW_3) -> Net-(J1A-SW_3)
- Z46 pad 2: Net-(U2D--) -> Net-(U3B--)
- Z47 pad 1: Net-(U3A--) -> Net-(U2A--)
- Z48 pad 1: Net-(U3C-+) -> Net-(U2C-+)
- Z49 pad 1: Net-(U2D--) -> Net-(U3B--)
- Z50 pad 1: Net-(J1D-Line_R-Pad19) -> Net-(J3D-Line_R-Pad13)
- Z54 pad 1: Net-(U3-Pad7) -> Net-(U2-Pad7)
- Z56 pad 1: Net-(U3-Pad7) -> Net-(U2-Pad7)
- Z56 pad 2: Net-(U3B--) -> Net-(U2B--)
- Z57 pad 1: Net-(U3B--) -> Net-(U2B--)
- Z7 pad 1: Net-(U1B--) -> Net-(U1D--)
- Z8 pad 1: Net-(U1-Pad7) -> Net-(U1-Pad14)
- Z9 pad 2: Net-(U2A-+) -> Net-(U3A-+)
Routing:
- net Net-(C1-Pad2): track 5.17 -> 0.00 mm
- net Net-(C7-Pad2): track 5.11 -> 0.00 mm
- net Net-(C6-Pad2): track 5.11 -> 0.00 mm
- net Net-(C4-Pad2): track 5.11 -> 0.00 mm
- net Net-(R3-Pad1): track 4.58 -> 0.00 mm
- net Net-(D3-A): track 4.55 -> 0.00 mm
- net Net-(D1-A): track 4.55 -> 0.00 mm
- net Net-(R8-Pad1): track 4.53 -> 0.00 mm
- net Net-(R15-Pad1): track 4.53 -> 0.00 mm
- net Net-(R12-Pad1): track 4.53 -> 0.00 mm
- net Net-(D5-A): track 4.51 -> 0.00 mm
- net Net-(D7-A): track 4.51 -> 0.00 mm
- net Net-(J1D-Line_R-Pad19): track 4.17 -> 0.00 mm
- net Net-(J1C-Line_L-Pad17): track 4.17 -> 0.00 mm
- net Net-(J1B-Phono_R-Pad3): track 4.17 -> 0.00 mm
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