File: KiCad/Designe_Blocks/Input_Phono_Line/Input_Phono_Line.kicad_sch (KiCad schematic)
At the start: 104 parts, among them J1 Conn_02x13_Odd_Even, J2 Stecker_In_Out_Switch, J603 Conn_02x07_Odd_Even, U101 TL074, U102 TL074, U103 TL074, U104 TL074, U105 TL074, U106 TL074, U107 TL074, U108 TL074

Commit message: Update
Parts:
- removed J1: Conn_02x13_Odd_Even, symbol Connector_Generic:Conn_02x13_Odd_Even
- J1: renamed from J2; footprint (none) -> PinHeader:PinHeader_2x013_P2.54mm_Vertical (Kopie)
- renumbered C101 to C1, C110 to C10, C111 to C11, C112 to C12, C113 to C13, C102 to C2, C103 to C3, C104 to C4, C105 to C5, C114 to C6, C115 to C7, C108 to C8, C109 to C9, D101 to D1, D102 to D2, D103 to D3, D104 to D4, D109 to D5, D111 to D6, D110 to D7, D112 to D8, J603 to J2, R101 to R1, R117 to R10, R110 to R11, R115 to R12, R119 to R13, R118 to R14, R116 to R15, R102 to R2, R103 to R3, R104 to R4, R105 to R5, R106 to R6, R108 to R7, R107 to R8, R109 to R9, U102 to U1, U101 to U1, U105 to U1, U106 to U1, U103 to U2, U101 to U2, U104 to U2, U103 to U3, U104 to U3, U107 to U3, U108 to U3, Z114 to Z1, Z109 to Z10, Z110 to Z11, Z111 to Z12, Z162 to Z13, Z112 to Z14, Z113 to Z15, Z163 to Z16, Z121 to Z17, Z138 to Z18, Z137 to Z19, Z101 to Z2, Z115 to Z20, Z116 to Z21, Z117 to Z22, Z118 to Z23, Z119 to Z24, Z141 to Z25, Z120 to Z26, Z164 to Z27, Z160 to Z28, Z165 to Z29, Z102 to Z3, Z161 to Z30, Z125 to Z31, Z143 to Z32, Z145 to Z33, Z147 to Z34, Z149 to Z35, Z151 to Z36, Z126 to Z37, Z140 to Z38, Z139 to Z39, Z103 to Z4, Z156 to Z40, Z155 to Z41, Z153 to Z42, Z166 to Z43, Z142 to Z44, Z157 to Z45, Z159 to Z46, Z167 to Z47, Z127 to Z48, Z158 to Z49, Z104 to Z5, Z144 to Z50, Z146 to Z51, Z148 to Z52, Z150 to Z53, Z152 to Z54, Z154 to Z55, Z168 to Z56, Z169 to Z57, Z105 to Z6, Z106 to Z7, Z107 to Z8, Z108 to Z9
Connections:
- net GND: now also J1.10 (GND), J1.11 (GND), J1.12 (GND), J1.13 (GND), J1.14 (GND), J1.9 (GND), U3.12 (+); no longer J1.3 (Pin_3), J1.3 (Pin_3), J1.3 (Pin_3), J1.3 (Pin_3), J1.4 (Pin_4), J1.4 (Pin_4), J1.4 (Pin_4), J1.4 (Pin_4), J1.5 (Pin_5), J1.5 (Pin_5), J1.5 (Pin_5), J1.6 (Pin_6), J1.6 (Pin_6), J1.6 (Pin_6), U3.5 (+)
- net at Z11.2: now also U2.5 (+); no longer U2.12 (+)
- net at U2.14, Z46.1: now also J1.21 (SW_In2), J1.22 (SW_3); no longer J1.11 (SW_In), J1.12 (Pin_12)
- net at Z18.2: now also U2.10 (+); no longer U2.12 (+)
- net at Z28.1: now also U2.9 (-); no longer U2.13 (-)
- net at C2.2, R4.1, Z10.1: now also U2.1; no longer U2.8
- net at R1.2, R2.1, R6.2: now also U1.9 (-); no longer U1.6 (-)
- net at R2.2, Z7.2: now also U1.8; no longer U1.7
- net at Z36.1, Z43.1: now also U3.1; no longer U3.14
- net at Z54.1, Z56.1: now also U3.7; no longer U3.14
- net at Z56.2, Z57.1: now also U3.6 (-); no longer U3.13 (-)
- net at Z31.2, Z37.1: now also U3.13 (-); no longer U3.6 (-)
- net at R11.2, Z37.2: now also U3.8; no longer U3.7
- net at Z9.2: now also U2.3 (+); no longer U2.10 (+)
- net at C5.2, R7.2: now also U2.2 (-); no longer U2.9 (-)
- net at Z17.1: now also U1.10 (+); no longer U1.5 (+)
- net at R10.2, R11.1, R14.2: now also U3.9 (-); no longer U3.6 (-)
- net at D8.1 (K), Z53.2: now also U3.5 (+); no longer U3.12 (+)
- net at Z31.1, Z38.1: now also U3.14; no longer U3.7
- net at Z43.2, Z47.1: now also U3.2 (-); no longer U3.13 (-)
- net at D2.1 (K), Z5.2: now also U1.3 (+); no longer U1.12 (+)
- net at Z40.2, Z45.1: now also J1.25 (SW_Out), J1.26 (SW_Out); no longer J1.11 (SW_In), J1.12 (Pin_12)
- net at D6.1 (K), Z35.2: now also U3.3 (+); no longer U3.12 (+)
- net at Z13.1, Z6.1: now also U1.1; no longer U1.14
- net at Z48.1: now also U3.10 (+); no longer U3.5 (+)
- net at Z13.2, Z16.1: now also U1.2 (-); no longer U1.13 (-)
- new net: J1.23 (SW_In1), J1.24 (SW_2), U2.8, Z28.2, Z30.1
- new net: J1.17 (Line_L), J1.18 (Line_L), Z32.1
- new net: J1.3 (Phono_R), J1.4 (Phono_R), Z20.1
- new net: J1.19 (Line_R), J1.20 (Line_R), Z50.1
- new net: U2.6 (-), U2.7, Z19.1
- new net: J1.15 (Out), J1.16 (Out_1), Z41.1

Commit message: Update
Parts:
- removed J1: Stecker_In_Out_Switch, PinHeader:PinHeader_2x013_P2.54mm_Vertical (Kopie), symbol Stecker_4In_1Out_Switch:Stecker_In_Out_Switch
- added J1: Stecker_1Out_Switch, PinHeader:PinHeader_2x07_P2.54mm_Vertical, symbol Stecker_1Out_Switch:Stecker_1Out_Switch
- added J3: Stecker_4In, PinHeader:PinHeader_2x07_P2.54mm_Vertical, symbol Stecker_4In:Stecker_4In
- C1, C10, C11, C12, C13, C2, C3, C4, C5, C6, C7, C8, C9: footprint (none) -> Capacitor_SMD:C_0805_2012Metric
- D1, D2, D3, D4, D5, D6, D7, D8: footprint (none) -> Diode_SMD:D_0805_2012Metric
- J2: footprint (none) -> PinHeader:PinHeader_2x07_P2.54mm_Vertical
- R1, R10, R11, R12, R13, R14, R15, R2, R3, R4, R5, R6, R7, R8, R9, Z1, Z10, Z11, Z12, Z13, Z14, Z15, Z16, Z17, Z18, Z19, Z2, Z20, Z21, Z22, Z23, Z24, Z25, Z26, Z27, Z28, Z29, Z3, Z30, Z31, Z32, Z33, Z34, Z35, Z36, Z37, Z38, Z39, Z4, Z40, Z41, Z42, Z43, Z44, Z45, Z46, Z47, Z48, Z49, Z5, Z50, Z51, Z52, Z53, Z54, Z55, Z56, Z57, Z6, Z7, Z8, Z9: footprint (none) -> Resistor_SMD:R_0805_2012Metric
- U1, U2, U3: footprint (none) -> TL074CN:DIP794W53P254L1930H508Q14N
- U2: renamed from U3; footprint (none) -> TL074CN:DIP794W53P254L1930H508Q14N
- U3: renamed from U2; footprint (none) -> TL074CN:DIP794W53P254L1930H508Q14N
Connections:
- net GND: now also U1.12 (+), J1.3 (GND), J1.4 (GND), J1.5 (GND), J1.6 (GND), J1.7 (GND), J1.8 (GND), J3.10 (GND), J3.5 (GND), J3.6 (GND), J3.7 (GND), J3.8 (GND), J3.9 (GND), J3.9 (GND); no longer U1.5 (+)
- net at Z11.2: now also U3.12 (+); no longer U3.5 (+)
- net at Z46.1: now also U3.7, J1.11 (SW_In2), J1.12 (SW_3); no longer U3.14
- net at Z46.2, Z49.1: now also U3.6 (-); no longer U3.13 (-)
- net at U3.8, Z28.2, Z30.1: now also J1.10 (SW_2), J1.9 (SW_In1)
- net at Z32.1: now also J3.11 (Line_L), J3.12 (Line_L)
- net at Z24.1, Z27.1: now also U1.7; no longer U1.14
- net at Z39.2: now also U3.5 (+); no longer U3.12 (+)
- net at Z20.1: now also J3.3 (Phono_R), J3.4 (Phono_R)
- net at D4.1 (K), Z23.2: now also U1.5 (+); no longer U1.12 (+)
- net at Z2.1: now also J3.1 (Phono_L), J3.2 (Pin_2)
- net at Z40.2, Z45.1: now also J1.13 (SW_Out), J1.14 (SW_Out)
- net at Z50.1: now also J3.13 (Line_R), J3.14 (Line_R)
- net at Z1.1, Z8.1: now also U1.14; no longer U1.7
- net at Z1.2, Z7.1: now also U1.13 (-); no longer U1.6 (-)
- net at Z41.1: now also J1.1 (Out), J1.2 (Out)
- net at Z27.2, Z29.1: now also U1.6 (-); no longer U1.13 (-)
- new net: U3.13 (-), U3.14, Z19.1
